File: Arduino.kicad_sch (KiCad schematic)
At the start: 1 part

Commit message: schamtic Update
Changed lines of the file:
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@@
+		)
+	)
+	(text_box ""
+		(exclude_from_sim no)
+		(at 92.71 52.07 0)
+		(size 104.14 80.01)
+		(stroke
+			(width 0.0508)
+			(type dash)
+			(color 0 0 0 1)
+		)
+		(fill
+			(type none)
+		)
+		(effects
+			(font
+				(size 1.27 1.27)
+			)
+			(justify left top)
 		)
 	)
 	(text "ARDUINO"
 		(exclude_from_sim no)
-		(at 97.536 48.006 0)
+		(at 101.092 49.784 0)
 		(effects
 			(font

Commit message: verification
Parts:
- added R36, R37: 4.7K, Resistor_SMD:R_0805_2012Metric, symbol Device:R_Small_US
- added R38, R39, R40, R41: 10]K, Resistor_SMD:R_0805_2012Metric, symbol Device:R_Small_US
- added TP10, TP11, TP6, TP7, TP8, TP9: TestPoint, TestPoint:TestPoint_Pad_D2.0mm, symbol Connector:TestPoint
Connections:
- net AR_MISO: now also R40.1, TP9.1
- net AR_MOSI: now also R39.1, TP10.1
- net AR_SCK: now also R41.1, TP8.1
- net AR_SCL: now also R36.1, TP7.1
- net AR_SDA: now also R37.1, TP6.1
- net AR_SS: now also R38.1, TP11.1
- new net +3.3V: R36.2, R37.2, R38.2, R39.2, R40.2, R41.2

Commit message: new
Parts:
- added C80: 100nF, C0402C104K4RAC:CAPC1005X55N, symbol C0402C104K4RAC:C0402C104K4RAC
Connections:
- net +3.3V: now also A1.4 (3V3)
- net GND: now also C80.1
- net VIN: now also A1.2 (IOREF), A1.5 (+5V)
- net JTCK/SWCLK: now reaches A1.17 (D2)
- net JTMS/SWDIO: now reaches A1.18 (D3)
- net RST_BUT: now reaches A1.3 (~{RESET})
- net at A1.30 (AREF): now also C80.2
- no-connect marks 7 -> 0

Commit message: new
Parts:
- added FL12: BLM21PG221SN1D, BLM21PG221SN1D:BEADC2012X105N, symbol BLM21PG221SN1D:BLM21PG221SN1D
Connections:
- net +3.3V: now also FL12.2; no longer A1.4 (3V3)
- net VIN: no longer A1.2 (IOREF)
- net RST_BUT renamed ARDUINO_RST_BUT
- new net +3.3V_ARDUINO: A1.2 (IOREF), A1.4 (3V3), FL12.1
Other:
- moved on the sheet: R36, R37, R38, R39, R40, R41, TP10, TP11, TP6, TP7, TP8, TP9

Commit message: new
Parts:
- R38, R39, R40, R41: value 10]K -> 10K
Connections:
- net VIN: no longer A1.8 (VIN)
- no-connect marks 0 -> 1

Commit message: new placed
Parts:
- removed TP10, TP11, TP8, TP9: TestPoint, TestPoint:TestPoint_Pad_D2.0mm, symbol Connector:TestPoint
- R36, R37, R38, R39, R40, R41: footprint Resistor_SMD:R_0805_2012Metric -> Resistor_SMD:R_0402_1005Metric

Commit message: usb
Parts:
- C80: value 100nF -> 100n
- R36, R37: value 4.7K -> 4K7
Changed lines of the file:
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@@
 			)
 		)
-		(property "Value" "4.7K"
+		(property "Value" "4K7"
 			(at 189.23 119.38 90)
 			(effects
@@
 			)
 		)
-		(property "Value" "4.7K"
+		(property "Value" "4K7"
 			(at 181.61 119.38 90)
 			(effects
@@
 			)
 		)
-		(property "Value" "100nF"
+		(property "Value" "100n"
 			(at 168.402 86.868 0)
 			(effects
