File: Arduino.kicad_sch (KiCad schematic)
At the start: 11 parts

Commit message: full
Other:
- moved on the sheet: R36, R37, R38, R39, R40, R41, TP6, TP7

Commit message: 16.09.2026
Parts:
- FL12: footprint BLM21PG221SN1D:BEADC2012X105N -> GNSS:BEADC2012X105N
Changed lines of the file:
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@@
 			)
 		)
-		(property "Footprint" "BLM21PG221SN1D:BEADC2012X105N"
+		(property "Footprint" "GNSS:BEADC2012X105N"
 			(at 212.598 38.354 0)
 			(effects

Commit message: 18.09.2026
Connections:
- net +3.3V renamed +3V3
- net +3.3V_ARDUINO renamed +3V3_ARDUINO
Changed lines of the file:
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@@
 			)
 		)
-		(property "Value" "+3.3V"
+		(property "Value" "+3V3"
 			(at 215.9 44.45 0)
 			(effects
@@
 			)
 		)
-		(property "Value" "+3.3V_ARDUINO"
+		(property "Value" "+3V3_ARDUINO"
 			(at 147.32 52.578 0)
 			(effects
@@
 			)
 		)
-		(property "Value" "+3.3V"
+		(property "Value" "+3V3"
 			(at 205.74 80.01 0)
 			(effects
@@
 			)
 		)
-		(property "Value" "+3.3V_ARDUINO"
+		(property "Value" "+3V3_ARDUINO"
 			(at 181.61 44.45 0)
 			(effects
@@
 			)
 		)
-		(property "Value" "+3.3V"
+		(property "Value" "+3V3"
 			(at 78.74 68.58 0)
 			(effects
@@
 			)
 		)
-		(property "Value" "+3.3V_ARDUINO"
+		(property "Value" "+3V3_ARDUINO"
 			(at 169.164 80.01 90)
 			(effects

Commit message: 22.09.26
Connections:
- net +3V3_ARDUINO: no longer A1.2 (IOREF)
- no-connect marks 1 -> 2
Changed lines of the file:
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@@
+	)
+	(no_connect
+		(at 157.48 80.01)
 	)
 	(no_connect
@@
 					(unit 1)
 				)
-			)
-		)
-	)
-	(symbol
-		(lib_id "power:+3.3V")
-		(at 157.48 80.01 270)
-		(unit 1)
-		(exclude_from_sim no)
-		(in_bom yes)
-		(on_board yes)
-		(dnp no)
-		(property "Reference" "#PWR0224"
-			(at 153.67 80.01 0)
-			(effects
-				(font
-					(size 1.27 1.27)
-				)
-				(hide yes)
-			)
-		)
-		(property "Value" "+3V3_ARDUINO"
-			(at 169.164 80.01 90)
-			(effects
-				(font
-					(size 1.27 1.27)
-				)
-			)
-		)
-		(property "Footprint" ""
-			(at 157.48 80.01 0)
-			(effects
-				(font
-					(size 1.27 1.27)
-				)
-				(hide yes)
-			)
-		)
-		(property "Datasheet" ""
-			(at 157.48 80.01 0)
-			(effects
-				(font
-					(size 1.27 1.27)
-				)
-				(hide yes)
-			)
-		)
-		(property "Description" "Power symbol creates a global label with name \"+3.3V\""
-			(at 157.48 80.01 0)
-			(effects
-				(font
-					(size 1.27 1.27)
-				)
-				(hide yes)
-			)
-		)
-		(pin "1"
-		)
-		(instances
-			(project "GNSS"
-				(path "/a70dad34-b24c-4b58-b91c-f14576b5da7d/c129ce73-fc4e-459a-b7eb-49148af5c1a5"
-					(reference "#PWR0224")
-					(unit 1)
-				)

Commit message: 123
Parts:
- removed FL12: BLM21PG221SN1D, GNSS:BEADC2012X105N, symbol BLM21PG221SN1D:BLM21PG221SN1D
- removed R39, R40, R41: 10K, Resistor_SMD:R_0402_1005Metric, symbol Device:R_Small_US
- added FB12: FerriteBead, GNSS:BEADC2012X105N, symbol Device:FerriteBead
Connections:
- net +3V3: now also FB12.1
- net +3V3_ARDUINO: now also FB12.2
Other:
- moved on the sheet: R38

Commit message: new
Parts:
- FB12: footprint GNSS:BEADC2012X105N -> Inductor_SMD:L_0805_2012Metric
Changed lines of the file:
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@@
 			)
 		)
-		(property "Footprint" "GNSS:BEADC2012X105N"
+		(property "Footprint" "Inductor_SMD:L_0805_2012Metric"
 			(at 203.2 51.308 90)
 			(effects
