File: ESP.kicad_sch (KiCad schematic)
At the start: 1 part, among them U3 ESP32-C3-MINI-1-N4

Commit message: Add the STM
Parts:
- added C27: 47uF, Capacitor_SMD:C_0805_2012Metric, symbol Device:C_Small
- added C28, C31: 0.1uF, C0402C104K4RAC:CAPC1005X55N, symbol C0402C104K4RAC:C0402C104K4RAC
- added R17: 10K, symbol Device:R_Small_US
Connections:
- net +3.3V: now also C27.1, C28.2, C31.2, R17.1
- net GND: now also C27.2, C28.1, C31.1
- net ESP_D_N: now reaches U3.26 (IO18)
- net ESP_D_P: now reaches U3.27 (IO19)
- net at U3.8 (EN): now also R17.2

Commit message: new
Parts:
- removed R17: 10K, symbol Device:R_Small_US
Connections:
- net ESP_EN: now reaches U3.8 (EN)
- net ESP_BOOT: now reaches U3.23 (IO9)
- net ESP_TXD: now reaches U3.30 (RXD0)
- net ESP_RXD: now reaches U3.31 (TXD0)
- no-connect marks 0 -> 10
Changed lines of the file:
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@@
 		(color 0 0 0 0)
+	)
+	(no_connect
+		(at 148.59 95.25)
+	)
+	(no_connect
+		(at 113.03 87.63)
+	)
+	(no_connect
+		(at 113.03 92.71)
+	)
+	(no_connect
+		(at 113.03 90.17)
+	)
+	(no_connect
+		(at 113.03 100.33)
+	)
+	(no_connect
+		(at 148.59 87.63)
+	)
+	(no_connect
+		(at 113.03 97.79)
+	)
+	(no_connect
+		(at 113.03 102.87)
+	)
+	(no_connect
+		(at 148.59 90.17)
+	)
+	(no_connect
+		(at 113.03 95.25)
 	)
 	(wire
@@
 	(wire
 		(pts
-			(xy 110.49 82.55) (xy 113.03 82.55)
-		)
-		(stroke
-			(width 0)
-			(type default)
-		)
-	)
-	(wire
-		(pts
-			(xy 102.87 81.28) (xy 102.87 82.55)
-		)
-		(stroke
-			(width 0)
-			(type default)
-		)
-	)
-	(wire
-		(pts
 			(xy 173.99 80.01) (xy 182.88 80.01)
-		)
-		(stroke
-			(width 0)
-			(type default)
-		)
-	)
-	(wire
-		(pts
-			(xy 102.87 82.55) (xy 105.41 82.55)
 		)
 		(stroke
@@
 		)
 	)
-	(label "ESP_D_N"
-		(at 158.75 97.79 0)
+	(text_box "IN THIS ESP THERE NO PIN FOR RESET. "
+		(exclude_from_sim no)
+		(at 66.04 48.26 0)
+		(size 40.64 13.97)
+		(stroke
+			(width 0)
+			(type default)
+		)
+		(fill
+			(type none)
+		)
+		(effects
+			(font
+				(size 2.54 2.54)
+				(thickness 0.508)
+				(bold yes)
+			)
+			(justify left top)
+		)
+	)
+	(global_label "ESP_TXD"
+		(shape input)
+		(at 113.03 107.95 180)
+		(fields_autoplaced yes)
 		(effects
 			(font
 				(size 1.27 1.27)
-				(color 18 255 0 1)
-			)
-			(justify left bottom)
-		)
-	)
-	(label "ESP_D_P"
-		(at 160.02 100.33 0)
+			)
+			(justify right)
+		)
+		(property "Intersheetrefs" "${INTERSHEET_REFS}"
+			(at 102.0016 107.95 0)
+			(effects
+				(font
+					(size 1.27 1.27)
+				)
+				(justify right)
+				(hide yes)
+			)
+		)
+	)
+	(global_label "ESP_D_N"
+		(shape input)
+		(at 158.75 97.79 0)
+		(fields_autoplaced yes)
 		(effects
 			(font
 				(size 1.27 1.27)
-				(color 18 255 0 1)
-			)
-			(justify left bottom)
+				(color 0 0 0 1)
+			)
+			(justify left)
+		)
+		(property "Intersheetrefs" "${INTERSHEET_REFS}"
+			(at 169.8994 97.79 0)
+			(effects
+				(font
+					(size 1.27 1.27)
+				)
+				(justify left)
+				(hide yes)
+			)
+		)
+	)
+	(global_label "ESP_RXD"
+		(shape input)
+		(at 113.03 110.49 180)
+		(fields_autoplaced yes)
+		(effects
+			(font
+				(size 1.27 1.27)
+			)
+			(justify right)
+		)
+		(property "Intersheetrefs" "${INTERSHEET_REFS}"
+			(at 101.6992 110.49 0)
+			(effects
+				(font
+					(size 1.27 1.27)
+				)
+				(justify right)
+				(hide yes)
+			)
+		)
+	)
+	(global_label "ESP_BOOT"
+		(shape input)
+		(at 148.59 92.71 0)
+		(fields_autoplaced yes)
+		(effects
+			(font
+				(size 1.27 1.27)
+			)
+			(justify left)
+		)
+		(property "Intersheetrefs" "${INTERSHEET_REFS}"
+			(at 161.0699 92.71 0)
+			(effects
+				(font
+					(size 1.27 1.27)
+				)
+				(justify left)
+				(hide yes)
+			)
+		)
+	)
+	(global_label "ESP_EN"
+		(shape input)
+		(at 113.03 82.55 180)
+		(fields_autoplaced yes)
+		(effects
+			(font
+				(size 1.27 1.27)
+			)
+			(justify right)
+		)
+		(property "Intersheetrefs" "${INTERSHEET_REFS}"
+			(at 102.9692 82.55 0)
+			(effects
+				(font
+					(size 1.27 1.27)
+				)
+				(justify right)
+				(hide yes)
+			)
+		)
+	)
+	(global_label "ESP_D_P"
+		(shape input)
+		(at 160.02 100.33 0)
+		(fields_autoplaced yes)
+		(effects
+			(font
+				(size 1.27 1.27)
+				(color 0 0 0 1)
+			)
+			(justify left)
+		)
+		(property "Intersheetrefs" "${INTERSHEET_REFS}"
+			(at 171.1089 100.33 0)
+			(effects
+				(font
+					(size 1.27 1.27)
+				)
+				(justify left)
+				(hide yes)
+			)
 		)
 	)
@@
 	)
 	(symbol
-		(lib_id "Device:R_Small_US")
-		(at 107.95 82.55 90)
-		(unit 1)
-		(exclude_from_sim no)
-		(in_bom yes)
-		(on_board yes)
-		(dnp no)
-		(property "Reference" "R17"
-			(at 106.172 80.772 0)
-			(effects
-				(font
-					(size 1.27 1.27)
-				)
-				(justify left)
-			)
-		)
-		(property "Value" "10K"
-			(at 109.474 81.28 0)
-			(effects
-				(font
-					(size 1.27 1.27)
-				)
-				(justify left)
-			)
-		)
-		(property "Footprint" ""
-			(at 107.95 82.55 0)
-			(effects
-				(font
-					(size 1.27 1.27)
-				)
-				(hide yes)
-			)
-		)
-		(property "Datasheet" "~"
-			(at 107.95 82.55 0)
-			(effects
-				(font
-					(size 1.27 1.27)
-				)
-				(hide yes)
-			)
-		)
-		(property "Description" "Resistor, small US symbol"
-			(at 107.95 82.55 0)
-			(effects
-				(font
-					(size 1.27 1.27)
-				)
-				(hide yes)
-			)
-		)
-		(pin "2"
-		)
-		(pin "1"
-		)
-		(instances
-			(project "GNSS"
-				(path "/a70dad34-b24c-4b58-b91c-f14576b5da7d/cd83e7ab-22db-42ff-a7e6-36d43df00222"
-					(reference "R17")
-					(unit 1)
-				)
-			)
-		)
-	)
-	(symbol
 		(lib_id "Device:C_Small")
 		(at 165.1 83.82 0)
@@
 					(unit 1)
 				)
-			)
-		)
-	)
-	(symbol
-		(lib_id "power:+3.3V")
-		(at 102.87 81.28 0)
-		(unit 1)
-		(exclude_from_sim no)
-		(in_bom yes)
-		(on_board yes)
-		(dnp no)
-		(fields_autoplaced yes)
-		(property "Reference" "#PWR053"
-			(at 102.87 85.09 0)
-			(effects
-				(font
-					(size 1.27 1.27)
-				)
-				(hide yes)
-			)
-		)
-		(property "Value" "+3.3V"
-			(at 102.87 76.2 0)
-			(effects
-				(font
-					(size 1.27 1.27)
-				)
-			)
-		)
-		(property "Footprint" ""
-			(at 102.87 81.28 0)
-			(effects
-				(font
-					(size 1.27 1.27)
-				)
-				(hide yes)
-			)
-		)
-		(property "Datasheet" ""
-			(at 102.87 81.28 0)
-			(effects
-				(font
-					(size 1.27 1.27)
-				)
-				(hide yes)
-			)
-		)
-		(property "Description" "Power symbol creates a global label with name \"+3.3V\""
-			(at 102.87 81.28 0)
-			(effects
-				(font
-					(size 1.27 1.27)
-				)
-				(hide yes)
-			)
-		)
-		(pin "1"
-		)
-		(instances
-			(project "GNSS"
-				(path "/a70dad34-b24c-4b58-b91c-f14576b5da7d/cd83e7ab-22db-42ff-a7e6-36d43df00222"
-					(reference "#PWR053")
-					(unit 1)
-				)

Commit message: new table
Changed lines of the file:
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@@
-		)
-	)
-	(text_box "IN THIS ESP THERE NO PIN FOR RESET. "
-		(exclude_from_sim no)
-		(at 66.04 48.26 0)
-		(size 40.64 13.97)
-		(stroke
-			(width 0)
-			(type default)
-		)
-		(fill
-			(type none)
-		)
-		(effects
-			(font
-				(size 2.54 2.54)
-				(thickness 0.508)
-				(bold yes)
-			)
-			(justify left top)
 		)
 	)

Commit message: new
Connections:
- net ESP_INT: now reaches U3.18 (IO4)
- no-connect marks 10 -> 9
Changed lines of the file:
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@@
-	)
-	(no_connect
-		(at 113.03 97.79)
 	)
 	(no_connect
@@
 			(effects
 				(font
+					(size 1.27 1.27)
+				)
+				(justify right)
+				(hide yes)
+			)
+		)
+	)
+	(global_label "ESP_INT"
+		(shape input)
+		(at 113.03 97.79 180)
+		(fields_autoplaced yes)
+		(effects
+			(font
+				(size 1.27 1.27)
+			)
+			(justify right)
+		)
+		(property "Intersheetrefs" "${INTERSHEET_REFS}"
+			(at 102.5458 97.79 0)
+			(effects
+				(font

Commit message: new can
Parts:
- added C68: 4.7nF, C0402C104K4RAC:CAPC1005X55N, symbol C0402C104K4RAC:C0402C104K4RAC
- added C69, C71: 100nF, C0402C104K4RAC:CAPC1005X55N, symbol C0402C104K4RAC:C0402C104K4RAC
- added C70, C72: 4.7uF, Capacitor_SMD:C_0805_2012Metric, symbol Device:C_Small
- added C73, C74: 100pF, C0402C104K4RAC:CAPC1005X55N, symbol C0402C104K4RAC:C0402C104K4RAC
- added D5, D6: ESD5V0D5-TP, ESD5V0D5TP, symbol ESD5V0D5-TP:ESD5V0D5-TP
- added R16, R26: 60R, Resistor_SMD:R_0805_2012Metric, symbol Device:R_Small_US
- added U5: TCAN1042VDRBRQ1, GNSS_Library:DRB0008F, symbol 2026-08-14_04-42-40:TCAN1042VDRBRQ1
Connections:
- net GND: now also C68.1, C69.1, C70.2, C71.1, C72.2, C73.1, C74.1, D5.1 (K), D6.1 (K), U5.2 (GND), U5.9 (PAD)
- new net: C68.2, R16.1, R26.1
- new net: C74.2, D6.2 (A), R26.2, U5.6 (CANL)
- new net: C73.2, D5.2 (A), R16.2, U5.7 (CANH)
- new net CAN_RXD: U5.4 (RXD)
- new net CAN_STB: U5.8 (STB)
- new net CAN_TXD: U5.1 (TXD)
- new net VIN: C69.2, C70.1, C71.2, C72.1, U5.3 (VCC), U5.5 (VIO)
Other:
- note added: "CAN_TRANS"
- note added: "WIFI"
- moved on the sheet: C27, C28, C31, U3
