File: ESP.kicad_sch (KiCad schematic)
At the start: 16 parts, among them U3 ESP32-C3-MINI-1-N4, U5 TCAN1042VDRBRQ1

Commit message: schamtic Update
Parts:
- removed D5, D6: ESD5V0D5-TP, ESD5V0D5TP, symbol ESD5V0D5-TP:ESD5V0D5-TP
- added D7: PESD2CANFD24V-TR, SOT95P230X110-3N, symbol PESD2CANFD24V-TR:PESD2CANFD24V-TR
Connections:
- net GND: now also D7.3 (CC)
- net at C74.2, R26.2, U5.6 (CANL): now also D7.2 (K2)
- net at C73.2, R16.2, U5.7 (CANH): now also D7.1 (K1)

Commit message: changed
Changed lines of the file:
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@@
 	(wire
 		(pts
-			(xy 220.98 102.87) (xy 209.55 102.87)
+			(xy 219.71 102.87) (xy 209.55 102.87)
 		)
 		(stroke
@@
 	(global_label "ESP_D_P"
 		(shape input)
-		(at 220.98 102.87 0)
+		(at 219.71 102.87 0)
 		(fields_autoplaced yes)
 		(effects
@@
 		)
 		(property "Intersheetrefs" "${INTERSHEET_REFS}"
-			(at 232.0689 102.87 0)
-			(effects
-				(font
+			(at 230.7989 102.87 0)
+			(effects
+				(font

Commit message: changed
Parts:
- removed C27: 47uF, Capacitor_SMD:C_0805_2012Metric, symbol Device:C_Small
- added C79: 10uF, Capacitor_SMD:C_0805_2012Metric, symbol Device:C_Small
- added L4: WE-CBF_0603, GNSS_Library:WE-CBF_0603_W2.6, symbol WE-CBF_0603:WE-CBF_0603
Connections:
- net +3.3V: now also C79.1, L4.1; no longer C31.2
- net GND: now also C79.2
- new net: C31.2, L4.2
Other:
- moved on the sheet: C31

Commit message: verification
Parts:
- added J7: Conn, Connector_PinHeader_1.00mm:PinHeader_1x03_P1.00mm_Vertical, symbol Connector:Conn_01x03_Pin
- added R43, R44, R45: 10K, Resistor_SMD:R_0805_2012Metric, symbol Device:R_Small_US
- added TP1: TestPoint, TestPoint:TestPoint_Pad_D2.0mm, symbol Connector:TestPoint
Connections:
- net +3.3V: now also L4.2, R43.1, R44.1, R45.1; no longer C28.2, C79.1, L4.1, U3.3 (3V3)
- net ESP_EN: now also R43.2
- net GND: now also J7.3 (Pin_3)
- net CANL: now reaches C74.2, D7.2 (K2), R26.2, U5.6 (CANL)
- net CANL: now also J7.2 (Pin_2)
- net at C31.2: now also C28.2, C79.1, L4.1, U3.3 (3V3); no longer L4.2
- net CANH: now reaches C73.2, D7.1 (K1), R16.2, U5.7 (CANH)
- net CANH: now also J7.1 (Pin_1)
- net IO8: now reaches U3.22 (IO8)
- net IO8: now also R45.2
- net at U3.5 (IO2): now also R44.2
- no-connect marks 9 -> 7
Other:
- moved on the sheet: C28, C79

Commit message: new
Parts:
- removed TP1: TestPoint, TestPoint:TestPoint_Pad_D2.0mm, symbol Connector:TestPoint
Changed lines of the file:
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@@
-		)
-	)
-	(text_box "C27 47uF 10uF is enough,fb included"
-		(exclude_from_sim no)
-		(at 214.63 64.77 0)
-		(size 21.59 11.43)
-		(stroke
-			(width 0)
-			(type default)
-		)
-		(fill
-			(type none)
-		)
-		(effects
-			(font
-				(size 1.27 1.27)
-			)
-			(justify left top)
 		)
 	)
@@
 					(unit 1)
 				)
-			)
-		)
-	)
-	(symbol
-		(lib_id "Connector:TestPoint")
-		(at 158.75 41.91 0)
-		(unit 1)
-		(exclude_from_sim no)
-		(in_bom yes)
-		(on_board yes)
-		(dnp no)
-		(fields_autoplaced yes)
-		(property "Reference" "TP1"
-			(at 161.29 37.3379 0)
-			(effects
-				(font
-					(size 1.27 1.27)
-				)
-				(justify left)
-			)
-		)
-		(property "Value" "TestPoint"
-			(at 161.29 39.8779 0)
-			(effects
-				(font
-					(size 1.27 1.27)
-				)
-				(justify left)
-			)
-		)
-		(property "Footprint" "TestPoint:TestPoint_Pad_D2.0mm"
-			(at 163.83 41.91 0)
-			(effects
-				(font
-					(size 1.27 1.27)
-				)
-				(hide yes)
-			)
-		)
-		(property "Datasheet" "~"
-			(at 163.83 41.91 0)
-			(effects
-				(font
-					(size 1.27 1.27)
-				)
-				(hide yes)
-			)
-		)
-		(property "Description" "test point"
-			(at 158.75 41.91 0)
-			(effects
-				(font
-					(size 1.27 1.27)
-				)
-				(hide yes)
-			)
-		)
-		(pin "1"
-		)
-		(instances
-			(project "GNSS"
-				(path "/a70dad34-b24c-4b58-b91c-f14576b5da7d/cd83e7ab-22db-42ff-a7e6-36d43df00222"
-					(reference "TP1")
-					(unit 1)
-				)

Commit message: new
Parts:
- removed C71: 100nF, C0402C104K4RAC:CAPC1005X55N, symbol C0402C104K4RAC:C0402C104K4RAC
- removed C72: 4.7uF, Capacitor_SMD:C_0805_2012Metric, symbol Device:C_Small
Connections:
- net +3.3V renamed +3.3V_ESP
- net VIN renamed VIN_CAN
Other:
- moved on the sheet: J7

Commit message: new
Parts:
- removed L4: WE-CBF_0603, GNSS_Library:WE-CBF_0603_W2.6, symbol WE-CBF_0603:WE-CBF_0603
- added C81: 1uF, Capacitor_SMD:C_0805_2012Metric, symbol Device:C_Small
- added FL1, FL2, FL3: BLM21PG221SN1D, BLM21PG221SN1D:BEADC2012X105N, symbol BLM21PG221SN1D:BLM21PG221SN1D
- added R70, R71, R74, R75: 10K, Resistor_SMD:R_0805_2012Metric, symbol Device:R_Small_US
- added R72, R73: 22E, Resistor_SMD:R_0805_2012Metric, symbol Device:R_Small_US
- added TP3: TestPoint, TestPoint:TestPoint_Pad_D2.0mm, symbol Connector:TestPoint
- U3: footprint Module:XCVR_ESP32-C3-MINI-1-N4 -> GNSS:XCVR_ESP32-C3-MINI-1-N4
- U5: footprint GNSS_Library:DRB0008F -> GNSS:DRB0008F
Connections:
- net +3.3V_ESP: now also C28.2, C31.2, C79.1, U3.3 (3V3), FL1.1, R70.2, R71.1, R74.2, R75.2
- net ESP_BOOT: now also TP3.1
- net ESP_EN: now also C81.1, R70.1
- net ESP_INT: now also R71.2
- net ESP_RXD: now also R73.1, R75.1; no longer U3.31 (TXD0)
- net ESP_TXD: now also R72.1, R74.1; no longer U3.30 (RXD0)
- net GND: now also C81.2
- net VIN_CAN: now also FL2.1; no longer U5.5 (VIO)
- new net: R73.2, U3.31 (TXD0)
- new net: R72.2, U3.30 (RXD0)
- new net +3.3V: FL1.2, FL3.2
- new net +3.3V_CAN: FL3.1, U5.5 (VIO)
- new net VIN: FL2.2
- no-connect marks 7 -> 8
Other:
- moved on the sheet: C28, C31, C68, C69, C70, C73, C74, C79, D7, J7, R16, R26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

Commit message: new
Parts:
- removed R43: 10K, Resistor_SMD:R_0805_2012Metric, symbol Device:R_Small_US
- added R94: 10K, Resistor_SMD:R_0805_2012Metric, symbol Device:R_Small_US
Connections:
- net +3.3V_ESP: now also R94.2
- net ESP_BOOT: now also R94.1
Other:
- moved on the sheet: C81, R70, TP3
