File: ESP.kicad_sch (KiCad schematic)
At the start: 28 parts, among them J7 Conn, U3 ESP32-C3-MINI-1-N4, U5 TCAN1042VDRBRQ1

Commit message: schematics
Parts:
- C69: footprint C0402C104K4RAC:CAPC1005X55N -> Capacitor_SMD:C_0402_1005Metric
Connections:
- net GND: no longer C69.1
Changed lines of the file:
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@@
 	)
 	(junction
+		(at 34.29 58.42)
+		(diameter 0)
+		(color 0 0 0 0)
+	)
+	(junction
 		(at 111.76 101.6)
 		(diameter 0)
@@
 	(wire
 		(pts
-			(xy 34.29 55.88) (xy 34.29 59.69)
+			(xy 34.29 55.88) (xy 34.29 58.42)
 		)
 		(stroke
@@
 	(wire
 		(pts
+			(xy 34.29 58.42) (xy 34.29 59.69)
+		)
+		(stroke
+			(width 0)
+			(type default)
+		)
+	)
+	(wire
+		(pts
 			(xy 111.76 119.38) (xy 115.57 119.38)
 		)
@@
 	)
 	(symbol
-		(lib_id "C0402C104K4RAC:C0402C104K4RAC")
-		(at 34.29 64.77 90)
-		(unit 1)
-		(exclude_from_sim no)
-		(in_bom yes)
-		(on_board yes)
-		(dnp no)
-		(property "Reference" "C69"
-			(at 29.972 61.214 90)
-			(effects
-				(font
-					(size 1.27 1.27)
-				)
-			)
-		)
-		(property "Value" "100nF"
-			(at 29.718 65.786 90)
-			(effects
-				(font
-					(size 1.27 1.27)
-				)
-			)
-		)
-		(property "Footprint" "C0402C104K4RAC:CAPC1005X55N"
-			(at 34.29 64.77 0)
-			(effects
-				(font
-					(size 1.27 1.27)
-				)
-				(justify bottom)
-				(hide yes)
-			)
-		)
-		(property "Datasheet" ""
-			(at 34.29 64.77 0)
-			(effects
-				(font
-					(size 1.27 1.27)
-				)
-				(hide yes)
-			)
-		)
-		(property "Description" "0.1 µF ±10% 16V Ceramic Capacitor X7R 0402 (1005 Metric)"
-			(at 34.29 64.77 0)
-			(effects
-				(font
-					(size 1.27 1.27)
-				)
-				(justify bottom)
-				(hide yes)
-			)
-		)
-		(property "MF" "KEMET"
-			(at 34.29 64.77 0)
-			(effects
-				(font
-					(size 1.27 1.27)
-				)
-				(justify bottom)
-				(hide yes)
-			)
-		)
-		(property "PACKAGE" "0402 KEMET"
-			(at 34.29 64.77 0)
-			(effects
-				(font
-					(size 1.27 1.27)
-				)
-				(justify bottom)
-				(hide yes)
-			)
-		)
-		(property "PRICE" "None"
-			(at 34.29 64.77 0)
-			(effects
-				(font
-					(size 1.27 1.27)
-				)
-				(justify bottom)
-				(hide yes)
-			)
-		)
-		(property "Package" "402-2 KEMET"
-			(at 34.29 64.77 0)
-			(effects
-				(font
-					(size 1.27 1.27)
-				)
-				(justify bottom)
-				(hide yes)
-			)
-		)
-		(property "Check_prices" "https://www.snapeda.com/parts/C0402C104K4RAC/Kemet/view-part/?ref=eda"
-			(at 34.29 64.77 0)
-			(effects
-				(font
-					(size 1.27 1.27)
-				)
-				(justify bottom)
-				(hide yes)
-			)
-		)
-		(property "Price" "None"
-			(at 34.29 64.77 0)
-			(effects
-				(font
-					(size 1.27 1.27)
-				)
-				(justify bottom)
-				(hide yes)
-			)
-		)
-		(property "SnapEDA_Link" "https://www.snapeda.com/parts/C0402C104K4RAC/Kemet/view-part/?ref=snap"
-			(at 34.29 64.77 0)
-			(effects
-				(font
-					(size 1.27 1.27)
-				)
-				(justify bottom)
-				(hide yes)
-			)
-		)
-		(property "MP" "C0402C104K4RAC"
-			(at 34.29 64.77 0)
-			(effects
-				(font
-					(size 1.27 1.27)
-				)
-				(justify bottom)
-				(hide yes)
-			)
-		)
-		(property "Purchase-URL" "https://www.snapeda.com/api/url_track_click_mouser/?unipart_id=1766586&manufacturer=KEMET&part_name=C0402C104K4RAC&search_term=None"
-			(at 34.29 64.77 0)
-			(effects
-				(font
-					(size 1.27 1.27)
-				)
-				(justify bottom)
-				(hide yes)
-			)
-		)
-		(property "Description_1" "\n                        \n                            0.1 µF ±10% 16V Ceramic Capacitor X7R 0402 (1005 Metric)\n                        \n"
-			(at 34.29 64.77 0)
-			(effects
-				(font
-					(size 1.27 1.27)
-				)
-				(justify bottom)
-				(hide yes)
-			)
-		)
-		(property "Availability" "In Stock"
-			(at 34.29 64.77 0)
-			(effects
-				(font
-					(size 1.27 1.27)
-				)
-				(justify bottom)
-				(hide yes)
-			)
-		)
-		(property "AVAILABILITY" "In Stock"
-			(at 34.29 64.77 0)
-			(effects
-				(font
-					(size 1.27 1.27)
-				)
-				(justify bottom)
-				(hide yes)
-			)
-		)
-		(property "PURCHASE-URL" "https://pricing.snapeda.com/search/part/C0402C104K4RAC/?ref=eda"
-			(at 34.29 64.77 0)
-			(effects
-				(font
-					(size 1.27 1.27)
-				)
-				(justify bottom)
-				(hide yes)
-			)
-		)
-		(pin "1"
-		)
-		(pin "2"
-		)
-		(instances
-			(project "GNSS"
-				(path "/a70dad34-b24c-4b58-b91c-f14576b5da7d/cd83e7ab-22db-42ff-a7e6-36d43df00222"
-					(reference "C69")
-					(unit 1)
-				)
-			)
-		)
-	)
-	(symbol
 		(lib_id "power:PWR_FLAG")
 		(at 38.1 106.68 0)
@@
 					(unit 1)
 				)
+			)
+		)
+	)
+	(symbol
+		(lib_id "C0402C104K4RAC:C0402C104K4RAC")
+		(at 34.29 63.5 90)
+		(unit 1)
+		(exclude_from_sim no)
+		(in_bom yes)
+		(on_board yes)
+		(dnp no)
+		(property "Reference" "C69"
+			(at 30.734 59.944 90)
+			(effects
+				(font
+					(size 1.27 1.27)
+				)
+			)
+		)
+		(property "Value" "100nF"
+			(at 30.48 64.516 90)
+			(effects
+				(font
+					(size 1.27 1.27)
+				)
+			)
+		)
+		(property "Footprint" "Capacitor_SMD:C_0402_1005Metric"
+			(at 34.29 63.5 0)
+			(effects
+				(font
+					(size 1.27 1.27)
+				)
+				(justify bottom)
+				(hide yes)
+			)
+		)
+		(property "Datasheet" ""
+			(at 34.29 63.5 0)
+			(effects
+				(font
+					(size 1.27 1.27)
+				)
+				(hide yes)
+			)
+		)
+		(property "Description" "0.1 µF ±10% 16V Ceramic Capacitor X7R 0402 (1005 Metric)"
+			(at 34.29 63.5 0)
+			(effects
+				(font
+					(size 1.27 1.27)
+				)
+				(justify bottom)
+				(hide yes)
+			)
+		)
+		(property "MF" "KEMET"
+			(at 34.29 63.5 0)
+			(effects
+				(font
+					(size 1.27 1.27)
+				)
+				(justify bottom)
+				(hide yes)
+			)
+		)
+		(property "PACKAGE" "0402 KEMET"
+			(at 34.29 63.5 0)
+			(effects
+				(font
+					(size 1.27 1.27)
+				)
+				(justify bottom)
+				(hide yes)
+			)
+		)
+		(property "PRICE" "None"
+			(at 34.29 63.5 0)
+			(effects
+				(font
+					(size 1.27 1.27)
+				)
+				(justify bottom)
+				(hide yes)
+			)
+		)
+		(property "Package" "402-2 KEMET"
+			(at 34.29 63.5 0)
+			(effects
+				(font
+					(size 1.27 1.27)
+				)
+				(justify bottom)
+				(hide yes)
+			)
+		)
+		(property "Check_prices" "https://www.snapeda.com/parts/C0402C104K4RAC/Kemet/view-part/?ref=eda"
+			(at 34.29 63.5 0)
+			(effects
+				(font
+					(size 1.27 1.27)
+				)
+				(justify bottom)
+				(hide yes)
+			)
+		)
+		(property "Price" "None"
+			(at 34.29 63.5 0)
+			(effects
+				(font
+					(size 1.27 1.27)
+				)
+				(justify bottom)
+				(hide yes)
+			)
+		)
+		(property "SnapEDA_Link" "https://www.snapeda.com/parts/C0402C104K4RAC/Kemet/view-part/?ref=snap"
+			(at 34.29 63.5 0)
+			(effects
+				(font
+					(size 1.27 1.27)
+				)
+				(justify bottom)
+				(hide yes)
+			)
+		)
+		(property "MP" "C0402C104K4RAC"
+			(at 34.29 63.5 0)
+			(effects
+				(font
+					(size 1.27 1.27)
+				)
+				(justify bottom)
+				(hide yes)
+			)
+		)
+		(property "Purchase-URL" "https://www.snapeda.com/api/url_track_click_mouser/?unipart_id=1766586&manufacturer=KEMET&part_name=C0402C104K4RAC&search_term=None"
+			(at 34.29 63.5 0)
+			(effects
+				(font
+					(size 1.27 1.27)
+				)
+				(justify bottom)
+				(hide yes)
+			)
+		)
+		(property "Description_1" "\n                        \n                            0.1 µF ±10% 16V Ceramic Capacitor X7R 0402 (1005 Metric)\n                        \n"
+			(at 34.29 63.5 0)
+			(effects
+				(font
+					(size 1.27 1.27)
+				)
+				(justify bottom)
+				(hide yes)
+			)
+		)
+		(property "Availability" "In Stock"
+			(at 34.29 63.5 0)
+			(effects
+				(font
+					(size 1.27 1.27)
+				)
+				(justify bottom)
+				(hide yes)
+			)
+		)
+		(property "AVAILABILITY" "In Stock"
+			(at 34.29 63.5 0)
+			(effects
+				(font
+					(size 1.27 1.27)
+				)
+				(justify bottom)
+				(hide yes)
+			)
+		)
+		(property "PURCHASE-URL" "https://pricing.snapeda.com/search/part/C0402C104K4RAC/?ref=eda"
+			(at 34.29 63.5 0)
+			(effects
+				(font
+					(size 1.27 1.27)
+				)
+				(justify bottom)
+				(hide yes)
+			)
+		)
+		(pin "1"
+		)
+		(pin "2"
+		)
+		(instances
+			(project "GNSS"
+				(path "/a70dad34-b24c-4b58-b91c-f14576b5da7d/cd83e7ab-22db-42ff-a7e6-36d43df00222"
+					(reference "C69")
+					(unit 1)
+				)

Commit message: placed
Parts:
- C28, C31: footprint C0402C104K4RAC:CAPC1005X55N -> Capacitor_SMD:C_0402_1005Metric
- C79: footprint Capacitor_SMD:C_0805_2012Metric -> Capacitor_SMD:C_0402_1005Metric
- R16, R26, R44, R45, R70, R71, R72, R73, R74, R75, R94: footprint Resistor_SMD:R_0805_2012Metric -> Resistor_SMD:R_0402_1005Metric
Changed lines of the file:
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@@
 	(text "WIFI"
 		(exclude_from_sim no)
-		(at 155.448 38.862 0)
+		(at 156.21 40.132 0)
 		(effects
 			(font
@@
 			)
 		)
-		(property "Footprint" "Resistor_SMD:R_0805_2012Metric"
+		(property "Footprint" "Resistor_SMD:R_0402_1005Metric"
 			(at 171.45 107.95 0)
 			(effects
@@
 			)
 		)
-		(property "Footprint" "Resistor_SMD:R_0805_2012Metric"
+		(property "Footprint" "Resistor_SMD:R_0402_1005Metric"
 			(at 243.84 106.68 0)
 			(effects
@@
 			)
 		)
-		(property "Footprint" "C0402C104K4RAC:CAPC1005X55N"
+		(property "Footprint" "Capacitor_SMD:C_0402_1005Metric"
 			(at 228.6 78.74 0)
 			(effects
@@
 			)
 		)
-		(property "Footprint" "Resistor_SMD:R_0805_2012Metric"
+		(property "Footprint" "Resistor_SMD:R_0402_1005Metric"
 			(at 90.17 113.03 0)
 			(effects
@@
 			)
 		)
-		(property "Footprint" "Capacitor_SMD:C_0805_2012Metric"
+		(property "Footprint" "Capacitor_SMD:C_0402_1005Metric"
 			(at 219.71 77.47 0)
 			(effects
@@
 			)
 		)
-		(property "Footprint" "Resistor_SMD:R_0805_2012Metric"
+		(property "Footprint" "Resistor_SMD:R_0402_1005Metric"
 			(at 90.17 105.41 0)
 			(effects
@@
 			)
 		)
-		(property "Footprint" "Resistor_SMD:R_0805_2012Metric"
+		(property "Footprint" "Resistor_SMD:R_0402_1005Metric"
 			(at 168.91 106.68 0)
 			(effects
@@
 			)
 		)
-		(property "Footprint" "C0402C104K4RAC:CAPC1005X55N"
+		(property "Footprint" "Capacitor_SMD:C_0402_1005Metric"
 			(at 240.03 78.74 0)
 			(effects
@@
 			)
 		)
-		(property "Footprint" "Resistor_SMD:R_0805_2012Metric"
+		(property "Footprint" "Resistor_SMD:R_0402_1005Metric"
 			(at 170.18 95.25 0)
 			(effects
@@
 			)
 		)
-		(property "Footprint" "Resistor_SMD:R_0805_2012Metric"
+		(property "Footprint" "Resistor_SMD:R_0402_1005Metric"
 			(at 223.52 128.27 0)
 			(effects
@@
 			)
 		)
-		(property "Footprint" "Resistor_SMD:R_0805_2012Metric"
+		(property "Footprint" "Resistor_SMD:R_0402_1005Metric"
 			(at 171.45 86.36 0)
 			(effects
@@
 			)
 		)
-		(property "Footprint" "Resistor_SMD:R_0805_2012Metric"
+		(property "Footprint" "Resistor_SMD:R_0402_1005Metric"
 			(at 196.85 123.19 0)
 			(effects
@@
 			)
 		)
-		(property "Footprint" "Resistor_SMD:R_0805_2012Metric"
+		(property "Footprint" "Resistor_SMD:R_0402_1005Metric"
 			(at 189.23 123.19 0)
 			(effects
@@
 			)
 		)
-		(property "Footprint" "Resistor_SMD:R_0805_2012Metric"
+		(property "Footprint" "Resistor_SMD:R_0402_1005Metric"
 			(at 252.73 87.63 0)
 			(effects

Commit message: usb
Parts:
- removed C68: 4.7nF, C0402C104K4RAC:CAPC1005X55N, symbol C0402C104K4RAC:C0402C104K4RAC
- removed C69: 100nF, Capacitor_SMD:C_0402_1005Metric, symbol C0402C104K4RAC:C0402C104K4RAC
- removed C70: 4.7uF, Capacitor_SMD:C_0805_2012Metric, symbol Device:C_Small
- removed C73, C74: 100pF, C0402C104K4RAC:CAPC1005X55N, symbol C0402C104K4RAC:C0402C104K4RAC
- removed D7: PESD2CANFD24V-TR, SOT95P230X110-3N, symbol PESD2CANFD24V-TR:PESD2CANFD24V-TR
- removed FL2, FL3: BLM21PG221SN1D, BLM21PG221SN1D:BEADC2012X105N, symbol BLM21PG221SN1D:BLM21PG221SN1D
- removed J7: Conn, Connector_PinHeader_1.00mm:PinHeader_1x03_P1.00mm_Vertical, symbol Connector:Conn_01x03_Pin
- removed R16, R26: 60R, Resistor_SMD:R_0402_1005Metric, symbol Device:R_Small_US
- removed U5: TCAN1042VDRBRQ1, GNSS:DRB0008F, symbol 2026-08-14_04-42-40:TCAN1042VDRBRQ1
- C28, C31: value 0.1uF -> 0.1u
- C79: value 10uF -> 10u
- C81: value 1uF -> 1u
- R72, R73: value 22E -> 22R
Other:
- note removed: "CAN_TRANS"
- moved on the sheet: C28, C31, C79, C81, FL1, R44, R45, R70, R71, R72, R73, R74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

Commit message: can
Parts:
- removed C28, C31: 0.1u, Capacitor_SMD:C_0402_1005Metric, symbol C0402C104K4RAC:C0402C104K4RAC
- removed C79: 10u, Capacitor_SMD:C_0402_1005Metric, symbol Device:C_Small
- removed C81: 1u, Capacitor_SMD:C_0805_2012Metric, symbol Device:C_Small
- removed FL1: BLM21PG221SN1D, BLM21PG221SN1D:BEADC2012X105N, symbol BLM21PG221SN1D:BLM21PG221SN1D
- removed R44, R45, R70, R71, R74, R75, R94: 10K, Resistor_SMD:R_0402_1005Metric, symbol Device:R_Small_US
- removed R72, R73: 22R, Resistor_SMD:R_0402_1005Metric, symbol Device:R_Small_US
- removed TP3: TestPoint, TestPoint:TestPoint_Pad_D2.0mm, symbol Connector:TestPoint
- removed U3: ESP32-C3-MINI-1-N4, GNSS:XCVR_ESP32-C3-MINI-1-N4, symbol ESP32-C3-MINI-1-N4:ESP32-C3-MINI-1-N4
- added C27: 100n, Capacitor_SMD:C_0402_1005Metric, symbol C0402C104K4RAC:C0402C104K4RAC
- added C65: 4u7, Capacitor_SMD:C_0805_2012Metric, symbol Device:C_Small
- added C68: 4n7, C0402C104K4RAC:CAPC1005X55N, symbol C0402C104K4RAC:C0402C104K4RAC
- added C69, C70: 100p, C0402C104K4RAC:CAPC1005X55N, symbol C0402C104K4RAC:C0402C104K4RAC
- added C73: 10uF, Capacitor_SMD:C_0805_2012Metric, symbol Device:C_Small
- added C74, C78: 0.1uF, C0402C104K4RAC:CAPC1005X55N, symbol C0402C104K4RAC:C0402C104K4RAC
- added C85: 1uF, Capacitor_SMD:C_0805_2012Metric, symbol Device:C_Small
- added FL2, FL3, FL9: BLM21PG221SN1D, BLM21PG221SN1D:BEADC2012X105N, symbol BLM21PG221SN1D:BLM21PG221SN1D
- added J2: Conn, Connector_PinHeader_1.00mm:PinHeader_1x03_P1.00mm_Vertical, symbol Connector:Conn_01x03_Pin
- added R16, R26: 60R, Resistor_SMD:R_0805_2012Metric, symbol Device:R_Small_US
- added R66, R92: 22E, Resistor_SMD:R_0805_2012Metric, symbol Device:R_Small_US
- added R77, R78, R93, R95, R96, R97, R98: 10K, Resistor_SMD:R_0805_2012Metric, symbol Device:R_Small_US
- added TP8: TestPoint, TestPoint:TestPoint_Pad_D2.0mm, symbol Connector:TestPoint
- added U15: ESP32-C3-MINI-1-N4, GNSS:XCVR_ESP32-C3-MINI-1-N4, symbol ESP32-C3-MINI-1-N4:ESP32-C3-MINI-1-N4
- added U5: TCAN1042VDRBRQ1, GNSS:DRB0008F, symbol 2026-08-14_04-42-40:TCAN1042VDRBRQ1
- added U8: TPD2EUSB30ADRTR, GNSS:SOTFL35P100X50-3N, symbol TPD2EUSB30ADRTR:TPD2EUSB30ADRTR
Connections:
- net +3.3V: now also FL3.2, FL9.2
- net +3.3V_ESP: now also C73.1, C74.2, C78.2, FL9.1, R77.1, R78.1, R93.2, R95.2, R96.2, R97.2, R98.1, U15.3 (3V3)
- net ESP_BOOT: now also R96.1, TP8.1, U15.23 (IO9)
- net ESP_D_N: now also U15.26 (IO18)
- net ESP_D_P: now also U15.27 (IO19)
- net ESP_EN: now also C85.1, R97.1, U15.8 (EN)
- net ESP_INT: now also R77.2, U15.18 (IO4)
- net ESP_RXD: now also R92.1, R95.1
- net ESP_TXD: now also R66.1, R93.1
- net GND: now also C27.1, C65.2, C68.1, C69.1, C70.1, C73.2, C74.1, C78.1, C85.2, J2.3 (Pin_3), U15.1 (GND), U15.11 (GND), U15.14 (GND), U15.2 (GND), U15.36 (GND), U15.37 (GND), U15.38 (GND), U15.39 (GND), U15.40 (GND), U15.41 (GND), U15.42 (GND), U15.43 (GND), U15.44 (GND), U15.45 (GND), U15.46 (GND), U15.47 (GND), U15.48 (GND), U15.49_1 (GND), U15.49_2 (GND), U15.49_3 (GND), U15.49_4 (GND), U15.49_5 (GND), U15.49_6 (GND), U15.49_7 (GND), U15.49_8 (GND), U15.49_9 (GND), U15.50 (GND), U15.51 (GND), U15.52 (GND), U15.53 (GND), U5.2 (GND), U5.9 (PAD), U8.3 (GND)
- net IO8: now also R98.2, U15.22 (IO8)
- new net: R78.2, U15.5 (IO2)
- new net: R92.2, U15.31 (TXD0)
- new net: C68.2, R16.1, R26.1
- new net: R66.2, U15.30 (RXD0)
- new net: U15.10 (NC), U15.15 (NC), U15.17 (NC), U15.24 (NC), U15.25 (NC), U15.28 (NC), U15.29 (NC), U15.32 (NC), U15.33 (NC), U15.34 (NC), U15.35 (NC), U15.4 (NC), U15.7 (NC), U15.9 (NC)
- new net +3.3V_CAN: FL3.1, U5.5 (VIO)
- new net CANH: C69.2, J2.1 (Pin_1), R16.2, U5.7 (CANH), U8.1 (D+)
- new net CANL: C70.2, J2.2 (Pin_2), R26.2, U5.6 (CANL), U8.2 (D-)
- new net CAN_RXD: U5.4 (RXD)
- new net CAN_STB: U5.8 (STB)
- new net CAN_TXD: U5.1 (TXD)
- new net VIN: FL2.2
- new net VIN_CAN: C27.2, C65.1, FL2.1, U5.3 (VCC)
Other:
- note added: "CAN_TRANS"
