File: Ethernet.kicad_sch (KiCad schematic)
At the start: 0 parts

Commit message: new update
Parts:
- added T1: WE-RJ45_7499010211A, Module:7499010211A, symbol WE-RJ45_7499010211A:WE-RJ45_7499010211A
Connections:
- new net GND: T1.S1 (SHIELD1), T1.S2 (SHIELD2)
- no-connect marks 0 -> 1

Commit message: new
Parts:
- added U4: DP83825IRMQR, GNSS_Library:XCVR_DP83825IRMQR, symbol DP83825IRMQR:DP83825IRMQR
Connections:
- net GND renamed EXP
- net EXP: now also U4.21 (GND), U4.25 (EXP), U4.26 (EXP), U4.27 (EXP), U4.28 (EXP), U4.29 (EXP), U4.30 (EXP), U4.9 (GND)
Other:
- moved on the sheet: T1

Commit message: new
Parts:
- added C53, C59, C61, C64: 100nF, C0402C104K4RAC:CAPC1005X55N, symbol C0402C104K4RAC:C0402C104K4RAC
- added C54, C60: 10nF, C0402C104K4RAC:CAPC1005X55N, symbol C0402C104K4RAC:C0402C104K4RAC
- added C55, C58, C62, C63: 1uF, Capacitor_SMD:C_0805_2012Metric, symbol Device:C_Small
- added C56, C57: 10uF, Capacitor_SMD:C_0805_2012Metric, symbol Device:C_Small
- added C65, C66: 20pF, C0402C104K4RAC:CAPC1005X55N, symbol C0402C104K4RAC:C0402C104K4RAC
- added L2, L3: WE-CBF_0603, GNSS_Library:WE-CBF_0603_W2.6, symbol WE-CBF_0603:WE-CBF_0603
- added R21: 6.49K, symbol Device:R_Small_US
- added R22, R23: 470R, symbol Device:R_Small_US
- added R24: 10K, symbol Device:R_Small_US
- added Y3: ECS-250-12-33-AGN-TR, GNSS_Library:XTAL_ECS-250-12-33-AGN-TR, symbol ECS-250-12-33-AGN-TR:ECS-250-12-33-AGN-TR
Connections:
- net EXP: now also T1.8, C53.1, C54.1, C55.2, C56.2, C57.2, C58.2, C59.1, C60.1, C61.1, C62.2, C63.2, C64.1, C65.1, C66.1, R21.1, Y3.2 (GND), Y3.4 (GND)
- net ETH_TX_EN: now reaches U4.1 (TX_EN)
- net at U4.10 (TD_M): now also T1.2 (TD-)
- net at U4.11 (TD_P): now also T1.1 (TD+)
- net CLK_XI: now reaches U4.13 (XI/50MHZIN)
- net CLK_XI: now also C66.2, Y3.3 (OUT/IN)
- net at U4.14 (RBIAS): now also R21.2
- net ETH_MDIO: now reaches U4.15 (MDIO)
- net ETH_MDC: now reaches U4.16 (MDC)
- net ETH_RX_D1: now reaches U4.17 (RX_D1/S(MASTER/SLAVE))
- net ETH_RX_D0: now reaches U4.18 (RX_D0/S(PHYADD0))
- net VDDIO: now reaches U4.19 (VDDIO)
- net VDDIO: now also C53.2, C54.2, C55.1, C56.1, L3.1
- net 50MHZOUT: now reaches U4.2 (50MHZOUT/LED2/S(RX_DV_EN))
- net 50MHZOUT: now also C65.2, R22.2, Y3.1 (IN/OUT)
- net ETH_CRS_DV: now reaches U4.20 (CRS_DV/S(PHYADD1))
- net ETH_TX_D0: now reaches U4.23 (TX_D0)
- net ETH_TX_D1: now reaches U4.24 (TX_D1)
- net LED_LINK: now reaches U4.4 (LED0/S(ANEG_DIS))
- net LED_LINK: now also R23.1
- net ETH_RST_N: now reaches U4.5 (~{RST})
- net ETH_RST_N: now also R24.1
- net VDDA3V3: now reaches U4.6 (VDDA3V3)
- net VDDA3V3: now also C57.1, C58.1, C59.2, C60.2, L2.1
- net at U4.7 (RD_M): now also T1.6 (RD-)
- net at U4.8 (RD_P): now also T1.3 (RD+)
- net at T1.10: now also R23.2
- net at T1.11: now also R22.1
- net +3.3V: now reaches T1.12
- net +3.3V: now also T1.9, L2.2, L3.2
- net CTD: now reaches T1.4 (CTD)
- net CTD: now also C63.1, C64.2
- net CRD: now reaches T1.5 (CRD)
- net CRD: now also C61.2, C62.1
- no-connect marks 1 -> 4
Other:
- moved on the sheet: T1, U4

Commit message: new can
Connections:
- net +3.3V: now also R24.2
- net ETH_RST_N: no longer R24.1, U4.5 (~{RST})
- new net: R24.1, U4.5 (~{RST})
Other:
- note added: "ETHERNET"
Changed lines of the file:
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@@
-	)
-	(junction
-		(at 118.11 97.79)
-		(diameter 0)
-		(color 0 0 0 0)
 	)
 	(junction
@@
 	(wire
 		(pts
+			(xy 118.11 86.36) (xy 118.11 88.9)
+		)
+		(stroke
+			(width 0)
+			(type default)
+		)
+	)
+	(wire
+		(pts
 			(xy 48.26 110.49) (xy 54.61 110.49)
 		)
@@
 	(wire
 		(pts
-			(xy 115.57 97.79) (xy 118.11 97.79)
-		)
-		(stroke
-			(width 0)
-			(type default)
-		)
-	)
-	(wire
-		(pts
 			(xy 99.06 118.11) (xy 102.87 118.11)
 		)
@@
 			(width 0)
 			(type default)
+		)
+	)
+	(text "ETHERNET"
+		(exclude_from_sim no)
+		(at 37.084 34.798 0)
+		(effects
+			(font
+				(size 2.54 2.54)
+				(bold yes)
+			)
 		)
 	)
@@
 	(global_label "ETH_RST_N"
 		(shape input)
-		(at 115.57 97.79 180)
+		(at 118.11 71.12 180)
 		(fields_autoplaced yes)
 		(effects
@@
 		)
 		(property "Intersheetrefs" "${INTERSHEET_REFS}"
-			(at 102.4249 97.79 0)
+			(at 104.9649 71.12 0)
 			(effects
 				(font
@@
 					(unit 1)
 				)
+			)
+		)
+	)
+	(symbol
+		(lib_id "power:+3.3V")
+		(at 118.11 86.36 0)
+		(unit 1)
+		(exclude_from_sim no)
+		(in_bom yes)
+		(on_board yes)
+		(dnp no)
+		(fields_autoplaced yes)
+		(property "Reference" "#PWR0129"
+			(at 118.11 90.17 0)
+			(effects
+				(font
+					(size 1.27 1.27)
+				)
+				(hide yes)
+			)
+		)
+		(property "Value" "+3.3V"
+			(at 118.11 81.28 0)
+			(effects
+				(font
+					(size 1.27 1.27)
+				)
+			)
+		)
+		(property "Footprint" ""
+			(at 118.11 86.36 0)
+			(effects
+				(font
+					(size 1.27 1.27)
+				)
+				(hide yes)
+			)
+		)
+		(property "Datasheet" ""
+			(at 118.11 86.36 0)
+			(effects
+				(font
+					(size 1.27 1.27)
+				)
+				(hide yes)
+			)
+		)
+		(property "Description" "Power symbol creates a global label with name \"+3.3V\""
+			(at 118.11 86.36 0)
+			(effects
+				(font
+					(size 1.27 1.27)
+				)
+				(hide yes)
+			)
+		)
+		(pin "1"
+		)
+		(instances
+			(project "GNSS"
+				(path "/a70dad34-b24c-4b58-b91c-f14576b5da7d/a33a7fbe-117f-40f3-9eeb-50ee11d7c18f"
+					(reference "#PWR0129")
+					(unit 1)
+				)

Commit message: schamtic Update
Connections:
- net ETH_RST_N: now also R24.1, U4.5 (~{RST})
Other:
- note added: "DE-CAPS"
- moved on the sheet: C53, C54, C55, C56, C57, C58, C59, C60, C61, C62, C63, C64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

Commit message: changed
Parts:
- removed C66: 20pF, C0402C104K4RAC:CAPC1005X55N, symbol C0402C104K4RAC:C0402C104K4RAC
- removed Y3: ECS-250-12-33-AGN-TR, GNSS_Library:XTAL_ECS-250-12-33-AGN-TR, symbol ECS-250-12-33-AGN-TR:ECS-250-12-33-AGN-TR
- added C27: 20pF, C0402C104K4RAC:CAPC1005X55N, symbol C0402C104K4RAC:C0402C104K4RAC
- added R35: 330R, symbol Device:R_Small_US
- added Y2: ECS-250-12-33-AGN-TR, GNSS_Library:XTAL_ECS-250-12-33-AGN-TR, symbol ECS-250-12-33-AGN-TR:ECS-250-12-33-AGN-TR
Connections:
- net 50MHZOUT: no longer C65.2
- net CLK_XI: now also C27.2, Y2.3 (OUT/IN)
- net EXP: now also C27.1, Y2.2 (GND), Y2.4 (GND)
- net CLK_XO: now reaches U4.12 (XO)
- net CLK_XO: now also C65.2, R35.2
- new net: R35.1, Y2.1 (IN/OUT)
- no-connect marks 4 -> 3
Other:
- moved on the sheet: C65
