File: Ethernet.kicad_sch (KiCad schematic)
At the start: 24 parts, among them T1 WE-RJ45_7499010211A, U4 DP83825IRMQR, Y2 ECS-250-12-33-AGN-TR

Commit message: new
Changed lines of the file:
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@@
-		)
-	)
-	(text_box "OSCILLATOR CHANGED TO XO FROM 50MHZOUT"
-		(exclude_from_sim no)
-		(at 209.55 62.23 0)
-		(size 31.75 20.32)
-		(stroke
-			(width 0)
-			(type default)
-		)
-		(fill
-			(type none)
-		)
-		(effects
-			(font
-				(size 1.27 1.27)
-			)
-			(justify left top)
 		)
 	)

Commit message: new
Parts:
- removed C53: 100nF, C0402C104K4RAC:CAPC1005X55N, symbol C0402C104K4RAC:C0402C104K4RAC
- removed C54: 10nF, C0402C104K4RAC:CAPC1005X55N, symbol C0402C104K4RAC:C0402C104K4RAC
- removed C55: 1uF, Capacitor_SMD:C_0805_2012Metric, symbol Device:C_Small
- removed C56: 10uF, Capacitor_SMD:C_0805_2012Metric, symbol Device:C_Small
- removed L3: WE-CBF_0603, GNSS_Library:WE-CBF_0603_W2.6, symbol WE-CBF_0603:WE-CBF_0603
Connections:
- net +3.3V: no longer L2.2
- net VDDA3V3: no longer names the net of C57.1, C58.1, C59.2, C60.2, L2.1
- net VDDA3V3: no longer U4.6 (VDDA3V3)
- net VDDIO renamed +3.3V_ETH
- net +3.3V_ETH: now also L2.2, U4.6 (VDDA3V3)
Other:
- moved on the sheet: C57, C58, C59, C60, L2

Commit message: change
Parts:
- removed C62, C63: 1uF, Capacitor_SMD:C_0805_2012Metric, symbol Device:C_Small
- removed R24: 10K, symbol Device:R_Small_US
- added R48, R49, R50, R51: 10K, Resistor_SMD:R_0805_2012Metric, symbol Device:R_Small_US
- C61, C64: value 100nF -> 10nF
Connections:
- net +3.3V_ETH: now also R48.1, R49.1, R50.1, R51.1
- net ETH_MDC: now also R49.2
- net ETH_MDIO: now also R50.2
- net ETH_RST_N: now also R48.2
- net ETH_INTR: now reaches U4.3 (INTR/PWRDN)
- net ETH_INTR: now also R51.2
- no-connect marks 3 -> 2

Commit message: new
Parts:
- removed L2: WE-CBF_0603, GNSS_Library:WE-CBF_0603_W2.6, symbol WE-CBF_0603:WE-CBF_0603
- removed R22: 470R, symbol Device:R_Small_US
- removed R35: 330R, symbol Device:R_Small_US
- added FL11: BLM21PG221SN1D, BLM21PG221SN1D:BEADC2012X105N, symbol BLM21PG221SN1D:BLM21PG221SN1D
- added L4: WE-CBF_0603, GNSS_Library:WE-CBF_0603_W2.6, symbol WE-CBF_0603:WE-CBF_0603
- C27, C65: value 20pF -> 27pF
- C57: value 10uF -> 1uF
- C60: value 10nF -> 100nF
- R49, R50: value 10K -> 2.2K
- T1: footprint Module:7499010211A -> GNSS:7499010211A
- U4: footprint GNSS_Library:XCVR_DP83825IRMQR -> GNSS:XCVR_DP83825IRMQR
- Y2: footprint GNSS_Library:XTAL_ECS-250-12-33-AGN-TR -> GNSS:XTAL_ECS-250-12-33-AGN-TR
Connections:
- net CLK_XO is gone; now on net XTAL_OUT: C65.2, U4.12 (XO)
- net +3.3V: now also FL11.2; no longer T1.12, T1.9
- net +3.3V_ETH: now also C57.1, C58.1, C59.2, C60.2, T1.9, FL11.1
- net EXP: no longer C27.1, C57.2, C58.2, C59.1, C60.1, C61.1, C64.1, C65.1, R21.1, T1.8, T1.S1 (SHIELD1), T1.S2 (SHIELD2), U4.21 (GND), U4.9 (GND), Y2.2 (GND), Y2.4 (GND)
- net XTAL_OUT: now reaches Y2.1 (IN/OUT)
- net 50MHZOUT renamed ETH_REFCLK
- net CLK_XI renamed XTAL_IN
- net CRD: no longer names the net of C61.2, T1.5 (CRD)
- net CTD: no longer names the net of C64.2, T1.4 (CTD)
- new net: L4.1, T1.8, T1.S1 (SHIELD1), T1.S2 (SHIELD2)
- new net GND: C27.1, C57.2, C58.2, C59.1, C60.1, C61.1, C64.1, C65.1, L4.2, R21.1, U4.21 (GND), U4.9 (GND), Y2.2 (GND), Y2.4 (GND)
- no-connect marks 2 -> 4
Other:
- note added: "CRYSTAL"
- note removed: "DE-CAPS"
- moved on the sheet: C27, C57, C58, C59, C60, C61, C64, C65, R21, R48, R49, R50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

Commit message: new
Connections:
- net GND is gone; now on net EXP: C27.1, C57.2, C58.2, C59.1, C60.1, C61.1, C64.1, C65.1, L4.2, R21.1, U4.21 (GND), U4.9 (GND), Y2.2 (GND), Y2.4 (GND)
Changed lines of the file:
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@@
 	(paper "A4")
 	(junction
-		(at 223.52 109.22)
+		(at 233.68 64.77)
 		(diameter 0)
 		(color 0 0 0 0)
@@
 		(color 0 0 0 0)
 	)
+	(junction
+		(at 208.28 109.22)
+		(diameter 0)
+		(color 0 0 0 0)
+	)
+	(junction
+		(at 180.34 106.68)
+		(diameter 0)
+		(color 0 0 0 0)
+	)
 	(no_connect
 		(at 67.31 76.2)
@@
 	(wire
 		(pts
-			(xy 223.52 109.22) (xy 228.6 109.22)
+			(xy 242.57 109.22) (xy 242.57 107.95)
 		)
 		(stroke
@@
 	(wire
 		(pts
-			(xy 242.57 109.22) (xy 242.57 107.95)
+			(xy 229.87 90.17) (xy 233.68 90.17)
 		)
 		(stroke
@@
 	(wire
 		(pts
-			(xy 229.87 90.17) (xy 233.68 90.17)
+			(xy 87.63 170.18) (xy 88.9 170.18)
 		)
 		(stroke
@@
 	(wire
 		(pts
-			(xy 87.63 170.18) (xy 88.9 170.18)
+			(xy 96.52 60.96) (xy 96.52 52.07)
 		)
 		(stroke
@@
 	(wire
 		(pts
-			(xy 96.52 60.96) (xy 96.52 52.07)
+			(xy 218.44 68.58) (xy 224.79 68.58)
 		)
 		(stroke
@@
 	(wire
 		(pts
-			(xy 218.44 68.58) (xy 224.79 68.58)
+			(xy 176.53 104.14) (xy 180.34 104.14)
 		)
 		(stroke
@@
 	(wire
 		(pts
-			(xy 217.17 109.22) (xy 223.52 109.22)
+			(xy 217.17 109.22) (xy 228.6 109.22)
 		)
 		(stroke
@@
 	(wire
 		(pts
-			(xy 245.11 100.33) (xy 242.57 100.33)
+			(xy 246.38 100.33) (xy 242.57 100.33)
 		)
 		(stroke
@@
 	(wire
 		(pts
+			(xy 180.34 104.14) (xy 180.34 106.68)
+		)
+		(stroke
+			(width 0)
+			(type default)
+		)
+	)
+	(wire
+		(pts
 			(xy 96.52 52.07) (xy 66.04 52.07)
 		)
@@
 	(symbol
 		(lib_id "power:GND")
-		(at 223.52 109.22 0)
+		(at 208.28 109.22 0)
 		(unit 1)
 		(exclude_from_sim no)
@@
 		(fields_autoplaced yes)
 		(property "Reference" "#PWR099"
-			(at 223.52 115.57 0)
+			(at 208.28 115.57 0)
 			(effects
 				(font
@@
 		)
 		(property "Value" "GND"
-			(at 223.52 114.3 0)
+			(at 208.28 114.3 0)
 			(effects
 				(font
@@
 		)
 		(property "Footprint" ""
-			(at 223.52 109.22 0)
+			(at 208.28 109.22 0)
 			(effects
 				(font
@@
 		)
 		(property "Datasheet" ""
-			(at 223.52 109.22 0)
+			(at 208.28 109.22 0)
 			(effects
 				(font
@@
 		)
 		(property "Description" "Power symbol creates a global label with name \"GND\" , ground"
-			(at 223.52 109.22 0)
+			(at 208.28 109.22 0)
 			(effects
 				(font
@@
 	)
 	(symbol
+		(lib_id "power:PWR_FLAG")
+		(at 233.68 64.77 90)
+		(unit 1)
+		(exclude_from_sim no)
+		(in_bom yes)
+		(on_board yes)
+		(dnp no)
+		(fields_autoplaced yes)
+		(property "Reference" "#FLG013"
+			(at 231.775 64.77 0)
+			(effects
+				(font
+					(size 1.27 1.27)
+				)
+				(hide yes)
+			)
+		)
+		(property "Value" "PWR_FLAG"
+			(at 228.6 64.77 0)
+			(effects
+				(font
+					(size 1.27 1.27)
+				)
+				(hide yes)
+			)
+		)
+		(property "Footprint" ""
+			(at 233.68 64.77 0)
+			(effects
+				(font
+					(size 1.27 1.27)
+				)
+				(hide yes)
+			)
+		)
+		(property "Datasheet" "~"
+			(at 233.68 64.77 0)
+			(effects
+				(font
+					(size 1.27 1.27)
+				)
+				(hide yes)
+			)
+		)
+		(property "Description" "Special symbol for telling ERC where power comes from"
+			(at 233.68 64.77 0)
+			(effects
+				(font
+					(size 1.27 1.27)
+				)
+				(hide yes)
+			)
+		)
+		(pin "1"
+		)
+		(instances
+			(project "GNSS"
+				(path "/a70dad34-b24c-4b58-b91c-f14576b5da7d/a33a7fbe-117f-40f3-9eeb-50ee11d7c18f"
+					(reference "#FLG013")
+					(unit 1)
+				)
+			)
+		)
+	)
+	(symbol
 		(lib_id "DP83825IRMQR:DP83825IRMQR")
 		(at 146.05 81.28 0)
@@
 	(symbol
 		(lib_id "power:+3.3V")
-		(at 245.11 100.33 0)
+		(at 246.38 100.33 0)
 		(unit 1)
 		(exclude_from_sim no)
@@
 		(fields_autoplaced yes)
 		(property "Reference" "#PWR0100"
-			(at 245.11 104.14 0)
+			(at 246.38 104.14 0)
 			(effects
 				(font
@@
 		)
 		(property "Value" "+3.3V_ETH"
-			(at 245.11 95.25 0)
+			(at 246.38 95.25 0)
 			(effects
 				(font
@@
 		)
 		(property "Footprint" ""
-			(at 245.11 100.33 0)
+			(at 246.38 100.33 0)
 			(effects
 				(font
@@
 		)
 		(property "Datasheet" ""
-			(at 245.11 100.33 0)
+			(at 246.38 100.33 0)
 			(effects
 				(font
@@
 		)
 		(property "Description" "Power symbol creates a global label with name \"+3.3V\""
-			(at 245.11 100.33 0)
+			(at 246.38 100.33 0)
 			(effects
 				(font

Commit message: placed
Parts:
- C27, C59, C60, C61, C64, C65: footprint C0402C104K4RAC:CAPC1005X55N -> Capacitor_SMD:C_0402_1005Metric
- R21, R23: footprint (none) -> Resistor_SMD:R_0402_1005Metric
- R48, R49, R50, R51: footprint Resistor_SMD:R_0805_2012Metric -> Resistor_SMD:R_0402_1005Metric
Changed lines of the file:
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@@
 			)
 		)
-		(property "Footprint" "Resistor_SMD:R_0805_2012Metric"
+		(property "Footprint" "Resistor_SMD:R_0402_1005Metric"
 			(at 227.33 90.17 0)
 			(effects
@@
 			)
 		)
-		(property "Footprint" ""
+		(property "Footprint" "Resistor_SMD:R_0402_1005Metric"
 			(at 53.34 78.74 0)
 			(effects
@@
 			)
 		)
-		(property "Footprint" "Resistor_SMD:R_0805_2012Metric"
+		(property "Footprint" "Resistor_SMD:R_0402_1005Metric"
 			(at 227.33 74.93 0)
 			(effects
@@
 			)
 		)
-		(property "Footprint" "Resistor_SMD:R_0805_2012Metric"
+		(property "Footprint" "Resistor_SMD:R_0402_1005Metric"
 			(at 227.33 82.55 0)
 			(effects
@@
 			)
 		)
-		(property "Footprint" "C0402C104K4RAC:CAPC1005X55N"
+		(property "Footprint" "Capacitor_SMD:C_0402_1005Metric"
 			(at 96.52 100.33 0)
 			(effects
@@
 			)
 		)
-		(property "Footprint" "C0402C104K4RAC:CAPC1005X55N"
+		(property "Footprint" "Capacitor_SMD:C_0402_1005Metric"
 			(at 104.14 100.33 0)
 			(effects
@@
 			)
 		)
-		(property "Footprint" "C0402C104K4RAC:CAPC1005X55N"
+		(property "Footprint" "Capacitor_SMD:C_0402_1005Metric"
 			(at 99.06 171.45 0)
 			(effects
@@
 			)
 		)
-		(property "Footprint" "C0402C104K4RAC:CAPC1005X55N"
+		(property "Footprint" "Capacitor_SMD:C_0402_1005Metric"
 			(at 228.6 105.41 0)
 			(effects
@@
 			)
 		)
-		(property "Footprint" ""
+		(property "Footprint" "Resistor_SMD:R_0402_1005Metric"
 			(at 115.57 101.6 0)
 			(effects
@@
 			)
 		)
-		(property "Footprint" "Resistor_SMD:R_0805_2012Metric"
+		(property "Footprint" "Resistor_SMD:R_0402_1005Metric"
 			(at 227.33 68.58 0)
 			(effects
@@
 			)
 		)
-		(property "Footprint" "C0402C104K4RAC:CAPC1005X55N"
+		(property "Footprint" "Capacitor_SMD:C_0402_1005Metric"
 			(at 41.91 171.45 0)
 			(effects
@@
 			)
 		)
-		(property "Description" "0.1 µF ±10% 16V Ceramic Capacitor X7R 0402 (1005 Metric)"
+		(property "Description" "Capacitor_SMD:C_0402_1005Metric"
 			(at 41.91 171.45 0)
 			(effects
@@
 			)
 		)
-		(property "Footprint" "C0402C104K4RAC:CAPC1005X55N"
+		(property "Footprint" "Capacitor_SMD:C_0402_1005Metric"
 			(at 242.57 105.41 0)
 			(effects

Commit message: Almost Placed file
Parts:
- L4: footprint GNSS_Library:WE-CBF_0603_W2.6 -> Resistor_SMD:R_0201_0603Metric
Changed lines of the file:
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@@
 			)
 		)
-		(property "Footprint" "GNSS_Library:WE-CBF_0603_W2.6"
+		(property "Footprint" "Resistor_SMD:R_0201_0603Metric"
 			(at 83.82 106.68 0)
 			(effects

Commit message: usb
Parts:
- removed C27, C65: 27pF, Capacitor_SMD:C_0402_1005Metric, symbol C0402C104K4RAC:C0402C104K4RAC
- removed Y2: ECS-250-12-33-AGN-TR, GNSS:XTAL_ECS-250-12-33-AGN-TR, symbol ECS-250-12-33-AGN-TR:ECS-250-12-33-AGN-TR
- added C66, C77: 18p, C0402C104K4RAC:CAPC1005X55N, symbol C0402C104K4RAC:C0402C104K4RAC
- added R22: 1M, Resistor_SMD:R_0402_1005Metric, symbol Device:R_Small_US
- added Y4: MURATA_XRCGB24M000FFS1DR0, GNSS:MURATA_XRCGB24M000FFS1DR0_0, symbol MURATA_XRCGB24M000FFS1DR0:MURATA_XRCGB24M000FFS1DR0
- C57, C58: value 1uF -> 1u
- C59, C60: value 100nF -> 100n
- C61, C64: value 10nF -> 10n
- R21: value 6.49K -> 6K49
- R49, R50: value 2.2K -> 2K2
Connections:
- net EXP: now also C66.2, C77.2
- net XTAL_IN: now also C77.1, R22.1, Y4.3
- net XTAL_OUT: now also C66.1, R22.2, Y4.1
- no-connect marks 4 -> 6
