File: Ethernet.kicad_sch (KiCad schematic)
At the start: 20 parts, among them T1 WE-RJ45_7499010211A, U4 DP83825IRMQR, Y4 MURATA_XRCGB24M000FFS1DR0

Commit message: full
Changed lines of the file:
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@@
 		)
 	)
-	(text_box ""
-		(exclude_from_sim no)
-		(at 25.4 144.78 0)
-		(size 99.06 49.53)
+	(rectangle
+		(start 30.48 148.59)
+		(end 115.57 195.58)
 		(stroke
 			(width 0.0508)
@@
 			(type none)
 		)
-		(effects
-			(font
-				(size 1.27 1.27)
-			)
-			(justify left top)
-		)
 	)
-	(text_box ""
-		(exclude_from_sim no)
-		(at 22.86 38.1 0)
-		(size 233.68 87.63)
+	(rectangle
+		(start 25.4 38.1)
+		(end 256.54 123.19)
 		(stroke
 			(width 0.0508)
@@
 		(fill
 			(type none)
-		)
-		(effects
-			(font
-				(size 1.27 1.27)
-			)
-			(justify left top)
 		)
 	)
@@
 	(text "CRYSTAL"
 		(exclude_from_sim no)
-		(at 33.02 140.97 0)
+		(at 38.354 144.78 0)
 		(effects
 			(font

Commit message: 16.09.2026
Parts:
- C66, C77: footprint C0402C104K4RAC:CAPC1005X55N -> Capacitor_SMD:C_0402_1005Metric
- FL11: footprint BLM21PG221SN1D:BEADC2012X105N -> GNSS:BEADC2012X105N
- Y4: footprint GNSS:MURATA_XRCGB24M000FFS1DR0_0 -> GNSS:XTAL_ECS-250-12-33-AGN-TR
Changed lines of the file:
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@@
 			)
 		)
-		(property "Footprint" "BLM21PG221SN1D:BEADC2012X105N"
+		(property "Footprint" "GNSS:BEADC2012X105N"
 			(at 236.728 40.894 0)
 			(effects
@@
 				)
 				(justify bottom)
-				(hide yes)
 			)
 		)
@@
 			)
 		)
-		(property "Footprint" "GNSS:MURATA_XRCGB24M000FFS1DR0_0"
+		(property "Footprint" "GNSS:XTAL_ECS-250-12-33-AGN-TR"
 			(at 64.77 165.1 0)
 			(effects
@@
 			)
 		)
-		(property "Footprint" "C0402C104K4RAC:CAPC1005X55N"
+		(property "Footprint" "Capacitor_SMD:C_0402_1005Metric"
 			(at 57.15 172.72 0)
 			(effects
@@
 			)
 		)
-		(property "Footprint" "C0402C104K4RAC:CAPC1005X55N"
+		(property "Footprint" "Capacitor_SMD:C_0402_1005Metric"
 			(at 93.98 172.72 0)
 			(effects

Commit message: we
Parts:
- removed Y4: MURATA_XRCGB24M000FFS1DR0, GNSS:XTAL_ECS-250-12-33-AGN-TR, symbol MURATA_XRCGB24M000FFS1DR0:MURATA_XRCGB24M000FFS1DR0
- added Y2: ECS-250-18-33-JGN-TR, ECS-250-18-33-JGN-TR:XTAL_ECS-250-18-33-JGN-TR, symbol ECS-250-18-33-JGN-TR:ECS-250-18-33-JGN-TR
- C66, C77: value 18p -> 20p
Connections:
- net EXP: now also C66.1, C77.1, Y2.2 (GND), Y2.4 (GND); no longer C66.2, C77.2
- net XTAL_IN: now also C77.2, Y2.3 (OUT/IN); no longer C77.1
- net XTAL_OUT: now also C66.2, Y2.1 (IN/OUT); no longer C66.1
- net +3.3V renamed +3V3
- net +3.3V_ETH renamed +3V3_ETH
- no-connect marks 6 -> 4
Other:
- moved on the sheet: C66, C77, R22

Commit message: 22.09.26
Parts:
- removed FL11: BLM21PG221SN1D, GNSS:BEADC2012X105N, symbol BLM21PG221SN1D:BLM21PG221SN1D
- added FB8: FerriteBead, GNSS:BEADC2012X105N, symbol Device:FerriteBead
Connections:
- net +3V3: now also FB8.2
- net +3V3_ETH: now also FB8.1
Changed lines of the file:
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@@
 	(wire
 		(pts
-			(xy 214.63 52.07) (xy 218.44 52.07)
+			(xy 214.63 52.07) (xy 224.79 52.07)
 		)
 		(stroke
@@
 	(wire
 		(pts
-			(xy 236.22 52.07) (xy 241.3 52.07)
+			(xy 232.41 52.07) (xy 241.3 52.07)
 		)
 		(stroke
@@
 	)
 	(symbol
-		(lib_id "BLM21PG221SN1D:BLM21PG221SN1D")
-		(at 233.68 52.07 0)
-		(unit 1)
-		(exclude_from_sim no)
-		(in_bom yes)
-		(on_board yes)
-		(dnp no)
-		(property "Reference" "FL11"
-			(at 227.33 45.72 0)
-			(effects
-				(font
-					(size 1.27 1.27)
-				)
-			)
-		)
-		(property "Value" "BLM21PG221SN1D"
-			(at 227.33 48.26 0)
-			(effects
-				(font
-					(size 1.27 1.27)
-				)
-			)
-		)
-		(property "Footprint" "GNSS:BEADC2012X105N"
-			(at 236.728 40.894 0)
-			(effects
-				(font
-					(size 1.27 1.27)
-				)
-				(justify bottom)
-			)
-		)
-		(property "Datasheet" ""
-			(at 233.68 52.07 0)
-			(effects
-				(font
-					(size 1.27 1.27)
-				)
-				(hide yes)
-			)
-		)
-		(property "Description" ""
-			(at 233.68 52.07 0)
-			(effects
-				(font
-					(size 1.27 1.27)
-				)
-				(hide yes)
-			)
-		)
-		(property "MF" "Murata"
-			(at 251.206 46.228 0)
-			(effects
-				(font
-					(size 1.27 1.27)
-				)
-				(justify bottom)
-				(hide yes)
-			)
-		)
-		(property "Description_1" "\n                        \n                            220 Ohms @ 100 MHz 1 Power Line Ferrite Bead 0805 (2012 Metric) 2A 45mOhm\n                        \n"
-			(at 233.426 43.942 0)
-			(effects
-				(font
-					(size 1.27 1.27)
-				)
-				(justify bottom)
-				(hide yes)
-			)
-		)
-		(property "Package" "2012 Murata"
-			(at 235.458 46.482 0)
-			(effects
-				(font
-					(size 1.27 1.27)
-				)
-				(justify bottom)
-				(hide yes)
-			)
-		)
-		(property "Price" "None"
-			(at 244.856 46.99 0)
-			(effects
-				(font
-					(size 1.27 1.27)
-				)
-				(justify bottom)
-				(hide yes)
-			)
-		)
-		(property "SnapEDA_Link" "https://www.snapeda.com/parts/BLM21PG221SN1D/Murata/view-part/?ref=snap"
-			(at 236.728 43.688 0)
-			(effects
-				(font
-					(size 1.27 1.27)
-				)
-				(justify bottom)
-				(hide yes)
-			)
-		)
-		(property "MP" "BLM21PG221SN1D"
-			(at 242.062 39.37 0)
-			(effects
-				(font
-					(size 1.27 1.27)
-				)
-				(justify bottom)
-				(hide yes)
-			)
-		)
-		(property "Availability" "In Stock"
-			(at 258.572 46.99 0)
-			(effects
-				(font
-					(size 1.27 1.27)
-				)
-				(justify bottom)
-				(hide yes)
-			)
-		)
-		(property "Check_prices" "https://www.snapeda.com/parts/BLM21PG221SN1D/Murata/view-part/?ref=eda"
-			(at 239.776 37.592 0)
-			(effects
-				(font
-					(size 1.27 1.27)
-				)
-				(justify bottom)
-				(hide yes)
-			)
-		)
-		(pin "1"
-		)
-		(pin "2"
-		)
-		(instances
-			(project "GNSS"
-				(path "/a70dad34-b24c-4b58-b91c-f14576b5da7d/a33a7fbe-117f-40f3-9eeb-50ee11d7c18f"
-					(reference "FL11")
-					(unit 1)
-				)
-			)
-		)
-	)
-	(symbol
 		(lib_id "Device:R_Small_US")
 		(at 227.33 90.17 270)
@@
 					(unit 1)
 				)
+			)
+		)
+	)
+	(symbol
+		(lib_id "Device:FerriteBead")
+		(at 228.6 52.07 90)
+		(unit 1)
+		(exclude_from_sim no)
+		(in_bom yes)
+		(on_board yes)
+		(dnp no)
+		(fields_autoplaced yes)
+		(property "Reference" "FB8"
+			(at 228.5492 44.45 90)
+			(effects
+				(font
+					(size 1.27 1.27)
+				)
+			)
+		)
+		(property "Value" "FerriteBead"
+			(at 228.5492 46.99 90)
+			(effects
+				(font
+					(size 1.27 1.27)
+				)
+			)
+		)
+		(property "Footprint" "GNSS:BEADC2012X105N"
+			(at 228.6 53.848 90)
+			(effects
+				(font
+					(size 1.27 1.27)
+				)
+				(hide yes)
+			)
+		)
+		(property "Datasheet" "~"
+			(at 228.6 52.07 0)
+			(effects
+				(font
+					(size 1.27 1.27)
+				)
+				(hide yes)
+			)
+		)
+		(property "Description" "Ferrite bead"
+			(at 228.6 52.07 0)
+			(effects
+				(font
+					(size 1.27 1.27)
+				)
+				(hide yes)
+			)
+		)
+		(pin "1"
+		)
+		(pin "2"
+		)
+		(instances
+			(project "GNSS"
+				(path "/a70dad34-b24c-4b58-b91c-f14576b5da7d/a33a7fbe-117f-40f3-9eeb-50ee11d7c18f"
+					(reference "FB8")
+					(unit 1)
+				)

Commit message: 123
Connections:
- net +3V3: now also FB8.1; no longer FB8.2
- net +3V3_ETH: now also FB8.2; no longer FB8.1
Changed lines of the file:
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@@
 		(dnp no)
 		(property "Reference" "R51"
-			(at 227.076 92.202 90)
+			(at 225.298 86.36 90)
 			(effects
 				(font
@@
 		)
 		(property "Value" "10K"
-			(at 221.996 91.948 90)
+			(at 225.044 88.392 90)
 			(effects
 				(font
@@
 		(dnp no)
 		(property "Reference" "R23"
-			(at 49.784 81.026 90)
+			(at 55.372 73.406 90)
 			(effects
 				(font
@@
 		)
 		(property "Value" "470R"
-			(at 56.134 81.28 90)
+			(at 55.372 75.692 90)
 			(effects
 				(font
@@
 		(dnp no)
 		(property "Reference" "L4"
-			(at 83.058 111.252 0)
+			(at 83.058 109.728 0)
 			(effects
 				(font
@@
 		)
 		(property "Value" "WE-CBF_0603"
-			(at 82.55 108.712 0)
+			(at 82.55 111.76 0)
 			(effects
 				(font
@@
 	)
 	(symbol
-		(lib_id "power:+3.3V")
-		(at 241.3 50.8 0)
-		(unit 1)
-		(exclude_from_sim no)
-		(in_bom yes)
-		(on_board yes)
-		(dnp no)
-		(fields_autoplaced yes)
-		(property "Reference" "#PWR0103"
-			(at 241.3 54.61 0)
-			(effects
-				(font
-					(size 1.27 1.27)
-				)
-				(hide yes)
-			)
-		)
-		(property "Value" "+3V3"
-			(at 241.3 45.72 0)
-			(effects
-				(font
-					(size 1.27 1.27)
-				)
-			)
-		)
-		(property "Footprint" ""
-			(at 241.3 50.8 0)
-			(effects
-				(font
-					(size 1.27 1.27)
-				)
-				(hide yes)
-			)
-		)
-		(property "Datasheet" ""
-			(at 241.3 50.8 0)
-			(effects
-				(font
-					(size 1.27 1.27)
-				)
-				(hide yes)
-			)
-		)
-		(property "Description" "Power symbol creates a global label with name \"+3.3V\""
-			(at 241.3 50.8 0)
-			(effects
-				(font
-					(size 1.27 1.27)
-				)
-				(hide yes)
-			)
-		)
-		(pin "1"
-		)
-		(instances
-			(project "GNSS"
-				(path "/a70dad34-b24c-4b58-b91c-f14576b5da7d/a33a7fbe-117f-40f3-9eeb-50ee11d7c18f"
-					(reference "#PWR0103")
-					(unit 1)
-				)
-			)
-		)
-	)
-	(symbol
 		(lib_id "Device:R_Small_US")
 		(at 227.33 74.93 270)
@@
 		(dnp no)
 		(property "Reference" "R49"
-			(at 227.076 76.962 90)
+			(at 224.536 71.12 90)
 			(effects
 				(font
@@
 		)
 		(property "Value" "2K2"
-			(at 221.996 76.708 90)
+			(at 224.282 72.898 90)
 			(effects
 				(font
@@
 		(dnp no)
 		(property "Reference" "R50"
-			(at 227.076 84.582 90)
+			(at 225.298 78.486 90)
 			(effects
 				(font
@@
 		)
 		(property "Value" "2K2"
-			(at 221.996 84.328 90)
+			(at 225.298 80.518 90)
 			(effects
 				(font
@@
 	)
 	(symbol
-		(lib_id "power:+3.3V")
-		(at 214.63 50.8 0)
-		(unit 1)
-		(exclude_from_sim no)
-		(in_bom yes)
-		(on_board yes)
-		(dnp no)
-		(fields_autoplaced yes)
-		(property "Reference" "#PWR095"
-			(at 214.63 54.61 0)
-			(effects
-				(font
-					(size 1.27 1.27)
-				)
-				(hide yes)
-			)
-		)
-		(property "Value" "+3V3_ETH"
-			(at 214.63 45.72 0)
-			(effects
-				(font
-					(size 1.27 1.27)
-				)
-			)
-		)
-		(property "Footprint" ""
-			(at 214.63 50.8 0)
-			(effects
-				(font
-					(size 1.27 1.27)
-				)
-				(hide yes)
-			)
-		)
-		(property "Datasheet" ""
-			(at 214.63 50.8 0)
-			(effects
-				(font
-					(size 1.27 1.27)
-				)
-				(hide yes)
-			)
-		)
-		(property "Description" "Power symbol creates a global label with name \"+3.3V\""
-			(at 214.63 50.8 0)
-			(effects
-				(font
-					(size 1.27 1.27)
-				)
-				(hide yes)
-			)
-		)
-		(pin "1"
-		)
-		(instances
-			(project "GNSS"
-				(path "/a70dad34-b24c-4b58-b91c-f14576b5da7d/a33a7fbe-117f-40f3-9eeb-50ee11d7c18f"
-					(reference "#PWR095")
-					(unit 1)
-				)
-			)
-		)
-	)
-	(symbol
 		(lib_id "C0402C104K4RAC:C0402C104K4RAC")
 		(at 96.52 100.33 90)
@@
 	)
 	(symbol
+		(lib_id "power:+3.3V")
+		(at 241.3 50.8 0)
+		(unit 1)
+		(exclude_from_sim no)
+		(in_bom yes)
+		(on_board yes)
+		(dnp no)
+		(fields_autoplaced yes)
+		(property "Reference" "#PWR095"
+			(at 241.3 54.61 0)
+			(effects
+				(font
+					(size 1.27 1.27)
+				)
+				(hide yes)
+			)
+		)
+		(property "Value" "+3V3_ETH"
+			(at 241.3 45.72 0)
+			(effects
+				(font
+					(size 1.27 1.27)
+				)
+			)
+		)
+		(property "Footprint" ""
+			(at 241.3 50.8 0)
+			(effects
+				(font
+					(size 1.27 1.27)
+				)
+				(hide yes)
+			)
+		)
+		(property "Datasheet" ""
+			(at 241.3 50.8 0)
+			(effects
+				(font
+					(size 1.27 1.27)
+				)
+				(hide yes)
+			)
+		)
+		(property "Description" "Power symbol creates a global label with name \"+3.3V\""
+			(at 241.3 50.8 0)
+			(effects
+				(font
+					(size 1.27 1.27)
+				)
+				(hide yes)
+			)
+		)
+		(pin "1"
+		)
+		(instances
+			(project "GNSS"
+				(path "/a70dad34-b24c-4b58-b91c-f14576b5da7d/a33a7fbe-117f-40f3-9eeb-50ee11d7c18f"
+					(reference "#PWR095")
+					(unit 1)
+				)
+			)
+		)
+	)
+	(symbol
 		(lib_id "Device:R_Small_US")
 		(at 67.31 179.07 270)
@@
 		(dnp no)
 		(property "Reference" "R22"
-			(at 68.326 180.848 90)
+			(at 65.278 175.006 90)
 			(effects
 				(font
@@
 		)
 		(property "Value" "1M"
-			(at 60.198 180.34 90)
+			(at 65.532 176.784 90)
 			(effects
 				(font
@@
 		)
 		(property "Value" "6K49"
-			(at 114.3 100.076 0)
+			(at 114.3 105.664 0)
 			(effects
 				(font
@@
 		(dnp no)
 		(property "Reference" "R48"
-			(at 227.076 70.612 90)
+			(at 224.79 64.008 90)
 			(effects
 				(font
@@
 		)
 		(property "Value" "10K"
-			(at 221.996 70.358 90)
+			(at 224.536 66.294 90)
 			(effects
 				(font
@@
 					(unit 1)
 				)
+			)
+		)
+	)
+	(symbol
+		(lib_id "power:+3.3V")
+		(at 214.63 50.8 0)
+		(unit 1)
+		(exclude_from_sim no)
+		(in_bom yes)
+		(on_board yes)
+		(dnp no)
+		(fields_autoplaced yes)
+		(property "Reference" "#PWR0103"
+			(at 214.63 54.61 0)
+			(effects
+				(font
+					(size 1.27 1.27)
+				)
+				(hide yes)
+			)
+		)
+		(property "Value" "+3V3"
+			(at 214.63 45.72 0)
+			(effects
+				(font
+					(size 1.27 1.27)
+				)
+			)
+		)
+		(property "Footprint" ""
+			(at 214.63 50.8 0)
+			(effects
+				(font
+					(size 1.27 1.27)
+				)
+				(hide yes)
+			)
+		)
+		(property "Datasheet" ""
+			(at 214.63 50.8 0)
+			(effects
+				(font
+					(size 1.27 1.27)
+				)
+				(hide yes)
+			)
+		)
+		(property "Description" "Power symbol creates a global label with name \"+3.3V\""
+			(at 214.63 50.8 0)
+			(effects
+				(font
+					(size 1.27 1.27)
+				)
+				(hide yes)
+			)
+		)
+		(pin "1"
+		)
+		(instances
+			(project "GNSS"
+				(path "/a70dad34-b24c-4b58-b91c-f14576b5da7d/a33a7fbe-117f-40f3-9eeb-50ee11d7c18f"
+					(reference "#PWR0103")
+					(unit 1)
+				)
