File: Content_sch.kicad_sch (KiCad schematic)
At the start: 0 parts

Commit message: new table
Other:
- note added: "10"
- note added: "11"
- note added: "3"
- note added: "4"
- note added: "5"
- note added: "6"
- note added: "7"
- note added: "8"
- note added: "9"
- note added: "ARDUINO"
- note added: "BLOCK DIAGRAM"
- note added: "CONTENT"
- note added: "CONTROLLER"
- note added: "ESP"
- note added: "ETHERNET"
- note added: "GNSS DEV BOARD"
- note added: "IMU"
- note added: "PAGE NO"
- note added: "POWER"
- note added: "USB_HUB"
- note added: "ZED_F9P"

Commit message: changed
Changed lines of the file:
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@@
 			(font
 				(size 1.778 1.778)
+				(bold yes)
 			)
 		)
@@
 			(font
 				(size 1.778 1.778)
+				(bold yes)
 			)
 		)
@@
 			(font
 				(size 1.778 1.778)
+				(bold yes)
 			)
 		)
@@
 			(font
 				(size 1.778 1.778)
+				(bold yes)
 			)
 		)
@@
 			(font
 				(size 1.778 1.778)
+				(bold yes)
 			)
 		)
@@
 			(font
 				(size 1.778 1.778)
+				(bold yes)
 			)
 		)
@@
 			(font
 				(size 1.778 1.778)
+				(bold yes)
 			)
 		)
@@
 			(font
 				(size 1.778 1.778)
+				(bold yes)
 			)
 		)
@@
 			(font
 				(size 1.778 1.778)
+				(bold yes)
 			)
 		)
@@
 			(font
 				(size 1.778 1.778)
+				(bold yes)
 			)
 		)
@@
 			(font
 				(size 3.81 3.81)
+				(bold yes)
 			)
 		)
@@
 			(font
 				(size 1.778 1.778)
+				(bold yes)
 			)
 		)
@@
 			(font
 				(size 1.778 1.778)
+				(bold yes)
 			)
 		)
@@
 			(font
 				(size 2.54 2.54)
+				(bold yes)
 			)
 		)
@@
 			(font
 				(size 1.778 1.778)
+				(bold yes)
 			)
 		)
@@
 			(font
 				(size 1.778 1.778)
+				(bold yes)
 			)
 		)
@@
 			(font
 				(size 1.778 1.778)
+				(bold yes)
 			)
 		)
@@
 			(font
 				(size 1.778 1.778)
+				(bold yes)
 			)
 		)
@@
 			(font
 				(size 2.54 2.54)
+				(bold yes)
 			)
 		)
@@
 			(font
 				(size 1.778 1.778)
+				(bold yes)
 			)
 		)
@@
 			(font
 				(size 1.778 1.778)
-			)
-		)
+				(bold yes)
+			)
+		)

Commit message: new
Other:
- note removed: "10"
- note removed: "11"
- note removed: "3"
- note removed: "4"
- note removed: "5"
- note removed: "6"
- note removed: "7"
- note removed: "8"
- note removed: "9"
- note removed: "ARDUINO"
- note removed: "BLOCK DIAGRAM"
- note removed: "CONTENT"
- note removed: "CONTROLLER"
- note removed: "ESP"
- note removed: "ETHERNET"
- note removed: "GNSS DEV BOARD"
- note removed: "IMU"
- note removed: "PAGE NO"
- note removed: "POWER"
- note removed: "USB_HUB"
- note removed: "ZED_F9P"
