File: Content_sch.kicad_sch (KiCad schematic)
At the start: 0 parts

Commit message: can
Other:
- note added: "1"
- note added: "10"
- note added: "11"
- note added: "12"
- note added: "2"
- note added: "3"
- note added: "4"
- note added: "5"
- note added: "6"
- note added: "7"
- note added: "8"
- note added: "9"
- note added: "ARDUINO"
- note added: "BLOCK_DIAGRAM"
- note added: "CONTROLLER"
- note added: "DESCRIPTION"
- note added: "ESP & CAN"
- note added: "ETHERNET"
- note added: "IMU & SDCARD"
- note added: "PAGE"
- note added: "POWER"
- note added: "POWER_ARCHITECTURE"
- note added: "SECTION"
- note added: "TABLE OF CONTENT"
- note added: "USB_HUB"
- note added: "ZED_F9P"

Commit message: block
Changed lines of the file:
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@@
 	(polyline
 		(pts
-			(xy 82.296 88.646) (xy 214.376 88.646)
-		)
-		(stroke
-			(width 0)
-			(type default)
-		)
-	)
-	(polyline
-		(pts
-			(xy 82.296 103.886) (xy 214.376 103.886)
-		)
-		(stroke
-			(width 0)
-			(type default)
-		)
-	)
-	(polyline
-		(pts
-			(xy 82.296 114.046) (xy 214.376 114.046)
-		)
-		(stroke
-			(width 0)
-			(type default)
-		)
-	)
-	(polyline
-		(pts
-			(xy 82.296 93.726) (xy 214.376 93.726)
-		)
-		(stroke
-			(width 0)
-			(type default)
-		)
-	)
-	(polyline
-		(pts
-			(xy 82.296 78.486) (xy 214.376 78.486)
-		)
-		(stroke
-			(width 0)
-			(type default)
-		)
-	)
-	(polyline
-		(pts
-			(xy 82.296 83.566) (xy 214.376 83.566)
-		)
-		(stroke
-			(width 0)
-			(type default)
-		)
-	)
-	(polyline
-		(pts
-			(xy 82.296 73.406) (xy 214.376 73.406)
-		)
-		(stroke
-			(width 0)
-			(type default)
-		)
-	)
-	(polyline
-		(pts
-			(xy 82.296 98.806) (xy 214.376 98.806)
-		)
-		(stroke
-			(width 0)
-			(type default)
-		)
-	)
-	(polyline
-		(pts
-			(xy 106.426 59.436) (xy 106.426 119.126)
-		)
-		(stroke
-			(width 0)
-			(type default)
-		)
-	)
-	(polyline
-		(pts
-			(xy 185.166 59.436) (xy 185.166 119.126)
-		)
-		(stroke
-			(width 0)
-			(type default)
-		)
-	)
-	(polyline
-		(pts
-			(xy 82.296 108.966) (xy 214.376 108.966)
-		)
-		(stroke
-			(width 0)
-			(type default)
-		)
-	)
-	(polyline
-		(pts
-			(xy 82.296 68.326) (xy 214.376 68.326)
+			(xy 83.82 100.33) (xy 215.9 100.33)
+		)
+		(stroke
+			(width 0)
+			(type default)
+		)
+	)
+	(polyline
+		(pts
+			(xy 83.82 115.57) (xy 215.9 115.57)
+		)
+		(stroke
+			(width 0)
+			(type default)
+		)
+	)
+	(polyline
+		(pts
+			(xy 83.82 125.73) (xy 215.9 125.73)
+		)
+		(stroke
+			(width 0)
+			(type default)
+		)
+	)
+	(polyline
+		(pts
+			(xy 83.82 105.41) (xy 215.9 105.41)
+		)
+		(stroke
+			(width 0)
+			(type default)
+		)
+	)
+	(polyline
+		(pts
+			(xy 83.82 90.17) (xy 215.9 90.17)
+		)
+		(stroke
+			(width 0)
+			(type default)
+		)
+	)
+	(polyline
+		(pts
+			(xy 83.82 95.25) (xy 215.9 95.25)
+		)
+		(stroke
+			(width 0)
+			(type default)
+		)
+	)
+	(polyline
+		(pts
+			(xy 83.82 85.09) (xy 215.9 85.09)
+		)
+		(stroke
+			(width 0)
+			(type default)
+		)
+	)
+	(polyline
+		(pts
+			(xy 83.82 110.49) (xy 215.9 110.49)
+		)
+		(stroke
+			(width 0)
+			(type default)
+		)
+	)
+	(polyline
+		(pts
+			(xy 107.95 71.12) (xy 107.95 130.81)
+		)
+		(stroke
+			(width 0)
+			(type default)
+		)
+	)
+	(polyline
+		(pts
+			(xy 186.69 71.12) (xy 186.69 130.81)
+		)
+		(stroke
+			(width 0)
+			(type default)
+		)
+	)
+	(polyline
+		(pts
+			(xy 83.82 120.65) (xy 215.9 120.65)
+		)
+		(stroke
+			(width 0)
+			(type default)
+		)
+	)
+	(polyline
+		(pts
+			(xy 83.82 80.01) (xy 215.9 80.01)
 		)
 		(stroke
@@
 	)
 	(rectangle
-		(start 82.296 59.436)
-		(end 214.376 119.126)
+		(start 83.82 71.12)
+		(end 215.9 130.81)
 		(stroke
 			(width 0)
@@
 	(text "12"
 		(exclude_from_sim no)
-		(at 197.866 116.84 0)
+		(at 199.39 128.524 0)
 		(effects
 			(font
@@
 	(text "7"
 		(exclude_from_sim no)
-		(at 198.882 91.44 0)
+		(at 200.406 103.124 0)
 		(effects
 			(font
@@
 	(text "7"
 		(exclude_from_sim no)
-		(at 93.472 101.6 0)
+		(at 94.996 113.284 0)
 		(effects
 			(font
@@
 	(text "5"
 		(exclude_from_sim no)
-		(at 199.136 81.534 0)
+		(at 200.66 93.218 0)
 		(effects
 			(font
@@
 	(text "TABLE OF CONTENT"
 		(exclude_from_sim no)
-		(at 145.034 52.578 0)
+		(at 143.002 64.262 0)
 		(effects
 			(font
@@
 	(text "4"
 		(exclude_from_sim no)
-		(at 199.136 76.962 0)
+		(at 200.66 88.646 0)
 		(effects
 			(font
@@
 	(text "2\n"
 		(exclude_from_sim no)
-		(at 93.726 76.708 0)
+		(at 95.25 88.392 0)
 		(effects
 			(font
@@
 	(text "BLOCK_DIAGRAM"
 		(exclude_from_sim no)
-		(at 143.256 71.12 0)
+		(at 144.78 82.804 0)
 		(effects
 			(font
@@
 	(text "POWER_ARCHITECTURE"
 		(exclude_from_sim no)
-		(at 143.51 117.094 0)
+		(at 145.034 128.778 0)
 		(effects
 			(font
@@
 	(text "ARDUINO"
 		(exclude_from_sim no)
-		(at 143.256 101.854 0)
+		(at 144.78 113.538 0)
 		(effects
 			(font
@@
 	(text "10"
 		(exclude_from_sim no)
-		(at 92.964 116.586 0)
+		(at 94.488 128.27 0)
 		(effects
 			(font
@@
 	(text "8"
 		(exclude_from_sim no)
-		(at 93.726 106.68 0)
+		(at 95.25 118.364 0)
 		(effects
 			(font
@@
 	(text "PAGE"
 		(exclude_from_sim no)
-		(at 199.644 64.516 0)
+		(at 201.168 76.2 0)
 		(effects
 			(font
@@
 	(text "SECTION"
 		(exclude_from_sim no)
-		(at 94.488 64.77 0)
+		(at 96.012 76.454 0)
 		(effects
 			(font
@@
 	(text "POWER"
 		(exclude_from_sim no)
-		(at 143.51 75.946 0)
+		(at 145.034 87.63 0)
 		(effects
 			(font
@@
 	(text "3"
 		(exclude_from_sim no)
-		(at 199.136 71.12 0)
+		(at 200.66 82.804 0)
 		(effects
 			(font
@@
 	(text "USB_HUB"
 		(exclude_from_sim no)
-		(at 143.51 81.28 0)
+		(at 145.034 92.964 0)
 		(effects
 			(font
@@
 	(text "3"
 		(exclude_from_sim no)
-		(at 93.726 81.788 0)
+		(at 95.25 93.472 0)
 		(effects
 			(font
@@
 	(text "9"
 		(exclude_from_sim no)
-		(at 93.472 112.014 0)
+		(at 94.996 123.698 0)
 		(effects
 			(font
@@
 	(text "4"
 		(exclude_from_sim no)
-		(at 93.472 86.36 0)
+		(at 94.996 98.044 0)
 		(effects
 			(font
@@
 	(text "8"
 		(exclude_from_sim no)
-		(at 198.628 96.774 0)
+		(at 200.152 108.458 0)
 		(effects
 			(font
@@
 	(text "1"
 		(exclude_from_sim no)
-		(at 93.98 71.12 0)
+		(at 95.504 82.804 0)
 		(effects
 			(font
@@
 	(text "9"
 		(exclude_from_sim no)
-		(at 198.628 101.346 0)
+		(at 200.152 113.03 0)
 		(effects
 			(font
@@
 	(text "6"
 		(exclude_from_sim no)
-		(at 93.472 96.774 0)
+		(at 94.996 108.458 0)
 		(effects
 			(font
@@
 	(text "10"
 		(exclude_from_sim no)
-		(at 197.866 106.68 0)
+		(at 199.39 118.364 0)
 		(effects
 			(font
@@
 	(text "6"
 		(exclude_from_sim no)
-		(at 199.136 86.36 0)
+		(at 200.66 98.044 0)
 		(effects
 			(font
@@
 	(text "ETHERNET"
 		(exclude_from_sim no)
-		(at 143.256 106.934 0)
+		(at 144.78 118.618 0)
 		(effects
 			(font
@@
 	(text "11"
 		(exclude_from_sim no)
-		(at 197.866 111.506 0)
+		(at 199.39 123.19 0)
 		(effects
 			(font
@@
 	(text "ESP & CAN"
 		(exclude_from_sim no)
-		(at 143.256 96.52 0)
+		(at 144.78 108.204 0)
 		(effects
 			(font
@@
 	(text "CONTROLLER"
 		(exclude_from_sim no)
-		(at 143.51 91.44 0)
+		(at 145.034 103.124 0)
 		(effects
 			(font
@@
 	(text "5"
 		(exclude_from_sim no)
-		(at 93.472 91.694 0)
+		(at 94.996 103.378 0)
 		(effects
 			(font
@@
 	(text "IMU & SDCARD"
 		(exclude_from_sim no)
-		(at 143.256 112.014 0)
+		(at 144.78 123.698 0)
 		(effects
 			(font
@@
 	(text "ZED_F9P"
 		(exclude_from_sim no)
-		(at 143.51 86.36 0)
+		(at 145.034 98.044 0)
 		(effects
 			(font
@@
 	(text "DESCRIPTION"
 		(exclude_from_sim no)
-		(at 144.018 64.516 0)
-		(effects
-			(font
+		(at 145.542 76.2 0)
+		(effects
+			(font

Commit message: full
Other:
- note added: "13"
- note added: "14"
- note added: "ANTENNA"
- note added: "LEDs & BUTTONs"
- note removed: "BLOCK_DIAGRAM"

Commit message: 18.09.2026
Other:
- note added: "ZED_ZF9P"
- note removed: "ZED_F9P"
