File: ZED_Z9P.kicad_sch (KiCad schematic)
At the start: 6 parts, among them IC2 ZED-F9P-05B

Commit message: changed
Connections:
- net +3V3_GNSS: now also IC2.36 (V_BCKP)
- net GND: now also IC2.1 (GND_1), IC2.12 (GND_3), IC2.14 (GND_4), IC2.3 (GND_2), IC2.32 (GND_5), IC2.37 (GND_6), IC2.41 (GND_7), IC2.47 (D_SEL), IC2.48 (GND_8)

Commit message: zed
Connections:
- net +3V3_GNSS: no longer IC2.36 (V_BCKP)
Changed lines of the file:
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@@
-	)
-	(junction
-		(at 101.6 107.95)
-		(diameter 0)
-		(color 0 0 0 0)
 	)
 	(junction
@@
 	(wire
 		(pts
-			(xy 101.6 107.95) (xy 101.6 113.03)
-		)
-		(stroke
-			(width 0)
-			(type default)
-		)
-	)
-	(wire
-		(pts
 			(xy 163.83 100.33) (xy 163.83 102.87)
 		)
@@
 		)
 		(stroke
-			(width 0)
-			(type default)
-		)
-	)
-	(wire
-		(pts
-			(xy 101.6 113.03) (xy 113.03 113.03)
-		)
-		(stroke

Commit message: verification
Other:
- moved on the sheet: R15
Changed lines of the file:
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@@
 	)
 	(junction
-		(at 99.06 146.05)
+		(at 80.01 146.05)
 		(diameter 0)
 		(color 0 0 0 0)
@@
 	(wire
 		(pts
-			(xy 99.06 146.05) (xy 95.25 146.05)
+			(xy 80.01 146.05) (xy 76.2 146.05)
 		)
 		(stroke
@@
 	(wire
 		(pts
-			(xy 99.06 146.05) (xy 113.03 146.05)
+			(xy 80.01 146.05) (xy 113.03 146.05)
 		)
 		(stroke
@@
 	(wire
 		(pts
-			(xy 99.06 138.43) (xy 99.06 140.97)
+			(xy 80.01 138.43) (xy 80.01 140.97)
 		)
 		(stroke
@@
 	(global_label "RESET_GNSS"
 		(shape input)
-		(at 95.25 146.05 180)
+		(at 76.2 146.05 180)
 		(fields_autoplaced yes)
 		(effects
@@
 		)
 		(property "Intersheetrefs" "${INTERSHEET_REFS}"
-			(at 80.5326 146.05 0)
+			(at 61.4826 146.05 0)
 			(effects
 				(font
@@
 	(symbol
 		(lib_id "Device:R_Small_US")
-		(at 99.06 143.51 0)
+		(at 80.01 143.51 0)
 		(unit 1)
 		(exclude_from_sim no)
@@
 		(dnp no)
 		(property "Reference" "R15"
-			(at 93.98 139.954 0)
+			(at 74.93 139.954 0)
 			(effects
 				(font
@@
 		)
 		(property "Value" "10K"
-			(at 94.234 142.24 0)
+			(at 75.184 142.24 0)
 			(effects
 				(font
@@
 		)
 		(property "Footprint" "Resistor_SMD:R_0402_1005Metric"
-			(at 99.06 143.51 0)
+			(at 80.01 143.51 0)
 			(effects
 				(font
@@
 		)
 		(property "Datasheet" "~"
-			(at 99.06 143.51 0)
+			(at 80.01 143.51 0)
 			(effects
 				(font
@@
 		)
 		(property "Description" "Resistor, small US symbol"
-			(at 99.06 143.51 0)
+			(at 80.01 143.51 0)
 			(effects
 				(font
@@
 	(symbol
 		(lib_id "power:+3V3")
-		(at 99.06 138.43 0)
+		(at 80.01 138.43 0)
 		(unit 1)
 		(exclude_from_sim no)
@@
 		(fields_autoplaced yes)
 		(property "Reference" "#PWR047"
-			(at 99.06 142.24 0)
+			(at 80.01 142.24 0)
 			(effects
 				(font
@@
 		)
 		(property "Value" "+3V3_GNSS"
-			(at 99.06 133.35 0)
+			(at 80.01 133.35 0)
 			(effects
 				(font
@@
 		)
 		(property "Footprint" ""
-			(at 99.06 138.43 0)
+			(at 80.01 138.43 0)
 			(effects
 				(font
@@
 		)
 		(property "Datasheet" ""
-			(at 99.06 138.43 0)
+			(at 80.01 138.43 0)
 			(effects
 				(font
@@
 		)
 		(property "Description" "Power symbol creates a global label with name \"+3V3\""
-			(at 99.06 138.43 0)
-			(effects
-				(font
+			(at 80.01 138.43 0)
+			(effects
+				(font

Commit message: new
Changed lines of the file:
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@@
-		)
-	)
-	(text_box "V_USB LEFT"
-		(exclude_from_sim no)
-		(at 31.75 97.79 0)
-		(size 13.97 10.16)
-		(stroke
-			(width 0)
-			(type default)
-		)
-		(fill
-			(type none)
-		)
-		(effects
-			(font
-				(size 1.27 1.27)
-			)
-			(justify left top)
-		)
-	)
-	(text_box "GND1 2 3 4 5 6 7 8 CONNECTED \nV_BCKP TO VCC\nD_SEL TO GND\n\n \n       DONE"
-		(exclude_from_sim no)
-		(at 30.48 78.74 0)
-		(size 38.1 15.24)
-		(stroke
-			(width 0)
-			(type default)
-		)
-		(fill
-			(type none)
-		)
-		(effects
-			(font
-				(size 1.27 1.27)
-			)
-			(justify left top)
 		)
 	)

Commit message: new
Parts:
- removed R31: 560R, Resistor_SMD:R_0805_2012Metric, symbol Device:R_Small_US
- removed R32: SML-P12U2TT86R, GNSS_Library:LED_SML-P11D_ROM, symbol 2026-08-14_04-34-19:SML-P12U2TT86R
- added BT1: 1056, 1056:BAT_1056, symbol 1056:1056
- added C53, C55, C62: 1uF, Capacitor_SMD:C_0805_2012Metric, symbol Device:C_Small
- added C54, C56, C63: 100nF, C0402C104K4RAC:CAPC1005X55N, symbol C0402C104K4RAC:C0402C104K4RAC
- added C71: GRM033R71C103KE14D, GRM033R71C103KE14D:CAPC0603X33N, symbol GRM033R71C103KE14D:GRM033R71C103KE14D
- added D1: PESD0402-140, PESD0402-140:DIO_PESD0402-140, symbol PESD0402-140:PESD0402-140
- added FL9: BLM21PG221SN1D, BLM21PG221SN1D:BEADC2012X105N, symbol BLM21PG221SN1D:BLM21PG221SN1D
- added J4: SMA-J-P-X-RA-TH1, SMA-J-P-X-RA-TH1:SAMTEC_SMA-J-P-X-RA-TH1, symbol SMA-J-P-X-RA-TH1:SMA-J-P-X-RA-TH1
- added JP1: SolderJumper_3_Open, symbol Jumper:SolderJumper_3_Open
- added L3: LQG15HS47NJ02D, LQG15HS47NJ02D:INDC1005X55N, symbol LQG15HS47NJ02D:LQG15HS47NJ02D
- added Q1: SI1016CX-T1-GE3, SOTFL50P160X60-6N, symbol SI1016CX-T1-GE3:SI1016CX-T1-GE3
- added Q2: MMBT3904LT1G, MMBT3904LT1G:SOT95P240X111-3N, symbol MMBT3904LT1G:MMBT3904LT1G
- added R32: 10E, Resistor_SMD:R_0402_1005Metric, symbol Device:R_Small_US
- added R62, R63, R64, R65, R68, R69: 10]K, Resistor_SMD:R_0805_2012Metric, symbol Device:R_Small_US
- added R66, R78: SML-P12U2TT86R, GNSS_Library:LED_SML-P11D_ROM, symbol 2026-08-14_04-34-19:SML-P12U2TT86R
- added R67, R79: 560R, Resistor_SMD:R_0805_2012Metric, symbol Device:R_Small_US
- added R80, R81, R82: 10K, Resistor_SMD:R_0402_1005Metric, symbol Device:R_Small_US
- added R83, R84, R85, R86: 10K, Resistor_SMD:R_0805_2012Metric, symbol Device:R_Small_US
- added U13: LT6000IDCB_TRMPBF, LT6000IDCB_TRMPBF:DFN-6_DCB, symbol LT6000IDCB_TRMPBF:LT6000IDCB_TRMPBF
- added U14: TPS22946YZPR, TPS22946YZPR:BGA6C50P2X3_140X90X50, symbol TPS22946YZPR:TPS22946YZPR
- IC2: footprint Module:ZEDF9P05B -> GNSS:ZEDF9P05B
Connections:
- net +3V3_GNSS: now also FL9.2; no longer IC2.33 (VCC_1), IC2.34 (VCC_2), R15.1
- net GND: now also BT1.N, C53.2, C54.1, C55.2, C56.1, C62.2, C63.1, C71.1, D1.1, J4.2, J4.3, J4.4, J4.5, Q2.2 (E), R66.1, R69.2, R78.1, R82.1, U13.5 (V-), U13.7 (EPAD), U14.B1 (GND)
- net GN_CS: now also R64.1
- net GN_SCK: now also R65.1
- net GN_SDI: now also R63.1
- net GN_SDO: now also R62.1
- net GEOFENCE: now reaches IC2.19 (GEOFENCE_STAT)
- net GEOFENCE: now also R67.1
- net at IC2.2 (RF_IN): now also D1.2, J4.1, L3.1
- net RTK_STAT: now reaches IC2.20 (RTK_STAT)
- net RTK_STAT: now also R79.1
- net V_BCKP: now reaches IC2.36 (V_BCKP)
- net V_BCKP: now also BT1.P
- net PG_VBUS: now reaches IC2.38 (V_USB)
- net at IC2.4 (ANT_DETECT): now also U13.4 (OUT)
- net ANT_OFF: now reaches IC2.5 (ANT_OFF_)
- net ANT_OFF: now also Q1.5 (G2), R80.1, R83.2
- net SAFE_BOOT: now reaches IC2.50 (SAFEBOOT_N)
- net SAFE_BOOT: now also JP1.2 (C)
- net ANT_SHORT_N: now reaches IC2.6 (ANT_SHORT_N)
- net ANT_SHORT_N: now also R81.1, R82.2, U13.3 (+IN)
- net RF_VCC: now reaches IC2.7 (VCC_RF)
- net RF_VCC: now also R84.1, R85.1, R86.2, U13.1 (*SHDN), U13.6 (V+), U14.A2 (VIN)
- new net: C71.2, L3.2, R32.1, U13.2 (-IN)
- new net: Q2.1 (B), R83.1
- new net: Q1.3 (D2), R32.2, R81.2
- new net: R78.2, R79.2
- new net: R66.2, R67.2
- new net: JP1.1 (A), R68.1
- new net: Q1.4 (S2), R80.2, U14.A1 (VOUT)
- new net: R86.1, U14.B2 (CL)
- new net: JP1.3 (B), R69.1
- new net +3V3_GN: C53.1, C54.2, C55.1, C56.2, C62.1, C63.2, FL9.1, IC2.33 (VCC_1), IC2.34 (VCC_2), R15.1, R62.2, R63.2, R64.2, R65.2, R68.2
- new net ANT_FAULT: R85.2, U14.C1 (OC)
- new net ON/OFF: Q2.3 (C), R84.2, U14.C2 (ON)
- no-connect marks 25 -> 26
Other:
- moved on the sheet: IC2, R33, R34
