File: ZED_Z9P.kicad_sch (KiCad schematic)
At the start: 39 parts, among them IC2 ZED-F9P-05B, J4 SMA-J-P-X-RA-TH1, Q1 SI1016CX-T1-GE3, Q2 MMBT3904LT1G, U13 LT6000IDCB_TRMPBF, U14 TPS22946YZPR

Commit message: schematics
Parts:
- C54, C56, C63: footprint C0402C104K4RAC:CAPC1005X55N -> Capacitor_SMD:C_0402_1005Metric

Commit message: placed
Parts:
- removed C53: 1uF, Capacitor_SMD:C_0805_2012Metric, symbol Device:C_Small
- removed C54: 100nF, Capacitor_SMD:C_0402_1005Metric, symbol C0402C104K4RAC:C0402C104K4RAC
- J4: footprint SMA-J-P-X-RA-TH1:SAMTEC_SMA-J-P-X-RA-TH1 -> GNSS:SAMTEC_SMA-J-P-X-RA-TH1
- JP1: footprint (none) -> Jumper:SolderJumper-3_P2.0mm_Open_TrianglePad1.0x1.5mm
- R33, R62, R63, R64, R65, R67, R68, R69, R79, R83, R84, R85, R86: footprint Resistor_SMD:R_0805_2012Metric -> Resistor_SMD:R_0402_1005Metric
- R34, R66, R78: footprint GNSS_Library:LED_SML-P11D_ROM -> LED_SMD:LED_0402_1005Metric

Commit message: Almost Placed file
Parts:
- Q1: footprint SOTFL50P160X60-6N -> GNSS:SOTFL50P160X60-6N
- U13: footprint LT6000IDCB_TRMPBF:DFN-6_DCB -> GNSS:DFN-6_DCB
- renumbered R66 to D12, R78 to D13, R34 to D14
Changed lines of the file:
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@@
 			)
 		)
-		(property "Footprint" "LT6000IDCB_TRMPBF:DFN-6_DCB"
+		(property "Footprint" "GNSS:DFN-6_DCB"
 			(at 45.72 102.87 0)
 			(effects
@@
 		(dnp no)
 		(fields_autoplaced yes)
-		(property "Reference" "R78"
+		(property "Reference" "D13"
 			(at 33.02 138.43 0)
 			(effects
@@
 			(project "GNSS"
 				(path "/a70dad34-b24c-4b58-b91c-f14576b5da7d/3ceb85b8-7c9a-4fa2-96e5-dbe80db6ac49"
-					(reference "R78")
+					(reference "D13")
 					(unit 1)
 				)
@@
 		(dnp no)
 		(fields_autoplaced yes)
-		(property "Reference" "R66"
+		(property "Reference" "D12"
 			(at 31.75 116.84 0)
 			(effects
@@
 			(project "GNSS"
 				(path "/a70dad34-b24c-4b58-b91c-f14576b5da7d/3ceb85b8-7c9a-4fa2-96e5-dbe80db6ac49"
-					(reference "R66")
+					(reference "D12")
 					(unit 1)
 				)
@@
 			)
 		)
-		(property "Footprint" "SOTFL50P160X60-6N"
+		(property "Footprint" "GNSS:SOTFL50P160X60-6N"
 			(at 62.23 173.66 0)
 			(effects
@@
 		(dnp no)
 		(fields_autoplaced yes)
-		(property "Reference" "R34"
+		(property "Reference" "D14"
 			(at 219.71 16.51 0)
 			(effects
@@
 			(project "GNSS"
 				(path "/a70dad34-b24c-4b58-b91c-f14576b5da7d/3ceb85b8-7c9a-4fa2-96e5-dbe80db6ac49"
-					(reference "R34")
+					(reference "D14")
 					(unit 1)
 				)

Commit message: new placed
Parts:
- removed FL9: BLM21PG221SN1D, BLM21PG221SN1D:BEADC2012X105N, symbol BLM21PG221SN1D:BLM21PG221SN1D

Commit message: usb
Parts:
- C55, C62: value 1uF -> 1u
- C56, C63: value 100nF -> 100n
- R32: value 10E -> 10R
- R62, R63, R64, R65, R68, R69: value 10]K -> 10K
Changed lines of the file:
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@@
 			)
 		)
-		(property "Value" "100nF"
+		(property "Value" "100n"
 			(at 245.11 69.596 90)
 			(effects
@@
 			)
 		)
-		(property "Value" "10]K"
+		(property "Value" "10K"
 			(at 60.452 167.386 90)
 			(effects
@@
 			)
 		)
-		(property "Value" "10]K"
+		(property "Value" "10K"
 			(at 66.802 167.386 90)
 			(effects
@@
 		(dnp no)
 		(property "Reference" "C71"
-			(at 72.39 68.326 90)
+			(at 72.136 68.326 90)
 			(effects
 				(font
@@
 			)
 		)
-		(property "Value" "10E"
+		(property "Value" "10R"
 			(at 55.88 67.056 0)
 			(effects
@@
 			)
 		)
-		(property "Value" "1uF"
+		(property "Value" "1u"
 			(at 250.952 69.342 0)
 			(effects
@@
 			)
 		)
-		(property "Value" "10]K"
+		(property "Value" "10K"
 			(at 73.152 167.386 90)
 			(effects
@@
 			)
 		)
-		(property "Value" "100nF"
+		(property "Value" "100n"
 			(at 261.62 69.596 90)
 			(effects
@@
 			)
 		)
-		(property "Value" "10]K"
+		(property "Value" "10K"
 			(at 130.81 170.18 90)
 			(effects
@@
 			)
 		)
-		(property "Value" "10]K"
+		(property "Value" "10K"
 			(at 148.844 170.434 90)
 			(effects
@@
 			)
 		)
-		(property "Value" "1uF"
+		(property "Value" "1u"
 			(at 234.442 69.342 0)
 			(effects
@@
 			)
 		)
-		(property "Value" "10]K"
+		(property "Value" "10K"
 			(at 78.232 167.386 90)
 			(effects

Commit message: can
Parts:
- removed D12, D13, D14: SML-P12U2TT86R, LED_SMD:LED_0402_1005Metric, symbol 2026-08-14_04-34-19:SML-P12U2TT86R
- removed R79: 560R, Resistor_SMD:R_0402_1005Metric, symbol Device:R_Small_US
- added D10, D2, D9: SML-P12U2TT86R, LED_SMD:LED_0402_1005Metric, symbol 2026-08-14_04-34-19:SML-P12U2TT86R
- added Q7, Q8, Q9: BC849, Package_TO_SOT_SMD:SOT-23, symbol Transistor_BJT:BC849
- added R44, R71, R72: 10K, Resistor_SMD:R_0402_1005Metric, symbol Device:R_Small_US
- added R73: 560R, Resistor_SMD:R_0402_1005Metric, symbol Device:R_Small_US
Connections:
- net +3V3_GN: now also R33.1, R67.1, R73.1
- net GEOFENCE: now also R71.2; no longer R67.1
- net GND: now also Q7.2 (E), Q8.2 (E), Q9.2 (E)
- net GN_TIMEPULSE: now also D2.1, Q7.3 (C); no longer IC2.53 (TIMEPULSE), R33.1
- net RTK_STAT: now also R72.2
- net at R67.2: now also D9.2
- net at R33.2: now also D2.2
- new net: Q8.1 (B), R72.1
- new net: D10.1, Q8.3 (C)
- new net: Q7.1 (B), R44.1
- new net: IC2.53 (TIMEPULSE), R44.2
- new net: Q9.1 (B), R71.1
- new net: D9.1, Q9.3 (C)
- new net: D10.2, R73.2
Other:
- moved on the sheet: JP1, R15, R62, R63, R64, R65, R68, R69

Commit message: new
Parts:
- removed Q1: SI1016CX-T1-GE3, GNSS:SOTFL50P160X60-6N, symbol SI1016CX-T1-GE3:SI1016CX-T1-GE3
- removed U13: LT6000IDCB_TRMPBF, GNSS:DFN-6_DCB, symbol LT6000IDCB_TRMPBF:LT6000IDCB_TRMPBF
- added Q12: PMOS, symbol Simulation_SPICE:PMOS
- added U3: MCP6001-OT, Package_TO_SOT_SMD:SOT-23-5, symbol Amplifier_Operational:MCP6001-OT
Connections:
- net ANT_OFF: now also Q12.2 (G)
- net ANT_SHORT_N: now also U3.3 (+)
- net GND: now also U3.2 (V-)
- net RF_VCC: now also U3.5 (V+)
- net at C71.2, L3.2, R32.1: now also U3.4 (-)
- net at IC2.4 (ANT_DETECT): now also U3.1
- net at R32.2, R81.2: now also Q12.1 (D)
- net at R80.2, U14.A1 (VOUT): now also Q12.3 (S)
- no-connect marks 26 -> 23
Other:
- moved on the sheet: R80

Commit message: block
Parts:
- R33, R67, R73: value 560R -> 10K
Changed lines of the file:
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@@
 			)
 		)
-		(property "Value" "560R"
+		(property "Value" "10K"
 			(at 236.22 16.51 90)
 			(effects
@@
 			)
 		)
-		(property "Value" "560R"
+		(property "Value" "10K"
 			(at 35.56 132.08 90)
 			(effects
@@
 			)
 		)
-		(property "Value" "560R"
+		(property "Value" "10K"
 			(at 77.47 133.35 90)
 			(effects
