File: ZED_Z9P.kicad_sch (KiCad schematic)
At the start: 42 parts, among them IC2 ZED-F9P-05B, J4 SMA-J-P-X-RA-TH1, Q12 PMOS, Q2 MMBT3904LT1G, Q7 BC849, Q8 BC849, Q9 BC849, U14 TPS22946YZPR, U3 MCP6001-OT

Commit message: full
Parts:
- removed C71: GRM033R71C103KE14D, GRM033R71C103KE14D:CAPC0603X33N, symbol GRM033R71C103KE14D:GRM033R71C103KE14D
- removed D1: PESD0402-140, PESD0402-140:DIO_PESD0402-140, symbol PESD0402-140:PESD0402-140
- removed D10, D2, D9: SML-P12U2TT86R, LED_SMD:LED_0402_1005Metric, symbol 2026-08-14_04-34-19:SML-P12U2TT86R
- removed J4: SMA-J-P-X-RA-TH1, GNSS:SAMTEC_SMA-J-P-X-RA-TH1, symbol SMA-J-P-X-RA-TH1:SMA-J-P-X-RA-TH1
- removed L3: LQG15HS47NJ02D, LQG15HS47NJ02D:INDC1005X55N, symbol LQG15HS47NJ02D:LQG15HS47NJ02D
- removed Q12: PMOS, symbol Simulation_SPICE:PMOS
- removed Q2: MMBT3904LT1G, MMBT3904LT1G:SOT95P240X111-3N, symbol MMBT3904LT1G:MMBT3904LT1G
- removed Q7, Q8, Q9: BC849, Package_TO_SOT_SMD:SOT-23, symbol Transistor_BJT:BC849
- removed R32: 10R, Resistor_SMD:R_0402_1005Metric, symbol Device:R_Small_US
- removed R33, R44, R67, R71, R72, R73, R80, R81, R82, R83, R84, R85, R86: 10K, Resistor_SMD:R_0402_1005Metric, symbol Device:R_Small_US
- removed U14: TPS22946YZPR, TPS22946YZPR:BGA6C50P2X3_140X90X50, symbol TPS22946YZPR:TPS22946YZPR
- removed U3: MCP6001-OT, Package_TO_SOT_SMD:SOT-23-5, symbol Amplifier_Operational:MCP6001-OT
Connections:
- net GN_TIMEPULSE: now also IC2.53 (TIMEPULSE)
- net RF_IN: now reaches IC2.2 (RF_IN)
- net ANT_DETECT: now reaches IC2.4 (ANT_DETECT)
Other:
- moved on the sheet: BT1, C55, C56, C62, C63, IC2, JP1, R15, R62, R63, R64, R65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

Commit message: 16.09.2026
Parts:
- BT1: footprint 1056:BAT_1056 -> GNSS:BAT_1056
Connections:
- net +3V3_GN renamed +3V3_GNSS

Commit message: 22.09.26
Parts:
- added C85: 100n, Capacitor_SMD:C_0402_1005Metric, symbol C0402C104K4RAC:C0402C104K4RAC
- added C86: 2u2, Capacitor_SMD:C_0805_2012Metric, symbol Device:C_Small
- C62: value 1u -> 10u
Connections:
- net GND: now also C85.1, C86.2
- net V_BCKP: now also C85.2, C86.1
Other:
- moved on the sheet: BT1, C55, C56, C62, C63, IC2, JP1, R15, R62, R63, R64, R65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

Commit message: 123
Parts:
- removed R62, R63, R65: 10K, Resistor_SMD:R_0402_1005Metric, symbol Device:R_Small_US
Other:
- moved on the sheet: R64

Commit message: new
Parts:
- added U11: NC7SZ125M5X, SC-74A_318BQ_ONS, symbol 2026-09-29_16-21-45:NC7SZ125M5X
Connections:
- net +3V3_GNSS: now also U11.5 (VCC)
- net GND: now also U11.1 (*OE), U11.3 (GND)
- net GN_TIMEPULSE: now also U11.2 (A)
- new net TIMEPULSE_LED: U11.4 (Y)

Commit message: new
Parts:
- U11: footprint SC-74A_318BQ_ONS -> Package_TO_SOT_SMD:SOT-23-5
Changed lines of the file:
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@@
 			)
 		)
-		(property "Footprint" "SC-74A_318BQ_ONS"
+		(property "Footprint" "Package_TO_SOT_SMD:SOT-23-5"
 			(at 189.23 33.02 0)
 			(effects
