File: IMU.kicad_sch (KiCad schematic)
At the start: 22 parts, among them J3 5033981892, U1 ICM-42688-P

Commit message: placed
Parts:
- removed R77: 10K, Resistor_SMD:R_0805_2012Metric, symbol Device:R_Small_US
- added R43: 10K, Resistor_SMD:R_0402_1005Metric, symbol Device:R_Small_US
- R24, R52, R53, R54, R55, R56, R57, R58, R59, R60, R61: value 10]K -> 10K; footprint Resistor_SMD:R_0805_2012Metric -> Resistor_SMD:R_0402_1005Metric
- R76: footprint Resistor_SMD:R_0805_2012Metric -> Resistor_SMD:R_0402_1005Metric
Connections:
- net +3.3V_SD: now also R43.2; no longer R61.2
- net +3V3_IMU: now also R61.2
- net INT1_ACCEL: now also R61.1; no longer R76.1
- net INT1_GYRO: now also R76.1
- net SD_CLK: now also R57.1; no longer R58.1
- net SD_CMD: now also R56.1; no longer R57.1
- net SD_DAT0: now also R58.1; no longer R59.1
- net SD_DAT1: now also R59.1; no longer R60.1
- net SD_DAT3: now also R43.1; no longer R56.1
- net SD_DETECT: now also R60.1; no longer R61.1

Commit message: new commit
Connections:
- net +3V3_BMI renamed +3V3_ICM
Changed lines of the file:
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@@
 			)
 		)
-		(property "Value" "+3V3_BMI"
+		(property "Value" "+3V3_ICM"
 			(at 156.21 50.8 0)
 			(effects

Commit message: usb
Parts:
- removed C75: 100nF, Capacitor_SMD:C_0402_1005Metric, symbol C0402C104K4RAC:C0402C104K4RAC
- removed C76: 10uF, Capacitor_SMD:C_0805_2012Metric, symbol Device:C_Small
- removed FL5: BLM21PG221SN1D, BLM21PG221SN1D:BEADC2012X105N, symbol BLM21PG221SN1D:BLM21PG221SN1D
- removed J3: 5033981892, GNSS:CONN_503398-1892_MOL, symbol 5033981892:5033981892
- removed R43, R55, R56, R57, R58, R59, R60: 10K, Resistor_SMD:R_0402_1005Metric, symbol Device:R_Small_US
- C29: value 100nF -> 100n
- C30: value 10nF -> 10n
- C67: value 2.2uF -> 2u2
Other:
- note removed: "SD_CARD"
- moved on the sheet: C29, C30, C67, FL4, R24, R52, R53, R54, R61, R76, U1

Commit message: can
Parts:
- added C53: 100n, Capacitor_SMD:C_0402_1005Metric, symbol C0402C104K4RAC:C0402C104K4RAC
- added C54: 10u, Capacitor_SMD:C_0805_2012Metric, symbol Device:C_Small
- added FL5: BLM21PG221SN1D, BLM21PG221SN1D:BEADC2012X105N, symbol BLM21PG221SN1D:BLM21PG221SN1D
- added J3: 5033981892, GNSS:CONN_503398-1892_MOL, symbol 5033981892:5033981892
- added R17, R25, R34, R35, R43, R55, R56: 10K, Resistor_SMD:R_0402_1005Metric, symbol Device:R_Small_US
Connections:
- net GND: now also C53.1, C54.2, J3.6, J3.9
- new net +3.3V: FL5.2
- new net +3.3V_SD: C53.2, C54.1, FL5.1, J3.4, R17.2, R25.2, R34.2, R35.2, R43.2, R55.2, R56.2
- new net SD_CLK: J3.5, R35.1
- new net SD_CMD: J3.3, R34.1
- new net SD_DAT0: J3.7, R43.1
- new net SD_DAT1: J3.8, R55.1
- new net SD_DAT2: J3.1, R17.1
- new net SD_DAT3: J3.2, R25.1
- new net SD_DETECT: J3.10, R56.1
Other:
- note added: "SD_CARD"
- moved on the sheet: C29, C30, C67, FL4, R24, R52, R53, R54, R61, R76, U1
