File: USB_HUB_sch.kicad_sch (KiCad schematic)
At the start: 22 parts, among them IC1 USB2513B_M2, Y1 MURATA_XRCGB24M000FFS1DR0

Commit message: changed
Connections:
- net VBUS renamed PG_VBUS
Changed lines of the file:
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@@
+		)
+	)
+	(text_box "VBUS CHANGED TO PG_VBUS           DONE"
+		(exclude_from_sim no)
+		(at 71.12 59.69 0)
+		(size 19.05 13.97)
+		(stroke
+			(width 0)
+			(type default)
+		)
+		(fill
+			(type none)
+		)
+		(effects
+			(font
+				(size 1.27 1.27)
+			)
+			(justify left top)
 		)
 	)
@@
 		)
 	)
-	(label "VBUS"
+	(label "PG_VBUS"
 		(at 135.89 81.28 90)
 		(fields_autoplaced yes)

Commit message: new
Other:
- moved on the sheet: R6, R9

Commit message: new
Connections:
- net +3.3V: no longer C10.2, C4.2, C5.2, C6.2, C7.2, C8.2, C9.2, IC1.10 (VDDA33_2), IC1.15 (VDD33_1), IC1.23 (VDD33_2), IC1.29 (VDDA33_3), IC1.36 (VDDA33_4), IC1.5 (VDDA33_1)
- new net +3.3V_HUB: C10.2, C4.2, C5.2, C6.2, C7.2, C8.2, C9.2, IC1.10 (VDDA33_2), IC1.15 (VDD33_1), IC1.23 (VDD33_2), IC1.29 (VDDA33_3), IC1.36 (VDDA33_4), IC1.5 (VDDA33_1)
Changed lines of the file:
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@@
 	)
 	(junction
-		(at 148.59 72.39)
+		(at 237.49 39.37)
 		(diameter 0)
 		(color 0 0 0 0)
 	)
 	(junction
-		(at 237.49 39.37)
+		(at 143.51 69.85)
 		(diameter 0)
 		(color 0 0 0 0)
@@
 	)
 	(junction
-		(at 143.51 72.39)
-		(diameter 0)
-		(color 0 0 0 0)
-	)
-	(junction
 		(at 261.62 68.58)
 		(diameter 0)
@@
 	)
 	(junction
+		(at 148.59 69.85)
+		(diameter 0)
+		(color 0 0 0 0)
+	)
+	(junction
 		(at 242.57 55.88)
 		(diameter 0)
@@
 	(wire
 		(pts
-			(xy 143.51 72.39) (xy 148.59 72.39)
+			(xy 143.51 69.85) (xy 148.59 69.85)
 		)
 		(stroke
@@
 	(wire
 		(pts
-			(xy 78.74 121.92) (xy 74.93 121.92)
+			(xy 78.74 121.92) (xy 69.85 121.92)
 		)
 		(stroke
@@
 	(wire
 		(pts
+			(xy 143.51 69.85) (xy 143.51 72.39)
+		)
+		(stroke
+			(width 0)
+			(type default)
+		)
+	)
+	(wire
+		(pts
 			(xy 59.69 127) (xy 64.77 127)
 		)
@@
 	(wire
 		(pts
-			(xy 140.97 72.39) (xy 143.51 72.39)
+			(xy 140.97 69.85) (xy 143.51 69.85)
 		)
 		(stroke
@@
 	(wire
 		(pts
+			(xy 152.4 69.85) (xy 152.4 72.39)
+		)
+		(stroke
+			(width 0)
+			(type default)
+		)
+	)
+	(wire
+		(pts
 			(xy 243.84 68.58) (xy 243.84 69.85)
 		)
@@
 	(wire
 		(pts
-			(xy 186.69 114.3) (xy 184.15 114.3)
+			(xy 242.57 55.88) (xy 242.57 60.96)
 		)
 		(stroke
@@
 	(wire
 		(pts
-			(xy 242.57 55.88) (xy 242.57 60.96)
+			(xy 256.54 68.58) (xy 261.62 68.58)
 		)
 		(stroke
@@
 	(wire
 		(pts
-			(xy 256.54 68.58) (xy 261.62 68.58)
+			(xy 69.85 121.92) (xy 69.85 124.46)
 		)
 		(stroke
@@
 	(wire
 		(pts
-			(xy 74.93 121.92) (xy 74.93 124.46)
+			(xy 237.49 68.58) (xy 242.57 68.58)
 		)
 		(stroke
@@
 	(wire
 		(pts
-			(xy 237.49 68.58) (xy 242.57 68.58)
+			(xy 252.73 39.37) (xy 257.81 39.37)
 		)
 		(stroke
@@
 	(wire
 		(pts
-			(xy 252.73 39.37) (xy 257.81 39.37)
+			(xy 148.59 69.85) (xy 148.59 72.39)
 		)
 		(stroke
@@
 	(wire
 		(pts
-			(xy 148.59 72.39) (xy 152.4 72.39)
+			(xy 148.59 69.85) (xy 152.4 69.85)
 		)
 		(stroke
@@
 	(wire
 		(pts
+			(xy 140.97 69.85) (xy 140.97 72.39)
+		)
+		(stroke
+			(width 0)
+			(type default)
+		)
+	)
+	(wire
+		(pts
 			(xy 64.77 114.3) (xy 64.77 104.14)
 		)
@@
 		(exclude_from_sim no)
 		(at 34.29 49.53 0)
-		(size 166.37 115.57)
+		(size 167.64 115.57)
 		(stroke
 			(width 0.0508)
@@
 		)
 	)
-	(label "PG_VBUS"
-		(at 135.89 81.28 90)
-		(fields_autoplaced yes)
-		(effects
-			(font
-				(size 1.27 1.27)
-			)
-			(justify left bottom)
-		)
-	)
 	(label "PLL"
 		(at 88.9 119.38 180)
@@
 		)
 	)
+	(global_label "PG_VBUS"
+		(shape input)
+		(at 135.89 81.28 90)
+		(fields_autoplaced yes)
+		(effects
+			(font
+				(size 1.27 1.27)
+			)
+			(justify left)
+		)
+		(property "Intersheetrefs" "${INTERSHEET_REFS}"
+			(at 135.89 69.8886 90)
+			(effects
+				(font
+					(size 1.27 1.27)
+				)
+				(justify left)
+				(hide yes)
+			)
+		)
+	)
 	(global_label "ESP_D_N"
 		(shape input)
@@
 			)
 		)
-		(property "Value" "+3.3V"
+		(property "Value" "+3.3V_HUB"
 			(at 86.36 106.6799 90)
 			(effects
@@
 			)
 		)
-		(property "Value" "+3.3V"
+		(property "Value" "+3.3V_HUB"
 			(at 187.96 126.9999 90)
 			(effects
@@
 	(symbol
 		(lib_id "power:+3.3V")
-		(at 186.69 114.3 270)
+		(at 184.15 114.3 270)
 		(unit 1)
 		(exclude_from_sim no)
@@
 		(fields_autoplaced yes)
 		(property "Reference" "#PWR0153"
-			(at 182.88 114.3 0)
+			(at 180.34 114.3 0)
 			(effects
 				(font
@@
 			)
 		)
-		(property "Value" "+3.3V"
-			(at 190.5 114.2999 90)
+		(property "Value" "+3.3V_HUB"
+			(at 187.96 114.2999 90)
 			(effects
 				(font
@@
 		)
 		(property "Footprint" ""
-			(at 186.69 114.3 0)
+			(at 184.15 114.3 0)
 			(effects
 				(font
@@
 		)
 		(property "Datasheet" ""
-			(at 186.69 114.3 0)
+			(at 184.15 114.3 0)
 			(effects
 				(font
@@
 		)
 		(property "Description" "Power symbol creates a global label with name \"+3.3V\""
-			(at 186.69 114.3 0)
+			(at 184.15 114.3 0)
 			(effects
 				(font
@@
 	(symbol
 		(lib_id "power:GND")
-		(at 74.93 124.46 0)
+		(at 69.85 124.46 0)
 		(unit 1)
 		(exclude_from_sim no)
@@
 		(fields_autoplaced yes)
 		(property "Reference" "#PWR017"
-			(at 74.93 130.81 0)
+			(at 69.85 130.81 0)
 			(effects
 				(font
@@
 		)
 		(property "Value" "GND"
-			(at 74.93 129.54 0)
+			(at 69.85 129.54 0)
 			(effects
 				(font
@@
 		)
 		(property "Footprint" ""
-			(at 74.93 124.46 0)
+			(at 69.85 124.46 0)
 			(effects
 				(font
@@
 		)
 		(property "Datasheet" ""
-			(at 74.93 124.46 0)
+			(at 69.85 124.46 0)
 			(effects
 				(font
@@
 		)
 		(property "Description" "Power symbol creates a global label with name \"GND\" , ground"
-			(at 74.93 124.46 0)
+			(at 69.85 124.46 0)
 			(effects
 				(font
@@
 			)
 		)
-		(property "Value" "+3.3V"
+		(property "Value" "+3.3V_HUB"
 			(at 227.33 31.75 0)
 			(effects
@@
 			)
 		)
-		(property "Value" "+3.3V"
+		(property "Value" "+3.3V_HUB"
 			(at 146.05 157.48 90)
 			(effects
@@
 			)
 		)
-		(property "Value" "+3.3V"
-			(at 146.05 76.2 90)
+		(property "Value" "+3.3V_HUB"
+			(at 145.796 73.152 90)
 			(effects
 				(font
@@
 		(dnp no)
 		(property "Reference" "R6"
-			(at 77.724 120.904 90)
+			(at 78.232 120.904 90)
 			(effects
 				(font
@@
 		)
 		(property "Value" "12K"
-			(at 79.502 123.952 90)
+			(at 87.63 120.904 90)
 			(effects
 				(font
@@
 			)
 		)
-		(property "Value" "+3.3V"
+		(property "Value" "+3.3V_HUB"
 			(at 86.36 124.4599 90)
 			(effects

Commit message: new
Parts:
- added C72: 1uF, C0402C104K4RAC:CAPC1005X55N, symbol C0402C104K4RAC:C0402C104K4RAC
- added FL10: BLM21PG221SN1D, BLM21PG221SN1D:BEADC2012X105N, symbol BLM21PG221SN1D:BLM21PG221SN1D
- added R87, R88, R89, R90: 100K, Resistor_SMD:R_0402_1005Metric, symbol Device:R_Small_US
- added R91: 1Meg, Resistor_SMD:R_0402_1005Metric, symbol Device:R_Small_US
- added U10, U11, U12: TPD2EUSB30ADRTR, symbol TPD2EUSB30ADRTR:TPD2EUSB30ADRTR
- C11, C13: value 0.1uF -> 1uF
- IC1: footprint QFN50P600X600X100-37N-D -> GNSS:QFN50P600X600X100-37N-D
- R10, R8: value 100K -> 10K; now not fitted
Connections:
- net +3.3V: now also FL10.1; no longer R5.2
- net +3.3V_HUB: now also R10.1, R5.2, R8.2, FL10.2
- net ESP_D_N: now also U11.2 (D-)
- net ESP_D_P: now also U11.1 (D+)
- net GND: now also R8.1, C72.1, R87.1, R88.1, R90.2, U10.3 (GND), U11.3 (GND), U12.3 (GND); no longer R8.2
- net GNSS_D_N: now also U10.2 (D-)
- net GNSS_D_P: now also U10.1 (D+)
- net PG_VBUS: now also C72.2, R89.2; no longer IC1.27 (VBUS_DET)
- net STM_D_N: now also U12.2 (D-)
- net STM_D_P: now also U12.1 (D+)
- net USB_RST: now reaches C3.2, IC1.26 (RESET_N), R5.1
- net at IC1.22 (SDA/SMBDATA/NON_REM1): now also R88.2; no longer R10.1
- net at IC1.24 (SCL/SMBCLK/CFG_SEL0): now also R87.2; no longer R8.1
- net at C2.1, IC1.32 (XTALOUT), Y1.1: now also R91.2
- net at C1.1, IC1.33 (XTALIN/CLKIN), Y1.3: now also R91.1
- new net: IC1.27 (VBUS_DET), R89.1, R90.1
Other:
- moved on the sheet: C1, C10, C2, C3, C4, C5, C6, C7, C8, C9, R5

Commit message: new
Parts:
- R9: value 100K -> 10K; footprint Resistor_SMD:R_0402_1005Metric -> Resistor_SMD:R_0805_2012Metric
Connections:
- net +3.3V: now also R9.2
- net GND: no longer R10.2, R8.1, R9.1
- net USB_SDA: now reaches IC1.22 (SDA/SMBDATA/NON_REM1), R88.2
- net USB_SDA: now also R10.2
- net USB_SCL: now reaches IC1.24 (SCL/SMBCLK/CFG_SEL0), R87.2
- net USB_SCL: now also R8.1
- net at IC1.28 (SUSP_IND/LOCAL_PWR/NON_REM0): now also R9.1; no longer R9.2
Other:
- moved on the sheet: R87, R88, U11

Commit message: schematics
Parts:
- C11, C13: footprint C0402C104K4RAC:CAPC1005X55N -> Capacitor_SMD:C_0805_2012Metric
- C12, C14, C4, C5, C6, C7, C8, C9: footprint C0402C104K4RAC:CAPC1005X55N -> Capacitor_SMD:C_0402_1005Metric
- U10, U11, U12: footprint (none) -> GNSS:SOTFL35P100X50-3N
Connections:
- net CR: now also C12.2; no longer C14.2
- net ESP_D_N: now also U12.2 (D-); no longer U11.2 (D-)
- net ESP_D_P: now also U12.1 (D+); no longer U11.1 (D+)
- net PLL: now also C14.2; no longer C12.2
- net STM_D_N: now also U11.2 (D-); no longer U12.2 (D-)
- net STM_D_P: now also U11.1 (D+); no longer U12.1 (D+)

Commit message: placed
Parts:
- R9: footprint Resistor_SMD:R_0805_2012Metric -> Resistor_SMD:R_0402_1005Metric
Changed lines of the file:
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@@
 			)
 		)
-		(property "Footprint" "Resistor_SMD:R_0805_2012Metric"
+		(property "Footprint" "Resistor_SMD:R_0402_1005Metric"
 			(at 82.55 99.06 0)
 			(effects

Commit message: Almost Placed file
Parts:
- Y1: footprint Crystal:MURATA_XRCGB24M000FFS1DR0_0 -> GNSS:MURATA_XRCGB24M000FFS1DR0_0
Changed lines of the file:
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@@
 			)
 		)
-		(property "Footprint" "Crystal:MURATA_XRCGB24M000FFS1DR0_0"
+		(property "Footprint" "GNSS:MURATA_XRCGB24M000FFS1DR0_0"
 			(at 64.77 106.68 0)
 			(effects
