File: USB_HUB_sch.kicad_sch (KiCad schematic)
At the start: 32 parts, among them IC1 USB2513B_M2, U10 TPD2EUSB30ADRTR, U11 TPD2EUSB30ADRTR, U12 TPD2EUSB30ADRTR, Y1 MURATA_XRCGB24M000FFS1DR0

Commit message: usb
Parts:
- C1, C2: value 18pF -> 18p
- C10: value 4.7uF -> 4u7
- C11, C13, C72: value 1uF -> 1u
- C12, C14, C3, C4, C5, C6, C7, C8, C9: value 0.1uF -> 0.1u
- R91: value 1Meg -> 1M
Changed lines of the file:
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@@
 			)
 		)
-		(property "Value" "1Meg"
+		(property "Value" "1M"
 			(at 41.91 107.188 90)
 			(effects
@@
 			)
 		)
-		(property "Value" "0.1uF"
+		(property "Value" "0.1u"
 			(at 252.476 42.926 0)
 			(effects
@@
 			)
 		)
-		(property "Value" "0.1uF"
+		(property "Value" "0.1u"
 			(at 260.096 68.326 0)
 			(effects
@@
 			)
 		)
-		(property "Value" "0.1uF"
+		(property "Value" "0.1u"
 			(at 133.604 61.214 0)
 			(effects
@@
 			)
 		)
-		(property "Value" "1uF"
+		(property "Value" "1u"
 			(at 255.016 68.326 0)
 			(effects
@@
 			)
 		)
-		(property "Value" "4.7uF"
+		(property "Value" "4u7"
 			(at 230.886 42.926 0)
 			(effects
@@
 			)
 		)
-		(property "Value" "0.1uF"
+		(property "Value" "0.1u"
 			(at 242.316 42.926 0)
 			(effects
@@
 			)
 		)
-		(property "Value" "0.1uF"
+		(property "Value" "0.1u"
 			(at 237.236 42.926 0)
 			(effects
@@
 			)
 		)
-		(property "Value" "1uF"
+		(property "Value" "1u"
 			(at 117.094 74.676 0)
 			(effects
@@
 			)
 		)
-		(property "Value" "0.1uF"
+		(property "Value" "0.1u"
 			(at 241.046 68.326 0)
 			(effects
@@
 			)
 		)
-		(property "Value" "0.1uF"
+		(property "Value" "0.1u"
 			(at 247.396 42.926 0)
 			(effects
@@
 			)
 		)
-		(property "Value" "18pF"
+		(property "Value" "18p"
 			(at 60.96 138.4299 90)
 			(effects
@@
 			)
 		)
-		(property "Value" "18pF"
+		(property "Value" "18p"
 			(at 60.96 99.0599 90)
 			(effects
@@
 			)
 		)
-		(property "Value" "0.1uF"
+		(property "Value" "0.1u"
 			(at 262.636 42.926 0)
 			(effects
@@
 			)
 		)
-		(property "Value" "0.1uF"
+		(property "Value" "0.1u"
 			(at 257.556 42.926 0)
 			(effects
@@
 			)
 		)
-		(property "Value" "1uF"
+		(property "Value" "1u"
 			(at 235.966 68.326 0)
 			(effects

Commit message: new
Other:
- moved on the sheet: C1, C2, C3, C72, IC1, R10, R5, R6, R7, R8, R87, R88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

Commit message: full
Parts:
- removed U10, U11, U12: TPD2EUSB30ADRTR, GNSS:SOTFL35P100X50-3N, symbol TPD2EUSB30ADRTR:TPD2EUSB30ADRTR
- added U10, U12, U3: TPD2EUSB30A, Package_TO_SOT_SMD:Texas_DRT-3, symbol Power_Protection:TPD2EUSB30A
Connections:
- net ESP_D_N: now also U10.2 (D-)
- net ESP_D_P: now also U10.1 (D+)
- net GND: now also U10.3 (GND), U12.3 (GND), U3.3 (GND)
- net GNSS_D_N: now also U3.2 (D-)
- net GNSS_D_P: now also U3.1 (D+)
- net STM_D_N: now also U12.2 (D-)
- net STM_D_P: now also U12.1 (D+)

Commit message: 16.09.2026
Parts:
- FL10: footprint BLM21PG221SN1D:BEADC2012X105N -> GNSS:BEADC2012X105N
- R10, R8: now fitted
- R87, R88: now not fitted
Other:
- moved on the sheet: FL10
Changed lines of the file:
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@@
 	(wire
 		(pts
-			(xy 187.96 24.13) (xy 193.04 24.13)
+			(xy 158.75 41.91) (xy 163.83 41.91)
 		)
 		(stroke
@@
 	(wire
 		(pts
-			(xy 215.9 20.32) (xy 215.9 24.13)
+			(xy 186.69 38.1) (xy 186.69 41.91)
 		)
 		(stroke
@@
 	(wire
 		(pts
-			(xy 210.82 24.13) (xy 215.9 24.13)
+			(xy 181.61 41.91) (xy 186.69 41.91)
 		)
 		(stroke
@@
 	(wire
 		(pts
-			(xy 187.96 21.59) (xy 187.96 24.13)
+			(xy 158.75 39.37) (xy 158.75 41.91)
 		)
 		(stroke
@@
 	(symbol
 		(lib_id "BLM21PG221SN1D:BLM21PG221SN1D")
-		(at 208.28 24.13 0)
+		(at 179.07 41.91 0)
 		(unit 1)
 		(exclude_from_sim no)
@@
 		(fields_autoplaced yes)
 		(property "Reference" "FL10"
-			(at 201.93 17.78 0)
+			(at 172.72 35.56 0)
 			(effects
 				(font
@@
 		)
 		(property "Value" "BLM21PG221SN1D"
-			(at 201.93 20.32 0)
+			(at 172.72 38.1 0)
 			(effects
 				(font
@@
 			)
 		)
-		(property "Footprint" "BLM21PG221SN1D:BEADC2012X105N"
-			(at 211.328 12.954 0)
+		(property "Footprint" "GNSS:BEADC2012X105N"
+			(at 182.118 30.734 0)
 			(effects
 				(font
@@
 		)
 		(property "Datasheet" ""
-			(at 208.28 24.13 0)
+			(at 179.07 41.91 0)
 			(effects
 				(font
@@
 		)
 		(property "Description" ""
-			(at 208.28 24.13 0)
+			(at 179.07 41.91 0)
 			(effects
 				(font
@@
 		)
 		(property "MF" "Murata"
-			(at 225.806 18.288 0)
+			(at 196.596 36.068 0)
 			(effects
 				(font
@@
 		)
 		(property "Description_1" "\n                        \n                            220 Ohms @ 100 MHz 1 Power Line Ferrite Bead 0805 (2012 Metric) 2A 45mOhm\n                        \n"
-			(at 208.026 16.002 0)
+			(at 178.816 33.782 0)
 			(effects
 				(font
@@
 		)
 		(property "Package" "2012 Murata"
-			(at 210.058 18.542 0)
+			(at 180.848 36.322 0)
 			(effects
 				(font
@@
 		)
 		(property "Price" "None"
-			(at 219.456 19.05 0)
+			(at 190.246 36.83 0)
 			(effects
 				(font
@@
 		)
 		(property "SnapEDA_Link" "https://www.snapeda.com/parts/BLM21PG221SN1D/Murata/view-part/?ref=snap"
-			(at 211.328 15.748 0)
+			(at 182.118 33.528 0)
 			(effects
 				(font
@@
 		)
 		(property "MP" "BLM21PG221SN1D"
-			(at 216.662 11.43 0)
+			(at 187.452 29.21 0)
 			(effects
 				(font
@@
 		)
 		(property "Availability" "In Stock"
-			(at 233.172 19.05 0)
+			(at 203.962 36.83 0)
 			(effects
 				(font
@@
 		)
 		(property "Check_prices" "https://www.snapeda.com/parts/BLM21PG221SN1D/Murata/view-part/?ref=eda"
-			(at 214.376 9.652 0)
+			(at 185.166 27.432 0)
 			(effects
 				(font
@@
 		(in_bom yes)
 		(on_board yes)
-		(dnp yes)
+		(dnp no)
 		(property "Reference" "R10"
 			(at 136.906 65.532 90)
@@
 		(in_bom yes)
 		(on_board yes)
-		(dnp no)
+		(dnp yes)
 		(property "Reference" "R88"
 			(at 140.462 56.134 90)
@@
 	(symbol
 		(lib_id "power:+3.3V")
-		(at 215.9 20.32 0)
+		(at 186.69 38.1 0)
 		(unit 1)
 		(exclude_from_sim no)
@@
 		(dnp no)
 		(property "Reference" "#PWR0211"
-			(at 215.9 24.13 0)
+			(at 186.69 41.91 0)
 			(effects
 				(font
@@
 		)
 		(property "Value" "+3.3V_HUB"
-			(at 216.154 15.748 0)
+			(at 186.944 33.528 0)
 			(effects
 				(font
@@
 		)
 		(property "Footprint" ""
-			(at 215.9 20.32 0)
+			(at 186.69 38.1 0)
 			(effects
 				(font
@@
 		)
 		(property "Datasheet" ""
-			(at 215.9 20.32 0)
+			(at 186.69 38.1 0)
 			(effects
 				(font
@@
 		)
 		(property "Description" "Power symbol creates a global label with name \"+3.3V\""
-			(at 215.9 20.32 0)
+			(at 186.69 38.1 0)
 			(effects
 				(font
@@
 	(symbol
 		(lib_id "power:+3.3V")
-		(at 187.96 21.59 0)
+		(at 158.75 39.37 0)
 		(unit 1)
 		(exclude_from_sim no)
@@
 		(fields_autoplaced yes)
 		(property "Reference" "#PWR0210"
-			(at 187.96 25.4 0)
+			(at 158.75 43.18 0)
 			(effects
 				(font
@@
 		)
 		(property "Value" "+3.3V"
-			(at 187.96 16.51 0)
+			(at 158.75 34.29 0)
 			(effects
 				(font
@@
 		)
 		(property "Footprint" ""
-			(at 187.96 21.59 0)
+			(at 158.75 39.37 0)
 			(effects
 				(font
@@
 		)
 		(property "Datasheet" ""
-			(at 187.96 21.59 0)
+			(at 158.75 39.37 0)
 			(effects
 				(font
@@
 		)
 		(property "Description" "Power symbol creates a global label with name \"+3.3V\""
-			(at 187.96 21.59 0)
+			(at 158.75 39.37 0)
 			(effects
 				(font
@@
 		(in_bom yes)
 		(on_board yes)
-		(dnp no)
+		(dnp yes)
 		(property "Reference" "R87"
 			(at 140.462 49.784 90)
@@
 		(in_bom yes)
 		(on_board yes)
-		(dnp yes)
+		(dnp no)
 		(property "Reference" "R8"
 			(at 135.636 41.402 90)

Commit message: 18.09.2026
Connections:
- net +3.3V renamed +3V3
- net +3.3V_HUB renamed +3V3_HUB
Changed lines of the file:
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@@
 			)
 		)
-		(property "Value" "+3.3V"
+		(property "Value" "+3V3"
 			(at 72.39 87.63 0)
 			(effects
@@
 			)
 		)
-		(property "Value" "+3.3V_HUB"
+		(property "Value" "+3V3_HUB"
 			(at 76.2 104.1399 90)
 			(effects
@@
 			)
 		)
-		(property "Value" "+3.3V_HUB"
+		(property "Value" "+3V3_HUB"
 			(at 124.46 40.64 0)
 			(effects
@@
 			)
 		)
-		(property "Value" "+3.3V_HUB"
+		(property "Value" "+3V3_HUB"
 			(at 156.21 122.428 90)
 			(effects
@@
 			)
 		)
-		(property "Value" "+3.3V_HUB"
+		(property "Value" "+3V3_HUB"
 			(at 186.944 33.528 0)
 			(effects
@@
 			)
 		)
-		(property "Value" "+3.3V_HUB"
+		(property "Value" "+3V3_HUB"
 			(at 162.56 107.9499 90)
 			(effects
@@
 			)
 		)
-		(property "Value" "+3.3V"
+		(property "Value" "+3V3"
 			(at 158.75 34.29 0)
 			(effects
@@
 			)
 		)
-		(property "Value" "+3.3V_HUB"
+		(property "Value" "+3V3_HUB"
 			(at 227.838 26.67 0)
 			(effects
@@
 			)
 		)
-		(property "Value" "+3.3V_HUB"
+		(property "Value" "+3V3_HUB"
 			(at 119.38 157.988 90)
 			(effects
@@
 			)
 		)
-		(property "Value" "+3.3V_HUB"
+		(property "Value" "+3V3_HUB"
 			(at 144.272 71.882 90)
 			(effects
@@
 			)
 		)
-		(property "Value" "+3.3V_HUB"
+		(property "Value" "+3V3_HUB"
 			(at 118.872 61.468 90)
 			(effects
@@
 			)
 		)
-		(property "Value" "+3.3V_HUB"
+		(property "Value" "+3V3_HUB"
 			(at 140.208 38.608 0)
 			(effects
@@
 			)
 		)
-		(property "Value" "+3.3V_HUB"
+		(property "Value" "+3V3_HUB"
 			(at 76.2 121.9199 90)
 			(effects

Commit message: 22.09.26
Parts:
- removed FL10: BLM21PG221SN1D, GNSS:BEADC2012X105N, symbol BLM21PG221SN1D:BLM21PG221SN1D
- removed R91: 1M, Resistor_SMD:R_0402_1005Metric, symbol Device:R_Small_US
- added FB11: FerriteBead, GNSS:BEADC2012X105N, symbol Device:FerriteBead
Connections:
- net +3V3: now also FB11.1
- net +3V3_HUB: now also FB11.2
Other:
- moved on the sheet: C1, C2, C3, C72, IC1, R10, R5, R6, R7, R8, R87, R88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
