File: Power_sch.kicad_sch (KiCad schematic)
At the start: 38 parts, among them J1 USB4105-GF-A, J2 USB4105-GF-A, U2 TPD2EUSB30ADRTR, U6 ADP150WACBZ-3.3-R7, U7 IR3883MTRPBF

Commit message: new
Changed lines of the file:
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@@
-	(wire
-		(pts
-			(xy 29.21 58.42) (xy 38.1 58.42)
-		)
-		(stroke
-			(width 0)
-			(type default)
-		)
-	)
 	(wire
 		(pts
@@
 		)
 	)
-	(label "PG_VBUS"
-		(at 104.14 66.04 0)
-		(fields_autoplaced yes)
-		(effects
-			(font
-				(size 1.27 1.27)
-			)
-			(justify left bottom)
-		)
-	)
 	(label "EN"
 		(at 152.4 127 180)
@@
 	(label "VO"
 		(at 218.44 124.46 0)
-		(fields_autoplaced yes)
-		(effects
-			(font
-				(size 1.27 1.27)
-			)
-			(justify left bottom)
-		)
-	)
-	(label "PG_VBUS"
-		(at 29.21 58.42 0)
 		(fields_autoplaced yes)
 		(effects
@@
 			(effects
 				(font
+					(size 1.27 1.27)
+				)
+				(justify right)
+				(hide yes)
+			)
+		)
+	)
+	(global_label "PG_VBUS"
+		(shape input)
+		(at 104.14 66.04 0)
+		(fields_autoplaced yes)
+		(effects
+			(font
+				(size 1.27 1.27)
+			)
+			(justify left)
+		)
+		(property "Intersheetrefs" "${INTERSHEET_REFS}"
+			(at 115.5314 66.04 0)
+			(effects
+				(font
+					(size 1.27 1.27)
+				)
+				(justify left)
+				(hide yes)
+			)
+		)
+	)
+	(global_label "PG_VBUS"
+		(shape input)
+		(at 38.1 58.42 180)
+		(fields_autoplaced yes)
+		(effects
+			(font
+				(size 1.27 1.27)
+			)
+			(justify right)
+		)
+		(property "Intersheetrefs" "${INTERSHEET_REFS}"
+			(at 26.7086 58.42 0)
+			(effects
+				(font

Commit message: change
Parts:
- added R46: 32.4K, Resistor_SMD:R_0402_1005Metric, symbol Device:R_Small_US
- added R47: 47K, Resistor_SMD:R_0402_1005Metric, symbol Device:R_Small_US
Connections:
- net GND: now also R47.1
- net VIN: now also R46.1, R46.2, R47.2

Commit message: new
Parts:
- removed D1, D2: PMEG3030EP_115, PMEG3030EP_115:SOD128, symbol PMEG3030EP_115:PMEG3030EP_115
- removed TP3: TestPoint, TestPoint:TestPoint_Pad_D2.0mm, symbol Connector:TestPoint
- added FL6, FL7, FL8: BLM21PG221SN1D, BLM21PG221SN1D:BEADC2012X105N, symbol BLM21PG221SN1D:BLM21PG221SN1D
- added R18, R92: 560R, Resistor_SMD:R_0805_2012Metric, symbol Device:R_Small_US
- added R31: 10K, Resistor_SMD:R_0805_2012Metric, symbol Device:R_Small_US
- added R35, R93: SML-P12U2TT86R, GNSS_Library:LED_SML-P11D_ROM, symbol 2026-08-14_04-34-19:SML-P12U2TT86R
- added TP1: TestPoint, TestPoint:TestPoint_Pad_D2.0mm, symbol Connector:TestPoint
- added U9: LM66200DRLR, SOT-5X3_DRL_TEX, symbol 2026-08-30_06-28-01:LM66200DRLR
- C22, C23: value 1uF -> 10uF
- C24: value 0.47uF -> 0.47
- C25: value 2.7uF -> 4.7uF
- C26: value 2.7uF -> 10uF
- J1, J2: footprint USB4105_GCT -> GNSS:USB4105_GCT
- U6: footprint Module:CB-4-3_ADI -> GNSS:CB-4-3_ADI
- U7: footprint Module:VREG_IR3883MTRPBF -> GNSS:VREG_IR3883MTRPBF
- VR1: footprint Module:SON50P300X300X80-11N -> GNSS:SON50P300X300X80-11N
Connections:
- net +3.3V: now also R31.2
- net EX_VBUS: now also R92.1, U9.6 (VIN2)
- net GND: now also R35.1, R93.1, U9.1 (GND), U9.4 (ON), U9.5 (GND)
- net PG_VBUS: now also R18.1, U9.3 (VIN1)
- net VIN: now also FL6.1, FL7.1, FL8.1, U9.2 (VOUT), U9.7 (VOUT); no longer C19.1, C20.1, C21.2, C23.1, C25.1, R46.1, R46.2, R47.2, U6.A1 (VIN), U6.B1 (EN), U7.1 (VIN), U7.15_16 (PVIN), U7.2 (VCC), U7.5 (EN/FCCM), VR1.1 (IN_1), VR1.2 (IN_2), VR1.3 (EN/UV)
- new net: R31.1, TP1.1, U9.8 (ST)
- new net: R92.2, R93.2
- new net: R18.2, R35.2
- new net 5V: C19.1, C20.1, C21.2, FL8.2, R46.1, R46.2, R47.2, U7.1 (VIN), U7.15_16 (PVIN), U7.2 (VCC), U7.5 (EN/FCCM)
- new net VIN_BMI: C23.1, FL7.2, U6.A1 (VIN), U6.B1 (EN)
- new net VIN_GNSS: C25.1, FL6.2, VR1.1 (IN_1), VR1.2 (IN_2), VR1.3 (EN/UV)
Other:
- note added: "3.3V, 500mA"
- note added: "@5V, 1.5A DROP IS 60mV"
- moved on the sheet: C22, C25, TP12, TP2, U2

Commit message: new
Connections:
- net EX_VBUS: no longer J2.A4-B9 (VBUS)
- net PG_VBUS: no longer J1.A4-B9 (VBUS)
- net at D4.1 (K), F2.1, J2.B4-A9 (VBUS): now also J2.A4-B9 (VBUS)
- net at D3.1 (K), F1.1, J1.B4-A9 (VBUS): now also J1.A4-B9 (VBUS)
Other:
- note added: "3.3V, 150mA"
- note added: "3.3V, 3A"
- moved on the sheet: C15, C16, C17, C18, C19, C20, C21, C22, C23, C24, C25, C26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

Commit message: schematics
Parts:
- D4: footprint ESD5V0D5TP -> GNSS:ESD5V0D5TP
- F1, F2: footprint FUSC4632X85N -> GNSS:FUSC4632X85N
- U2: footprint (none) -> GNSS:SOTFL35P100X50-3N
Changed lines of the file:
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@@
 			)
 		)
-		(property "Footprint" "FUSC4632X85N"
+		(property "Footprint" "GNSS:FUSC4632X85N"
 			(at 100.33 202.87 0)
 			(effects
@@
 			)
 		)
-		(property "Footprint" ""
+		(property "Footprint" "GNSS:SOTFL35P100X50-3N"
 			(at 130.81 170.18 0)
 			(effects
@@
 			)
 		)
-		(property "Footprint" "FUSC4632X85N"
+		(property "Footprint" "GNSS:FUSC4632X85N"
 			(at 99.06 143.18 0)
 			(effects
@@
 			)
 		)
-		(property "Footprint" "ESD5V0D5TP"
+		(property "Footprint" "GNSS:ESD5V0D5TP"
 			(at -9.83 118.11 0)
 			(effects

Commit message: placed
Parts:
- added C83, C84: 0.1uF, C0402C104K4RAC:CAPC1005X55N, symbol C0402C104K4RAC:C0402C104K4RAC
- C24: footprint C0402C104K4RAC:CAPC1005X55N -> Capacitor_SMD:C_0402_1005Metric
- R18, R92: footprint Resistor_SMD:R_0805_2012Metric -> Resistor_SMD:R_0402_1005Metric
- R2, R3, R4: footprint (none) -> Resistor_SMD:R_0402_1005Metric
- R35, R93: footprint GNSS_Library:LED_SML-P11D_ROM -> LED_SMD:LED_0402_1005Metric
- U9: footprint SOT-5X3_DRL_TEX -> GNSS:SOT-5X3_DRL_TEX-M
Connections:
- net +3V3_GNSS: now also C83.2
- net GND: now also C83.1, C84.1
- net VIN_GNSS: now also C84.2
Other:
- moved on the sheet: TP12

Commit message: Almost Placed file
Parts:
- renumbered R35 to D15, R93 to D16
Connections:
- net 5V: no longer R46.1, R47.2, U7.5 (EN/FCCM)
- new net EN: R46.1, R47.2, U7.5 (EN/FCCM)
Changed lines of the file:
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@@
 		)
 	)
-	(label "EN"
-		(at 185.42 96.52 0)
-		(fields_autoplaced yes)
-		(effects
-			(font
-				(size 1.27 1.27)
-			)
-			(justify left bottom)
-		)
-	)
 	(label "SW"
 		(at 134.62 104.14 0)
@@
 		(on_board yes)
 		(dnp no)
-		(property "Reference" "R93"
+		(property "Reference" "D16"
 			(at 268.732 107.95 0)
 			(effects
@@
 			(project "GNSS"
 				(path "/a70dad34-b24c-4b58-b91c-f14576b5da7d/95adfb1d-f4b2-4924-8c0a-df43d58bdb39"
-					(reference "R93")
+					(reference "D16")
 					(unit 1)
 				)
@@
 		(on_board yes)
 		(dnp no)
-		(property "Reference" "R35"
+		(property "Reference" "D15"
 			(at 268.478 83.566 0)
 			(effects
@@
 			(project "GNSS"
 				(path "/a70dad34-b24c-4b58-b91c-f14576b5da7d/95adfb1d-f4b2-4924-8c0a-df43d58bdb39"
-					(reference "R35")
+					(reference "D15")
 					(unit 1)
 				)

Commit message: new commit
Connections:
- net +3V3_BMI renamed +3V3_ICM
- net VIN_BMI renamed VIN_ICM
Other:
- note added: "3V3_ICM"
- note removed: "3V3_BMI"
Changed lines of the file:
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@@
 		)
 	)
-	(text "3V3_BMI\n"
+	(text "3V3_ICM"
 		(exclude_from_sim no)
 		(at 202.438 16.764 0)
@@
 			)
 		)
-		(property "Value" "VIN_BMI"
+		(property "Value" "VIN_ICM"
 			(at 241.3 33.02 0)
 			(effects
@@
 			)
 		)
-		(property "Value" "VIN_BMI"
+		(property "Value" "VIN_ICM"
 			(at 255.778 50.292 90)
 			(effects
@@
 			)
 		)
-		(property "Value" "VIN_BMI"
+		(property "Value" "VIN_ICM"
 			(at 209.55 40.64 0)
 			(effects
@@
 			)
 		)
-		(property "Value" "+3V3_BMI"
+		(property "Value" "+3V3_ICM"
 			(at 265.43 40.64 0)
 			(effects
