File: Power_sch.kicad_sch (KiCad schematic)
At the start: 49 parts, among them J1 USB4105-GF-A, J2 USB4105-GF-A, U2 TPD2EUSB30ADRTR, U6 ADP150WACBZ-3.3-R7, U7 IR3883MTRPBF, U9 LM66200DRLR

Commit message: usb
Parts:
- removed J1, J2: USB4105-GF-A, GNSS:USB4105_GCT, symbol 2026-08-09_12-47-05:USB4105-GF-A
- added J1, J8: USB_C_Receptacle_USB2.0_16P, Connector_USB:USB_C_Receptacle_HCTL_HC-TYPE-C-16P-01A, symbol Connector:USB_C_Receptacle_USB2.0_16P
- C15, C16, C19, C20: value 22uF -> 22u
- C17: value 220pF -> 220p
- C18, C21, C83, C84: value 0.1uF -> 0.1u
- C22, C23, C26: value 10uF -> 10u
- C24: value 0.47 -> 0.47u
- C25: value 4.7uF -> 4u7
- L1: value 2.2uH -> 2.2u
- R1, R2, R3, R4: value 5.1K -> 5K1
- R11: value 16.5K -> 16K5
- R12: value 2.94K -> 2K94
- R13: value 49.9K -> 49K9
- R14: value 33.2K -> 33K2
- R46: value 32.4K -> 32K4
Connections:
- net DN: now also J8.A7 (D-), J8.B7 (D-)
- net DP: now also J8.A6 (D+), J8.B6 (D+)
- net GND: now also J1.A1 (GND), J1.A12 (GND), J1.B1 (GND), J1.B12 (GND), J1.S1 (SHIELD), J8.A1 (GND), J8.A12 (GND), J8.B1 (GND), J8.B12 (GND), J8.S1 (SHIELD)
- net at D4.1 (K), F2.1: now also J1.A4 (VBUS), J1.A9 (VBUS), J1.B4 (VBUS), J1.B9 (VBUS)
- net at R1.1: now also J8.B5 (CC2)
- net at R2.2: now also J8.A5 (CC1)
- net at R4.1: now also J1.B5 (CC2)
- net at D3.1 (K), F1.1: now also J8.A4 (VBUS), J8.A9 (VBUS), J8.B4 (VBUS), J8.B9 (VBUS)
- net at R3.1: now also J1.A5 (CC1)
Other:
- moved on the sheet: C15, C16, C17, C18, C19, C20, C21, FL8, L1, R11, R12, R13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

Commit message: can
Parts:
- removed D15, D16: SML-P12U2TT86R, LED_SMD:LED_0402_1005Metric, symbol 2026-08-14_04-34-19:SML-P12U2TT86R
- removed R92: 560R, Resistor_SMD:R_0402_1005Metric, symbol Device:R_Small_US
- added D5, D6: SML-P12U2TT86R, LED_SMD:LED_0402_1005Metric, symbol 2026-08-14_04-34-19:SML-P12U2TT86R
- added Q3, Q4: BC849, Package_TO_SOT_SMD:SOT-23, symbol Transistor_BJT:BC849
- added R58, R59: 10K, Resistor_SMD:R_0402_1005Metric, symbol Device:R_Small_US
- added R60: 560R, Resistor_SMD:R_0402_1005Metric, symbol Device:R_Small_US
Connections:
- net EX_VBUS: now also R59.2
- net GND: now also Q3.2 (E), Q4.2 (E)
- net PG_VBUS: now also R58.2; no longer R18.1
- net VIN: now also R18.1, R60.1
- net at R18.2: now also D5.2
- new net: Q3.1 (B), R58.1
- new net: D5.1, Q3.3 (C)
- new net: Q4.1 (B), R59.1
- new net: D6.1, Q4.3 (C)
- new net: D6.2, R60.2
Other:
- note added: "TYPE_C_1"
- note added: "TYPE_C_2"
- note removed: "POWER"
- note removed: "PROGRAMMING"
- moved on the sheet: C15, C16, C17, C18, C19, C20, C21, FL8, L1, R11, R12, R13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

Commit message: new
Parts:
- removed C22, C23: 10u, Capacitor_SMD:C_0805_2012Metric, symbol Device:C_Small
- removed F2: MF-MSMF200-2, GNSS:FUSC4632X85N, symbol MF-MSMF200-2:MF-MSMF200-2
- removed TP4: TestPoint, TestPoint:TestPoint_Pad_D2.0mm, symbol Connector:TestPoint
- removed U6: ADP150WACBZ-3.3-R7, GNSS:CB-4-3_ADI, symbol 2026-08-11_06-36-10:ADP150WACBZ-3.3-R7
- removed U9: LM66200DRLR, GNSS:SOT-5X3_DRL_TEX-M, symbol 2026-08-30_06-28-01:LM66200DRLR
- added C27: 470p, C0402C104K4RAC:CAPC1005X55N, symbol C0402C104K4RAC:C0402C104K4RAC
- added C28: 2u2, C0402C104K4RAC:CAPC1005X55N, symbol C0402C104K4RAC:C0402C104K4RAC
- added F3: MF-MSMF200-2, MF-MSMF200-2:FUSER_MF-MSMF200-2, symbol MF-MSMF200-2:MF-MSMF200-2
- added IC4: LM66200DRLR, LM66200DRLR:SOT8, symbol LM66200DRLR:LM66200DRLR
- added TP3: TestPoint, TestPoint:TestPoint_Pad_D2.0mm, symbol Connector:TestPoint
- added U1: MIC5205-3.3YM5, Package_TO_SOT_SMD:SOT-23-5, symbol Regulator_Linear:MIC5205-3.3YM5
- F1: footprint GNSS:FUSC4632X85N -> MF-MSMF200-2:FUSER_MF-MSMF200-2; ARROW_ELECTRONICS-PURCHASE-URL (none) -> https://snapeda.com/shop?store=Arrow+Electronics&id=143366; AVAILABILITY (none) -> Good; DESCRIPTION (none) -> Polymeric PTC Resettable Fuse 8V 2A Ih Surface Mount 1812 (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; DIGIKEY-PURCHASE-URL (none) -> https://snapeda.com/shop?store=DigiKey&id=143366; Height 0.85 -> (none); MF (none) -> Bourns; MOUSER-PURCHASE-URL (none) -> https://snapeda.com/shop?store=Mouser&id=143366; MP (none) -> MF-MSMF200-2; Manufacturer_Name Bourns -> (none); Manufacturer_Part_Number MF-MSMF200-2 -> (none); PACKAGE (none) -> 1812 Bourns; PRICE (none) -> None
Connections:
- net +3V3_ICM: now also C28.2, TP3.1, U1.5 (OUT)
- net EX_VBUS: now also F1.2, IC4.6 (VIN2)
- net GND: now also C27.1, C28.1, IC4.1 (GND@1), IC4.4 (ON), IC4.5 (GND@2), U1.2 (GND)
- net PG_VBUS: now also F3.2, IC4.3 (VIN1); no longer F1.2
- net VIN: now also IC4.2 (VOUT@1), IC4.7 (VOUT@2)
- net VIN_ICM: now also U1.1 (IN), U1.3 (EN)
- net at D3.1 (K), J8.A4 (VBUS), J8.A9 (VBUS)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: now also F3.1; no longer F1.1
- net at D4.1 (K), J1.A4 (VBUS), J1.A9 (VBUS)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: now also F1.1
- net at R31.1, TP1.1: now also IC4.8 (ST)
- new net: C27.2, U1.4 (BP)
Other:
- moved on the sheet: FL7

Commit message: block
Parts:
- R18, R60: value 560R -> 10K
Other:
- moved on the sheet: C15, C16, C17, C18, C19, C20, C21, C24, C25, C26, C27, C28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

Commit message: full
Parts:
- removed D5, D6: SML-P12U2TT86R, LED_SMD:LED_0402_1005Metric, symbol 2026-08-14_04-34-19:SML-P12U2TT86R
- removed Q3, Q4: BC849, Package_TO_SOT_SMD:SOT-23, symbol Transistor_BJT:BC849
- removed R18, R58, R59, R60: 10K, Resistor_SMD:R_0402_1005Metric, symbol Device:R_Small_US
- removed U2: TPD2EUSB30ADRTR, GNSS:SOTFL35P100X50-3N, symbol TPD2EUSB30ADRTR:TPD2EUSB30ADRTR
- added U2: TPD2EUSB30A, Package_TO_SOT_SMD:Texas_DRT-3, symbol Power_Protection:TPD2EUSB30A
Connections:
- net DN: now also U2.2 (D-)
- net DP: now also U2.1 (D+)
- net GND: now also U2.3 (GND)

Commit message: 16.09.2026
Parts:
- added C79, C82: 0.1u, Capacitor_SMD:C_0402_1005Metric, symbol C0402C104K4RAC:C0402C104K4RAC
- added C81: 10u, Capacitor_SMD:C_0805_2012Metric, symbol Device:C_Small
- C18, C21, C27, C83, C84: footprint C0402C104K4RAC:CAPC1005X55N -> Capacitor_SMD:C_0402_1005Metric
- C28: footprint C0402C104K4RAC:CAPC1005X55N -> Capacitor_SMD:C_0805_2012Metric
- FL6, FL7, FL8: footprint BLM21PG221SN1D:BEADC2012X105N -> GNSS:BEADC2012X105N
Connections:
- net +3V3_ICM: now also C82.2
- net GND: now also C79.1, C81.1, C82.1
- net VIN_ICM: now also C79.2, C81.2
Other:
- moved on the sheet: TP3

Commit message: 18.09.2026
Connections:
- net +3.3V renamed +3V3
Other:
- note added: "3V3, 150mA"
- note added: "3V3, 3A"
- note added: "3V3, 500mA"
- note removed: "3.3V, 150mA"
- note removed: "3.3V, 3A"
- note removed: "3.3V, 500mA"
- moved on the sheet: C15, C16, C17, C18, C19, C20, C21, FL8, L1, R11, R12, R13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

Commit message: 22.09.26
Parts:
- removed C15, C16, C19, C20: 22u, Capacitor_SMD:C_0805_2012Metric, symbol Device:C_Small
- removed C17: 220p, C0402C104K4RAC:CAPC1005X55N, symbol C0402C104K4RAC:C0402C104K4RAC
- removed C18, C21, C79, C82, C83, C84: 0.1u, Capacitor_SMD:C_0402_1005Metric, symbol C0402C104K4RAC:C0402C104K4RAC
- removed C24: 0.47u, Capacitor_SMD:C_0402_1005Metric, symbol C0402C104K4RAC:C0402C104K4RAC
- removed C25: 4u7, Capacitor_SMD:C_0805_2012Metric, symbol Device:C_Small
- removed C26, C81: 10u, Capacitor_SMD:C_0805_2012Metric, symbol Device:C_Small
- removed C27: 470p, Capacitor_SMD:C_0402_1005Metric, symbol C0402C104K4RAC:C0402C104K4RAC
- removed C28: 2u2, Capacitor_SMD:C_0805_2012Metric, symbol C0402C104K4RAC:C0402C104K4RAC
- removed FL6, FL7, FL8: BLM21PG221SN1D, GNSS:BEADC2012X105N, symbol BLM21PG221SN1D:BLM21PG221SN1D
- removed L1: 2.2u, ASPIAIG-F5030-2R2M-T:IND_ASPIAIG-F5030-2R2M-T, symbol ASPIAIG-F5030-2R2M-T:ASPIAIG-F5030-2R2M-T
- removed R11: 16K5, Resistor_SMD:R_0402_1005Metric, symbol Device:R_Small_US
- removed R12: 2K94, Resistor_SMD:R_0402_1005Metric, symbol Device:R_Small_US
- removed R13: 49K9, Resistor_SMD:R_0402_1005Metric, symbol Device:R_Small_US
- removed R14: 33K2, Resistor_SMD:R_0402_1005Metric, symbol Device:R_Small_US
- removed R46: 32K4, Resistor_SMD:R_0402_1005Metric, symbol Device:R_Small_US
- removed R47: 47K, Resistor_SMD:R_0402_1005Metric, symbol Device:R_Small_US
- removed TP12, TP3, TP5: TestPoint, TestPoint:TestPoint_Pad_D2.0mm, symbol Connector:TestPoint
- removed U1: MIC5205-3.3YM5, Package_TO_SOT_SMD:SOT-23-5, symbol Regulator_Linear:MIC5205-3.3YM5
- removed U7: IR3883MTRPBF, GNSS:VREG_IR3883MTRPBF, symbol IR3883MTRPBF:IR3883MTRPBF
- removed VR1: LT3045EDD_PBF, GNSS:SON50P300X300X80-11N, symbol LT3045EDD_PBF:LT3045EDD_PBF
- J1, J8: footprint Connector_USB:USB_C_Receptacle_HCTL_HC-TYPE-C-16P-01A -> GNSS:USB4105_GCT
Connections:
- no-connect marks 9 -> 8
Other:
- note added: "Ferrrite Beak Drop(hi0805r800r-10) --> 5mV @500mA"
- note removed: "3V3, 150mA"
- note removed: "3V3, 3A"
- note removed: "3V3, 500mA"
- note removed: "3V3_GNSS"
- note removed: "3V3_ICM"
- note removed: "Buck_Converter"
- moved on the sheet: D3, D4, F1, F3, IC4, J1, J8, R1, R2, R3, R31, R4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
