File: Controller.kicad_sch (KiCad schematic)
At the start: 40 parts, among them IC3 STM32H563VGT6, J5 Conn_01x05_Pin, J6 Conn, U8 ECS-TXO-2520-33-240-AN-TR

Commit message: new
Changed lines of the file:
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@@
 	(wire
 		(pts
-			(xy 232.41 44.45) (xy 231.14 44.45)
-		)
-		(stroke
-			(width 0)
-			(type default)
-		)
-	)
-	(wire
-		(pts
 			(xy 246.38 69.85) (xy 246.38 64.77)
 		)
@@
 	(wire
 		(pts
-			(xy 231.14 44.45) (xy 231.14 46.99)
-		)
-		(stroke
-			(width 0)
-			(type default)
-		)
-	)
-	(wire
-		(pts
 			(xy 81.28 64.77) (xy 81.28 60.96)
 		)
@@
 	(wire
 		(pts
-			(xy 238.76 67.31) (xy 252.73 67.31)
+			(xy 238.76 67.31) (xy 256.54 67.31)
 		)
 		(stroke
@@
 	(wire
 		(pts
-			(xy 232.41 43.18) (xy 232.41 44.45)
-		)
-		(stroke
-			(width 0)
-			(type default)
-		)
-	)
-	(wire
-		(pts
 			(xy 143.51 187.96) (xy 149.86 187.96)
 		)
@@
 	(wire
 		(pts
-			(xy 160.02 97.79) (xy 162.56 97.79)
-		)
-		(stroke
-			(width 0)
-			(type default)
-		)
-	)
-	(wire
-		(pts
 			(xy 205.74 35.56) (xy 205.74 46.99)
 		)
@@
 		)
 	)
-	(label "RST_BUT"
-		(at 260.35 43.18 0)
-		(fields_autoplaced yes)
-		(effects
-			(font
-				(size 1.27 1.27)
-			)
-			(justify left bottom)
-		)
-	)
 	(label "GN_LED"
 		(at 41.91 29.21 180)
@@
 		)
 	)
-	(label "RST_BUT"
-		(at 160.02 97.79 180)
-		(fields_autoplaced yes)
-		(effects
-			(font
-				(size 1.27 1.27)
-			)
-			(justify right bottom)
-		)
-	)
 	(label "USER_LED"
 		(at 85.09 29.21 180)
@@
 		)
 	)
-	(label "RST_BUT"
-		(at 81.28 64.77 180)
-		(fields_autoplaced yes)
-		(effects
-			(font
-				(size 1.27 1.27)
-			)
-			(justify right bottom)
-		)
-	)
-	(label "JTCK{slash}SWCLK"
-		(at 232.41 43.18 90)
-		(fields_autoplaced yes)
-		(effects
-			(font
-				(size 1.27 1.27)
-			)
-			(justify left bottom)
-		)
-	)
-	(label "JTMS{slash}SWDIO"
-		(at 260.35 48.26 0)
-		(fields_autoplaced yes)
-		(effects
-			(font
-				(size 1.27 1.27)
-			)
-			(justify left bottom)
-		)
-	)
-	(label "JTMS{slash}SWDIO"
-		(at 238.76 72.39 0)
-		(fields_autoplaced yes)
-		(effects
-			(font
-				(size 1.27 1.27)
-			)
-			(justify left bottom)
-		)
-	)
 	(label "GN_LED"
 		(at 210.82 35.56 90)
@@
 		)
 	)
-	(label "JTCK{slash}SWCLK"
-		(at 260.35 45.72 0)
-		(fields_autoplaced yes)
-		(effects
-			(font
-				(size 1.27 1.27)
-			)
-			(justify left bottom)
-		)
-	)
 	(label "USER_LED"
 		(at 205.74 35.56 90)
@@
 		)
 	)
+	(global_label "JTMS{slash}SWDIO"
+		(shape input)
+		(at 238.76 72.39 0)
+		(fields_autoplaced yes)
+		(effects
+			(font
+				(size 1.27 1.27)
+			)
+			(justify left)
+		)
+		(property "Intersheetrefs" "${INTERSHEET_REFS}"
+			(at 253.538 72.39 0)
+			(effects
+				(font
+					(size 1.27 1.27)
+				)
+				(justify left)
+				(hide yes)
+			)
+		)
+	)
 	(global_label "AR_RX"
 		(shape input)
@@
 		)
 	)
+	(global_label "JTMS{slash}SWDIO"
+		(shape input)
+		(at 260.35 48.26 0)
+		(fields_autoplaced yes)
+		(effects
+			(font
+				(size 1.27 1.27)
+			)
+			(justify left)
+		)
+		(property "Intersheetrefs" "${INTERSHEET_REFS}"
+			(at 275.128 48.26 0)
+			(effects
+				(font
+					(size 1.27 1.27)
+				)
+				(justify left)
+				(hide yes)
+			)
+		)
+	)
+	(global_label "RST_BUT"
+		(shape input)
+		(at 162.56 97.79 180)
+		(fields_autoplaced yes)
+		(effects
+			(font
+				(size 1.27 1.27)
+			)
+			(justify right)
+		)
+		(property "Intersheetrefs" "${INTERSHEET_REFS}"
+			(at 151.592 97.79 0)
+			(effects
+				(font
+					(size 1.27 1.27)
+				)
+				(justify right)
+				(hide yes)
+			)
+		)
+	)
 	(global_label "ETH_MDC"
 		(shape input)
@@
 		)
 	)
+	(global_label "JTCK{slash}SWCLK"
+		(shape input)
+		(at 231.14 46.99 90)
+		(fields_autoplaced yes)
+		(effects
+			(font
+				(size 1.27 1.27)
+			)
+			(justify left)
+		)
+		(property "Intersheetrefs" "${INTERSHEET_REFS}"
+			(at 231.14 31.9701 90)
+			(effects
+				(font
+					(size 1.27 1.27)
+				)
+				(justify left)
+				(hide yes)
+			)
+		)
+	)
 	(global_label "RESET_GNSS"
 		(shape input)
@@
 		)
 	)
+	(global_label "RST_BUT"
+		(shape input)
+		(at 81.28 64.77 180)
+		(fields_autoplaced yes)
+		(effects
+			(font
+				(size 1.27 1.27)
+			)
+			(justify right)
+		)
+		(property "Intersheetrefs" "${INTERSHEET_REFS}"
+			(at 70.312 64.77 0)
+			(effects
+				(font
+					(size 1.27 1.27)
+				)
+				(justify right)
+				(hide yes)
+			)
+		)
+	)
 	(global_label "SDI"
 		(shape input)
@@
 		)
 	)
+	(global_label "RST_BUT"
+		(shape input)
+		(at 260.35 43.18 0)
+		(fields_autoplaced yes)
+		(effects
+			(font
+				(size 1.27 1.27)
+			)
+			(justify left)
+		)
+		(property "Intersheetrefs" "${INTERSHEET_REFS}"
+			(at 271.318 43.18 0)
+			(effects
+				(font
+					(size 1.27 1.27)
+				)
+				(justify left)
+				(hide yes)
+			)
+		)
+	)
+	(global_label "JTCK{slash}SWCLK"
+		(shape input)
+		(at 260.35 45.72 0)
+		(fields_autoplaced yes)
+		(effects
+			(font
+				(size 1.27 1.27)
+			)
+			(justify left)
+		)
+		(property "Intersheetrefs" "${INTERSHEET_REFS}"
+			(at 275.3699 45.72 0)
+			(effects
+				(font
+					(size 1.27 1.27)
+				)
+				(justify left)
+				(hide yes)
+			)
+		)
+	)
 	(global_label "STM_D_N"
 		(shape input)
@@
 	(symbol
 		(lib_id "power:GND")
-		(at 252.73 67.31 0)
+		(at 256.54 67.31 0)
 		(unit 1)
 		(exclude_from_sim no)
@@
 		(fields_autoplaced yes)
 		(property "Reference" "#PWR073"
-			(at 252.73 73.66 0)
+			(at 256.54 73.66 0)
 			(effects
 				(font
@@
 		)
 		(property "Value" "GND"
-			(at 252.73 72.39 0)
+			(at 256.54 72.39 0)
 			(effects
 				(font
@@
 		)
 		(property "Footprint" ""
-			(at 252.73 67.31 0)
+			(at 256.54 67.31 0)
 			(effects
 				(font
@@
 		)
 		(property "Datasheet" ""
-			(at 252.73 67.31 0)
+			(at 256.54 67.31 0)
 			(effects
 				(font
@@
 		)
 		(property "Description" "Power symbol creates a global label with name \"GND\" , ground"
-			(at 252.73 67.31 0)
+			(at 256.54 67.31 0)
 			(effects
 				(font

Commit message: new
Parts:
- removed R18: 0R, Resistor_SMD:R_0805_2012Metric, symbol Device:R_Small_US
- added C82: 100nF, C0402C104K4RAC:CAPC1005X55N, symbol C0402C104K4RAC:C0402C104K4RAC
- added FL13: BLM21PG221SN1D, BLM21PG221SN1D:BEADC2012X105N, symbol BLM21PG221SN1D:BLM21PG221SN1D
- added R22: 22E, Resistor_SMD:R_0805_2012Metric, symbol Device:R_Small_US
- C66: now not fitted
- IC3: footprint Module:QFP50P1600X1600X160-100N -> GNSS:QFP50P1600X1600X160-100N
- S1: footprint gnss1_Library:SOIC450P1000X730-4N -> GNSS:SOIC450P1000X730-4N
- U8: footprint GNSS_Library:ECS-TXO-2520-33-240-AN-TR_ECS -> GNSS:ECS-TXO-2520-33-240-AN-TR_ECS
Connections:
- net AGND is gone; now on net GND: IC3.19 (VSSA)
- net +3.3V: now also FL13.2; no longer C77.2, C78.1, R27.2, R30.2, U8.1, U8.4
- net ETH_RST_N: now also IC3.40 (PE9)
- net GND: now also C82.1
- net OSC: now also R22.1; no longer C66.2, U8.3
- net RST_BUT: now also C82.2
- net STM_3.3V: now also C77.2, C78.1, R27.2, R30.2, U8.1, U8.4, FL13.1
- net ANT_FAULT: now reaches IC3.39 (PE8)
- net USB_RST: now reaches IC3.41 (PE10)
- net ARDUINO_RST_BUT: now reaches IC3.42 (PE11)
- net 50MHZOUT renamed ETH_REFCLK
- new net: C66.2, R22.2, U8.3
- no-connect marks 17 -> 13
Other:
- moved on the sheet: C32, C33, C34, C35, C36, C37, C38, C39, C40, C41, C42, C43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

Commit message: new
Parts:
- J6, R22: now not fitted
Connections:
- net AR_D4: now also IC3.62 (PD15); no longer IC3.57 (PD10)
- net AR_D5: now also IC3.61 (PD14); no longer IC3.58 (PD11)
- net AR_D6: now also IC3.57 (PD10); no longer IC3.59 (PD12)
- net AR_D7: now also IC3.63 (PC6); no longer IC3.60 (PD13)
- net AR_D8: now also IC3.58 (PD11); no longer IC3.61 (PD14)
- net AR_D9: now also IC3.64 (PC7); no longer IC3.62 (PD15)
- net BOOT0: now also IC3.94 (BOOT0), R42.1; no longer R42.2
- net ESP_BOOT: now also IC3.46 (PE15); no longer IC3.47 (PB10)
- net ETH_RST_N: no longer IC3.40 (PE9)
- net SD_DETECT: now also IC3.67 (PA8); no longer IC3.64 (PC7)
- net STM_3.3V: now also R42.2
- net USB_SCL: now also IC3.59 (PD12)
- net USB_SDA: now also IC3.60 (PD13)
- net GN_SDI renamed GN_MISO
- net GN_SDO renamed GN_MOSI
- net SCK renamed IMU_SCK
- net SDI renamed IMU_MISO
- net SDO renamed IMU_MOSI
- no-connect marks 13 -> 12

Commit message: schematics
Parts:
- C32, C33, C34, C35, C36, C37, C38, C39, C40, C41, C42: footprint C0402C104K4RAC:CAPC1005X55N -> Capacitor_SMD:C_0402_1005Metric
- C82: value 100nF -> 0.1uF; footprint C0402C104K4RAC:CAPC1005X55N -> Capacitor_SMD:C_0402_1005Metric

Commit message: placed
Parts:
- C52: value 1uF -> 100n; footprint Capacitor_SMD:C_0805_2012Metric -> Capacitor_SMD:C_0402_1005Metric
- R17, R25: footprint GNSS_Library:LED_SML-P11D_ROM -> LED_SMD:LED_0402_1005Metric
- R19, R20, R22, R27, R28, R29, R30, R42: footprint Resistor_SMD:R_0805_2012Metric -> Resistor_SMD:R_0402_1005Metric
Changed lines of the file:
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@@
 			)
 		)
-		(property "Footprint" "Resistor_SMD:R_0805_2012Metric"
+		(property "Footprint" "Resistor_SMD:R_0402_1005Metric"
 			(at 35.56 59.69 0)
 			(effects
@@
 			)
 		)
-		(property "Footprint" "Resistor_SMD:R_0805_2012Metric"
+		(property "Footprint" "Resistor_SMD:R_0402_1005Metric"
 			(at 82.55 58.42 0)
 			(effects
@@
 			)
 		)
-		(property "Footprint" "Resistor_SMD:R_0805_2012Metric"
+		(property "Footprint" "Resistor_SMD:R_0402_1005Metric"
 			(at 49.53 29.21 0)
 			(effects
@@
 			)
 		)
-		(property "Footprint" "Resistor_SMD:R_0805_2012Metric"
+		(property "Footprint" "Resistor_SMD:R_0402_1005Metric"
 			(at 85.09 114.3 0)
 			(effects
@@
 			)
 		)
-		(property "Footprint" "Resistor_SMD:R_0805_2012Metric"
+		(property "Footprint" "Resistor_SMD:R_0402_1005Metric"
 			(at 181.61 26.67 0)
 			(effects
@@
 			)
 		)
-		(property "Footprint" "Resistor_SMD:R_0805_2012Metric"
+		(property "Footprint" "Resistor_SMD:R_0402_1005Metric"
 			(at 105.41 147.32 0)
 			(effects
@@
 			)
 		)
-		(property "Footprint" "Resistor_SMD:R_0805_2012Metric"
+		(property "Footprint" "Resistor_SMD:R_0402_1005Metric"
 			(at 92.71 29.21 0)
 			(effects
@@
 			)
 		)
-		(property "Value" "1uF"
+		(property "Value" "100n"
 			(at 32.512 154.432 0)
 			(effects
@@
 			)
 		)
-		(property "Footprint" "Capacitor_SMD:C_0805_2012Metric"
+		(property "Footprint" "Capacitor_SMD:C_0402_1005Metric"
 			(at 38.1 152.4 0)
 			(effects
@@
 			)
 		)
-		(property "Footprint" "GNSS_Library:LED_SML-P11D_ROM"
+		(property "Footprint" "LED_SMD:LED_0402_1005Metric"
 			(at 99.06 29.21 0)
 			(effects
@@
 			)
 		)
-		(property "Footprint" "GNSS_Library:LED_SML-P11D_ROM"
+		(property "Footprint" "LED_SMD:LED_0402_1005Metric"
 			(at 57.15 29.21 0)
 			(effects
@@
 			)
 		)
-		(property "Footprint" "Resistor_SMD:R_0805_2012Metric"
+		(property "Footprint" "Resistor_SMD:R_0402_1005Metric"
 			(at 118.11 147.32 0)
 			(effects

Commit message: Almost Placed file
Parts:
- removed S1: TL3301EF100QG, GNSS:SOIC450P1000X730-4N, symbol TL3301EF100QG:TL3301EF100QG
- removed S2: TL3301EF100QG, gnss1_Library:SOIC450P1000X730-4N, symbol TL3301EF100QG:TL3301EF100QG
- added S1, S3: SKRPABE010, GNSS:SW_SKRPABE010, symbol SKRPABE010:SKRPABE010
- renumbered R17 to D10, R25 to D11
Connections:
- net GND: now also S1.3, S1.4, S3.3, S3.4
- net RST_BUT: now also S3.1, S3.2
- net USER_BUT: now also S1.1, S1.2
- no-connect marks 12 -> 8
Other:
- moved on the sheet: R30

Commit message: usb
Parts:
- removed C66: 15pF, C0402C104K4RAC:CAPC1005X55N, symbol C0402C104K4RAC:C0402C104K4RAC
- removed C77: 100nF, C0402C104K4RAC:CAPC1005X55N, symbol C0402C104K4RAC:C0402C104K4RAC
- removed C78: 10uF, Capacitor_SMD:C_0805_2012Metric, symbol Device:C_Small
- removed R22: 22E, Resistor_SMD:R_0402_1005Metric, symbol Device:R_Small_US
- removed U8: ECS-TXO-2520-33-240-AN-TR, GNSS:ECS-TXO-2520-33-240-AN-TR_ECS, symbol 2026-08-15_06-11-37:ECS-TXO-2520-33-240-AN-TR
- added C75, C76: 18p, C0402C104K4RAC:CAPC1005X55N, symbol C0402C104K4RAC:C0402C104K4RAC
- added R57: 1M, Resistor_SMD:R_0402_1005Metric, symbol Device:R_Small_US
- added Y3: MURATA_XRCGB24M000FFS1DR0, GNSS:MURATA_XRCGB24M000FFS1DR0_0, symbol MURATA_XRCGB24M000FFS1DR0:MURATA_XRCGB24M000FFS1DR0
- C32, C33, C34, C35, C36, C37, C38, C39, C40, C41, C42, C44, C47, C49, C50: value 100nF -> 100n
- C43: value 4.7uF -> 4u7
- C45, C46, C48, C51: value 1uF -> 1u
- C82: value 0.1uF -> 0.1u
Connections:
- net GND: now also C75.2, C76.2
- net OSC_OUT: now reaches IC3.13 (PH1-OSC_OUT)
- net OSC_OUT: now also C75.1, R57.2, Y3.1
- net OSC renamed OSC_IN
- net OSC_IN: now also C76.1, R57.1, Y3.3
- no-connect marks 8 -> 9

Commit message: can
Parts:
- removed D10, D11: SML-P12U2TT86R, LED_SMD:LED_0402_1005Metric, symbol 2026-08-14_04-34-19:SML-P12U2TT86R
- added D7, D8: SML-P12U2TT86R, LED_SMD:LED_0402_1005Metric, symbol 2026-08-14_04-34-19:SML-P12U2TT86R
- added Q5, Q6: BC849, Package_TO_SOT_SMD:SOT-23, symbol Transistor_BJT:BC849
- added R45, R70: 10K, Resistor_SMD:R_0402_1005Metric, symbol Device:R_Small_US
Connections:
- net GND: now also Q5.2 (E), Q6.2 (E)
- net GN_LED: now also R45.2; no longer R29.1
- net STM_3.3V: now also R28.1, R29.1
- net USER_LED: now also R70.2; no longer R28.1
- net at R29.2: now also D7.2
- net at R28.2: now also D8.2
- new net: Q5.1 (B), R45.1
- new net: D7.1, Q5.3 (C)
- new net: Q6.1 (B), R70.1
- new net: D8.1, Q6.3 (C)
