File: Controller.kicad_sch (KiCad schematic)
At the start: 31 parts, among them IC3 STM32H563VGT6, J5 Conn_01x05_Pin, J6 Conn

Commit message: we
Parts:
- added Y3: ECS-250-18-33-JGN-TR, ECS-250-18-33-JGN-TR:XTAL_ECS-250-18-33-JGN-TR, symbol ECS-250-18-33-JGN-TR:ECS-250-18-33-JGN-TR
- C51: value 1u -> 2.2u
- C52: value 100n -> 2.2u
- C75, C76: value 18p -> 20p
Connections:
- net GND: now also C76.1, Y3.2 (GND), Y3.4 (GND); no longer C76.2
- net OSC_IN: now also C76.2, Y3.3 (OUT/IN); no longer C76.1
- net OSC_OUT: now also Y3.1 (IN/OUT)
- net ETH_INTR: now reaches IC3.23 (PA0)
- net +3.3V renamed +3V3
- net STM_3.3V renamed STM_3V3
- no-connect marks 9 -> 6
Other:
- moved on the sheet: C75, C76, R57

Commit message: 132
Parts:
- removed IC3: STM32H563VGT6, GNSS:QFP50P1600X1600X160-100N, symbol STM32H563VGT6:STM32H563VGT6
- removed R42: 10K, Resistor_SMD:R_0402_1005Metric, symbol Device:R_Small_US
- added R67: 10K, Resistor_SMD:R_0402_1005Metric, symbol Device:R_Small_US
- added U11: STM32H563VGTx, Package_QFP:LQFP-100_14x14mm_P0.5mm, symbol MCU_ST_STM32H5:STM32H563VGTx
Connections:
- net ANT_FAULT: now also U11.39 (PE8)
- net ARDUINO_RST_BUT: now also U11.42 (PE11)
- net AR_A0: now also U11.29 (PA4)
- net AR_A1: now also U11.31 (PA6)
- net AR_A2: now also U11.35 (PB0)
- net AR_A3: now also U11.36 (PB1)
- net AR_A4: now also U11.15 (PC0)
- net AR_A5: now also U11.17 (PC2)
- net AR_D4: now also U11.62 (PD15)
- net AR_D5: now also U11.61 (PD14)
- net AR_D6: now also U11.57 (PD10)
- net AR_D7: now also U11.63 (PC6)
- net AR_D8: now also U11.58 (PD11)
- net AR_D9: now also U11.64 (PC7)
- net AR_MISO: now also U11.53 (PB14)
- net AR_MOSI: now also U11.18 (PC3)
- net AR_RX: now also U11.56 (PD9)
- net AR_SCK: now also U11.52 (PB13)
- net AR_SCL: now also U11.92 (PB6)
- net AR_SDA: now also U11.93 (PB7)
- net AR_SS: now also U11.26 (PA3)
- net AR_TX: now also U11.55 (PD8)
- net BOOT0: now also R67.2, U11.94 (BOOT0)
- net CAN_RXD: now also U11.81 (PD0)
- net CAN_STB: now also U11.88 (PD7)
- net CAN_TXD: now also U11.82 (PD1)
- net ESP_BOOT: now also U11.46 (PE15)
- net ESP_EN: now also U11.45 (PE14)
- net ESP_INT: now also U11.44 (PE13)
- net ESP_RXD: now also U11.69 (PA10)
- net ESP_TXD: now also U11.68 (PA9)
- net ETH_CRS_DV: now also U11.32 (PA7)
- net ETH_INTR: now also U11.23 (PA0)
- net ETH_MDC: now also U11.16 (PC1)
- net ETH_MDIO: now also U11.25 (PA2)
- net ETH_REFCLK: now also U11.24 (PA1)
- net ETH_RST_N: now also U11.38 (PE7)
- net ETH_RX_D0_N: now also U11.33 (PC4)
- net ETH_RX_D1_N: now also U11.34 (PC5)
- net ETH_TX_D0_P: now also U11.51 (PB12)
- net ETH_TX_D1_P: now also U11.54 (PB15)
- net ETH_TX_EN: now also U11.30 (PA5)
- net GND: now also U11.10 (VSS), U11.19 (VSSA), U11.20 (VREF-), U11.27 (VSS), U11.49 (VSS), U11.74 (VSS), U11.99 (VSS)
- net GN_CS: now also U11.77 (PA15(JTDI))
- net GN_EXINT: now also U11.96 (PB9)
- net GN_LED: now also U11.84 (PD3)
- net GN_MISO: now also U11.90 (PB4(NJTRST))
- net GN_MOSI: now also U11.87 (PD6)
- net GN_SCK: now also U11.89 (PB3(JTDO)
- net GN_TIMEPULSE: now also U11.91 (PB5)
- net IMU_CS: now also U11.3 (PE4)
- net IMU_MISO: now also U11.4 (PE5)
- net IMU_MOSI: now also U11.5 (PE6)
- net IMU_SCK: now also U11.1 (PE2)
- net INT1_ACCEL: now also U11.2 (PE3)
- net INT1_GYRO: now also U11.7 (PC13)
- net JTCK/SWCLK: now also U11.76 (PA14(JTCK)
- net JTMS/SWDIO: now also U11.72 (PA13(JTMS)
- net OSC_IN: now also U11.12 (PH0)
- net OSC_OUT: now also U11.13 (PH1)
- net RESET_GNSS: now also U11.97 (PE0)
- net RST_BUT: now also U11.14 (NRST)
- net SD_CLK: now also U11.80 (PC12)
- net SD_CMD: now also U11.37 (PB2)
- net SD_DAT0: now also U11.65 (PC8)
- net SD_DAT1: now also U11.66 (PC9)
- net SD_DAT2: now also U11.78 (PC10)
- net SD_DAT3: now also U11.79 (PC11)
- net SD_DETECT: now also U11.67 (PA8)
- net STM_3V3: now also R67.1, U11.100 (VDD), U11.11 (VDD), U11.21 (VREF+), U11.22 (VDDA), U11.28 (VDD), U11.50 (VDD), U11.73 (VDDUSB), U11.75 (VDD); no longer C48.1
- net STM_D_N: now also U11.70 (PA11)
- net STM_D_P: now also U11.71 (PA12)
- net TX_READY: now also U11.95 (PB8)
- net USB_RST: now also U11.41 (PE10)
- net USB_SCL: now also U11.59 (PD12)
- net USB_SDA: now also U11.60 (PD13)
- net USER_BUT: now also U11.85 (PD4)
- net USER_LED: now also U11.86 (PD5)
- net VCAP: now also U11.48 (VCAP), U11.98 (VCAP)
- new net VBAT: C48.1, U11.6 (VBAT)
Other:
- note removed: "DE-CAPS"
- moved on the sheet: C32, C33, C34, C35, C36, C37, C38, C39, C40, C41, C42, C43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

Commit message: 22.09.26
Parts:
- removed C39, C41, C47: 100n, Capacitor_SMD:C_0402_1005Metric, symbol C0402C104K4RAC:C0402C104K4RAC
- removed C45, C46: 1u, Capacitor_SMD:C_0805_2012Metric, symbol Device:C_Small
- removed C49: 100n, C0402C104K4RAC:CAPC1005X55N, symbol C0402C104K4RAC:C0402C104K4RAC
- removed C75, C76: 20p, C0402C104K4RAC:CAPC1005X55N, symbol C0402C104K4RAC:C0402C104K4RAC
- removed FL13: BLM21PG221SN1D, BLM21PG221SN1D:BEADC2012X105N, symbol BLM21PG221SN1D:BLM21PG221SN1D
- removed J6: Conn, Connector_PinHeader_1.00mm:PinHeader_1x03_P1.00mm_Vertical, symbol Connector:Conn_01x03_Pin
- removed R57: 1M, Resistor_SMD:R_0402_1005Metric, symbol Device:R_Small_US
- removed Y3: ECS-250-18-33-JGN-TR, ECS-250-18-33-JGN-TR:XTAL_ECS-250-18-33-JGN-TR, symbol ECS-250-18-33-JGN-TR:ECS-250-18-33-JGN-TR
- added C39, C41: 1u, Capacitor_SMD:C_0805_2012Metric, symbol Device:C_Small
- added FB10: FerriteBead, GNSS:BEADC2012X105N, symbol Device:FerriteBead
- added JP3: SolderJumper_2_Open, symbol Jumper:SolderJumper_2_Open
- added R82: 10K, Resistor_SMD:R_0402_1005Metric, symbol Device:R_Small_US
- added Y3: MURATA_XRCGB24M000FFS1DR0, GNSS:MURATA_XRCGB24M000FFS1DR0_0, symbol MURATA_XRCGB24M000FFS1DR0:MURATA_XRCGB24M000FFS1DR0
- C40: footprint Capacitor_SMD:C_0402_1005Metric -> C0402C104K4RAC:CAPC1005X55N
- C42: value 100n -> 18p; footprint Capacitor_SMD:C_0402_1005Metric -> C0402C104K4RAC:CAPC1005X55N
- C44: value 100n -> 18p
- J5: footprint Connector_PinHeader_1.00mm:PinHeader_1x05_P1.00mm_Vertical -> Connector_PinSocket_2.54mm:PinSocket_1x04_P2.54mm_Vertical
- R19, R20: value 0R -> 0E
- renumbered U11 to IC3
Connections:
- net VBAT is gone; now on net STM_3V3: C48.1, IC3.6 (VBAT)
- net +3V3: now also FB10.2
- net BOOT0: now also JP3.1 (A)
- net GND: now also C42.2, C44.2, C39.2, C41.2, R82.2; no longer C42.1, C44.1
- net STM_3V3: now also FB10.1; no longer C40.2, C42.2, C44.2, C50.2, IC3.21 (VREF+), IC3.22 (VDDA), R19.2, R20.1, R20.2
- net OSC_IN: no longer names the net of IC3.12 (PH0)
- net OSC_IN: now also C42.1, Y3.1
- net OSC_OUT: no longer names the net of IC3.13 (PH1)
- net OSC_OUT: now also C44.1, Y3.3
- net VCAP: no longer names the net of C51.1, C52.1, IC3.48 (VCAP), IC3.98 (VCAP)
- new net: JP3.2 (B), R82.1
- new net VDDA: C39.1, C40.2, IC3.22 (VDDA), R19.2, R20.2
- new net VREFP: C41.1, C50.2, IC3.21 (VREF+), R20.1
- no-connect marks 6 -> 8
Other:
- note added: "STM32H563VGTx"
- note removed: "OSCILLATOR"
- note removed: "STM"
- moved on the sheet: C32, C33, C34, C35, C36, C37, C38, C43, C48, C50, C51, C52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

Commit message: 123
Connections:
- net +3V3: now also FB10.1; no longer FB10.2
- net STM_3V3: now also FB10.2; no longer FB10.1

Commit message: new
Parts:
- C40, C42: footprint C0402C104K4RAC:CAPC1005X55N -> Capacitor_SMD:C_0402_1005Metric
- JP3: footprint (none) -> Jumper:SolderJumper-2_P1.3mm_Open_Pad1.0x1.5mm
- Y3: footprint GNSS:MURATA_XRCGB24M000FFS1DR0_0 -> Crystal:Crystal_SMD_2016-4Pin_2.0x1.6mm
