File: _autosave-ESP & CAN.kicad_sch (KiCad schematic)
At the start: 28 parts, among them J2 Conn, U5 TCAN1042VDRBRQ1, U6 TPD2EUSB30ADRTR, U8 ESP32-C3-MINI-1-N4

Commit message: block
Connections:
- net +3.3V_CAN: no longer U5.5 (VIO)
- net CANH: no longer U5.7 (CANH)
- net CANL: no longer U5.6 (CANL)
- net CAN_RXD: no longer U5.4 (RXD)
- net CAN_STB: no longer U5.8 (STB)
- net CAN_TXD: no longer U5.1 (TXD)
- net GND: no longer U5.2 (GND), U5.9 (PAD)
- net VIN_CAN: no longer U5.3 (VCC)
Changed lines of the file:
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@@
 		)
 		(property "Value" "TCAN1042VDRBRQ1"
-			(at 58.42 96.52 0)
+			(at 59.69 96.52 0)
 			(effects
 				(font
@@
 		)
 		(property "Footprint" "GNSS:DRB0008F"
-			(at 58.42 114.3 0)
+			(at 59.69 114.3 0)
 			(effects
 				(font
@@
 		)
 		(property "Datasheet" "https://www.ti.com/lit/gpn/tcan1042v-q1"
-			(at 58.42 114.3 0)
+			(at 59.69 114.3 0)
 			(effects
 				(font
@@
 		)
 		(property "Description" ""
-			(at 58.42 114.3 0)
+			(at 59.69 114.3 0)
 			(effects
 				(font
