File: GNSS.kicad_sch (KiCad schematic)
At the start: 0 parts

Commit message: usb
Other:
- added sheet CAN_TRANS (CAN_TRANS.kicad_sch)
- added sheet SD_CARD (SD_CARD.kicad_sch)
Changed lines of the file:
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@@
 	(sheet
 		(at 137.16 74.93)
-		(size 90.17 19.05)
+		(size 76.2 12.7)
 		(fields_autoplaced yes)
 		(stroke
@@
 		)
 		(property "Sheetfile" "IMU.kicad_sch"
-			(at 137.16 94.5646 0)
+			(at 137.16 88.2146 0)
 			(effects
 				(font
@@
 	)
 	(sheet
-		(at 48.26 101.6)
-		(size 80.01 19.05)
+		(at 48.26 93.98)
+		(size 66.04 12.7)
 		(fields_autoplaced yes)
 		(stroke
@@
 		)
 		(property "Sheetname" "ZED_Z9P"
-			(at 48.26 100.8884 0)
+			(at 48.26 93.2684 0)
 			(effects
 				(font
@@
 		)
 		(property "Sheetfile" "ZED_Z9P.kicad_sch"
-			(at 48.26 121.2346 0)
+			(at 48.26 107.2646 0)
 			(effects
 				(font
@@
 	(sheet
 		(at 48.26 74.93)
-		(size 80.01 19.05)
+		(size 66.04 12.7)
 		(fields_autoplaced yes)
 		(stroke
@@
 		)
 		(property "Sheetfile" "USB_HUB_sch.kicad_sch"
-			(at 48.26 94.5646 0)
+			(at 48.26 88.2146 0)
 			(effects
 				(font
@@
 	(sheet
 		(at 40.64 26.67)
-		(size 81.28 11.43)
+		(size 73.66 11.43)
 		(fields_autoplaced yes)
 		(stroke
@@
 	)
 	(sheet
-		(at 137.16 128.27)
-		(size 90.17 19.05)
+		(at 137.16 132.08)
+		(size 76.2 12.7)
 		(fields_autoplaced yes)
 		(stroke
@@
 		)
 		(property "Sheetname" "Ethernet"
-			(at 137.16 127.5584 0)
+			(at 137.16 131.3684 0)
 			(effects
 				(font
@@
 		)
 		(property "Sheetfile" "Ethernet.kicad_sch"
-			(at 137.16 147.9046 0)
+			(at 137.16 145.3646 0)
 			(effects
 				(font
@@
 	)
 	(sheet
-		(at 137.16 101.6)
-		(size 90.17 19.05)
+		(at 137.16 93.98)
+		(size 76.2 12.7)
 		(fields_autoplaced yes)
 		(stroke
@@
 		)
 		(property "Sheetname" "Arduino"
-			(at 137.16 100.8884 0)
+			(at 137.16 93.2684 0)
 			(effects
 				(font
@@
 		)
 		(property "Sheetfile" "Arduino.kicad_sch"
-			(at 137.16 121.2346 0)
+			(at 137.16 107.2646 0)
 			(effects
 				(font
@@
 	)
 	(sheet
-		(at 48.26 128.27)
-		(size 80.01 19.05)
+		(at 137.16 114.3)
+		(size 76.2 12.7)
+		(fields_autoplaced yes)
+		(stroke
+			(width 0.1524)
+			(type solid)
+		)
+		(fill
+			(color 0 0 0 0.0000)
+		)
+		(property "Sheetname" "SD_CARD"
+			(at 137.16 113.5884 0)
+			(effects
+				(font
+					(size 1.27 1.27)
+				)
+				(justify left bottom)
+			)
+		)
+		(property "Sheetfile" "SD_CARD.kicad_sch"
+			(at 137.16 127.5846 0)
+			(effects
+				(font
+					(size 1.27 1.27)
+				)
+				(justify left top)
+			)
+		)
+		(instances
+			(project "GNSS"
+				(path "/a70dad34-b24c-4b58-b91c-f14576b5da7d"
+					(page "14")
+				)
+			)
+		)
+	)
+	(sheet
+		(at 48.26 132.08)
+		(size 66.04 12.7)
 		(fields_autoplaced yes)
 		(stroke
@@
 		)
 		(property "Sheetname" "ESP"
-			(at 48.26 127.5584 0)
+			(at 48.26 131.3684 0)
 			(effects
 				(font
@@
 		)
 		(property "Sheetfile" "ESP.kicad_sch"
-			(at 48.26 147.9046 0)
+			(at 48.26 145.3646 0)
 			(effects
 				(font
@@
 				)
 			)
+		)
+	)
+	(sheet
+		(at 48.26 113.03)
+		(size 66.04 12.7)
+		(fields_autoplaced yes)
+		(stroke
+			(width 0.1524)
+			(type solid)
+		)
+		(fill
+			(color 0 0 0 0.0000)
+		)
+		(property "Sheetname" "CAN_TRANS"
+			(at 48.26 112.3184 0)
+			(effects
+				(font
+					(size 1.27 1.27)
+				)
+				(justify left bottom)
+			)
+		)
+		(property "Sheetfile" "CAN_TRANS.kicad_sch"
+			(at 48.26 126.3146 0)
+			(effects
+				(font
+					(size 1.27 1.27)
+				)
+				(justify left top)
+			)
+		)
+		(instances
+			(project "GNSS"
+				(path "/a70dad34-b24c-4b58-b91c-f14576b5da7d"
+					(page "13")
+				)
+			)

Commit message: can
Other:
- sheet Arduino renamed ARDUINO
- sheet Block_Diagram renamed BLOCK_DIAGRAM
- sheet Controller renamed CONTROLLER
- sheet ESP renamed ESP & CAN
- sheet Ethernet renamed ETHERNET
- sheet IMU renamed IMU & SDCARD
- sheet Power renamed POWER
- sheet Power_Architecture renamed POWER_ARCHITECTURE
- sheet Table_of_content renamed TABLE_OF_CONTENT
- removed sheet CAN_TRANS
- removed sheet SD_CARD
- sheet ARDUINO: file Arduino.kicad_sch -> ARDUINO.kicad_sch
- sheet BLOCK_DIAGRAM: file Block_Diagram_sch.kicad_sch -> BLOCK_DIAGRAM_sch.kicad_sch
- sheet CONTROLLER: file Controller.kicad_sch -> CONTROLLER.kicad_sch
- sheet ESP & CAN: file ESP.kicad_sch -> ESP & CAN.kicad_sch
- sheet ETHERNET: file Ethernet.kicad_sch -> ETHERNET.kicad_sch
- sheet IMU & SDCARD: file IMU.kicad_sch -> IMU & SDCARD.kicad_sch
- sheet POWER: file Power_sch.kicad_sch -> POWER_sch.kicad_sch
- sheet POWER_ARCHITECTURE: file Power_Architecture.kicad_sch -> POWER_ARCHITECTURE.kicad_sch
- sheet TABLE_OF_CONTENT: file Content_sch.kicad_sch -> CONTENT_sch.kicad_sch
Changed lines of the file:
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@@
 			(color 0 0 0 0.0000)
 		)
-		(property "Sheetname" "Table_of_content"
+		(property "Sheetname" "TABLE_OF_CONTENT"
 			(at 36.83 20.8784 0)
 			(effects
@@
 			)
 		)
-		(property "Sheetfile" "Content_sch.kicad_sch"
+		(property "Sheetfile" "CONTENT_sch.kicad_sch"
 			(at 36.83 159.3346 0)
 			(effects
@@
 	(sheet
 		(at 137.16 74.93)
-		(size 76.2 12.7)
-		(fields_autoplaced yes)
-		(stroke
-			(width 0.1524)
-			(type solid)
-		)
-		(fill
-			(color 0 0 0 0.0000)
-		)
-		(property "Sheetname" "IMU"
+		(size 76.2 15.24)
+		(fields_autoplaced yes)
+		(stroke
+			(width 0.1524)
+			(type solid)
+		)
+		(fill
+			(color 0 0 0 0.0000)
+		)
+		(property "Sheetname" "IMU & SDCARD"
 			(at 137.16 74.2184 0)
 			(effects
@@
 			)
 		)
-		(property "Sheetfile" "IMU.kicad_sch"
-			(at 137.16 88.2146 0)
+		(property "Sheetfile" "IMU & SDCARD.kicad_sch"
+			(at 137.16 90.7546 0)
 			(effects
 				(font
@@
 	)
 	(sheet
-		(at 48.26 93.98)
-		(size 66.04 12.7)
+		(at 48.26 100.33)
+		(size 67.31 16.51)
 		(fields_autoplaced yes)
 		(stroke
@@
 		)
 		(property "Sheetname" "ZED_Z9P"
-			(at 48.26 93.2684 0)
+			(at 48.26 99.6184 0)
 			(effects
 				(font
@@
 		)
 		(property "Sheetfile" "ZED_Z9P.kicad_sch"
-			(at 48.26 107.2646 0)
+			(at 48.26 117.4246 0)
 			(effects
 				(font
@@
 	(sheet
 		(at 48.26 74.93)
-		(size 66.04 12.7)
+		(size 66.04 16.51)
 		(fields_autoplaced yes)
 		(stroke
@@
 		)
 		(property "Sheetfile" "USB_HUB_sch.kicad_sch"
-			(at 48.26 88.2146 0)
+			(at 48.26 92.0246 0)
 			(effects
 				(font
@@
 			(color 0 0 0 0.0000)
 		)
-		(property "Sheetname" "Power_Architecture"
+		(property "Sheetname" "POWER_ARCHITECTURE"
 			(at 43.18 52.6284 0)
 			(effects
@@
 			)
 		)
-		(property "Sheetfile" "Power_Architecture.kicad_sch"
+		(property "Sheetfile" "POWER_ARCHITECTURE.kicad_sch"
 			(at 43.18 65.3546 0)
 			(effects
@@
 			(color 0 0 0 0.0000)
 		)
-		(property "Sheetname" "Controller"
+		(property "Sheetname" "CONTROLLER"
 			(at 41.91 70.4084 0)
 			(effects
@@
 			)
 		)
-		(property "Sheetfile" "Controller.kicad_sch"
+		(property "Sheetfile" "CONTROLLER.kicad_sch"
 			(at 41.91 151.7146 0)
 			(effects
@@
 			(color 0 0 0 0.0000)
 		)
-		(property "Sheetname" "Block_Diagram"
+		(property "Sheetname" "BLOCK_DIAGRAM"
 			(at 40.64 25.9584 0)
 			(effects
@@
 			)
 		)
-		(property "Sheetfile" "Block_Diagram_sch.kicad_sch"
+		(property "Sheetfile" "BLOCK_DIAGRAM_sch.kicad_sch"
 			(at 40.64 38.6846 0)
 			(effects
@@
 			(color 0 0 0 0.0000)
 		)
-		(property "Sheetname" "Power"
+		(property "Sheetname" "POWER"
 			(at 39.37 46.2784 0)
 			(effects
@@
 			)
 		)
-		(property "Sheetfile" "Power_sch.kicad_sch"
+		(property "Sheetfile" "POWER_sch.kicad_sch"
 			(at 39.37 154.2546 0)
 			(effects
@@
 	)
 	(sheet
-		(at 137.16 132.08)
-		(size 76.2 12.7)
-		(fields_autoplaced yes)
-		(stroke
-			(width 0.1524)
-			(type solid)
-		)
-		(fill
-			(color 0 0 0 0.0000)
-		)
-		(property "Sheetname" "Ethernet"
-			(at 137.16 131.3684 0)
-			(effects
-				(font
-					(size 1.27 1.27)
-				)
-				(justify left bottom)
-			)
-		)
-		(property "Sheetfile" "Ethernet.kicad_sch"
-			(at 137.16 145.3646 0)
+		(at 137.16 127)
+		(size 76.2 16.51)
+		(fields_autoplaced yes)
+		(stroke
+			(width 0.1524)
+			(type solid)
+		)
+		(fill
+			(color 0 0 0 0.0000)
+		)
+		(property "Sheetname" "ETHERNET"
+			(at 137.16 126.2884 0)
+			(effects
+				(font
+					(size 1.27 1.27)
+				)
+				(justify left bottom)
+			)
+		)
+		(property "Sheetfile" "ETHERNET.kicad_sch"
+			(at 137.16 144.0946 0)
 			(effects
 				(font
@@
 	)
 	(sheet
-		(at 137.16 93.98)
-		(size 76.2 12.7)
-		(fields_autoplaced yes)
-		(stroke
-			(width 0.1524)
-			(type solid)
-		)
-		(fill
-			(color 0 0 0 0.0000)
-		)
-		(property "Sheetname" "Arduino"
-			(at 137.16 93.2684 0)
-			(effects
-				(font
-					(size 1.27 1.27)
-				)
-				(justify left bottom)
-			)
-		)
-		(property "Sheetfile" "Arduino.kicad_sch"
-			(at 137.16 107.2646 0)
+		(at 137.16 100.33)
+		(size 76.2 16.51)
+		(fields_autoplaced yes)
+		(stroke
+			(width 0.1524)
+			(type solid)
+		)
+		(fill
+			(color 0 0 0 0.0000)
+		)
+		(property "Sheetname" "ARDUINO"
+			(at 137.16 99.6184 0)
+			(effects
+				(font
+					(size 1.27 1.27)
+				)
+				(justify left bottom)
+			)
+		)
+		(property "Sheetfile" "ARDUINO.kicad_sch"
+			(at 137.16 117.4246 0)
 			(effects
 				(font
@@
 	)
 	(sheet
-		(at 137.16 114.3)
-		(size 76.2 12.7)
-		(fields_autoplaced yes)
-		(stroke
-			(width 0.1524)
-			(type solid)
-		)
-		(fill
-			(color 0 0 0 0.0000)
-		)
-		(property "Sheetname" "SD_CARD"
-			(at 137.16 113.5884 0)
-			(effects
-				(font
-					(size 1.27 1.27)
-				)
-				(justify left bottom)
-			)
-		)
-		(property "Sheetfile" "SD_CARD.kicad_sch"
-			(at 137.16 127.5846 0)
-			(effects
-				(font
-					(size 1.27 1.27)
-				)
-				(justify left top)
-			)
-		)
-		(instances
-			(project "GNSS"
-				(path "/a70dad34-b24c-4b58-b91c-f14576b5da7d"
-					(page "14")
-				)
-			)
-		)
-	)
-	(sheet
-		(at 48.26 132.08)
-		(size 66.04 12.7)
-		(fields_autoplaced yes)
-		(stroke
-			(width 0.1524)
-			(type solid)
-		)
-		(fill
-			(color 0 0 0 0.0000)
-		)
-		(property "Sheetname" "ESP"
-			(at 48.26 131.3684 0)
-			(effects
-				(font
-					(size 1.27 1.27)
-				)
-				(justify left bottom)
-			)
-		)
-		(property "Sheetfile" "ESP.kicad_sch"
-			(at 48.26 145.3646 0)
+		(at 48.26 128.27)
+		(size 67.31 15.24)
+		(fields_autoplaced yes)
+		(stroke
+			(width 0.1524)
+			(type solid)
+		)
+		(fill
+			(color 0 0 0 0.0000)
+		)
+		(property "Sheetname" "ESP & CAN"
+			(at 48.26 127.5584 0)
+			(effects
+				(font
+					(size 1.27 1.27)
+				)
+				(justify left bottom)
+			)
+		)
+		(property "Sheetfile" "ESP & CAN.kicad_sch"
+			(at 48.26 144.0946 0)
 			(effects
 				(font
@@
 				)
 			)
-		)
-	)
-	(sheet
-		(at 48.26 113.03)
-		(size 66.04 12.7)
-		(fields_autoplaced yes)
-		(stroke
-			(width 0.1524)
-			(type solid)
-		)
-		(fill
-			(color 0 0 0 0.0000)
-		)
-		(property "Sheetname" "CAN_TRANS"
-			(at 48.26 112.3184 0)
-			(effects
-				(font
-					(size 1.27 1.27)
-				)
-				(justify left bottom)
-			)
-		)
-		(property "Sheetfile" "CAN_TRANS.kicad_sch"
-			(at 48.26 126.3146 0)
-			(effects
-				(font
-					(size 1.27 1.27)
-				)
-				(justify left top)
-			)
-		)
-		(instances
-			(project "GNSS"
-				(path "/a70dad34-b24c-4b58-b91c-f14576b5da7d"
-					(page "13")
-				)
-			)

Commit message: full
Other:
- removed sheet BLOCK_DIAGRAM
- added sheet ANTENNA (ANTENNA.kicad_sch)
- added sheet LEDs & BUTTONs (LEDs & BUTTONs.kicad_sch)
- note added: "ANALOG"
- note added: "ANT_DETECT"
- note added: "ANT_OFF"
- note added: "ANT_SHORT_N"
- note added: "BOOT"
- note added: "CAN_RXD"
- note added: "CAN_STD"
- note added: "CAN_TXD"
- note added: "CS"
- note added: "Connections Overview"
- note added: "DIGITAL"
- note added: "DN"
- note added: "DP"
- note added: "EN"
- note added: "ETH_RST"
- note added: "EXTINT"
- note added: "GNSS_LED"
- note added: "I2C"
- note added: "INT"
- note added: "INT1"
- note added: "INT2"
- note added: "MDC"
- note added: "MDIO"
- note added: "MISO"
- note added: "MOSI"
- note added: "RESET_N"
- note added: "RF_IN"
- note added: "RMII_CRS_DV"
- note added: "RMII_REF_CLK"
- note added: "RMII_RXD0"
- note added: "RMII_RXD1"
- note added: "RMII_TXD0"
- note added: "RMII_TXD1"
- note added: "RMII_TX_EN"
- note added: "RST_BUT"
- note added: "RXD"
- note added: "SCK"
- note added: "SD_CLK"
- note added: "SD_CMD"
- note added: "SD_D0"
- note added: "SD_D1"
- note added: "SD_D2"
- note added: "SD_D3"
- note added: "SD_DETECT"
- note added: "SPI"
- note added: "STM32H563VGT6"
- note added: "TIMEPULSE"
- note added: "TXD"
- note added: "TX_READY"
- note added: "UART"
- note added: "USER_BUT"
- note added: "USER_LED"
- note added: "VCC_RF"
