File: GNSS.kicad_sch (KiCad schematic)
At the start: 0 parts

Commit message: 18.09.2026
Other:
- added sheet BLOCK_DIAGRAM (BLOCK_DIAGRAM.kicad_sch)
- note added: "ANT_FAULT"
- note added: "GND"
- note added: "I2C_1"
- note added: "I2C_4"
- note added: "SDMMC1"
- note added: "SPI_2"
- note added: "SPI_3"
- note added: "SPI_4"
- note added: "USART_1"
- note added: "USART_3"
- note added: "VBUS"
Changed lines of the file:
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@@
 	(polyline
 		(pts
-			(xy 167.64 45.212) (xy 167.64 31.496)
+			(xy 167.64 45.72) (xy 167.64 31.496)
 		)
 		(stroke
@@
 		)
 	)
-	(text "DP"
-		(exclude_from_sim no)
-		(at 116.332 46.482 0)
+	(text "VBUS"
+		(exclude_from_sim no)
+		(at 115.57 46.99 0)
 		(effects
 			(font
@@
 		)
 	)
+	(text "SPI_4"
+		(exclude_from_sim no)
+		(at 204.216 85.852 0)
+		(effects
+			(font
+				(size 1.778 1.778)
+				(bold yes)
+			)
+		)
+	)
 	(text "MISO"
 		(exclude_from_sim no)
@@
 		)
 	)
+	(text "I2C_1"
+		(exclude_from_sim no)
+		(at 162.56 121.666 90)
+		(effects
+			(font
+				(size 1.778 1.778)
+				(bold yes)
+			)
+		)
+	)
 	(text "TXD"
 		(exclude_from_sim no)
@@
 		(exclude_from_sim no)
 		(at 242.189 85.725 0)
+		(effects
+			(font
+				(size 1.778 1.778)
+				(bold yes)
+			)
+		)
+	)
+	(text "ANT_FAULT"
+		(exclude_from_sim no)
+		(at 42.418 108.204 0)
 		(effects
 			(font
@@
 		)
 	)
+	(text "SPI_2"
+		(exclude_from_sim no)
+		(at 159.512 121.666 90)
+		(effects
+			(font
+				(size 1.778 1.778)
+				(bold yes)
+			)
+		)
+	)
 	(text "DP"
 		(exclude_from_sim no)
@@
 		)
 	)
+	(text "RST_BUT"
+		(exclude_from_sim no)
+		(at 173.736 136.652 90)
+		(effects
+			(font
+				(size 1.778 1.778)
+				(bold yes)
+			)
+		)
+	)
 	(text "SD_D3"
 		(exclude_from_sim no)
@@
 		)
 	)
-	(text "DN"
+	(text "GND"
 		(exclude_from_sim no)
 		(at 116.332 49.53 0)
@@
 		)
 	)
+	(text "SDMMC1"
+		(exclude_from_sim no)
+		(at 204.216 89.154 0)
+		(effects
+			(font
+				(size 1.778 1.778)
+				(bold yes)
+			)
+		)
+	)
 	(text "RST_BUT"
 		(exclude_from_sim no)
@@
 		)
 	)
+	(text "USART_3"
+		(exclude_from_sim no)
+		(at 156.21 121.158 90)
+		(effects
+			(font
+				(size 1.778 1.778)
+				(bold yes)
+			)
+		)
+	)
 	(text "CAN_TXD"
 		(exclude_from_sim no)
@@
 		)
 	)
+	(text "SPI_3"
+		(exclude_from_sim no)
+		(at 116.332 80.264 0)
+		(effects
+			(font
+				(size 1.778 1.778)
+				(bold yes)
+			)
+		)
+	)
 	(text "MDIO"
 		(exclude_from_sim no)
@@
 		)
 	)
+	(text "I2C_4"
+		(exclude_from_sim no)
+		(at 159.766 64.77 90)
+		(effects
+			(font
+				(size 1.778 1.778)
+				(bold yes)
+			)
+		)
+	)
+	(text "USART_1"
+		(exclude_from_sim no)
+		(at 112.522 127.762 0)
+		(effects
+			(font
+				(size 1.778 1.778)
+				(bold yes)
+			)
+		)
+	)
 	(text "INT1"
 		(exclude_from_sim no)
@@
 	)
 	(sheet
-		(at 20.828 24.13)
+		(at 19.304 24.638)
 		(size 256.794 139.192)
 		(fields_autoplaced yes)
@@
 		)
 		(property "Sheetname" "TABLE_OF_CONTENT"
-			(at 20.828 23.4184 0)
+			(at 19.304 23.9264 0)
 			(effects
 				(font
@@
 		)
 		(property "Sheetfile" "CONTENT_sch.kicad_sch"
-			(at 20.828 163.9066 0)
+			(at 19.304 164.4146 0)
 			(effects
 				(font
@@
 	)
 	(sheet
+		(at 22.86 44.45)
+		(size 13.97 10.16)
+		(fields_autoplaced yes)
+		(stroke
+			(width 0.1524)
+			(type solid)
+		)
+		(fill
+			(color 0 0 0 0.0000)
+		)
+		(property "Sheetname" "BLOCK_DIAGRAM"
+			(at 22.86 43.7384 0)
+			(effects
+				(font
+					(size 1.27 1.27)
+				)
+				(justify left bottom)
+			)
+		)
+		(property "Sheetfile" "BLOCK_DIAGRAM.kicad_sch"
+			(at 22.86 55.1946 0)
+			(effects
+				(font
+					(size 1.27 1.27)
+				)
+				(justify left top)
+			)
+		)
+		(instances
+			(project "GNSS"
+				(path "/a70dad34-b24c-4b58-b91c-f14576b5da7d"
+					(page "15")
+				)
+			)
+		)
+	)
+	(sheet
 		(at 59.69 73.66)
 		(size 38.1 29.21)
@@
 	)
 	(sheet
-		(at 22.098 28.194)
-		(size 27.94 11.43)
+		(at 23.368 28.194)
+		(size 14.732 9.906)
 		(fields_autoplaced yes)
 		(stroke
@@
 		)
 		(property "Sheetname" "POWER_ARCHITECTURE"
-			(at 22.098 27.4824 0)
+			(at 23.368 27.4824 0)
 			(effects
 				(font
@@
 		)
 		(property "Sheetfile" "POWER_ARCHITECTURE.kicad_sch"
-			(at 22.098 40.2086 0)
+			(at 23.368 38.6846 0)
 			(effects
 				(font
@@
 	(sheet
 		(at 22.86 77.47)
-		(size 26.67 22.86)
+		(size 26.67 32.766)
 		(fields_autoplaced yes)
 		(stroke
@@
 		)
 		(property "Sheetfile" "ANTENNA.kicad_sch"
-			(at 22.86 100.9146 0)
-			(effects
-				(font
+			(at 22.86 110.8206 0)
+			(effects
+				(font

Commit message: 22.09.26
Other:
- sheet ESP & CAN renamed ESP 
- sheet IMU & SDCARD renamed IMU 
- added sheet CAN (CAN.kicad_sch)
- added sheet POWER_2 (POWER_2_sch.kicad_sch)
- added sheet SD_CARD (SD_CARD.kicad_sch)
- sheet ESP : file ESP & CAN.kicad_sch -> ESP .kicad_sch
- sheet IMU : file IMU & SDCARD.kicad_sch -> IMU .kicad_sch
Changed lines of the file:
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@@
+	)
+	(sheet
+		(at 62.23 38.1)
+		(size 20.32 17.78)
+		(fields_autoplaced yes)
+		(stroke
+			(width 0.1524)
+			(type solid)
+		)
+		(fill
+			(color 0 0 0 0.0000)
+		)
+		(property "Sheetname" "POWER_2"
+			(at 62.23 37.3884 0)
+			(effects
+				(font
+					(size 1.27 1.27)
+				)
+				(justify left bottom)
+			)
+		)
+		(property "Sheetfile" "POWER_2_sch.kicad_sch"
+			(at 62.23 56.4646 0)
+			(effects
+				(font
+					(size 1.27 1.27)
+				)
+				(justify left top)
+			)
+		)
+		(instances
+			(project "GNSS"
+				(path "/a70dad34-b24c-4b58-b91c-f14576b5da7d"
+					(page "5")
+				)
+			)
+		)
 	)
 	(sheet
@@
 			(color 0 0 0 0.0000)
 		)
-		(property "Sheetname" "IMU & SDCARD"
+		(property "Sheetname" "IMU "
 			(at 219.71 69.1384 0)
 			(effects
@@
 			)
 		)
-		(property "Sheetfile" "IMU & SDCARD.kicad_sch"
+		(property "Sheetfile" "IMU .kicad_sch"
 			(at 219.71 109.1696 0)
 			(effects
@@
 			(project "GNSS"
 				(path "/a70dad34-b24c-4b58-b91c-f14576b5da7d"
-					(page "12")
-				)
-			)
-		)
-	)
-	(sheet
-		(at 22.86 44.45)
+					(page "11")
+				)
+			)
+		)
+	)
+	(sheet
+		(at 29.21 54.61)
 		(size 13.97 10.16)
 		(fields_autoplaced yes)
@@
 		)
 		(property "Sheetname" "BLOCK_DIAGRAM"
-			(at 22.86 43.7384 0)
+			(at 29.21 53.8984 0)
 			(effects
 				(font
@@
 		)
 		(property "Sheetfile" "BLOCK_DIAGRAM.kicad_sch"
-			(at 22.86 55.1946 0)
-			(effects
-				(font
-					(size 1.27 1.27)
-				)
-				(justify left top)
-			)
-		)
-		(instances
-			(project "GNSS"
-				(path "/a70dad34-b24c-4b58-b91c-f14576b5da7d"
-					(page "15")
+			(at 29.21 65.3546 0)
+			(effects
+				(font
+					(size 1.27 1.27)
+				)
+				(justify left top)
+			)
+		)
+		(instances
+			(project "GNSS"
+				(path "/a70dad34-b24c-4b58-b91c-f14576b5da7d"
+					(page "16")
 				)
 			)
@@
 			(project "GNSS"
 				(path "/a70dad34-b24c-4b58-b91c-f14576b5da7d"
-					(page "6")
+					(page "8")
 				)
 			)
@@
 			(project "GNSS"
 				(path "/a70dad34-b24c-4b58-b91c-f14576b5da7d"
-					(page "5")
+					(page "6")
 				)
 			)
@@
 			(project "GNSS"
 				(path "/a70dad34-b24c-4b58-b91c-f14576b5da7d"
-					(page "14")
+					(page "17")
 				)
 			)
@@
 			(project "GNSS"
 				(path "/a70dad34-b24c-4b58-b91c-f14576b5da7d"
-					(page "8")
+					(page "7")
 				)
 			)
@@
 			(project "GNSS"
 				(path "/a70dad34-b24c-4b58-b91c-f14576b5da7d"
-					(page "13")
+					(page "15")
 				)
 			)
@@
 	)
 	(sheet
+		(at 186.69 135.89)
+		(size 19.05 17.78)
+		(fields_autoplaced yes)
+		(stroke
+			(width 0.1524)
+			(type solid)
+		)
+		(fill
+			(color 0 0 0 0.0000)
+		)
+		(property "Sheetname" "SD_CARD"
+			(at 186.69 135.1784 0)
+			(effects
+				(font
+					(size 1.27 1.27)
+				)
+				(justify left bottom)
+			)
+		)
+		(property "Sheetfile" "SD_CARD.kicad_sch"
+			(at 186.69 154.2546 0)
+			(effects
+				(font
+					(size 1.27 1.27)
+				)
+				(justify left top)
+			)
+		)
+		(instances
+			(project "GNSS"
+				(path "/a70dad34-b24c-4b58-b91c-f14576b5da7d"
+					(page "12")
+				)
+			)
+		)
+	)
+	(sheet
 		(at 219.075 119.38)
 		(size 30.099 35.306)
@@
 			(project "GNSS"
 				(path "/a70dad34-b24c-4b58-b91c-f14576b5da7d"
-					(page "11")
+					(page "10")
 				)
 			)
@@
 			(project "GNSS"
 				(path "/a70dad34-b24c-4b58-b91c-f14576b5da7d"
-					(page "7")
+					(page "9")
 				)
 			)
@@
 			(project "GNSS"
 				(path "/a70dad34-b24c-4b58-b91c-f14576b5da7d"
-					(page "10")
+					(page "14")
 				)
 			)
@@
 			(color 0 0 0 0.0000)
 		)
-		(property "Sheetname" "ESP & CAN"
+		(property "Sheetname" "ESP "
 			(at 58.166 121.3354 0)
 			(effects
@@
 			)
 		)
-		(property "Sheetfile" "ESP & CAN.kicad_sch"
+		(property "Sheetfile" "ESP .kicad_sch"
 			(at 58.166 156.7946 0)
 			(effects
@@
 				)
 			)
+		)
+	)
+	(sheet
+		(at 106.68 137.16)
+		(size 24.13 15.24)
+		(fields_autoplaced yes)
+		(stroke
+			(width 0.1524)
+			(type solid)
+		)
+		(fill
+			(color 0 0 0 0.0000)
+		)
+		(property "Sheetname" "CAN"
+			(at 106.68 136.4484 0)
+			(effects
+				(font
+					(size 1.27 1.27)
+				)
+				(justify left bottom)
+			)
+		)
+		(property "Sheetfile" "CAN.kicad_sch"
+			(at 106.68 152.9846 0)
+			(effects
+				(font
+					(size 1.27 1.27)
+				)
+				(justify left top)
+			)
+		)
+		(instances
+			(project "GNSS"
+				(path "/a70dad34-b24c-4b58-b91c-f14576b5da7d"
+					(page "13")
+				)
+			)
