File: GNSS.kicad_sch (KiCad schematic)
At the start: 0 parts

Commit message: 132
Other:
- added sheet BLOCK_DIAGRAM (BLOCK_DIAGRAM.kicad_sch)
Changed lines of the file:
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@@
+	)
+	(sheet
+		(at 22.86 44.45)
+		(size 13.97 10.16)
+		(fields_autoplaced yes)
+		(stroke
+			(width 0.1524)
+			(type solid)
+		)
+		(fill
+			(color 0 0 0 0.0000)
+		)
+		(property "Sheetname" "BLOCK_DIAGRAM"
+			(at 22.86 43.7384 0)
+			(effects
+				(font
+					(size 1.27 1.27)
+				)
+				(justify left bottom)
+			)
+		)
+		(property "Sheetfile" "BLOCK_DIAGRAM.kicad_sch"
+			(at 22.86 55.1946 0)
+			(effects
+				(font
+					(size 1.27 1.27)
+				)
+				(justify left top)
+			)
+		)
+		(instances
+			(project "GNSS"
+				(path "/a70dad34-b24c-4b58-b91c-f14576b5da7d"
+					(page "14")
+				)
+			)
+		)
 	)
 	(sheet
@@
 	)
 	(sheet
-		(at 22.098 28.194)
-		(size 27.94 11.43)
+		(at 23.368 28.194)
+		(size 14.732 9.906)
 		(fields_autoplaced yes)
 		(stroke
@@
 		)
 		(property "Sheetname" "POWER_ARCHITECTURE"
-			(at 22.098 27.4824 0)
+			(at 23.368 27.4824 0)
 			(effects
 				(font
@@
 		)
 		(property "Sheetfile" "POWER_ARCHITECTURE.kicad_sch"
-			(at 22.098 40.2086 0)
+			(at 23.368 38.6846 0)
 			(effects
 				(font

Commit message: 22.09.26
Other:
- sheet ESP & CAN renamed ESP 
- sheet IMU & SDCARD renamed IMU 
- added sheet CAN (CAN.kicad_sch)
- added sheet POWER_2 (POWER_2_sch.kicad_sch)
- added sheet SD_CARD (SD_CARD.kicad_sch)
- sheet ESP : file ESP & CAN.kicad_sch -> ESP .kicad_sch
- sheet IMU : file IMU & SDCARD.kicad_sch -> IMU .kicad_sch
Changed lines of the file:
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@@
+	)
+	(sheet
+		(at 62.23 38.1)
+		(size 20.32 17.78)
+		(fields_autoplaced yes)
+		(stroke
+			(width 0.1524)
+			(type solid)
+		)
+		(fill
+			(color 0 0 0 0.0000)
+		)
+		(property "Sheetname" "POWER_2"
+			(at 62.23 37.3884 0)
+			(effects
+				(font
+					(size 1.27 1.27)
+				)
+				(justify left bottom)
+			)
+		)
+		(property "Sheetfile" "POWER_2_sch.kicad_sch"
+			(at 62.23 56.4646 0)
+			(effects
+				(font
+					(size 1.27 1.27)
+				)
+				(justify left top)
+			)
+		)
+		(instances
+			(project "GNSS"
+				(path "/a70dad34-b24c-4b58-b91c-f14576b5da7d"
+					(page "5")
+				)
+			)
+		)
 	)
 	(sheet
@@
 			(color 0 0 0 0.0000)
 		)
-		(property "Sheetname" "IMU & SDCARD"
+		(property "Sheetname" "IMU "
 			(at 219.71 69.1384 0)
 			(effects
@@
 			)
 		)
-		(property "Sheetfile" "IMU & SDCARD.kicad_sch"
+		(property "Sheetfile" "IMU .kicad_sch"
 			(at 219.71 109.1696 0)
 			(effects
@@
 			(project "GNSS"
 				(path "/a70dad34-b24c-4b58-b91c-f14576b5da7d"
-					(page "12")
-				)
-			)
-		)
-	)
-	(sheet
-		(at 22.86 44.45)
+					(page "11")
+				)
+			)
+		)
+	)
+	(sheet
+		(at 29.21 54.61)
 		(size 13.97 10.16)
 		(fields_autoplaced yes)
@@
 		)
 		(property "Sheetname" "BLOCK_DIAGRAM"
-			(at 22.86 43.7384 0)
+			(at 29.21 53.8984 0)
 			(effects
 				(font
@@
 		)
 		(property "Sheetfile" "BLOCK_DIAGRAM.kicad_sch"
-			(at 22.86 55.1946 0)
-			(effects
-				(font
-					(size 1.27 1.27)
-				)
-				(justify left top)
-			)
-		)
-		(instances
-			(project "GNSS"
-				(path "/a70dad34-b24c-4b58-b91c-f14576b5da7d"
-					(page "14")
+			(at 29.21 65.3546 0)
+			(effects
+				(font
+					(size 1.27 1.27)
+				)
+				(justify left top)
+			)
+		)
+		(instances
+			(project "GNSS"
+				(path "/a70dad34-b24c-4b58-b91c-f14576b5da7d"
+					(page "16")
 				)
 			)
@@
 			(project "GNSS"
 				(path "/a70dad34-b24c-4b58-b91c-f14576b5da7d"
-					(page "6")
+					(page "8")
 				)
 			)
@@
 			(project "GNSS"
 				(path "/a70dad34-b24c-4b58-b91c-f14576b5da7d"
-					(page "5")
+					(page "6")
 				)
 			)
@@
 			(project "GNSS"
 				(path "/a70dad34-b24c-4b58-b91c-f14576b5da7d"
-					(page "14")
+					(page "17")
 				)
 			)
@@
 			(project "GNSS"
 				(path "/a70dad34-b24c-4b58-b91c-f14576b5da7d"
-					(page "8")
+					(page "7")
 				)
 			)
@@
 			(project "GNSS"
 				(path "/a70dad34-b24c-4b58-b91c-f14576b5da7d"
-					(page "13")
+					(page "15")
 				)
 			)
@@
 	)
 	(sheet
+		(at 186.69 135.89)
+		(size 19.05 17.78)
+		(fields_autoplaced yes)
+		(stroke
+			(width 0.1524)
+			(type solid)
+		)
+		(fill
+			(color 0 0 0 0.0000)
+		)
+		(property "Sheetname" "SD_CARD"
+			(at 186.69 135.1784 0)
+			(effects
+				(font
+					(size 1.27 1.27)
+				)
+				(justify left bottom)
+			)
+		)
+		(property "Sheetfile" "SD_CARD.kicad_sch"
+			(at 186.69 154.2546 0)
+			(effects
+				(font
+					(size 1.27 1.27)
+				)
+				(justify left top)
+			)
+		)
+		(instances
+			(project "GNSS"
+				(path "/a70dad34-b24c-4b58-b91c-f14576b5da7d"
+					(page "12")
+				)
+			)
+		)
+	)
+	(sheet
 		(at 219.075 119.38)
 		(size 30.099 35.306)
@@
 			(project "GNSS"
 				(path "/a70dad34-b24c-4b58-b91c-f14576b5da7d"
-					(page "11")
+					(page "10")
 				)
 			)
@@
 			(project "GNSS"
 				(path "/a70dad34-b24c-4b58-b91c-f14576b5da7d"
-					(page "7")
+					(page "9")
 				)
 			)
@@
 			(project "GNSS"
 				(path "/a70dad34-b24c-4b58-b91c-f14576b5da7d"
-					(page "10")
+					(page "14")
 				)
 			)
@@
 			(color 0 0 0 0.0000)
 		)
-		(property "Sheetname" "ESP & CAN"
+		(property "Sheetname" "ESP "
 			(at 58.166 121.3354 0)
 			(effects
@@
 			)
 		)
-		(property "Sheetfile" "ESP & CAN.kicad_sch"
+		(property "Sheetfile" "ESP .kicad_sch"
 			(at 58.166 156.7946 0)
 			(effects
@@
 				)
 			)
+		)
+	)
+	(sheet
+		(at 106.68 137.16)
+		(size 24.13 15.24)
+		(fields_autoplaced yes)
+		(stroke
+			(width 0.1524)
+			(type solid)
+		)
+		(fill
+			(color 0 0 0 0.0000)
+		)
+		(property "Sheetname" "CAN"
+			(at 106.68 136.4484 0)
+			(effects
+				(font
+					(size 1.27 1.27)
+				)
+				(justify left bottom)
+			)
+		)
+		(property "Sheetfile" "CAN.kicad_sch"
+			(at 106.68 152.9846 0)
+			(effects
+				(font
+					(size 1.27 1.27)
+				)
+				(justify left top)
+			)
+		)
+		(instances
+			(project "GNSS"
+				(path "/a70dad34-b24c-4b58-b91c-f14576b5da7d"
+					(page "13")
+				)
+			)

Commit message: 123
Other:
- note added: "CAN"

Commit message: uty
Changed lines of the file:
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@@
 	(polyline
 		(pts
-			(xy 95.25 161.29) (xy 261.112 161.036)
+			(xy 93.98 160.02) (xy 259.842 159.766)
 		)
 		(stroke
@@
 	(polyline
 		(pts
-			(xy 261.112 31.496) (xy 261.112 161.036)
+			(xy 259.842 31.496) (xy 259.842 159.766)
 		)
 		(stroke
@@
 		(pts
 			(xy 127.254 54.356) (xy 127.254 74.168)
+		)
+		(stroke
+			(width 0.254)
+			(type default)
+			(color 0 0 0 1)
+		)
+	)
+	(polyline
+		(pts
+			(xy 71.12 46.99) (xy 77.47 46.99)
 		)
 		(stroke
@@
 	)
 	(sheet
-		(at 72.39 44.45)
-		(size 25.4 19.05)
+		(at 77.47 40.64)
+		(size 20.32 13.97)
 		(fields_autoplaced yes)
 		(stroke
@@
 		)
 		(property "Sheetname" "POWER_2"
-			(at 72.39 43.7384 0)
+			(at 77.47 39.9284 0)
 			(effects
 				(font
@@
 		)
 		(property "Sheetfile" "POWER_2_sch.kicad_sch"
-			(at 72.39 64.0846 0)
+			(at 77.47 55.1946 0)
 			(effects
 				(font
@@
 	)
 	(sheet
-		(at 72.39 33.02)
-		(size 25.4 19.05)
+		(at 50.8 40.64)
+		(size 20.32 13.97)
 		(fields_autoplaced yes)
 		(stroke
@@
 		)
 		(property "Sheetname" "POWER"
-			(at 72.39 32.3084 0)
+			(at 50.8 39.9284 0)
 			(effects
 				(font
@@
 		)
 		(property "Sheetfile" "POWER_sch.kicad_sch"
-			(at 72.39 52.6546 0)
+			(at 50.8 55.1946 0)
 			(effects
 				(font
@@
 	)
 	(sheet
-		(at 69.596 138.557)
-		(size 25.654 25.273)
+		(at 69.85 140.97)
+		(size 25.4 19.05)
 		(fields_autoplaced yes)
 		(stroke
@@
 		)
 		(property "Sheetname" "ESP "
-			(at 69.596 137.8454 0)
+			(at 69.85 140.2584 0)
 			(effects
 				(font
@@
 		)
 		(property "Sheetfile" "ESP .kicad_sch"
-			(at 69.596 164.4146 0)
-			(effects
-				(font
+			(at 69.85 160.6046 0)
+			(effects
+				(font

Commit message: new
Other:
- note added: "CONNECTIONS OVERVIEW"
- note removed: "Connections Overview"
Changed lines of the file:
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@@
 		)
 	)
-	(text "Connections Overview"
+	(text "CONNECTIONS OVERVIEW"
 		(exclude_from_sim no)
 		(at 145.796 18.288 0)

Commit message: 02.10.26
Other:
- sheet ANTENNA renamed antenna
- sheet ARDUINO renamed arduino
- sheet BLOCK_DIAGRAM renamed block_diagram
- sheet CAN renamed can
- sheet CONTROLLER renamed controller
- sheet ESP  renamed esp
- sheet ETHERNET renamed ethernet
- sheet IMU  renamed imu
- sheet LEDs & BUTTONs renamed led&button
- sheet POWER renamed power_1
- sheet POWER_2 renamed power_2
- sheet POWER_ARCHITECTURE renamed power_arch
- sheet SD_CARD renamed sd_card
- sheet TABLE_OF_CONTENT renamed content
- sheet USB_HUB renamed usb_hub
- sheet ZED_Z9P renamed zed_z9p
- sheet antenna: file ANTENNA.kicad_sch -> antenna.kicad_sch
- sheet arduino: file ARDUINO.kicad_sch -> arduino.kicad_sch
- sheet block_diagram: file BLOCK_DIAGRAM.kicad_sch -> block_diagram.kicad_sch
- sheet can: file CAN.kicad_sch -> can.kicad_sch
- sheet content: file CONTENT_sch.kicad_sch -> content.kicad_sch
- sheet controller: file CONTROLLER.kicad_sch -> controller.kicad_sch
- sheet esp: file ESP .kicad_sch -> esp.kicad_sch
- sheet ethernet: file ETHERNET.kicad_sch -> ethernet.kicad_sch
- sheet imu: file IMU .kicad_sch -> imu.kicad_sch
- sheet led&button: file LEDs & BUTTONs.kicad_sch -> led&button.kicad_sch
- sheet power_1: file POWER_sch.kicad_sch -> power_1.kicad_sch
- sheet power_2: file POWER_2_sch.kicad_sch -> power_2_sch.kicad_sch
- sheet power_arch: file POWER_ARCHITECTURE.kicad_sch -> power_arch.kicad_sch
- sheet sd_card: file SD_CARD.kicad_sch -> sd_card.kicad_sch
- sheet usb_hub: file USB_HUB_sch.kicad_sch -> usb_hub.kicad_sch
- sheet zed_z9p: file ZED_Z9P.kicad_sch -> zed_z9p.kicad_sch
Changed lines of the file:
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@@
 			(color 0 0 0 0.0000)
 		)
-		(property "Sheetname" "TABLE_OF_CONTENT"
+		(property "Sheetname" "content"
 			(at 15.24 20.8784 0)
 			(effects
@@
 			)
 		)
-		(property "Sheetfile" "CONTENT_sch.kicad_sch"
+		(property "Sheetfile" "content.kicad_sch"
 			(at 15.24 174.5746 0)
 			(effects
@@
 			(color 0 0 0 0.0000)
 		)
-		(property "Sheetname" "POWER_2"
+		(property "Sheetname" "power_2"
 			(at 77.47 39.9284 0)
 			(effects
@@
 			)
 		)
-		(property "Sheetfile" "POWER_2_sch.kicad_sch"
+		(property "Sheetfile" "power_2_sch.kicad_sch"
 			(at 77.47 55.1946 0)
 			(effects
@@
 			(color 0 0 0 0.0000)
 		)
-		(property "Sheetname" "IMU "
+		(property "Sheetname" "imu"
 			(at 219.71 65.3284 0)
 			(effects
@@
 			)
 		)
-		(property "Sheetfile" "IMU .kicad_sch"
+		(property "Sheetfile" "imu.kicad_sch"
 			(at 219.71 85.6746 0)
 			(effects
@@
 			(color 0 0 0 0.0000)
 		)
-		(property "Sheetname" "BLOCK_DIAGRAM"
+		(property "Sheetname" "block_diagram"
 			(at 17.78 24.6884 0)
 			(effects
@@
 			)
 		)
-		(property "Sheetfile" "BLOCK_DIAGRAM.kicad_sch"
+		(property "Sheetfile" "block_diagram.kicad_sch"
 			(at 17.78 170.7646 0)
 			(effects
@@
 			(color 0 0 0 0.0000)
 		)
-		(property "Sheetname" "ZED_Z9P"
+		(property "Sheetname" "zed_z9p"
 			(at 59.69 72.9484 0)
 			(effects
@@
 			)
 		)
-		(property "Sheetfile" "ZED_Z9P.kicad_sch"
+		(property "Sheetfile" "zed_z9p.kicad_sch"
 			(at 59.69 103.4546 0)
 			(effects
@@
 			(color 0 0 0 0.0000)
 		)
-		(property "Sheetname" "USB_HUB"
+		(property "Sheetname" "usb_hub"
 			(at 149.86 45.0084 0)
 			(effects
@@
 			)
 		)
-		(property "Sheetfile" "USB_HUB_sch.kicad_sch"
+		(property "Sheetfile" "usb_hub.kicad_sch"
 			(at 149.86 59.0046 0)
 			(effects
@@
 			(color 0 0 0 0.0000)
 		)
-		(property "Sheetname" "POWER_ARCHITECTURE"
+		(property "Sheetname" "power_arch"
 			(at 20.828 28.7524 0)
 			(effects
@@
 			)
 		)
-		(property "Sheetfile" "POWER_ARCHITECTURE.kicad_sch"
+		(property "Sheetfile" "power_arch.kicad_sch"
 			(at 20.828 166.9546 0)
 			(effects
@@
 			(color 0 0 0 0.0000)
 		)
-		(property "Sheetname" "CONTROLLER"
+		(property "Sheetname" "controller"
 			(at 140.97 70.4084 0)
 			(effects
@@
 			)
 		)
-		(property "Sheetfile" "CONTROLLER.kicad_sch"
+		(property "Sheetfile" "controller.kicad_sch"
 			(at 140.97 111.0746 0)
 			(effects
@@
 			(color 0 0 0 0.0000)
 		)
-		(property "Sheetname" "LEDs & BUTTONs"
+		(property "Sheetname" "led&button"
 			(at 219.71 42.4684 0)
 			(effects
@@
 			)
 		)
-		(property "Sheetfile" "LEDs & BUTTONs.kicad_sch"
+		(property "Sheetfile" "led&button.kicad_sch"
 			(at 219.71 56.4646 0)
 			(effects
@@
 			(color 0 0 0 0.0000)
 		)
-		(property "Sheetname" "POWER"
+		(property "Sheetname" "power_1"
 			(at 50.8 39.9284 0)
 			(effects
@@
 			)
 		)
-		(property "Sheetfile" "POWER_sch.kicad_sch"
+		(property "Sheetfile" "power_1.kicad_sch"
 			(at 50.8 55.1946 0)
 			(effects
@@
 			(color 0 0 0 0.0000)
 		)
-		(property "Sheetname" "SD_CARD"
+		(property "Sheetname" "sd_card"
 			(at 219.71 89.4584 0)
 			(effects
@@
 			)
 		)
-		(property "Sheetfile" "SD_CARD.kicad_sch"
+		(property "Sheetfile" "sd_card.kicad_sch"
 			(at 219.71 112.3446 0)
 			(effects
@@
 			(color 0 0 0 0.0000)
 		)
-		(property "Sheetname" "ETHERNET"
+		(property "Sheetname" "ethernet"
 			(at 219.075 118.6684 0)
 			(effects
@@
 			)
 		)
-		(property "Sheetfile" "ETHERNET.kicad_sch"
+		(property "Sheetfile" "ethernet.kicad_sch"
 			(at 219.075 155.2706 0)
 			(effects
@@
 			(color 0 0 0 0.0000)
 		)
-		(property "Sheetname" "ANTENNA"
+		(property "Sheetname" "antenna"
 			(at 22.86 76.7584 0)
 			(effects
@@
 			)
 		)
-		(property "Sheetfile" "ANTENNA.kicad_sch"
+		(property "Sheetfile" "antenna.kicad_sch"
 			(at 22.86 110.8206 0)
 			(effects
@@
 			(color 0 0 0 0.0000)
 		)
-		(property "Sheetname" "ARDUINO"
+		(property "Sheetname" "arduino"
 			(at 151.13 130.0984 0)
 			(effects
@@
 			)
 		)
-		(property "Sheetfile" "ARDUINO.kicad_sch"
+		(property "Sheetfile" "arduino.kicad_sch"
 			(at 151.13 147.9046 0)
 			(effects
@@
 			(color 0 0 0 0.0000)
 		)
-		(property "Sheetname" "ESP "
+		(property "Sheetname" "esp"
 			(at 69.85 140.2584 0)
 			(effects
@@
 			)
 		)
-		(property "Sheetfile" "ESP .kicad_sch"
+		(property "Sheetfile" "esp.kicad_sch"
 			(at 69.85 160.6046 0)
 			(effects
@@
 			(color 0 0 0 0.0000)
 		)
-		(property "Sheetname" "CAN"
+		(property "Sheetname" "can"
 			(at 73.66 112.3184 0)
 			(effects
@@
 			)
 		)
-		(property "Sheetfile" "CAN.kicad_sch"
+		(property "Sheetfile" "can.kicad_sch"
 			(at 73.66 126.3146 0)
 			(effects

Commit message: new
Changed lines of the file:
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@@
 	(polyline
 		(pts
-			(xy 167.64 31.496) (xy 261.112 31.496)
+			(xy 167.64 31.496) (xy 260.35 31.75)
 		)
 		(stroke
