File: ESP & CAN.kicad_sch (KiCad schematic)
At the start: 28 parts, among them J2 Conn, U5 TCAN1042VDRBRQ1, U6 TPD2EUSB30ADRTR, U8 ESP32-C3-MINI-1-N4

Commit message: full
Parts:
- removed U6: TPD2EUSB30ADRTR, GNSS:SOTFL35P100X50-3N, symbol TPD2EUSB30ADRTR:TPD2EUSB30ADRTR
- added U6: TPD2EUSB30A, Package_TO_SOT_SMD:Texas_DRT-3, symbol Power_Protection:TPD2EUSB30A
Connections:
- net +3.3V_CAN: no longer U5.5 (VIO)
- net CANH: now also U6.1 (D+); no longer U5.7 (CANH)
- net CANL: now also U6.2 (D-); no longer U5.6 (CANL)
- net CAN_RXD: no longer U5.4 (RXD)
- net CAN_STB: no longer U5.8 (STB)
- net CAN_TXD: no longer U5.1 (TXD)
- net GND: now also U6.3 (GND); no longer U5.2 (GND), U5.9 (PAD)
- net VIN_CAN: no longer U5.3 (VCC)
Other:
- moved on the sheet: C31

Commit message: 16.09.2026
Parts:
- removed U6: TPD2EUSB30A, Package_TO_SOT_SMD:Texas_DRT-3, symbol Power_Protection:TPD2EUSB30A
- C29: footprint C0402C104K4RAC:CAPC1005X55N -> Capacitor_SMD:C_0805_2012Metric
- C30, C31, C54, C65: footprint C0402C104K4RAC:CAPC1005X55N -> Capacitor_SMD:C_0402_1005Metric
- FL1, FL2: footprint BLM21PG221SN1D:BEADC2012X105N -> GNSS:BEADC2012X105N
- R16, R17, R24, R25, R26, R34, R43, R52, R53: footprint Resistor_SMD:R_0805_2012Metric -> Resistor_SMD:R_0402_1005Metric
- R35, R54: footprint Resistor_SMD:R_0805_2012Metric -> Capacitor_SMD:C_0402_1005Metric
Connections:
- net +3.3V_CAN: now also U5.5 (VIO)
- net CANH: now also U5.7 (CANH)
- net CANL: now also U5.6 (CANL)
- net CAN_RXD: now also U5.4 (RXD)
- net CAN_STB: now also U5.8 (STB)
- net CAN_TXD: now also U5.1 (TXD)
- net GND: now also U5.2 (GND), U5.9 (PAD)
- net VIN_CAN: now also U5.3 (VCC)
Other:
- moved on the sheet: U5
Changed lines of the file:
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@@
 	)
 	(symbol
-		(lib_id "Power_Protection:TPD2EUSB30A")
-		(at 121.92 104.14 0)
-		(unit 1)
-		(exclude_from_sim no)
-		(in_bom yes)
-		(on_board yes)
-		(dnp no)
-		(fields_autoplaced yes)
-		(property "Reference" "U6"
-			(at 121.92 93.98 0)
-			(effects
-				(font
-					(size 1.27 1.27)
-				)
-			)
-		)
-		(property "Value" "TPD2EUSB30A"
-			(at 121.92 96.52 0)
-			(effects
-				(font
-					(size 1.27 1.27)
-				)
-			)
-		)
-		(property "Footprint" "Package_TO_SOT_SMD:Texas_DRT-3"
-			(at 102.87 111.76 0)
-			(effects
-				(font
-					(size 1.27 1.27)
-				)
-				(hide yes)
-			)
-		)
-		(property "Datasheet" "http://www.ti.com/lit/ds/symlink/tpd2eusb30a.pdf"
-			(at 121.92 104.14 0)
-			(effects
-				(font
-					(size 1.27 1.27)
-				)
-				(hide yes)
-			)
-		)
-		(property "Description" "2-Channel ESD Protection for Super-Speed USB 3.0 Interface, DRT-3"
-			(at 121.92 104.14 0)
-			(effects
-				(font
-					(size 1.27 1.27)
-				)
-				(hide yes)
-			)
-		)
-		(pin "2"
-		)
-		(pin "1"
-		)
-		(pin "3"
-		)
-		(instances
-			(project "GNSS"
-				(path "/a70dad34-b24c-4b58-b91c-f14576b5da7d/cd83e7ab-22db-42ff-a7e6-36d43df00222"
-					(reference "U6")
-					(unit 1)
-				)
-			)
-		)
-	)
-	(symbol
 		(lib_id "Device:R_Small_US")
 		(at 172.72 109.22 180)
@@
 			)
 		)
-		(property "Footprint" "Resistor_SMD:R_0805_2012Metric"
+		(property "Footprint" "Resistor_SMD:R_0402_1005Metric"
 			(at 172.72 109.22 0)
 			(effects
@@
 			)
 		)
-		(property "Footprint" "Resistor_SMD:R_0805_2012Metric"
+		(property "Footprint" "Resistor_SMD:R_0402_1005Metric"
 			(at 173.99 97.79 0)
 			(effects
@@
 			)
 		)
-		(property "Footprint" "C0402C104K4RAC:CAPC1005X55N"
+		(property "Footprint" "Capacitor_SMD:C_0805_2012Metric"
 			(at 97.79 115.57 0)
 			(effects
@@
 			)
 		)
-		(property "Footprint" "Resistor_SMD:R_0805_2012Metric"
+		(property "Footprint" "Resistor_SMD:R_0402_1005Metric"
 			(at 86.36 107.95 0)
 			(effects
@@
 			)
 		)
-		(property "Footprint" "Resistor_SMD:R_0805_2012Metric"
+		(property "Footprint" "Capacitor_SMD:C_0402_1005Metric"
 			(at 256.54 90.17 0)
 			(effects
@@
 			)
 		)
-		(property "Footprint" "Resistor_SMD:R_0805_2012Metric"
+		(property "Footprint" "Resistor_SMD:R_0402_1005Metric"
 			(at 227.33 130.81 0)
 			(effects
@@
 			)
 		)
-		(property "Footprint" "Resistor_SMD:R_0805_2012Metric"
+		(property "Footprint" "Capacitor_SMD:C_0402_1005Metric"
 			(at 193.04 125.73 0)
 			(effects
@@
 			)
 		)
-		(property "Footprint" "C0402C104K4RAC:CAPC1005X55N"
+		(property "Footprint" "Capacitor_SMD:C_0402_1005Metric"
 			(at 243.84 81.28 0)
 			(effects
@@
 			)
 		)
-		(property "Footprint" "BLM21PG221SN1D:BEADC2012X105N"
+		(property "Footprint" "GNSS:BEADC2012X105N"
 			(at 124.968 59.944 0)
 			(effects
@@
 			)
 		)
-		(property "Footprint" "BLM21PG221SN1D:BEADC2012X105N"
+		(property "Footprint" "GNSS:BEADC2012X105N"
 			(at 123.698 49.784 0)
 			(effects
@@
 	(symbol
 		(lib_id "2026-08-14_04-42-40:TCAN1042VDRBRQ1")
-		(at 58.42 114.3 0)
+		(at 57.15 114.3 0)
 		(unit 1)
 		(exclude_from_sim no)
@@
 		(fields_autoplaced yes)
 		(property "Reference" "U5"
-			(at 58.42 93.98 0)
+			(at 57.15 93.98 0)
 			(effects
 				(font
@@
 		)
 		(property "Value" "TCAN1042VDRBRQ1"
-			(at 59.69 96.52 0)
+			(at 58.42 96.52 0)
 			(effects
 				(font
@@
 		)
 		(property "Footprint" "GNSS:DRB0008F"
-			(at 59.69 114.3 0)
+			(at 58.42 114.3 0)
 			(effects
 				(font
@@
 		)
 		(property "Datasheet" "https://www.ti.com/lit/gpn/tcan1042v-q1"
-			(at 59.69 114.3 0)
+			(at 58.42 114.3 0)
 			(effects
 				(font
@@
 		)
 		(property "Description" ""
-			(at 59.69 114.3 0)
+			(at 58.42 114.3 0)
 			(effects
 				(font
@@
 			)
 		)
-		(property "Footprint" "Resistor_SMD:R_0805_2012Metric"
+		(property "Footprint" "Resistor_SMD:R_0402_1005Metric"
 			(at 200.66 125.73 0)
 			(effects
@@
 			)
 		)
-		(property "Footprint" "Resistor_SMD:R_0805_2012Metric"
+		(property "Footprint" "Resistor_SMD:R_0402_1005Metric"
 			(at 247.65 109.22 0)
 			(effects
@@
 			)
 		)
-		(property "Footprint" "C0402C104K4RAC:CAPC1005X55N"
+		(property "Footprint" "Capacitor_SMD:C_0402_1005Metric"
 			(at 107.95 109.22 0)
 			(effects
@@
 			)
 		)
-		(property "Footprint" "Resistor_SMD:R_0805_2012Metric"
+		(property "Footprint" "Resistor_SMD:R_0402_1005Metric"
 			(at 175.26 110.49 0)
 			(effects
@@
 			)
 		)
-		(property "Footprint" "Resistor_SMD:R_0805_2012Metric"
+		(property "Footprint" "Resistor_SMD:R_0402_1005Metric"
 			(at 86.36 115.57 0)
 			(effects
@@
 			)
 		)
-		(property "Footprint" "Resistor_SMD:R_0805_2012Metric"
+		(property "Footprint" "Resistor_SMD:R_0402_1005Metric"
 			(at 175.26 88.9 0)
 			(effects
@@
 			)
 		)
-		(property "Footprint" "C0402C104K4RAC:CAPC1005X55N"
+		(property "Footprint" "Capacitor_SMD:C_0402_1005Metric"
 			(at 232.41 81.28 0)
 			(effects
@@
 			)
 		)
-		(property "Footprint" "C0402C104K4RAC:CAPC1005X55N"
+		(property "Footprint" "Capacitor_SMD:C_0402_1005Metric"
 			(at 113.03 132.08 0)
 			(effects

Commit message: 18.09.2026
Parts:
- added D10, D12: PESD0402-140, PESD0402-140:DIO_PESD0402-140, symbol PESD0402-140:PESD0402-140
Connections:
- net CANH: now also D10.2
- net CANL: now also D12.1
- net GND: now also D10.1, D12.2
- net +3.3V renamed +3V3
- net +3.3V_CAN renamed +3V3_CAN
- net +3.3V_ESP renamed +3V3_ESP
Other:
- moved on the sheet: C30
