File: GNSS.kicad_pcb (KiCad board)
At the start: 2 copper layers, 101 x 53.3 mm, 243 parts, among them IC1 USB2513B_M2, IC2 ZED-F9P-05B, IC3 STM32H563VGT6, J1 USB_C_Receptacle_USB2.0_16P, J2 Conn, J3 5033981892, J5 Conn_01x05_Pin, J6 Conn, J7 SMA-J-P-X-RA-TH1, J8 USB_C_Receptacle_USB2.0_16P, Q1 SI1016CX-T1-GE3, Q3 BC849, Q5 BC849, Q6 BC849, Q7 BC849, Q8 BC849, T1 WE-RJ45_7499010211A, U1 MIC5205-3.3YM5, U10 TPD2EUSB30A, U12 TPD2EUSB30A, U13 ICM-42688-P, U2 TPD2EUSB30A, U3 TPD2EUSB30A, U4 DP83825IRMQR, U5 TCAN1042VDRBRQ1, U6 TPD2EUSB30A, U7 IR3883MTRPBF, U8 ESP32-C3-MINI-1-N4, U9 MCP6001-OT, Y1 MURATA_XRCGB24M000FFS1DR0, Y4 MURATA_XRCGB24M000FFS1DR0

Commit message: 18.09.2026
Parts:
- moved U6 15.2 mm to (141.9, 67.1)
- moved C22 1.38 mm to (142.4, 83.8)
- moved C23 1.38 mm to (144.8, 83.7)
- moved C30 1.38 mm to (140.3, 78.7)
- moved C31 1.38 mm to (140.4, 81.9)
- moved R16 1.38 mm to (140.3, 79.7)
- moved C29 1.38 mm to (135.8, 80.4)
- moved FL2 1.38 mm to (142.2, 77.1)
- moved R17 1.38 mm to (140.3, 80.8)
- moved FL1 1.38 mm to (145.9, 77.1)
- moved J2 1.38 mm to (150.3, 84.3)
- moved U5 1.38 mm to (143.9, 81.0)
- moved FL12 1.35 mm to (149.6, 77.0)
Changed lines of the file:
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@@
 	(footprint "Connector_PinHeader_1.00mm:PinHeader_1x03_P1.00mm_Vertical"
 		(layer "F.Cu")
-		(at 150.125 82.95 -90)
+		(at 150.275 84.324998 -90)
 		(descr "Through hole straight pin header, 1x03, 1.00mm pitch, single row")
 		(tags "Through hole pin header THT 1x03 1.00mm single row")
@@
 	(footprint "Capacitor_SMD:C_0805_2012Metric"
 		(layer "B.Cu")
-		(at 144.7 82.375)
+		(at 144.85 83.749998)
 		(descr "Capacitor SMD 0805 (2012 Metric), square (rectangular) end terminal, IPC_7351 nominal, (Body size source: IPC-SM-782 page 76, https://www.pcb-3d.com/wordpress/wp-content/uploads/ipc-sm-782a_amendment_1_and_2.pdf, https://docs.google.com/spreadsheets/d/1BsfQQcO9C6DZCsRaXUlFlo91Tg2WpOkGARC1WS5S8t0/edit?usp=sharing), generated with kicad-footprint-generator")
 		(tags "capacitor")
@@
 	(footprint "GNSS:DRB0008F"
 		(layer "B.Cu")
-		(at 143.8 79.650001 180)
+		(at 143.95 81.024999 180)
 		(tags "TCAN1042VDRBRQ1 ")
 		(property "Reference" "U5"
-			(at 0 0 0)
+			(at 1.8 2.374999 0)
 			(unlocked yes)
 			(layer "B.SilkS")
@@
 	(footprint "Capacitor_SMD:C_0402_1005Metric"
 		(layer "B.Cu")
-		(at 142.25 82.425 90)
+		(at 142.4 83.799998 90)
 		(descr "Capacitor SMD 0402 (1005 Metric), square (rectangular) end terminal, IPC_7351 nominal, (Body size source: IPC-SM-782 page 76, https://www.pcb-3d.com/wordpress/wp-content/uploads/ipc-sm-782a_amendment_1_and_2.pdf), generated with kicad-footprint-generator")
 		(tags "capacitor")
@@
 	(footprint "GNSS:BEADC2012X105N"
 		(layer "B.Cu")
-		(at 149.625 75.7 180)
+		(at 149.6 77.05 180)
 		(property "Reference" "FL12"
-			(at -2.925 0 180)
+			(at -0.15 1.575 180)
 			(layer "B.SilkS")
 			(effects
@@
 	(footprint "Capacitor_SMD:C_0402_1005Metric"
 		(layer "B.Cu")
-		(at 140.22 80.55)
+		(at 140.37 81.924998)
 		(descr "Capacitor SMD 0402 (1005 Metric), square (rectangular) end terminal, IPC_7351 nominal, (Body size source: IPC-SM-782 page 76, https://www.pcb-3d.com/wordpress/wp-content/uploads/ipc-sm-782a_amendment_1_and_2.pdf), generated with kicad-footprint-generator")
 		(tags "capacitor")
@@
 	(footprint "GNSS:BEADC2012X105N"
 		(layer "B.Cu")
-		(at 145.75 75.7 180)
+		(at 145.9 77.074998 180)
 		(property "Reference" "FL1"
 			(at 0.25 1.5 180)
@@
 	(footprint "Resistor_SMD:R_0402_1005Metric"
 		(layer "B.Cu")
-		(at 140.125 78.375)
+		(at 140.275 79.749998)
 		(descr "Resistor SMD 0402 (1005 Metric), square (rectangular) end terminal, IPC_7351 nominal, (Body size source: IPC-SM-782 page 72, https://www.pcb-3d.com/wordpress/wp-content/uploads/ipc-sm-782a_amendment_1_and_2.pdf), generated with kicad-footprint-generator")
 		(tags "resistor")
@@
 	(footprint "Capacitor_SMD:C_0805_2012Metric"
 		(layer "B.Cu")
-		(at 135.675 79)
+		(at 135.825 80.374998)
 		(descr "Capacitor SMD 0805 (2012 Metric), square (rectangular) end terminal, IPC_7351 nominal, (Body size source: IPC-SM-782 page 76, https://www.pcb-3d.com/wordpress/wp-content/uploads/ipc-sm-782a_amendment_1_and_2.pdf, https://docs.google.com/spreadsheets/d/1BsfQQcO9C6DZCsRaXUlFlo91Tg2WpOkGARC1WS5S8t0/edit?usp=sharing), generated with kicad-footprint-generator")
 		(tags "capacitor")
@@
 	(footprint "Package_TO_SOT_SMD:Texas_DRT-3"
 		(layer "B.Cu")
-		(at 140.1875 82.2225)
+		(at 141.9 67.125)
 		(descr "Texas Instrument DRT-3 1x0.8mm Pitch 0.7mm http://www.ti.com/lit/ds/symlink/tpd2eusb30.pdf")
 		(tags "DRT-3 1x0.8mm Pitch 0.7mm")
@@
 	(footprint "Capacitor_SMD:C_0402_1005Metric"
 		(layer "B.Cu")
-		(at 140.125 77.3)
+		(at 140.275 78.674998)
 		(descr "Capacitor SMD 0402 (1005 Metric), square (rectangular) end terminal, IPC_7351 nominal, (Body size source: IPC-SM-782 page 76, https://www.pcb-3d.com/wordpress/wp-content/uploads/ipc-sm-782a_amendment_1_and_2.pdf), generated with kicad-footprint-generator")
 		(tags "capacitor")
@@
 	(footprint "Resistor_SMD:R_0402_1005Metric"
 		(layer "B.Cu")
-		(at 140.175 79.475)
+		(at 140.325 80.849998)
 		(descr "Resistor SMD 0402 (1005 Metric), square (rectangular) end terminal, IPC_7351 nominal, (Body size source: IPC-SM-782 page 72, https://www.pcb-3d.com/wordpress/wp-content/uploads/ipc-sm-782a_amendment_1_and_2.pdf), generated with kicad-footprint-generator")
 		(tags "resistor")
@@
 	(footprint "GNSS:BEADC2012X105N"
 		(layer "B.Cu")
-		(at 142.05 75.725 180)
+		(at 142.2 77.099998 180)
 		(property "Reference" "FL2"
-			(at 3 0.05 180)
+			(at -0.175 1.549998 180)
 			(layer "B.SilkS")
 			(effects
