File: GNSS.kicad_pcb (KiCad board)
At the start: 2 copper layers, 101 x 53.3 mm, 240 parts, among them IC1 USB2513B_M2, IC2 ZED-F9P-05B, IC3 STM32H563VGT6, J1 USB_C_Receptacle_USB2.0_16P, J2 Conn, J3 5033981892, J5 Conn_01x05_Pin, J6 Conn, J7 SMA-J-P-X-RA-TH1, J8 USB_C_Receptacle_USB2.0_16P, Q1 SI1016CX-T1-GE3, Q3 BC849, Q5 BC849, Q6 BC849, Q7 BC849, Q8 BC849, T1 WE-RJ45_7499010211A, U1 MIC5205-3.3YM5, U10 TPD2EUSB30A, U12 TPD2EUSB30A, U13 ICM-42688-P, U2 TPD2EUSB30A, U3 TPD2EUSB30A, U4 DP83825IRMQR, U5 TCAN1042VDRBRQ1, U6 TPD2EUSB30A, U7 IR3883MTRPBF, U8 ESP32-C3-MINI-1-N4, U9 MCP6001-OT, Y1 MURATA_XRCGB24M000FFS1DR0

Commit message: 16.09.2026
Parts:
- removed C75: 100nF, Capacitor_SMD:C_0402_1005Metric
- removed C76: 10uF, Capacitor_SMD:C_0805_2012Metric
- removed D11: SML-P12U2TT86R, LED_SMD:LED_0402_1005Metric
- added C54: 0.1uF, Capacitor_SMD:C_0402_1005Metric, F.Cu at (122.1, 117.0)
- added C79: 0.1u, Capacitor_SMD:C_0402_1005Metric, B.Cu at (125.0, 96.0)
- added C81: 10u, Capacitor_SMD:C_0805_2012Metric, B.Cu at (127.0, 95.0)
- added C82: 0.1u, Capacitor_SMD:C_0402_1005Metric, B.Cu at (124.9, 89.3)
- added S2: SKRPABE010, GNSS:SW_SKRPABE010, F.Cu at (153.7, 115.1)
- added Y4: MURATA_XRCGB24M000FFS1DR0, GNSS:XTAL_ECS-250-12-33-AGN-TR, F.Cu at (167.3, 107.3)
- BT1: footprint 1056:BAT_1056 -> GNSS:BAT_1056
- C18, C21, C47, C66, C77, C83, C84: footprint C0402C104K4RAC:CAPC1005X55N -> Capacitor_SMD:C_0402_1005Metric
- C27: value 27pF -> 470p; moved to B.Cu
- C28: value 0.1uF -> 2u2; footprint Capacitor_SMD:C_0402_1005Metric -> Capacitor_SMD:C_0805_2012Metric; moved to B.Cu
- C29: value 100nF -> 4n7; footprint Capacitor_SMD:C_0402_1005Metric -> Capacitor_SMD:C_0805_2012Metric; moved to B.Cu
- C3, C68, C69, C70, D7, FL3, R13, R48, R51, R55, R56, R57, R7, R74, R75: moved to F.Cu
- C30: value 10nF -> 100p; moved to B.Cu
- C31: value 0.1uF -> 100p; moved to B.Cu
- C53, C58, C71, C72, L4, Q3, Q5, Q6, Q7, Q8, R18, R28, R29, R32, R33, R71, R76, R77, R78, R79, R92, R93, U1: moved to B.Cu
- C65: value 27pF -> 0.1uF
- FL1: footprint BLM21PG221SN1D:BEADC2012X105N -> GNSS:BEADC2012X105N; moved to B.Cu
- FL10, FL11, FL12, FL2, FL5, FL6, FL7, FL8: footprint BLM21PG221SN1D:BEADC2012X105N -> GNSS:BEADC2012X105N
- FL4: footprint BLM21PG221SN1D:BEADC2012X105N -> GNSS:BEADC2012X105N; moved to F.Cu
- R16, R26, R43, R53: footprint Resistor_SMD:R_0805_2012Metric -> Resistor_SMD:R_0402_1005Metric
- R17, R24, R25, R34, R52: footprint Resistor_SMD:R_0805_2012Metric -> Resistor_SMD:R_0402_1005Metric; moved to B.Cu
- R35, R54: footprint Resistor_SMD:R_0805_2012Metric -> Capacitor_SMD:C_0402_1005Metric; moved to B.Cu
- moved R57 129.9 mm to (242.2, 117.3), turned to 0 degrees
- moved R31 112.4 mm to (49.1, 122.5)
- moved U10 110.7 mm to (30.9, 102.3)
- moved TP4 109.7 mm to (32.3, 112.0)
- moved TP3 100.6 mm to (263.9, 70.3)
- moved D1 89.6 mm to (98.2, 95.6), turned to 0 degrees
- moved U9 84.8 mm to (190.3, 93.2)
- moved R100 82.9 mm to (186.3, 96.9)
- moved R97 82.8 mm to (185.6, 90.1)
- moved R95 82.8 mm to (185.6, 86.2)
- moved R96 82.8 mm to (185.6, 88.1)
- moved R98 82.8 mm to (185.6, 92.1)
- moved R99 82.8 mm to (185.6, 94.1)
- moved R66 68.0 mm to (126.5, 79.2)
- moved R93 66.0 mm to (120.0, 86.5), turned to -90 degrees
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Connections:
- C27 pad 2: /Ethernet/XTAL_IN -> Net-(U1-BP)
- C28 pad 2: +3.3V_ESP -> +3V3_ICM
- C29 pad 2: +3V3_IMU -> Net-(C29-Pad2)
- C30 pad 2: +3V3_IMU -> /ESP & CAN/CANH
- C31 pad 2: +3.3V_ESP -> /ESP & CAN/CANL
- C65 pad 2: /Ethernet/XTAL_OUT -> +3.3V_ESP
- U5 pad 1: unconnected-(U5-TXD-Pad1) -> CAN_TXD
- U5 pad 2: unconnected-(U5-GND-Pad2) -> GND
- U5 pad 3: unconnected-(U5-VCC-Pad3) -> VIN_CAN
- U5 pad 4: unconnected-(U5-RXD-Pad4) -> CAN_RXD
- U5 pad 5: unconnected-(U5-VIO-Pad5) -> +3.3V_CAN
- U5 pad 6: unconnected-(U5-CANL-Pad6) -> /ESP & CAN/CANL
- U5 pad 7: unconnected-(U5-CANH-Pad7) -> /ESP & CAN/CANH
- U5 pad 8: unconnected-(U5-STB-Pad8) -> CAN_STB
- U5 pad 9: unconnected-(U5-PAD-Pad9) -> GND
Routing:
- net GN_TIMEPULSE: track 56.7 -> 0.00 mm
- net INT1_GYRO: track 74.4 -> 20.8 mm
- net TX_READY: track 91.6 -> 38.9 mm, vias 1 -> 0
- net +3.3V_ESP: track 2.31 -> 51.2 mm
- net SD_DAT2: track 46.2 -> 0.00 mm
- net ETH_MDC: track 45.3 -> 0.00 mm
- net SD_DAT3: track 41.8 -> 0.00 mm
- net ETH_RX_D1_N: track 32.1 -> 0.00 mm
- net ETH_RX_D0_N: track 29.7 -> 0.00 mm
- net ETH_TX_EN: track 28.7 -> 0.00 mm
- net ETH_CRS_DV: track 28.3 -> 0.00 mm
- net SD_DAT0: track 27.5 -> 0.00 mm
- net INT1_ACCEL: track 62.3 -> 36.3 mm
- net Net-(IC2-RF_IN): track 25.4 -> 0.00 mm
- net SD_DAT1: track 24.3 -> 0.00 mm
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Other:
- board text removed: "USER BT1"

Commit message: 22.09.26
Parts:
- removed C45, C46: 1u, Capacitor_SMD:C_0805_2012Metric
- removed C47: 100n, Capacitor_SMD:C_0402_1005Metric
- removed C49: 100n, C0402C104K4RAC:CAPC1005X55N
- removed FL1, FL10, FL11, FL2, FL4, FL5, FL6, FL7, FL8: BLM21PG221SN1D, GNSS:BEADC2012X105N
- removed FL13, FL3: BLM21PG221SN1D, BLM21PG221SN1D:BEADC2012X105N
- removed J6: Conn, Connector_PinHeader_1.00mm:PinHeader_1x03_P1.00mm_Vertical
- removed R47: 47K, Resistor_SMD:R_0402_1005Metric
- removed R57, R91: 1M, Resistor_SMD:R_0402_1005Metric
- removed R92, R93, R94: 10K, Resistor_SMD:R_0402_1005Metric
- removed TP12: TestPoint, TestPoint:TestPoint_Pad_D2.0mm
- removed Y4: MURATA_XRCGB24M000FFS1DR0, GNSS:XTAL_ECS-250-12-33-AGN-TR
- added C85: 100n, Capacitor_SMD:C_0402_1005Metric, F.Cu at (232.9, 104.5)
- added C86: 2u2, Capacitor_SMD:C_0805_2012Metric, F.Cu at (233.7, 102.0)
- added FB1: FerriteBead, GNSS:BEADC2012X105N, F.Cu at (162.3, 49.9)
- added FB10: FerriteBead, GNSS:BEADC2012X105N, F.Cu at (227.2, 102.0)
- added FB11: FerriteBead, GNSS:BEADC2012X105N, F.Cu at (233.7, 114.0)
- added FB2: FerriteBead, GNSS:BEADC2012X105N, F.Cu at (201.3, 26.8)
- added FB3: FerriteBead, GNSS:BEADC2012X105N, B.Cu at (122.5, 88.5)
- added FB4: FerriteBead, GNSS:BEADC2012X105N, F.Cu at (230.1, 94.0)
- added FB5: FerriteBead, GNSS:BEADC2012X105N, F.Cu at (227.2, 111.0)
- added FB6: FerriteBead, GNSS:BEADC2012X105N, F.Cu at (227.2, 114.0)
- added FB7: FerriteBead, GNSS:BEADC2012X105N, F.Cu at (233.7, 109.0)
- added FB8: FerriteBead, GNSS:BEADC2012X105N, F.Cu at (236.6, 94.0)
- added FB9: FerriteBead, GNSS:BEADC2012X105N, F.Cu at (220.8, 105.1)
- added R67: 10K, Resistor_SMD:R_0402_1005Metric, F.Cu at (226.4, 104.5)
- added R73: 10K, Resistor_SMD:R_0402_1005Metric, B.Cu at (117.8, 86.8)
- added R80: 10K, Resistor_SMD:R_0402_1005Metric, B.Cu at (107.7, 86.8)
- added R81: 10K, Resistor_SMD:R_0402_1005Metric, B.Cu at (113.5, 86.7)
- added R82: 10K, Resistor_SMD:R_0402_1005Metric, F.Cu at (226.4, 106.5)
- added TP10: TestPoint, TestPoint:TestPoint_Pad_D2.0mm, F.Cu at (216.5, 109.7)
- added TP8: TestPoint, TestPoint:TestPoint_Pad_D2.0mm, F.Cu at (107.3, 153.8)
- added TP9: TestPoint, TestPoint:TestPoint_Pad_D2.0mm, F.Cu at (216.5, 105.6)
- C15, C19, C20: value 22u -> 0.1u; footprint Capacitor_SMD:C_0805_2012Metric -> Capacitor_SMD:C_0402_1005Metric
- C16: value 22u -> 0.47u; footprint Capacitor_SMD:C_0805_2012Metric -> Capacitor_SMD:C_0402_1005Metric
- C17: value 220p -> 4u7; footprint C0402C104K4RAC:CAPC1005X55N -> Capacitor_SMD:C_0805_2012Metric
- C18: value 0.1u -> 10u; footprint Capacitor_SMD:C_0402_1005Metric -> Capacitor_SMD:C_0805_2012Metric
- C24: value 0.47u -> 10u; footprint Capacitor_SMD:C_0402_1005Metric -> Capacitor_SMD:C_0805_2012Metric; moved to B.Cu
- C25: value 4u7 -> 0.1u; footprint Capacitor_SMD:C_0805_2012Metric -> Capacitor_SMD:C_0402_1005Metric; moved to B.Cu
- C26: value 10u -> 22u/25V
- C27: value 470p -> 22u/25V; footprint Capacitor_SMD:C_0402_1005Metric -> Capacitor_SMD:C_0805_2012Metric; moved to F.Cu
- C28: value 2u2 -> 22u/25V; moved to F.Cu
- C39, C41: value 100n -> 1u; footprint Capacitor_SMD:C_0402_1005Metric -> Capacitor_SMD:C_0805_2012Metric
- C44: value 100n -> 18p
- C51: value 1u -> 2.2u
- C52: value 100n -> 2.2u
- C62: value 1u -> 10u
- C66, C77: value 18p -> 20p
- C79: value 0.1u -> 22u/25V; footprint Capacitor_SMD:C_0402_1005Metric -> Capacitor_SMD:C_0805_2012Metric; moved to F.Cu
- C81: value 10u -> 0.1u/50V; footprint Capacitor_SMD:C_0805_2012Metric -> Capacitor_SMD:C_0402_1005Metric; moved to F.Cu
- C82: value 0.1u -> 470p
- C83: value 0.1u -> 2u2; footprint Capacitor_SMD:C_0402_1005Metric -> Capacitor_SMD:C_0805_2012Metric; moved to B.Cu
- C84: moved to B.Cu
- IC3: value STM32H563VGT6 -> STM32H563VGTx; footprint GNSS:QFP50P1600X1600X160-100N -> Package_QFP:LQFP-100_14x14mm_P0.5mm
- J1, J8: footprint Connector_USB:USB_C_Receptacle_HCTL_HC-TYPE-C-16P-01A -> GNSS:USB4105_GCT
- J5: footprint Connector_PinHeader_1.00mm:PinHeader_1x05_P1.00mm_Vertical -> Connector_PinSocket_2.54mm:PinSocket_1x04_P2.54mm_Vertical
- R11: value 16K5 -> 32K4
- R12: value 2K94 -> 47K
- R13: value 49K9 -> 33K2
- R14: value 33K2 -> 49K9
- R19, R20: value 0R -> 0E
- R42: value 10K -> 16K5; moved to F.Cu
- R46: value 32K4 -> 2K94
- moved C18 100.7 mm to (196.3, 25.7)
- moved R13 100.1 mm to (192.8, 32.2)
- moved C17 98.1 mm to (196.4, 35.2)
- moved C15 95.1 mm to (196.3, 31.1)
- moved C16 95.1 mm to (196.3, 28.9)
- moved C19 95.1 mm to (192.7, 28.9)
- moved C26 95.1 mm to (70.0, 32.9)
- moved R14 95.1 mm to (61.9, 33.0)
- moved R42 79.5 mm to (67.7, 51.0), turned to 90 degrees
- moved TP3 75.8 mm to (204.6, 23.2)
- moved VR1 73.2 mm to (205.6, 31.9)
- moved R11 70.1 mm to (61.0, 47.7)
- moved R12 70.1 mm to (58.6, 47.0)
- moved C21 70.1 mm to (59.9, 40.3)
- moved L1 70.1 mm to (66.4, 41.1)
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Connections:
- net +3.3V_ESP renamed +3V3_ESP
- net +3.3V_ETH renamed +3V3_ETH
- net +3.3V_HUB renamed +3V3_HUB
- net +3.3V_SD renamed +3V3_SD
- net /ESP & CAN/IO8 renamed /ESP /IO8
- net VCAP renamed Net-(C51-Pad1)
- A1 pad 2: +3.3V_ARDUINO -> unconnected-(A1-IOREF-Pad2)
- A1 pad 4: +3.3V_ARDUINO -> +3V3_ARDUINO
- C15 pad 1: +3.3V -> GND
- C15 pad 2: GND -> VIN_GNSS
- C16 pad 1: +3.3V -> GND
- C16 pad 2: GND -> Net-(VR1-SET)
- C17 pad 1: Net-(U7-FB) -> VIN_GNSS
- C17 pad 2: +3.3V -> GND
- C18 pad 1: /POWER/SW -> GND
- C18 pad 2: Net-(U7-BOOT) -> +3V3_GNSS
- C19 pad 1: 5V -> GND
- C19 pad 2: GND -> +3V3_GNSS
- C20 pad 1: 5V -> /POWER_2/SW
- C20 pad 2: GND -> Net-(U7-BOOT)
- C24 pad 2: Net-(VR1-SET) -> VIN_ICM
- C25 pad 1: VIN_GNSS -> GND
- C25 pad 2: GND -> VIN_ICM
- C26 pad 1: GND -> +3V3
- C26 pad 2: +3V3_GNSS -> GND
- C27 pad 1: GND -> 5V
- C27 pad 2: Net-(U1-BP) -> GND
- C28 pad 1: GND -> +3V3
- C28 pad 2: +3V3_ICM -> GND
- C30 pad 2: /ESP & CAN/CANH -> /CAN/CANH
- C31 pad 2: /ESP & CAN/CANL -> /CAN/CANL
- C32 pad 2: STM_3.3V -> STM_3V3
- C33 pad 2: STM_3.3V -> STM_3V3
- C34 pad 2: STM_3.3V -> STM_3V3
- C35 pad 2: STM_3.3V -> STM_3V3
- C36 pad 2: STM_3.3V -> STM_3V3
- C37 pad 2: STM_3.3V -> STM_3V3
- C38 pad 2: STM_3.3V -> STM_3V3
- C39 pad 1: GND -> VDDA
- C39 pad 2: STM_3.3V -> GND
- C41 pad 1: GND -> VREFP
- C41 pad 2: STM_3.3V -> GND
- C43 pad 1: STM_3.3V -> STM_3V3
- C44 pad 1: GND -> Net-(IC3-PH1)
- C44 pad 2: STM_3.3V -> GND
- C48 pad 1: STM_3.3V -> STM_3V3
- C50 pad 2: STM_3.3V -> VREFP
- C55 pad 1: +3V3_GN -> +3V3_GNSS
- C56 pad 2: +3V3_GN -> +3V3_GNSS
- C62 pad 1: +3V3_GN -> +3V3_GNSS
- C63 pad 2: +3V3_GN -> +3V3_GNSS
- C66 pad 1: /ETHERNET/XTAL_OUT -> GND
- C66 pad 2: GND -> /ETHERNET/XTAL_OUT
- C77 pad 1: /ETHERNET/XTAL_IN -> GND
- C77 pad 2: GND -> /ETHERNET/XTAL_IN
- C79 pad 1: GND -> 5V
- C79 pad 2: VIN_ICM -> GND
- C81 pad 2: VIN_ICM -> 5V
- C82 pad 2: +3V3_ICM -> Net-(U1-BP)
- C83 pad 2: +3V3_GNSS -> +3V3_ICM
- C84 pad 2: VIN_GNSS -> +3V3_ICM
- FL12 pad 1: +3.3V_ARDUINO -> +3V3_ARDUINO
- FL12 pad 2: +3.3V -> +3V3
- IC2 pad 33: +3V3_GN -> +3V3_GNSS
- IC2 pad 34: +3V3_GN -> +3V3_GNSS
- IC2 pad 38: +3V3_GN -> +3V3_GNSS
- IC3 pad 100: STM_3.3V -> STM_3V3
- IC3 pad 11: STM_3.3V -> STM_3V3
- IC3 pad 12: /CONTROLLER/OSC_IN -> Net-(IC3-PH0)
- IC3 pad 13: /CONTROLLER/OSC_OUT -> Net-(IC3-PH1)
- IC3 pad 21: STM_3.3V -> VREFP
- IC3 pad 22: STM_3.3V -> VDDA
- IC3 pad 23: unconnected-(IC3-PA0-Pad23) -> ETH_INTR
- IC3 pad 28: STM_3.3V -> STM_3V3
- IC3 pad 50: STM_3.3V -> STM_3V3
- IC3 pad 6: STM_3.3V -> STM_3V3
- IC3 pad 73: STM_3.3V -> STM_3V3
- IC3 pad 75: STM_3.3V -> STM_3V3
- J2 pad 1: /ESP & CAN/CANH -> /CAN/CANH
- J2 pad 2: /ESP & CAN/CANL -> /CAN/CANL
- J5 pad 1: STM_3.3V -> STM_3V3
- L1 pad 1: /POWER/SW -> /POWER_2/SW
- L1 pad 2: +3.3V -> +3V3
- R11 pad 1: +3.3V -> Net-(U7-EN/FCCM)
- R11 pad 2: Net-(U7-FB) -> 5V
- R12 pad 1: Net-(U7-FB) -> GND
- R12 pad 2: GND -> Net-(U7-EN/FCCM)
- R13 pad 1: +3.3V -> Net-(VR1-SET)
- R13 pad 2: Net-(U7-PGOOD) -> GND
- R14 pad 1: Net-(VR1-SET) -> +3V3
- R14 pad 2: GND -> Net-(U7-PGOOD)
- R15 pad 1: +3V3_GN -> +3V3_GNSS
- R16 pad 2: /ESP & CAN/CANH -> /CAN/CANH
- R17 pad 2: /ESP & CAN/CANL -> /CAN/CANL
- R18 pad 1: STM_3.3V -> STM_3V3
- R19 pad 1: STM_3.3V -> STM_3V3
- R19 pad 2: STM_3.3V -> VDDA
- R20 pad 1: STM_3.3V -> VREFP
- R20 pad 2: STM_3.3V -> VDDA
- R29 pad 1: STM_3.3V -> STM_3V3
- R30 pad 1: +3V3_GN -> +3V3_GNSS
- R31 pad 2: +3.3V -> +3V3
- R36 pad 2: +3.3V -> +3V3
- R37 pad 2: +3.3V -> +3V3
- R38 pad 2: +3.3V -> +3V3
- R39 pad 2: +3.3V -> +3V3
- R40 pad 2: +3.3V -> +3V3
- R41 pad 2: +3.3V -> +3V3
- R42 pad 1: /CONTROLLER/BOOT0 -> +3V3
- R42 pad 2: STM_3.3V -> Net-(U7-FB)
- R44 pad 1: +3V3_GN -> +3V3_GNSS
- R46 pad 1: /POWER/EN -> Net-(U7-FB)
- R46 pad 2: 5V -> GND
- R58 pad 2: STM_3.3V -> STM_3V3
- R59 pad 1: +3V3_GN -> +3V3_GNSS
- R62 pad 2: +3V3_GN -> +3V3_GNSS
- R63 pad 2: +3V3_GN -> +3V3_GNSS
- R64 pad 2: +3V3_GN -> +3V3_GNSS
- R65 pad 2: +3V3_GN -> +3V3_GNSS
- R68 pad 2: +3V3_GN -> +3V3_GNSS
- R70 pad 2: STM_3.3V -> STM_3V3
- R76 pad 1: SD_DAT2 -> SD_DAT3
- R77 pad 1: SD_DAT3 -> SD_CMD
- R78 pad 1: SD_CMD -> SD_CLK
- R79 pad 1: SD_CLK -> SD_DAT0
- R9 pad 2: +3.3V -> +3V3
- TP3 pad 1: +3V3_ICM -> +3V3_GNSS
- TP5 pad 1: +3.3V -> +3V3
- U5 pad 5: +3.3V_CAN -> +3V3_CAN
- U5 pad 6: /ESP & CAN/CANL -> /CAN/CANL
- U5 pad 7: /ESP & CAN/CANH -> /CAN/CANH
- U7 pad 10_11_12: /POWER/SW -> /POWER_2/SW
- U7 pad 5: /POWER/EN -> Net-(U7-EN/FCCM)
- U7 pad 8: +3.3V -> +3V3
- VR1 pad 6: VIN -> VIN_GNSS
Routing:
- net ESP_RXD: track 0.00 -> 51.2 mm
- net +3V3_ESP: track 51.2 -> 0.00 mm
- net SD_DAT2: track 0.00 -> 15.8 mm
- net SD_CMD: track 6.83 -> 22.4 mm
- net SD_DAT3: track 0.00 -> 15.4 mm
- net SD_CLK: track 0.00 -> 14.8 mm
- net SD_DAT0: track 0.00 -> 14.7 mm
- net SD_DAT1: track 0.00 -> 14.6 mm
- net +3V3_SD: track 0.21 -> 14.7 mm
- net INT1_GYRO: track 20.8 -> 31.8 mm, vias 1 -> 0
- net IMU_MOSI: track 0.00 -> 10.1 mm
- net IMU_MISO: track 0.00 -> 9.54 mm
- net INT1_ACCEL: track 36.3 -> 45.2 mm
- net IMU_SCK: track 0.00 -> 8.20 mm
- net SD_DETECT: track 0.00 -> 2.33 mm
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Other:
- copper layers 2 -> 4
- board text added: "PPS"
- board text added: "USER"

Commit message: uty
Parts:
- added R39: 5K1, Resistor_SMD:R_0402_1005Metric, F.Cu at (135.5, 127.5)
- added R40: 5K1, Resistor_SMD:R_0402_1005Metric, F.Cu at (135.5, 129.5)
Connections:
- FB10 pad 1: STM_3V3 -> +3V3
- FB10 pad 2: +3V3 -> STM_3V3
- FB5 pad 1: VIN_CAN -> VIN
- FB5 pad 2: VIN -> VIN_CAN
- FB6 pad 1: +3V3_CAN -> +3V3
- FB6 pad 2: +3V3 -> +3V3_CAN
- FB7 pad 1: +3V3_IMU -> +3V3_ICM
- FB7 pad 2: +3V3_ICM -> +3V3_IMU
- FB8 pad 1: +3V3_ETH -> +3V3
- FB8 pad 2: +3V3 -> +3V3_ETH
- R1 pad 1: Net-(J8-CC2) -> Net-(J4-CC2)
- R2 pad 2: Net-(J8-CC1) -> Net-(J4-CC1)
