File: GNSS.kicad_pcb (KiCad board)
At the start: 4 copper layers, 101 x 53.3 mm, 242 parts, among them IC1 USB2513B_M2, IC2 ZED-F9P-05B, IC3 STM32H563VGTx, J1 USB_C_Receptacle_USB2.0_16P, J2 Conn, J3 5033981892, J5 Conn_01x05_Pin, J7 SMA-J-P-X-RA-TH1, J8 USB_C_Receptacle_USB2.0_16P, Q1 SI1016CX-T1-GE3, Q3 BC849, Q5 BC849, Q6 BC849, Q7 BC849, Q8 BC849, T1 WE-RJ45_7499010211A, U1 MIC5205-3.3YM5, U10 TPD2EUSB30A, U12 TPD2EUSB30A, U13 ICM-42688-P, U2 TPD2EUSB30A, U3 TPD2EUSB30A, U4 DP83825IRMQR, U5 TCAN1042VDRBRQ1, U6 TPD2EUSB30A, U7 IR3883MTRPBF, U8 ESP32-C3-MINI-1-N4, U9 MCP6001-OT, Y1 MURATA_XRCGB24M000FFS1DR0

Commit message: uy
Parts:
- added C21: 220p, Capacitor_SMD:C_0402_1005Metric, F.Cu at (274.5, 81.5)
- added C40: 100n, Capacitor_SMD:C_0402_1005Metric, F.Cu at (280.0, 75.0)
- added C42: 18p, Capacitor_SMD:C_0402_1005Metric, F.Cu at (278.0, 81.5)
- added D10: PESD0402-140, Diode_SMD:D_0402_1005Metric, F.Cu at (257.5, 42.4)
- added D11: PESD0402-140, Diode_SMD:D_0402_1005Metric, F.Cu at (257.5, 47.0)
- added D12: PESD0402-140, Diode_SMD:D_0402_1005Metric, F.Cu at (257.5, 44.4)
- added D13: ESD5V0D5-TP, Diode_SMD:D_SOD-523, F.Cu at (274.3, 77.5)
- added F2: MF-MSMF200-2, Fuse:Fuse_1812_4532Metric, F.Cu at (241.3, 19.6)
- added F3: MF-MSMF200-2, Fuse:Fuse_1812_4532Metric, F.Cu at (241.9, 26.0)
- added FB12: FerriteBead, Inductor_SMD:L_0805_2012Metric, F.Cu at (274.5, 88.0)
- added IC4: LM66200DRLR, Package_SO:SOIC-8_3.9x4.9mm_P1.27mm, F.Cu at (275.5, 71.0)
- added J4: 2036150003, Connector_USB:USB_C_Receptacle_GCT_USB4085, F.Cu at (223.9, 19.6)
- added J6: 2036150003, Connector_USB:USB_C_Receptacle_GCT_USB4085, F.Cu at (223.7, 35.6)
- added JP3: SolderJumper_2_Open, Jumper:SolderJumper-2_P1.3mm_Open_Pad1.0x1.5mm, F.Cu at (242.9, 39.0)
- added L2: LQG15HS47NJ02D, Inductor_SMD:L_0402_1005Metric, F.Cu at (276.0, 57.5)
- added Q1: MMBT3904LT1G, Package_TO_SOT_SMD:SOT-23, F.Cu at (275.0, 39.0)
- added U11: TPS22918DBVR, Package_TO_SOT_SMD:SOT-23-6, F.Cu at (274.5, 47.0)
- added U15: TPS22946YZPR, Package_BGA:Texas_DSBGA-6_0.704x1.054mm_Layout2x3_P0.35mm, F.Cu at (252.8, 37.1)
- added U6: BSS84DW-7-F, Package_TO_SOT_SMD:SOT-323_SC-70, F.Cu at (275.0, 53.0)
- added Y2: ECS-250-18-33-JGN-TR, Crystal:Crystal_SMD_3225-4Pin_3.2x2.5mm, F.Cu at (275.6, 62.9)
- added Y3: MURATA_XRCGB24M000FFS1DR0, Crystal:Crystal_SMD_2016-4Pin_2.0x1.6mm, F.Cu at (242.2, 49.5)
- D3: footprint GNSS:ESD5V0D5TP -> Diode_SMD:D_SOD-523
- Y1: footprint GNSS:MURATA_XRCGB24M000FFS1DR0_0 -> Crystal:Crystal_SMD_2016-4Pin_2.0x1.6mm
- moved C17 13.0 mm to (183.7, 32.3)
- moved FB2 13.0 mm to (188.6, 23.9)
- moved TP3 13.0 mm to (191.9, 20.3)
- moved C15 13.0 mm to (183.6, 28.2)
- moved C16 13.0 mm to (183.6, 26.0)
- moved C18 13.0 mm to (183.6, 22.8)
- moved C19 13.0 mm to (180.0, 26.0)
- moved R13 13.0 mm to (180.1, 29.3)
- moved VR1 13.0 mm to (192.9, 29.0)
- moved C40 6.99 mm to (220.4, 104.9)
- moved C86 6.99 mm to (233.7, 109.0)
- moved FB10 6.99 mm to (227.2, 109.0)
- moved FB4 6.99 mm to (230.1, 101.0)
- moved FB6 6.99 mm to (227.2, 121.0)
- moved FB8 6.99 mm to (236.6, 101.0)
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
Commit message: new
Parts:
- added C45: 1u, Capacitor_SMD:C_0805_2012Metric, F.Cu at (92.2, 132.8)
- added C46: 1u, Capacitor_SMD:C_0805_2012Metric, F.Cu at (92.2, 135.8)
- added TP11: TestPoint, TestPoint:TestPoint_Pad_D2.0mm, F.Cu at (96.5, 138.0)
- added U14: NCV8705ML33TCG, Package_DFN_QFN:DFN-8-1EP_3x3mm_P0.65mm_EP1.55x2.4mm, F.Cu at (97.6, 133.7)

Commit message: new
Parts:
- removed J1, J8: USB_C_Receptacle_USB2.0_16P, GNSS:USB4105_GCT
- added L3: 22uH, footprints:IND_MSS1278T-223MLD_COC, F.Cu at (54.3, 83.0)
- added U11: NC7SZ125M5X, Package_TO_SOT_SMD:SOT-23-5, F.Cu at (62.9, 104.9)
- J4, J6: footprint Connector_USB:USB_C_Receptacle_GCT_USB4085 -> GNSS_Library:USB4105_GCT
- moved J6 145.3 mm to (97.5, 107.8), turned to -90 degrees
- moved J4 141.6 mm to (97.7, 83.6), turned to -90 degrees
- moved F3 60.6 mm to (228.1, 85.0)
- moved F2 60.6 mm to (227.6, 78.6)
- moved D13 46.5 mm to (252.3, 118.5)
- moved FB12 46.5 mm to (252.4, 129.0)
- moved IC4 46.5 mm to (253.5, 112.0)
- moved L2 46.5 mm to (254.0, 98.5)
- moved Q1 46.5 mm to (253.0, 80.0)
- moved U11 46.5 mm to (252.5, 88.0)
- moved U6 46.5 mm to (253.0, 94.0)
- moved C21 46.5 mm to (252.5, 122.5)
- moved C42 46.5 mm to (256.0, 122.5)
- moved C40 46.5 mm to (257.9, 116.0)
- moved Y2 46.5 mm to (253.6, 103.8)
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Connections:
- R45 pad 2: GN_TIMEPULSE -> TIMEPULSE_LED

Commit message: new
Parts:
- moved D10 25.6 mm to (253.0, 67.5)
- moved D11 25.6 mm to (253.0, 72.1)
- moved D12 25.6 mm to (253.0, 69.5)
- moved U15 25.3 mm to (252.8, 61.6)
- moved Y3 15.3 mm to (251.8, 56.0)
Changed lines of the file:
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@@
 	(footprint "Package_BGA:Texas_DSBGA-6_0.704x1.054mm_Layout2x3_P0.35mm"
 		(layer "F.Cu")
-		(at 248.795 36.65)
+		(at 252.825 61.65)
 		(descr "Texas Instruments, DSBGA-6, 0.704x1.054mm, NSMD, YKA pad definition, 0.704x1.054mm, 6 Ball, 2x3 Layout, 0.35mm Pitch, https://www.ti.com/lit/ml/mxbg383/mxbg383.pdf, https://www.ti.com/lit/ds/symlink/tps62800.pdf")
 		(tags "BGA 6 0.35")
@@
 			(pintype "input")
 		)
-		(model "${KICAD8_3DMODEL_DIR}/Package_BGA.3dshapes/Texas_DSBGA-6_0.704x1.054mm_Layout2x3_P0.35mm.wrl"
+		(model "${KICAD8_3DMODEL_DIR}/TPS22946YZPR.step"
 			(offset
 				(xyz 0 0 0)
 			)
 			(scale
-				(xyz 1 1 1)
+				(xyz 0.7 0.6001 0.7001)
 			)
 			(rotate
-				(xyz 0 0 0)
+				(xyz 90 180 180)
 			)
 		)
@@
 	(footprint "Diode_SMD:D_0402_1005Metric"
 		(layer "F.Cu")
-		(at 253.485 46.5)
+		(at 253 72.09)
 		(descr "Diode SMD 0402 (1005 Metric), square (rectangular) end terminal, IPC_7351 nominal, (Body size source: http://www.tortai-tech.com/upload/download/2011102023233369053.pdf), generated with kicad-footprint-generator")
 		(tags "diode")
@@
 			(pintype "passive")
 		)
-		(model "${KICAD8_3DMODEL_DIR}/Diode_SMD.3dshapes/D_0402_1005Metric.wrl"
+		(model "${KICAD8_3DMODEL_DIR}/Diode_SMD.3dshapes/PESD0402-140.step"
 			(offset
 				(xyz 0 0 0)
 			)
 			(scale
-				(xyz 1 1 1)
+				(xyz 1.5 1.3001 0.9001)
 			)
 			(rotate
-				(xyz 0 0 0)
+				(xyz 90 -180 0)
 			)
 		)
@@
 	(footprint "Crystal:Crystal_SMD_2016-4Pin_2.0x1.6mm"
 		(layer "F.Cu")
-		(at 238.2 48.95)
+		(at 251.8 55.95)
 		(descr "SMD Crystal SERIES SMD2016/4 http://www.q-crystal.com/upload/5/2015552223166229.pdf, 2.0x1.6mm^2 package")
 		(tags "SMD SMT crystal")
@@
 			(pintype "passive+no_connect")
 		)
-		(model "${KICAD8_3DMODEL_DIR}/Crystal.3dshapes/Crystal_SMD_2016-4Pin_2.0x1.6mm.wrl"
+		(model "${KICAD8_3DMODEL_DIR}/Crystal.3dshapes/MURATA_XRCGB24M000FFS1DR0.step"
 			(offset
 				(xyz 0 0 0)
@@
 	(footprint "Diode_SMD:D_0402_1005Metric"
 		(layer "F.Cu")
-		(at 253.485 41.91)
+		(at 253 67.5)
 		(descr "Diode SMD 0402 (1005 Metric), square (rectangular) end terminal, IPC_7351 nominal, (Body size source: http://www.tortai-tech.com/upload/download/2011102023233369053.pdf), generated with kicad-footprint-generator")
 		(tags "diode")
@@
 			(pintype "passive")
 		)
-		(model "${KICAD8_3DMODEL_DIR}/Diode_SMD.3dshapes/D_0402_1005Metric.wrl"
+		(model "${KICAD8_3DMODEL_DIR}/Diode_SMD.3dshapes/PESD0402-140.step"
 			(offset
 				(xyz 0 0 0)
 			)
 			(scale
-				(xyz 1 1 1)
+				(xyz 1.5 1.3 1.1)
 			)
 			(rotate
-				(xyz 0 0 0)
+				(xyz 90 180 180)
 			)
 		)
@@
 			(pintype "passive")
 		)
+		(model "${KICAD8_3DMODEL_DIR}/Connector_PinSocket_2.54mm.3dshapes/PinSocket_1x02_P2.54mm_Vertical.step"
+			(offset
+				(xyz 0.5 0 0)
+			)
+			(scale
+				(xyz 0.5 0.5 0.8)
+			)
+			(rotate
+				(xyz 0 0 90)
+			)
+		)
 	)
 	(footprint "Capacitor_SMD:C_0402_1005Metric"
@@
 	(footprint "Diode_SMD:D_0402_1005Metric"
 		(layer "F.Cu")
-		(at 253.485 43.9)
+		(at 253 69.49)
 		(descr "Diode SMD 0402 (1005 Metric), square (rectangular) end terminal, IPC_7351 nominal, (Body size source: http://www.tortai-tech.com/upload/download/2011102023233369053.pdf), generated with kicad-footprint-generator")
 		(tags "diode")
@@
 			(pintype "passive")
 		)
-		(model "${KICAD8_3DMODEL_DIR}/Diode_SMD.3dshapes/D_0402_1005Metric.wrl"
+		(model "${KICAD8_3DMODEL_DIR}/Diode_SMD.3dshapes/PESD0402-140.step"
 			(offset
 				(xyz 0 0 0)
 			)
 			(scale
-				(xyz 1 1 1)
+				(xyz 1.5 1.3 1)
 			)
 			(rotate
-				(xyz 0 0 0)
+				(xyz 90 180 180)
 			)
 		)

Commit message: new
Parts:
- removed the U11 at (252.5, 88.0)
- added C15: 0.1u/50V, Capacitor_SMD:C_0402_1005Metric, B.Cu at (115.5, 110.5)
- added C16: 0.1u, Capacitor_SMD:C_0402_1005Metric, B.Cu at (175.0, 83.5)
- C15, C16, C20, C21 (x2), C26, C27, C28, C79, C81, D10, D12, D13, FB11, FB12, FB2, FB4, FB5, FB6, R11, R12, R14, R39, R40, R42, R46, U14, U7: moved to B.Cu
- C45, C46: value 1u -> 10u; moved to B.Cu
- J4, J6: footprint GNSS_Library:USB4105_GCT -> Connector_USB:USB_C_Receptacle_GCT_USB4085
- moved D13 152.4 mm to (100.0, 113.0), turned to 180 degrees
- moved IC4 138.9 mm to (117.0, 86.5)
- moved Y3 133.5 mm to (125.2, 98.5)
- moved C21 131.0 mm to (122.0, 110.5), turned to 180 degrees
- moved C40 128.2 mm to (131.0, 98.0)
- moved C42 127.2 mm to (131.0, 99.0), turned to 180 degrees
- moved F3 118.2 mm to (110.0, 81.5)
- moved F2 117.8 mm to (110.0, 86.5)
- moved U11 117.2 mm to (180.0, 100.5)
- moved FB4 114.1 mm to (116.5, 90.4), turned to -90 degrees
- moved FB7 113.9 mm to (126.6, 77.0)
- moved FB11 111.9 mm to (122.4, 109.0), turned to 180 degrees
- moved D12 109.8 mm to (143.5, 77.5), turned to 180 degrees
- moved D10 108.0 mm to (145.5, 77.5), turned to 180 degrees
- moved C15 106.1 mm to (115.5, 109.5), turned to 0 degrees
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Connections:
- net /CAN/CANH renamed /can/CANH
- net /CAN/CANL renamed /can/CANL
- net /CONTROLLER/BOOT0 renamed /controller/BOOT0
- net /ESP /IO8 renamed /esp/IO8
- net /ETHERNET/XTAL_IN renamed /ethernet/XTAL_IN
- net /ETHERNET/XTAL_OUT renamed /ethernet/XTAL_OUT
- net /USB_HUB/CR renamed /usb_hub/CR
- net /USB_HUB/PLL renamed /usb_hub/PLL
- net /ZED_Z9P/SAFE_BOOT renamed /zed_z9p/SAFE_BOOT
- net /ZED_Z9P/V_BCKP renamed /zed_z9p/V_BCKP
- C20 pad 1: /POWER_2/SW -> /power_2/SW
- L3 pad 2: /POWER_2/SW -> /power_2/SW
- U7 pad 10_11_12: /POWER_2/SW -> /power_2/SW
