File: IMU & SDCARD.kicad_sch (KiCad schematic)
At the start: 22 parts, among them J3 5033981892, U13 ICM-42688-P

Commit message: 16.09.2026
Parts:
- FL4, FL5: footprint BLM21PG221SN1D:BEADC2012X105N -> GNSS:BEADC2012X105N
Changed lines of the file:
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@@
 			)
 		)
-		(property "Footprint" "BLM21PG221SN1D:BEADC2012X105N"
+		(property "Footprint" "GNSS:BEADC2012X105N"
 			(at 254.508 47.244 0)
 			(effects
@@
 			)
 		)
-		(property "Footprint" "BLM21PG221SN1D:BEADC2012X105N"
+		(property "Footprint" "GNSS:BEADC2012X105N"
 			(at 150.368 51.054 0)
 			(effects

Commit message: 18.09.2026
Connections:
- net +3.3V renamed +3V3
- net +3.3V_SD renamed +3V3_SD
Changed lines of the file:
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@@
 			)
 		)
-		(property "Value" "+3.3V_SD"
+		(property "Value" "+3V3_SD"
 			(at 231.14 53.34 0)
 			(effects
@@
 			)
 		)
-		(property "Value" "+3.3V_SD"
+		(property "Value" "+3V3_SD"
 			(at 210.82 69.85 0)
 			(effects
@@
 			)
 		)
-		(property "Value" "+3.3V"
+		(property "Value" "+3V3"
 			(at 257.81 53.34 0)
 			(effects
@@
 			)
 		)
-		(property "Value" "+3.3V_SD"
+		(property "Value" "+3V3_SD"
 			(at 258.572 98.044 0)
 			(effects
