File: Power_Architecture.kicad_sch (KiCad schematic)
At the start: 0 parts

Commit message: block
Other:
- note added: "0.88mA"
- note added: "100mA"
- note added: "130mA"
- note added: "250mA"
- note added: "350mA"
- note added: "3V3"
- note added: "5V"
- note added: "65mA"
- note added: "70mA"
- note added: "ARDUINO"
- note added: "BUCK_LR3883MTRPBF"
- note added: "CAN"
- note added: "ESD"
- note added: "ESP"
- note added: "ETHERNET"
- note added: "FUSE"
- note added: "ICM_48688"
- note added: "LDO_ADP150WAC02"
- note added: "LDO_LT3045EDD"
- note added: "POWER_ARCHITECTURE"
- note added: "SCHOTTKY"
- note added: "SD_CARD"
- note added: "STM32"
- note added: "TYPE_C"
- note added: "USB_HUB"
- note added: "ZED_F9P"

Commit message: full
Other:
- note added: "POWER_PATH"
- note added: "PROTECTION"
- note added: "TYPE_C 1"
- note added: "TYPE_C 2"
- note removed: "ESD"
- note removed: "FUSE"
- note removed: "SCHOTTKY"
- note removed: "TYPE_C"

Commit message: insert
Other:
- note added: "PLY_OR_ing"
- note added: "POWER_SUP"
- note removed: "POWER_PATH"

Commit message: we
Other:
- note added: "ANTENNA"
- note added: "CAN_CONNECTOR"
- note added: "MAX_2A"
- note added: "OR_ing"
- note added: "POWER"
- note added: "PROG"
- note removed: "PLY_OR_ing"
- note removed: "POWER_SUP"

Commit message: 132
Other:
- note added: "ZED_ZF9P"
- note removed: "ZED_F9P"
Changed lines of the file:
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@@
+	(polyline
+		(pts
+			(xy 119.38 90.17) (xy 132.08 90.17)
+		)
+		(stroke
+			(width 0.254)
+			(type default)
+			(color 0 0 0 1)
+		)
+	)
 	(polyline
 		(pts
@@
 		(pts
 			(xy 283.21 25.4) (xy 283.21 152.4)
-		)
-		(stroke
-			(width 0.254)
-			(type default)
-			(color 0 0 0 1)
-		)
-	)
-	(polyline
-		(pts
-			(xy 119.38 91.44) (xy 132.08 90.932)
 		)
 		(stroke
@@
 		)
 	)
-	(text "ZED_F9P"
+	(text "ZED_ZF9P"
 		(exclude_from_sim no)
 		(at 230.378 21.844 0)

Commit message: 123
Other:
- note added: "ZED_F9P"
- note removed: "ZED_ZF9P"
Changed lines of the file:
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@@
 		)
 	)
-	(text "ZED_ZF9P"
+	(text "ZED_F9P"
 		(exclude_from_sim no)
 		(at 230.378 21.844 0)

Commit message: uyt
Other:
- note added: "3V3/150mA"
- note added: "3V3/3A"
- note added: "3V3/500mA"
- note added: "3V6"
- note added: "ACTIVE,3V3"
- note added: "ADP150WAC02"
- note added: "BUCK REGULATOR"
- note added: "CAN FD TRANSCEIVER"
- note added: "COIN CELL"
- note added: "DC INPUT"
- note added: "ESD"
- note added: "ESP32 C3 MINI 1"
- note added: "ETHERNET PHY"
- note added: "FUSE"
- note added: "GNSS RECEIVER"
- note added: "HEADERS"
- note added: "ICM_48688_P"
- note added: "IMU"
- note added: "INPUT"
- note added: "LAN8742A"
- note added: "LOW NOISE LDO"
- note added: "LR3883MTRPBF"
- note added: "LT3045EDD"
- note added: "MAX 2A"
- note added: "MCU"
- note added: "MICRO SD_CARD"
- note added: "STM32H563VGT6"
- note added: "SWD"
- note added: "TCAN1042HG"
- note added: "TYPE C"
- note added: "USB"
- note added: "USB HUB"
- note added: "USB2513B/M2"
- note added: "V_BCKP"
- note added: "WIFI/BLUETOOTH LE"
- note added: "ZED F9P 05B"
- note removed: "3V3"
- note removed: "BUCK_LR3883MTRPBF"
- note removed: "CAN"
- note removed: "ESP"
- note removed: "ETHERNET"
- note removed: "ICM_48688"
- note removed: "LDO_ADP150WAC02"
- note removed: "LDO_LT3045EDD"
- note removed: "MAX_2A"
- note removed: "POWER"
- note removed: "PROG"
- note removed: "SD_CARD"
- note removed: "STM32"
- note removed: "TYPE_C 1"
- note removed: "TYPE_C 2"
- note removed: "USB_HUB"
- note removed: "ZED_F9P"
