File: BLOCK_DIAGRAM.kicad_sch (KiCad schematic)
At the start: 0 parts

Commit message: 22.09.26
Other:
- note added: "25MHz_OSC"
- note added: "5V"
- note added: "ANTENNA"
- note added: "ARDUINO"
- note added: "BLOCK_DIAGRAM"
- note added: "CAN"
- note added: "CONNECTOR"
- note added: "ESP"
- note added: "ETHERNET"
- note added: "GPIO"
- note added: "ICM_48688"
- note added: "LEDs"
- note added: "MAX_2A"
- note added: "POWER"
- note added: "POWER_SUPPLY"
- note added: "PROG"
- note added: "SD_CARD"
- note added: "STM32"
- note added: "SWD"
- note added: "TYPE_C 1"
- note added: "TYPE_C 2"
- note added: "USB_HUB"
- note added: "USER_BUTTON"
- note added: "ZED_ZF9P"
