File: BLOCK_DIAGRAM.kicad_sch (KiCad schematic)
At the start: 0 parts

Commit message: 132
Other:
- note added: "ZED_ZF9P"
- note removed: "ETH_PHY"
- note removed: "ZED_F9P"
Changed lines of the file:
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@@
 	(polyline
 		(pts
-			(xy 145.796 113.03) (xy 144.526 111.76)
-		)
-		(stroke
-			(width 0.254)
-			(type default)
-			(color 0 0 0 1)
-		)
-	)
-	(polyline
-		(pts
-			(xy 144.526 119.38) (xy 144.526 123.19)
+			(xy 138.938 112.776) (xy 137.668 111.506)
+		)
+		(stroke
+			(width 0.254)
+			(type default)
+			(color 0 0 0 1)
+		)
+	)
+	(polyline
+		(pts
+			(xy 137.668 119.126) (xy 137.668 122.936)
 		)
 		(stroke
@@
 	(polyline
 		(pts
-			(xy 137.16 127) (xy 138.43 125.73)
-		)
-		(stroke
-			(width 0.254)
-			(type default)
-			(color 0 0 0 1)
-		)
-	)
-	(polyline
-		(pts
 			(xy 68.58 44.45) (xy 72.39 44.45)
 		)
@@
 	(polyline
 		(pts
-			(xy 129.286 121.92) (xy 128.016 123.19)
-		)
-		(stroke
-			(width 0.254)
-			(type default)
-			(color 0 0 0 1)
-		)
-	)
-	(polyline
-		(pts
 			(xy 57.15 34.29) (xy 57.15 44.45)
 		)
@@
 	(polyline
 		(pts
-			(xy 145.796 121.92) (xy 144.526 123.19)
+			(xy 138.938 121.666) (xy 137.668 122.936)
 		)
 		(stroke
@@
 	(polyline
 		(pts
-			(xy 135.89 124.46) (xy 134.62 125.73)
-		)
-		(stroke
-			(width 0.254)
-			(type default)
-			(color 0 0 0 1)
-		)
-	)
-	(polyline
-		(pts
 			(xy 90.17 102.87) (xy 86.36 102.87)
 		)
@@
 	(polyline
 		(pts
-			(xy 137.16 124.46) (xy 138.43 125.73)
-		)
-		(stroke
-			(width 0.254)
-			(type default)
-			(color 0 0 0 1)
-		)
-	)
-	(polyline
-		(pts
-			(xy 128.016 119.38) (xy 128.016 123.19)
-		)
-		(stroke
-			(width 0.254)
-			(type default)
-			(color 0 0 0 1)
-		)
-	)
-	(polyline
-		(pts
-			(xy 135.89 127) (xy 134.62 125.73)
-		)
-		(stroke
-			(width 0.254)
-			(type default)
-			(color 0 0 0 1)
-		)
-	)
-	(polyline
-		(pts
 			(xy 177.8 109.22) (xy 185.42 109.22)
 		)
@@
 	(polyline
 		(pts
-			(xy 129.286 113.03) (xy 128.016 111.76)
-		)
-		(stroke
-			(width 0.254)
-			(type default)
-			(color 0 0 0 1)
-		)
-	)
-	(polyline
-		(pts
 			(xy 187.96 100.33) (xy 189.23 101.6)
 		)
@@
 	(polyline
 		(pts
-			(xy 143.256 121.92) (xy 144.526 123.19)
+			(xy 136.398 121.666) (xy 137.668 122.936)
 		)
 		(stroke
@@
 	(polyline
 		(pts
-			(xy 126.746 113.03) (xy 128.016 111.76)
-		)
-		(stroke
-			(width 0.254)
-			(type default)
-			(color 0 0 0 1)
-		)
-	)
-	(polyline
-		(pts
 			(xy 57.15 44.45) (xy 57.15 55.88)
 		)
@@
 	(polyline
 		(pts
-			(xy 128.016 111.76) (xy 128.016 119.38)
-		)
-		(stroke
-			(width 0.254)
-			(type default)
-			(color 0 0 0 1)
-		)
-	)
-	(polyline
-		(pts
 			(xy 137.16 73.66) (xy 135.89 74.93)
 		)
@@
 	(polyline
 		(pts
-			(xy 144.526 111.76) (xy 144.526 119.38)
+			(xy 137.668 111.506) (xy 137.668 119.126)
 		)
 		(stroke
@@
 	(polyline
 		(pts
-			(xy 134.62 125.73) (xy 138.43 125.73)
-		)
-		(stroke
-			(width 0.254)
-			(type default)
-			(color 0 0 0 1)
-		)
-	)
-	(polyline
-		(pts
 			(xy 177.8 101.6) (xy 185.42 101.6)
 		)
@@
 	(polyline
 		(pts
-			(xy 126.746 121.92) (xy 128.016 123.19)
-		)
-		(stroke
-			(width 0.254)
-			(type default)
-			(color 0 0 0 1)
-		)
-	)
-	(polyline
-		(pts
-			(xy 143.256 113.03) (xy 144.526 111.76)
+			(xy 136.398 112.776) (xy 137.668 111.506)
 		)
 		(stroke
@@
 	)
 	(rectangle
-		(start 138.43 123.19)
-		(end 154.94 128.27)
+		(start 130.302 122.936)
+		(end 146.812 128.016)
 		(stroke
 			(width 0.508)
@@
 	)
 	(rectangle
-		(start 121.92 128.27)
-		(end 134.62 123.19)
-		(stroke
-			(width 0.508)
-			(type default)
-			(color 72 72 72 1)
-		)
-		(fill
-			(type none)
-		)
-	)
-	(rectangle
 		(start 154.94 83.82)
 		(end 177.8 90.17)
@@
 		)
 	)
-	(text "ZED_F9P"
+	(text "ZED_ZF9P"
 		(exclude_from_sim no)
 		(at 106.68 102.87 0)
@@
 	(text "25MHz_OSC"
 		(exclude_from_sim no)
-		(at 146.558 125.984 0)
+		(at 138.43 125.73 0)
 		(effects
 			(font
@@
 				(bold yes)
 				(color 72 72 72 1)
-			)
-		)
-	)
-	(text "ETH_PHY"
-		(exclude_from_sim no)
-		(at 128.016 125.73 0)
-		(effects
-			(font
-				(size 1.778 1.778)
-				(bold yes)
-				(color 72 72 72 1)

Commit message: 123
Other:
- note added: "2PIN_SCREW_TERMINAL"
- note added: "5PIN_PROGRAMMING_HEADER"
- note added: "HEADERS"
- note added: "SWD_INTERFACE"
- note added: "ZED_F9P"
- note removed: "SWD"
- note removed: "ZED_ZF9P"

Commit message: uyt
Other:
- note added: "10/100 ETHERNET PHY"
- note added: "10/100 MBPS"
- note added: "12V"
- note added: "25MHz OSC"
- note added: "3V3"
- note added: "4 BIT"
- note added: "6 AXIS IMU"
- note added: "ARDUINO COMPATIBLE HEADERS"
- note added: "CAN CONNECTOR"
- note added: "CAN FD"
- note added: "CAN TRANSCEIVER"
- note added: "DC IN"
- note added: "DIGITAL/ANALOG/PWM"
- note added: "ESP32 C3 MINI 1"
- note added: "GNSS RECEIVER"
- note added: "HEADER"
- note added: "ICM_48688_P"
- note added: "LAN8742A"
- note added: "LQFP-100"
- note added: "MAGNETICS"
- note added: "MAX 2A"
- note added: "MCU"
- note added: "MICRO SD CARD"
- note added: "POWER INPUT"
- note added: "POWER SUPPLY"
- note added: "PPS"
- note added: "RJ45 CONNECTOR"
- note added: "RMII"
- note added: "RST"
- note added: "RST BUTTON"
- note added: "SDMMC"
- note added: "SMA ACTIVE"
- note added: "SPI"
- note added: "STATUS LED"
- note added: "STM32H563VGT6"
- note added: "SWCLK"
- note added: "SWD"
- note added: "SWD PROGRAMMING"
- note added: "SWDIO"
- note added: "TCAN1042HG"
- note added: "TDK INVENSENSE"
- note added: "TIMER INPUT"
- note added: "TX/RX"
- note added: "UBLOX"
- note added: "USART"
- note added: "USB"
- note added: "USB 2.0"
- note added: "USB C"
- note added: "USB HUB"
- note added: "USB2513B/M2"
- note added: "USER BUTTON"
- note added: "USER INTERFACE"
- note added: "USER LED"
- note added: "WIFI/BLUETOOTH LE"
- note added: "ZED F9P 05B"
- note removed: "25MHz_OSC"
- note removed: "2PIN_SCREW_TERMINAL"
- note removed: "5PIN_PROGRAMMING_HEADER"
- note removed: "ARDUINO"
- note removed: "ESP"
- note removed: "HEADERS"
- note removed: "ICM_48688"
- note removed: "LEDs"
- note removed: "MAX_2A"
- note removed: "POWER"
- note removed: "POWER_SUPPLY"
- note removed: "PROG"
- note removed: "SD_CARD"
- note removed: "STM32"
- note removed: "SWD_INTERFACE"
- note removed: "TYPE_C 1"
- note removed: "TYPE_C 2"
- note removed: "USB_HUB"
- note removed: "USER_BUTTON"
- note removed: "ZED_F9P"

Commit message: new
Other:
- note added: "DP83825I"
- note removed: "LAN8742A"
Changed lines of the file:
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@@
 		)
 	)
-	(text "LAN8742A"
+	(text "DP83825I"
 		(exclude_from_sim no)
 		(at 213.36 126.746 0)

Commit message: new
Changed lines of the file:
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@@
+	(polyline
+		(pts
+			(xy 124.46 38.1) (xy 104.14 38.1)
+		)
+		(stroke
+			(width 0.254)
+			(type default)
+			(color 0 0 194 1)
+		)
+	)
 	(polyline
 		(pts
@@
 	(polyline
 		(pts
-			(xy 104.14 38.1) (xy 124.46 38.1)
-		)
-		(stroke
-			(width 0.254)
-			(type default)
-			(color 0 0 194 1)
-		)
-	)
-	(polyline
-		(pts
 			(xy 102.87 96.52) (xy 104.14 95.25)
 		)
@@
 		)
 		(stroke
-			(width 0.254)
-			(type default)
-			(color 0 0 0 1)
-		)
-	)
-	(polyline
-		(pts
-			(xy 104.14 38.1) (xy 116.84 38.1)
-		)
-		(stroke

Commit message: new
Changed lines of the file:
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@@
-	(polyline
-		(pts
-			(xy 261.62 12.7) (xy 260.35 13.97)
-		)
-		(stroke
-			(width 0.254)
-			(type default)
-			(color 0 0 0 1)
-		)
-	)
 	(polyline
 		(pts
@@
 	(polyline
 		(pts
-			(xy 278.13 15.24) (xy 276.86 13.97)
-		)
-		(stroke
-			(width 0.254)
-			(type default)
-			(color 0 0 0 1)
-		)
-	)
-	(polyline
-		(pts
 			(xy 81.28 71.12) (xy 96.52 71.12)
 		)
@@
 	(polyline
 		(pts
-			(xy 267.97 13.97) (xy 271.78 13.97)
-		)
-		(stroke
-			(width 0.254)
-			(type default)
-			(color 0 0 0 1)
-		)
-	)
-	(polyline
-		(pts
 			(xy 64.77 37.592) (xy 68.58 37.592)
 		)
@@
 	(polyline
 		(pts
-			(xy 270.51 12.7) (xy 271.78 13.97)
-		)
-		(stroke
-			(width 0.254)
-			(type default)
-			(color 0 0 0 1)
-		)
-	)
-	(polyline
-		(pts
 			(xy 118.11 156.21) (xy 118.11 160.02)
 		)
@@
 	(polyline
 		(pts
-			(xy 260.35 13.97) (xy 267.97 13.97)
-		)
-		(stroke
-			(width 0.254)
-			(type default)
-			(color 0 0 0 1)
-		)
-	)
-	(polyline
-		(pts
 			(xy 96.52 76.2) (xy 104.14 76.2)
 		)
@@
 	(polyline
 		(pts
-			(xy 261.62 15.24) (xy 260.35 13.97)
-		)
-		(stroke
-			(width 0.254)
-			(type default)
-			(color 0 0 0 1)
-		)
-	)
-	(polyline
-		(pts
 			(xy 195.58 107.95) (xy 196.85 109.22)
 		)
@@
 	(polyline
 		(pts
-			(xy 270.51 15.24) (xy 271.78 13.97)
-		)
-		(stroke
-			(width 0.254)
-			(type default)
-			(color 0 0 0 1)
-		)
-	)
-	(polyline
-		(pts
 			(xy 116.84 119.38) (xy 115.57 118.11)
 		)
@@
 		)
 		(stroke
-			(width 0.254)
-			(type default)
-			(color 0 0 0 1)
-		)
-	)
-	(polyline
-		(pts
-			(xy 275.59 15.24) (xy 276.86 13.97)
-		)
-		(stroke
