File: ESP .kicad_sch (KiCad schematic)
At the start: 18 parts, among them U8 ESP32-C3-MINI-1-N4

Commit message: 123
Changed lines of the file:
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@@
 		(dnp no)
 		(property "Reference" "R24"
-			(at 90.424 113.538 90)
+			(at 91.44 114.046 0)
 			(effects
 				(font
@@
 		)
 		(property "Value" "22E"
-			(at 92.202 113.538 90)
+			(at 91.694 115.824 0)
 			(effects
 				(font
@@
 		(dnp no)
 		(property "Reference" "R25"
-			(at 96.52 97.028 90)
+			(at 96.52 97.028 0)
 			(effects
 				(font
@@
 		)
 		(property "Value" "10K"
-			(at 101.6 97.79 90)
+			(at 96.774 98.806 0)
 			(effects
 				(font
@@
 		(dnp no)
 		(property "Reference" "R54"
-			(at 188.468 125.73 90)
+			(at 188.468 118.364 90)
 			(effects
 				(font
@@
 		)
 		(property "Value" "10K"
-			(at 189.23 120.65 90)
+			(at 188.468 120.142 90)
 			(effects
 				(font
@@
 		(dnp no)
 		(property "Reference" "R52"
-			(at 187.96 142.748 90)
+			(at 187.96 142.748 0)
 			(effects
 				(font
@@
 		)
 		(property "Value" "10K"
-			(at 193.04 143.002 90)
+			(at 187.96 144.78 0)
 			(effects
 				(font
@@
 		(dnp no)
 		(property "Reference" "R53"
-			(at 152.4 132.588 90)
+			(at 152.4 132.588 0)
 			(effects
 				(font
@@
 		)
 		(property "Value" "10K"
-			(at 157.48 133.35 90)
+			(at 152.654 134.62 0)
 			(effects
 				(font
@@
 		(dnp no)
 		(property "Reference" "R34"
-			(at 99.822 113.538 90)
+			(at 102.87 114.3 0)
 			(effects
 				(font
@@
 		)
 		(property "Value" "22E"
-			(at 101.854 113.538 90)
+			(at 102.87 116.332 0)
 			(effects
 				(font
@@
 		(dnp no)
 		(property "Reference" "R26"
+			(at 92.202 85.598 90)
+			(effects
+				(font
+					(size 1.27 1.27)
+				)
+				(justify left)
+			)
+		)
+		(property "Value" "10K"
 			(at 92.202 87.63 90)
 			(effects
 				(font
-					(size 1.27 1.27)
-				)
-				(justify left)
-			)
-		)
-		(property "Value" "10K"
-			(at 91.44 92.71 90)
-			(effects
-				(font
