File: IMU .kicad_sch (KiCad schematic)
At the start: 11 parts, among them U13 ICM-42688-P

Commit message: 123
Parts:
- removed R56, R61, R66: 10K, Resistor_SMD:R_0402_1005Metric, symbol Device:R_Small_US
Connections:
- net +3V3_ICM: now also FB7.1; no longer FB7.2
- net +3V3_IMU: now also FB7.2; no longer FB7.1
Other:
- moved on the sheet: R55, R75
