File: _autosave-POWER_ARCHITECTURE.kicad_sch (KiCad schematic)
At the start: 0 parts

Commit message: uty
Other:
- note added: "DP83825I"
- note removed: "LAN8742A"
Changed lines of the file:
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@@
 		)
 	)
-	(text "LAN8742A"
+	(text "DP83825I"
 		(exclude_from_sim no)
 		(at 230.632 136.398 0)
