File: _autosave-POWER_sch.kicad_sch (KiCad schematic)
At the start: 15 parts, among them IC4 LM66200DRLR, J4 2036150003, J6 2036150003, U2 TPD2EUSB30A

Commit message: uty
Other:
- note added: "Ferrite Bead Drop(hi0805r800r-10) --> 5mV @500mA"
- note removed: "Ferrrite Beak Drop(hi0805r800r-10) --> 5mV @500mA"
Changed lines of the file:
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@@
 		)
 	)
-	(text "Ferrrite Beak Drop(hi0805r800r-10)\n--> 5mV @500mA "
+	(text "Ferrite Bead Drop(hi0805r800r-10)\n--> 5mV @500mA "
 		(exclude_from_sim no)
 		(at 66.04 187.706 0)

Commit message: uy
Parts:
- D13, D3: footprint ESD5V0D5TP -> Diode_SMD:D_SOD-523
- F2, F3: footprint MF-MSMF200-2:FUSER_MF-MSMF200-2 -> Fuse:Fuse_1812_4532Metric
- IC4: footprint LM66200DRLR:SOT8 -> Package_SO:SOIC-8_3.9x4.9mm_P1.27mm
- J4, J6: footprint CONN_2036150003_MOL -> Connector_USB:USB_C_Receptacle_GCT_USB4085
Changed lines of the file:
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@@
 			)
 		)
-		(property "Footprint" "ESD5V0D5TP"
+		(property "Footprint" "Diode_SMD:D_SOD-523"
 			(at 11.76 82.55 0)
 			(effects
@@
 			)
 		)
-		(property "Footprint" "MF-MSMF200-2:FUSER_MF-MSMF200-2"
+		(property "Footprint" "Fuse:Fuse_1812_4532Metric"
 			(at 115.57 57.15 0)
 			(effects
@@
 			)
 		)
-		(property "Footprint" "LM66200DRLR:SOT8"
+		(property "Footprint" "Package_SO:SOIC-8_3.9x4.9mm_P1.27mm"
 			(at 67.31 147.32 0)
 			(effects
@@
 			)
 		)
-		(property "Footprint" "ESD5V0D5TP"
+		(property "Footprint" "Diode_SMD:D_SOD-523"
 			(at 143.84 85.09 0)
 			(effects
@@
 			)
 		)
-		(property "Footprint" "CONN_2036150003_MOL"
+		(property "Footprint" "Connector_USB:USB_C_Receptacle_GCT_USB4085"
 			(at 44.45 52.07 0)
 			(effects
@@
 			)
 		)
-		(property "Footprint" "MF-MSMF200-2:FUSER_MF-MSMF200-2"
+		(property "Footprint" "Fuse:Fuse_1812_4532Metric"
 			(at 247.65 59.69 0)
 			(effects
@@
 			)
 		)
-		(property "Footprint" "CONN_2036150003_MOL"
+		(property "Footprint" "Connector_USB:USB_C_Receptacle_GCT_USB4085"
 			(at 176.53 54.61 0)
 			(effects
