File: LEDs & BUTTONs.kicad_sch (KiCad schematic)
At the start: 33 parts, among them Q2 BC849, Q3 BC849, Q4 BC849, Q5 BC849, Q6 BC849, Q7 BC849, Q8 BC849

Commit message: 14.09.2026
Parts:
- removed Q2, Q4: BC849, Package_TO_SOT_SMD:SOT-23, symbol Transistor_BJT:BC849
- removed R67, R72: 10K, Resistor_SMD:R_0402_1005Metric, symbol Device:R_Small_US
- R18, R28, R29, R30, R33, R44, R59: value 10K -> 560E
Connections:
- net +3V3_GN: now also R30.1, R44.1
- net EX_VBUS: now also R28.1; no longer R18.2
- net GND: now also D1.1, D5.1
- net PG_VBUS: now also R33.1; no longer R30.2
- net STM_3.3V: now also R18.1, R29.1; no longer R29.2, R44.2
- net at D7.2: now also R30.2; no longer R59.2
- net at D2.2: now also R18.2; no longer R29.1
- net at D9.2: now also R59.2
- net at D6.2: now also R29.2; no longer R44.1
- net at D8.2: now also R44.2
- removed net VIN: R28.1, R33.1
Other:
- moved on the sheet: D1, D5, R28, R33

Commit message: 16.09.2026
Connections:
- net +3V3_GN renamed +3V3_GNSS

Commit message: 18.09.2026
Connections:
- net STM_3.3V renamed STM_3V3
Changed lines of the file:
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@@
 			)
 		)
-		(property "Value" "STM_3.3V"
+		(property "Value" "STM_3V3"
 			(at 165.1 106.68 0)
 			(effects
@@
 			)
 		)
-		(property "Value" "STM_3.3V"
+		(property "Value" "STM_3V3"
 			(at 101.6 92.71 0)
 			(effects
@@
 			)
 		)
-		(property "Value" "STM_3.3V"
+		(property "Value" "STM_3V3"
 			(at 210.82 102.87 0)
 			(effects
@@
 			)
 		)
-		(property "Value" "STM_3.3V"
+		(property "Value" "STM_3V3"
 			(at 60.96 92.71 0)
 			(effects

Commit message: 22.09.26
Other:
- note added: "POWER_INDICATION_LEDs"
- note removed: "POWER_LEDs"
- moved on the sheet: R58, S1
Changed lines of the file:
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@@
 	)
 	(junction
-		(at 165.1 124.46)
+		(at 153.67 124.46)
 		(diameter 0)
 		(color 0 0 0 0)
@@
 	(wire
 		(pts
-			(xy 165.1 124.46) (xy 170.18 124.46)
+			(xy 153.67 124.46) (xy 158.75 124.46)
 		)
 		(stroke
@@
 	(wire
 		(pts
-			(xy 162.56 124.46) (xy 165.1 124.46)
+			(xy 151.13 124.46) (xy 153.67 124.46)
 		)
 		(stroke
@@
 	(wire
 		(pts
-			(xy 189.23 127) (xy 189.23 124.46)
+			(xy 177.8 127) (xy 177.8 124.46)
 		)
 		(stroke
@@
 	(wire
 		(pts
-			(xy 185.42 124.46) (xy 189.23 124.46)
+			(xy 173.99 124.46) (xy 177.8 124.46)
 		)
 		(stroke
@@
 	(wire
 		(pts
-			(xy 165.1 115.57) (xy 165.1 111.76)
+			(xy 153.67 115.57) (xy 153.67 111.76)
 		)
 		(stroke
@@
 	(wire
 		(pts
-			(xy 165.1 124.46) (xy 165.1 120.65)
+			(xy 153.67 124.46) (xy 153.67 120.65)
 		)
 		(stroke
@@
 	)
 	(rectangle
-		(start 144.78 93.98)
+		(start 129.54 86.36)
 		(end 250.19 146.05)
 		(stroke
@@
 	)
 	(rectangle
-		(start 29.21 86.36)
-		(end 125.73 146.05)
+		(start 20.32 86.36)
+		(end 120.65 146.05)
 		(stroke
 			(width 0.0508)
@@
 	(text "GNSS"
 		(exclude_from_sim no)
-		(at 100.584 140.462 0)
+		(at 101.6 142.24 0)
 		(effects
 			(font
@@
 		)
 	)
-	(text "POWER_LEDs"
+	(text "POWER_INDICATION_LEDs"
 		(exclude_from_sim no)
-		(at 33.782 25.908 0)
+		(at 41.656 25.4 0)
 		(effects
 			(font
@@
 	(text "RST"
 		(exclude_from_sim no)
-		(at 213.868 142.748 0)
+		(at 221.488 141.986 0)
 		(effects
 			(font
@@
 	(text "STM_LEDs"
 		(exclude_from_sim no)
-		(at 42.672 90.17 0)
+		(at 30.734 89.154 0)
 		(effects
 			(font
@@
 	(text "STM_PUSH_BUTTONs"
 		(exclude_from_sim no)
-		(at 166.116 97.79 0)
+		(at 146.812 90.932 0)
 		(effects
 			(font
@@
 	(text "USER"
 		(exclude_from_sim no)
-		(at 179.832 141.986 0)
+		(at 154.686 141.224 0)
 		(effects
 			(font
@@
 	(text "USER"
 		(exclude_from_sim no)
-		(at 57.15 141.478 0)
+		(at 58.928 142.494 0)
 		(effects
 			(font
@@
 	(global_label "USER_BUT"
 		(shape input)
-		(at 162.56 124.46 180)
+		(at 151.13 124.46 180)
 		(fields_autoplaced yes)
 		(effects
@@
 		)
 		(property "Intersheetrefs" "${INTERSHEET_REFS}"
-			(at 150.0801 124.46 0)
+			(at 138.6501 124.46 0)
 			(effects
 				(font
@@
 		(dnp no)
 		(property "Reference" "D2"
-			(at 59.436 115.824 0)
+			(at 55.626 110.998 90)
 			(effects
 				(font
@@
 					(size 1.524 1.524)
 				)
+				(hide yes)
 			)
 		)
@@
 	(symbol
 		(lib_id "power:+3.3V")
-		(at 165.1 111.76 0)
+		(at 153.67 111.76 0)
 		(unit 1)
 		(exclude_from_sim no)
@@
 		(fields_autoplaced yes)
 		(property "Reference" "#PWR0110"
-			(at 165.1 115.57 0)
+			(at 153.67 115.57 0)
 			(effects
 				(font
@@
 		)
 		(property "Value" "STM_3V3"
-			(at 165.1 106.68 0)
+			(at 153.67 106.68 0)
 			(effects
 				(font
@@
 		)
 		(property "Footprint" ""
-			(at 165.1 111.76 0)
+			(at 153.67 111.76 0)
 			(effects
 				(font
@@
 		)
 		(property "Datasheet" ""
-			(at 165.1 111.76 0)
+			(at 153.67 111.76 0)
 			(effects
 				(font
@@
 		)
 		(property "Description" "Power symbol creates a global label with name \"+3.3V\""
-			(at 165.1 111.76 0)
+			(at 153.67 111.76 0)
 			(effects
 				(font
@@
 		(on_board yes)
 		(dnp no)
-		(fields_autoplaced yes)
 		(property "Reference" "D9"
-			(at 250.19 46.99 0)
+			(at 250.698 47.752 90)
 			(effects
 				(font
@@
 					(size 1.524 1.524)
 				)
+				(hide yes)
 			)
 		)
@@
 					(size 1.524 1.524)
 				)
+				(hide yes)
 			)
 		)
@@
 		(dnp no)
 		(property "Reference" "D6"
-			(at 102.87 106.934 0)
+			(at 96.012 111.506 90)
 			(effects
 				(font
@@
 					(size 1.524 1.524)
 				)
+				(hide yes)
 			)
 		)
@@
 	(symbol
 		(lib_id "SKRPABE010:SKRPABE010")
-		(at 177.8 124.46 0)
+		(at 166.37 124.46 0)
 		(unit 1)
 		(exclude_from_sim no)
@@
 		(fields_autoplaced yes)
 		(property "Reference" "S1"
-			(at 177.8 114.3 0)
+			(at 166.37 114.3 0)
 			(effects
 				(font
@@
 		)
 		(property "Value" "SKRPABE010"
-			(at 177.8 116.84 0)
+			(at 166.37 116.84 0)
 			(effects
 				(font
@@
 		)
 		(property "Footprint" "GNSS:SW_SKRPABE010"
-			(at 177.8 124.46 0)
+			(at 166.37 124.46 0)
 			(effects
 				(font
@@
 		)
 		(property "Datasheet" ""
-			(at 177.8 124.46 0)
+			(at 166.37 124.46 0)
 			(effects
 				(font
@@
 		)
 		(property "Description" ""
-			(at 177.8 124.46 0)
+			(at 166.37 124.46 0)
 			(effects
 				(font
@@
 		)
 		(property "MF" "ALPS"
-			(at 177.8 124.46 0)
+			(at 166.37 124.46 0)
 			(effects
 				(font
@@
 		)
 		(property "MAXIMUM_PACKAGE_HEIGHT" "2.5 mm"
-			(at 177.8 124.46 0)
+			(at 166.37 124.46 0)
 			(effects
 				(font
@@
 		)
 		(property "Package" "None"
-			(at 177.8 124.46 0)
+			(at 166.37 124.46 0)
 			(effects
 				(font
@@
 		)
 		(property "Price" "None"
-			(at 177.8 124.46 0)
+			(at 166.37 124.46 0)
 			(effects
 				(font
@@
 		)
 		(property "Check_prices" "https://www.snapeda.com/parts/SKRPABE010/ALPS/view-part/?ref=eda"
-			(at 177.8 124.46 0)
+			(at 166.37 124.46 0)
 			(effects
 				(font
@@
 		)
 		(property "STANDARD" "Manufacturer Recommendations"
-			(at 177.8 124.46 0)
+			(at 166.37 124.46 0)
 			(effects
 				(font
@@
 		)
 		(property "SnapEDA_Link" "https://www.snapeda.com/parts/SKRPABE010/ALPS/view-part/?ref=snap"
-			(at 177.8 124.46 0)
+			(at 166.37 124.46 0)
 			(effects
 				(font
@@
 		)
 		(property "MP" "SKRPABE010"
-			(at 177.8 124.46 0)
+			(at 166.37 124.46 0)
 			(effects
 				(font
@@
 		)
 		(property "Purchase-URL" "https://www.snapeda.com/api/url_track_click_mouser/?unipart_id=652544&manufacturer=ALPS&part_name=SKRPABE010&search_term= skrpabe010"
-			(at 177.8 124.46 0)
+			(at 166.37 124.46 0)
 			(effects
 				(font
@@
 		)
 		(property "Description_1" "\n                        \n                            Switch Tactile N.O. SPST Button J-Bend 0.05A 16VDC 1.57N SMD Automotive T/R\n                        \n"
-			(at 177.8 124.46 0)
+			(at 166.37 124.46 0)
 			(effects
 				(font
@@
 		)
 		(property "Availability" "In Stock"
-			(at 177.8 124.46 0)
+			(at 166.37 124.46 0)
 			(effects
 				(font
@@
 		)
 		(property "MANUFACTURER" "Alps"
-			(at 177.8 124.46 0)
+			(at 166.37 124.46 0)
 			(effects
 				(font
@@
 		(dnp no)
 		(property "Reference" "D7"
-			(at 170.434 42.672 0)
+			(at 161.544 48.006 90)
 			(effects
 				(font
@@
 					(size 1.524 1.524)
 				)
+				(hide yes)
 			)
 		)
@@
 		(dnp no)
 		(property "Reference" "D1"
-			(at 62.23 51.562 0)
+			(at 46.99 55.626 90)
 			(effects
 				(font
@@
 					(size 1.524 1.524)
 				)
+				(hide yes)
 			)
 		)
@@
 		(on_board yes)
 		(dnp no)
-		(fields_autoplaced yes)
 		(property "Reference" "D8"
-			(at 204.47 48.26 0)
+			(at 204.216 48.514 90)
 			(effects
 				(font
@@
 					(size 1.524 1.524)
 				)
+				(hide yes)
 			)
 		)
@@
 	(symbol
 		(lib_id "Device:R_Small_US")
-		(at 165.1 118.11 180)
+		(at 153.67 118.11 180)
 		(unit 1)
 		(exclude_from_sim no)
@@
 		(dnp no)
 		(property "Reference" "R58"
-			(at 162.56 116.078 90)
+			(at 151.13 116.078 90)
 			(effects
 				(font
@@
 		)
 		(property "Value" "10K"
-			(at 167.64 116.84 90)
+			(at 156.21 116.84 90)
 			(effects
 				(font
@@
 		)
 		(property "Footprint" "Resistor_SMD:R_0402_1005Metric"
-			(at 165.1 118.11 0)
+			(at 153.67 118.11 0)
 			(effects
 				(font
@@
 		)
 		(property "Datasheet" "~"
-			(at 165.1 118.11 0)
+			(at 153.67 118.11 0)
 			(effects
 				(font
@@
 		)
 		(property "Description" "Resistor, small US symbol"
-			(at 165.1 118.11 0)
+			(at 153.67 118.11 0)
 			(effects
 				(font
@@
 	(symbol
 		(lib_id "power:GND")
-		(at 189.23 127 0)
+		(at 177.8 127 0)
 		(unit 1)
 		(exclude_from_sim no)
@@
 		(fields_autoplaced yes)
 		(property "Reference" "#PWR0123"
-			(at 189.23 133.35 0)
+			(at 177.8 133.35 0)
 			(effects
 				(font
@@
 		)
 		(property "Value" "GND"
-			(at 189.23 132.08 0)
+			(at 177.8 132.08 0)
 			(effects
 				(font
@@
 		)
 		(property "Footprint" ""
-			(at 189.23 127 0)
+			(at 177.8 127 0)
 			(effects
 				(font
@@
 		)
 		(property "Datasheet" ""
-			(at 189.23 127 0)
+			(at 177.8 127 0)
 			(effects
 				(font
@@
 		)
 		(property "Description" "Power symbol creates a global label with name \"GND\" , ground"
-			(at 189.23 127 0)
+			(at 177.8 127 0)
 			(effects
 				(font

Commit message: 123
Changed lines of the file:
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@@
 		(dnp no)
 		(property "Reference" "R30"
-			(at 170.18 38.862 90)
+			(at 161.544 36.322 0)
 			(effects
 				(font
@@
 		)
 		(property "Value" "560E"
-			(at 165.1 38.1 90)
+			(at 160.528 38.354 0)
 			(effects
 				(font
@@
 		(dnp no)
 		(property "Reference" "R44"
-			(at 213.36 38.862 90)
+			(at 203.962 36.068 0)
 			(effects
 				(font
@@
 		)
 		(property "Value" "560E"
-			(at 208.28 38.1 90)
+			(at 203.708 37.846 0)
 			(effects
 				(font
@@
 		(dnp no)
 		(property "Reference" "D5"
-			(at 104.394 53.848 0)
+			(at 89.154 57.912 90)
 			(effects
 				(font
@@
 		(dnp no)
 		(property "Reference" "R70"
-			(at 208.28 114.808 90)
+			(at 208.28 114.808 0)
 			(effects
 				(font
@@
 		)
 		(property "Value" "10K"
-			(at 213.36 115.57 90)
+			(at 208.28 116.84 0)
 			(effects
 				(font
@@
 		(dnp no)
 		(property "Reference" "R45"
-			(at 155.956 60.452 90)
+			(at 153.924 54.102 90)
 			(effects
 				(font
@@
 		)
 		(property "Value" "10K"
-			(at 150.876 60.198 90)
+			(at 153.924 55.88 90)
 			(effects
 				(font
@@
 		(dnp no)
 		(property "Reference" "R59"
-			(at 259.08 37.592 90)
+			(at 250.698 35.052 0)
 			(effects
 				(font
@@
 		)
 		(property "Value" "560E"
-			(at 254 36.83 90)
+			(at 249.936 36.83 0)
 			(effects
 				(font
@@
 		(dnp no)
 		(property "Reference" "C71"
-			(at 205.232 128.016 0)
+			(at 203.962 128.016 90)
 			(effects
 				(font
@@
 		)
 		(property "Value" "0.1u"
-			(at 214.122 127 0)
+			(at 203.708 130.048 90)
 			(effects
 				(font
@@
 		(dnp no)
 		(property "Reference" "R28"
-			(at 54.61 49.022 90)
+			(at 45.466 46.736 0)
 			(effects
 				(font
@@
 		)
 		(property "Value" "560E"
-			(at 49.53 48.26 90)
+			(at 45.466 48.768 0)
 			(effects
 				(font
@@
 		(dnp no)
 		(property "Reference" "R27"
-			(at 45.72 124.206 90)
+			(at 45.974 117.602 90)
 			(effects
 				(font
@@
 		(dnp no)
 		(property "Reference" "R18"
-			(at 63.5 103.632 90)
+			(at 54.61 100.838 0)
 			(effects
 				(font
@@
 		)
 		(property "Value" "560E"
-			(at 58.42 102.87 90)
+			(at 54.102 102.616 0)
 			(effects
 				(font
@@
 		(dnp no)
 		(property "Reference" "D7"
-			(at 161.544 48.006 90)
+			(at 162.814 45.72 90)
 			(effects
 				(font
@@
 		(dnp no)
 		(property "Reference" "R32"
-			(at 87.63 124.206 90)
+			(at 88.138 117.602 90)
 			(effects
 				(font
@@
 		(dnp no)
 		(property "Reference" "R29"
-			(at 104.14 103.632 90)
+			(at 94.996 101.092 0)
 			(effects
 				(font
@@
 		)
 		(property "Value" "560E"
-			(at 99.06 102.87 90)
+			(at 94.996 102.87 0)
 			(effects
 				(font
@@
 		(dnp no)
 		(property "Reference" "R71"
-			(at 244.856 59.182 90)
+			(at 243.078 52.578 90)
 			(effects
 				(font
@@
 		)
 		(property "Value" "10K"
-			(at 239.776 58.928 90)
+			(at 243.078 54.356 90)
 			(effects
 				(font
@@
 		(dnp no)
 		(property "Reference" "R33"
-			(at 96.52 49.022 90)
+			(at 87.884 46.736 0)
 			(effects
 				(font
@@
 		)
 		(property "Value" "560E"
-			(at 91.44 48.26 90)
+			(at 87.122 48.768 0)
 			(effects
 				(font
@@
 		(dnp no)
 		(property "Reference" "R58"
-			(at 151.13 116.078 90)
+			(at 151.13 116.078 0)
 			(effects
 				(font
@@
 		)
 		(property "Value" "10K"
-			(at 156.21 116.84 90)
+			(at 151.13 117.856 0)
 			(effects
 				(font
@@
 		(dnp no)
 		(property "Reference" "R60"
-			(at 199.136 60.452 90)
+			(at 197.358 53.848 90)
 			(effects
 				(font
@@
 		)
 		(property "Value" "10K"
-			(at 194.056 60.198 90)
-			(effects
-				(font
+			(at 197.358 55.88 90)
+			(effects
+				(font

Commit message: new
Connections:
- net GN_TIMEPULSE renamed TIMEPULSE_LED
Changed lines of the file:
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@@
 		)
 	)
-	(global_label "GN_TIMEPULSE"
+	(global_label "TIMEPULSE_LED"
 		(shape input)
 		(at 149.86 58.42 180)
