File: POWER_2_sch.kicad_sch (KiCad schematic)
At the start: 33 parts, among them U1 MIC5205-3.3YM5, U7 IR3883MTRPBF

Commit message: 123
Changed lines of the file:
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@@
 		(dnp no)
 		(property "Reference" "R42"
-			(at 148.082 86.106 90)
+			(at 148.082 81.534 90)
 			(effects
 				(font
@@
 		)
 		(property "Value" "16K5"
-			(at 143.51 81.788 90)
+			(at 143.51 86.106 90)
 			(effects
 				(font
@@
 		(dnp no)
 		(property "Reference" "R14"
-			(at 118.364 87.122 90)
+			(at 115.316 87.122 0)
 			(effects
 				(font
@@
 		)
 		(property "Value" "49K9"
-			(at 115.57 92.202 90)
+			(at 110.49 89.408 0)
 			(effects
 				(font
@@
 		(dnp no)
 		(property "Reference" "C18"
-			(at 104.902 148.59 0)
+			(at 104.394 146.05 0)
 			(effects
 				(font
@@
 		)
 		(property "Value" "10u"
-			(at 104.394 146.05 0)
+			(at 104.394 148.082 0)
 			(effects
 				(font
@@
 		(dnp no)
 		(property "Reference" "R11"
-			(at 96.52 79.248 90)
+			(at 90.17 81.026 0)
 			(effects
 				(font
@@
 		)
 		(property "Value" "32K4"
-			(at 90.17 84.328 90)
+			(at 85.598 83.058 0)
 			(effects
 				(font
@@
 		(dnp no)
 		(property "Reference" "R12"
-			(at 96.52 86.868 90)
+			(at 90.678 88.9 0)
 			(effects
 				(font
@@
 		)
 		(property "Value" "47K"
-			(at 90.17 91.948 90)
+			(at 86.614 91.186 0)
 			(effects
 				(font
@@
 		)
 		(property "Value" "33K2"
-			(at 65.278 162.56 0)
+			(at 64.262 162.306 0)
 			(effects
 				(font
@@
 		(dnp no)
 		(property "Reference" "R46"
-			(at 159.004 86.868 90)
+			(at 159.512 81.788 90)
 			(effects
 				(font
@@
 		)
 		(property "Value" "2K94"
-			(at 154.432 81.28 90)
+			(at 154.94 86.106 90)
 			(effects
 				(font

Commit message: new
Parts:
- removed C15, C19: 0.1u, Capacitor_SMD:C_0402_1005Metric, symbol C0402C104K4RAC:C0402C104K4RAC
- removed C16: 0.47u, Capacitor_SMD:C_0402_1005Metric, symbol C0402C104K4RAC:C0402C104K4RAC
- removed C17: 4u7, Capacitor_SMD:C_0805_2012Metric, symbol Device:C_Small
- removed C18: 10u, Capacitor_SMD:C_0805_2012Metric, symbol Device:C_Small
- removed R13: 33K2, Resistor_SMD:R_0402_1005Metric, symbol Device:R_Small_US
- removed TP3: TestPoint, TestPoint:TestPoint_Pad_D2.0mm, symbol Connector:TestPoint
- removed VR1: LT3045EDD_PBF, GNSS:SON50P300X300X80-11N, symbol LT3045EDD_PBF:LT3045EDD_PBF
- added C45, C46: 1u, Capacitor_SMD:C_0805_2012Metric, symbol C0402C104K4RAC:C0402C104K4RAC
- added TP11: TestPoint, TestPoint:TestPoint_Pad_D2.0mm, symbol Connector:TestPoint
- added U14: NCV8705ML33TCG, DFNW8-3x3_ONS, symbol 2026-09-25_10-52-04:NCV8705ML33TCG
- C21: footprint C0402C104K4RAC:CAPC1005X55N -> Capacitor_SMD:C_0402_1005Metric
Connections:
- net +3V3_GNSS: now also C46.2, TP11.1, U14.8 (IN)
- net GND: now also C45.1, C46.1, U14.4 (GND), U14.9 (EXP)
- net VIN_GNSS: now also C45.2, U14.1 (OUT), U14.5 (EN)

Commit message: new
Parts:
- U14: footprint DFNW8-3x3_ONS -> Package_DFN_QFN:DFN-8-1EP_3x3mm_P0.65mm_EP1.55x2.4mm
Changed lines of the file:
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@@
 			)
 		)
-		(property "Footprint" "DFNW8-3x3_ONS"
+		(property "Footprint" "Package_DFN_QFN:DFN-8-1EP_3x3mm_P0.65mm_EP1.55x2.4mm"
 			(at 57.15 143.51 0)
 			(effects

Commit message: new
Parts:
- removed L1: 2.2u, ASPIAIG-F5030-2R2M-T:IND_ASPIAIG-F5030-2R2M-T, symbol ASPIAIG-F5030-2R2M-T:ASPIAIG-F5030-2R2M-T
- added L3: 22uH, IND_MSS1278T-223MLD_COC, symbol 2026-09-30_02-40-54:MSS1278T-223MLD
Connections:
- net +3V3: now also L3.1
- net SW: now also L3.2
Changed lines of the file:
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@@
 	(wire
 		(pts
-			(xy 134.62 59.69) (xy 138.43 59.69)
-		)
-		(stroke
-			(width 0)
-			(type default)
-		)
-	)
-	(wire
-		(pts
-			(xy 163.83 59.69) (xy 171.45 59.69)
+			(xy 134.62 59.69) (xy 143.51 59.69)
+		)
+		(stroke
+			(width 0)
+			(type default)
+		)
+	)
+	(wire
+		(pts
+			(xy 158.75 59.69) (xy 171.45 59.69)
 		)
 		(stroke
@@
 				(path "/a70dad34-b24c-4b58-b91c-f14576b5da7d/29ff9884-2eb8-4e05-9573-dea527771c4b"
 					(reference "R14")
+					(unit 1)
+				)
+			)
+		)
+	)
+	(symbol
+		(lib_id "2026-09-30_02-40-54:MSS1278T-223MLD")
+		(at 143.51 59.69 0)
+		(unit 1)
+		(exclude_from_sim no)
+		(in_bom yes)
+		(on_board yes)
+		(dnp no)
+		(fields_autoplaced yes)
+		(property "Reference" "L3"
+			(at 151.13 52.07 0)
+			(effects
+				(font
+					(size 1.524 1.524)
+				)
+			)
+		)
+		(property "Value" "22uH"
+			(at 151.13 54.61 0)
+			(effects
+				(font
+					(size 1.524 1.524)
+				)
+			)
+		)
+		(property "Footprint" "IND_MSS1278T-223MLD_COC"
+			(at 143.51 59.69 0)
+			(effects
+				(font
+					(size 1.27 1.27)
+					(italic yes)
+				)
+				(hide yes)
+			)
+		)
+		(property "Datasheet" "MSS1278T-223MLD"
+			(at 143.51 59.69 0)
+			(effects
+				(font
+					(size 1.27 1.27)
+					(italic yes)
+				)
+				(hide yes)
+			)
+		)
+		(property "Description" ""
+			(at 143.51 59.69 0)
+			(effects
+				(font
+					(size 1.27 1.27)
+				)
+				(hide yes)
+			)
+		)
+		(pin "2"
+		)
+		(pin "1"
+		)
+		(instances
+			(project "GNSS"
+				(path "/a70dad34-b24c-4b58-b91c-f14576b5da7d/29ff9884-2eb8-4e05-9573-dea527771c4b"
+					(reference "L3")
 					(unit 1)
 				)
@@
 					(unit 1)
 				)
-			)
-		)
-	)
-	(symbol
-		(lib_id "ASPIAIG-F5030-2R2M-T:ASPIAIG-F5030-2R2M-T")
-		(at 151.13 59.69 0)
-		(unit 1)
-		(exclude_from_sim no)
-		(in_bom yes)
-		(on_board yes)
-		(dnp no)
-		(fields_autoplaced yes)
-		(property "Reference" "L1"
-			(at 151.13 53.34 0)
-			(effects
-				(font
-					(size 1.27 1.27)
-				)
-			)
-		)
-		(property "Value" "2.2u"
-			(at 151.13 55.88 0)
-			(effects
-				(font
-					(size 1.27 1.27)
-				)
-			)
-		)
-		(property "Footprint" "ASPIAIG-F5030-2R2M-T:IND_ASPIAIG-F5030-2R2M-T"
-			(at 151.13 59.69 0)
-			(effects
-				(font
-					(size 1.27 1.27)
-				)
-				(justify bottom)
-				(hide yes)
-			)
-		)
-		(property "Datasheet" ""
-			(at 151.13 59.69 0)
-			(effects
-				(font
-					(size 1.27 1.27)
-				)
-				(hide yes)
-			)
-		)
-		(property "Description" ""
-			(at 151.13 59.69 0)
-			(effects
-				(font
-					(size 1.27 1.27)
-				)
-				(hide yes)
-			)
-		)
-		(property "MF" "Abracon Corporation"
-			(at 151.13 59.69 0)
-			(effects
-				(font
-					(size 1.27 1.27)
-				)
-				(justify bottom)
-				(hide yes)
-			)
-		)
-		(property "MAXIMUM_PACKAGE_HEIGHT" "3.1 mm"
-			(at 151.13 59.69 0)
-			(effects
-				(font
-					(size 1.27 1.27)
-				)
-				(justify bottom)
-				(hide yes)
-			)
-		)
-		(property "Package" "None"
-			(at 151.13 59.69 0)
-			(effects
-				(font
-					(size 1.27 1.27)
-				)
-				(justify bottom)
-				(hide yes)
-			)
-		)
-		(property "Price" "None"
-			(at 151.13 59.69 0)
-			(effects
-				(font
-					(size 1.27 1.27)
-				)
-				(justify bottom)
-				(hide yes)
-			)
-		)
-		(property "Check_prices" "https://www.snapeda.com/parts/ASPIAIG-F5030-2R2M-T/Abracon/view-part/?ref=eda"
-			(at 151.13 59.69 0)
-			(effects
-				(font
-					(size 1.27 1.27)
-				)
-				(justify bottom)
-				(hide yes)
-			)
-		)
-		(property "STANDARD" "Manufacturer Recommendations"
-			(at 151.13 59.69 0)
-			(effects
-				(font
-					(size 1.27 1.27)
-				)
-				(justify bottom)
-				(hide yes)
-			)
-		)
-		(property "PARTREV" "05.01.2019"
-			(at 151.13 59.69 0)
-			(effects
-				(font
-					(size 1.27 1.27)
-				)
-				(justify bottom)
-				(hide yes)
-			)
-		)
-		(property "SnapEDA_Link" "https://www.snapeda.com/parts/ASPIAIG-F5030-2R2M-T/Abracon/view-part/?ref=snap"
-			(at 151.13 59.69 0)
-			(effects
-				(font
-					(size 1.27 1.27)
-				)
-				(justify bottom)
-				(hide yes)
-			)
-		)
-		(property "MP" "ASPIAIG-F5030-2R2M-T"
-			(at 151.13 59.69 0)
-			(effects
-				(font
-					(size 1.27 1.27)
-				)
-				(justify bottom)
-				(hide yes)
-			)
-		)
-		(property "Purchase-URL" "https://www.snapeda.com/api/url_track_click_mouser/?unipart_id=11894085&manufacturer=Abracon Corporation&part_name=ASPIAIG-F5030-2R2M-T&search_term=aspiaig-f5030-2r2m-t"
-			(at 151.13 59.69 0)
-			(effects
-				(font
-					(size 1.27 1.27)
-				)
-				(justify bottom)
-				(hide yes)
-			)
-		)
-		(property "Description_1" "\n                        \n                            Inductor Power Shielded/Molded Wirewound 2.2uH 20% 100KHz 9.7A 0.0145Ohm DCR Automotive T/R\n                        \n"
-			(at 151.13 59.69 0)
-			(effects
-				(font
-					(size 1.27 1.27)
-				)
-				(justify bottom)
-				(hide yes)
-			)
-		)
-		(property "Availability" "In Stock"
-			(at 151.13 59.69 0)
-			(effects
-				(font
-					(size 1.27 1.27)
-				)
-				(justify bottom)
-				(hide yes)
-			)
-		)
-		(property "MANUFACTURER" "Abracon"
-			(at 151.13 59.69 0)
-			(effects
-				(font
-					(size 1.27 1.27)
-				)
-				(justify bottom)
-				(hide yes)
-			)
-		)
-		(pin "2"
-		)
-		(pin "1"
-		)
-		(instances
-			(project "GNSS"
-				(path "/a70dad34-b24c-4b58-b91c-f14576b5da7d/29ff9884-2eb8-4e05-9573-dea527771c4b"
-					(reference "L1")
-					(unit 1)
-				)

Commit message: 02.10.26
Parts:
- added C15: 0.1u/50V, Capacitor_SMD:C_0402_1005Metric, symbol C0402C104K4RAC:C0402C104K4RAC
- added C16: 0.1u, Capacitor_SMD:C_0402_1005Metric, symbol C0402C104K4RAC:C0402C104K4RAC
- C45, C46: value 1u -> 10u
Connections:
- net +3V3: now also C15.2
- net +3V3_GNSS: now also C16.2
- net GND: now also C15.1, C16.1
Other:
- note added: "Ripple: 300mA --> 21.25% 700mA --> 9.11% 1.3A --> 4.90%"
- moved on the sheet: TP5
