File: SD_CARD.kicad_sch (KiCad schematic)
At the start: 11 parts, among them J3 5033981892

Commit message: 123
Other:
- moved on the sheet: R73, R76, R77, R78, R81

Commit message: uty
Changed lines of the file:
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@@
+	(wire
+		(pts
+			(xy 195.58 95.25) (xy 195.58 97.79)
+		)
+		(stroke
+			(width 0)
+			(type default)
+		)
+	)
 	(wire
 		(pts
@@
 	(symbol
 		(lib_id "power:+3.3V")
-		(at 195.58 97.79 0)
+		(at 195.58 95.25 0)
 		(unit 1)
 		(exclude_from_sim no)
@@
 		(dnp no)
 		(property "Reference" "#PWR093"
-			(at 195.58 101.6 0)
+			(at 195.58 99.06 0)
 			(effects
 				(font
@@
 		)
 		(property "Value" "+3V3_SD"
-			(at 192.532 92.964 0)
+			(at 192.532 90.424 0)
 			(effects
 				(font
@@
 		)
 		(property "Footprint" ""
-			(at 195.58 97.79 0)
+			(at 195.58 95.25 0)
 			(effects
 				(font
@@
 		)
 		(property "Datasheet" ""
-			(at 195.58 97.79 0)
+			(at 195.58 95.25 0)
 			(effects
 				(font
@@
 		)
 		(property "Description" "Power symbol creates a global label with name \"+3.3V\""
-			(at 195.58 97.79 0)
-			(effects
-				(font
+			(at 195.58 95.25 0)
+			(effects
+				(font

Commit message: 02.10.26
Parts:
- R78: now not fitted
Changed lines of the file:
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@@
 		(in_bom yes)
 		(on_board yes)
-		(dnp no)
+		(dnp yes)
 		(property "Reference" "R78"
 			(at 176.022 102.87 0)
