File: ANTENNA.kicad_sch (KiCad schematic)
At the start: 16 parts, among them J7 SMA-J-P-X-RA-TH1, Q1 MMBT3904LT1G, Q9 PMOS, U15 TPS22946YZPR, U9 MCP6001-OT

Commit message: 18.09.2026
Parts:
- removed Q9: PMOS, symbol Simulation_SPICE:PMOS
- added U6: BSS84DW-7-F, SOT-363_DIO, symbol 2026-09-17_17-18-21:BSS84DW-7-F
Connections:
- net ANT_OFF: now also U6.5 (G1)
- net at R95.2, R97.2: now also U6.3 (D1)
- net at R99.2, U15.A1 (VOUT): now also U6.4 (S1)
- no-connect marks 0 -> 3
Other:
- moved on the sheet: R99, U9

Commit message: 123
Changed lines of the file:
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@@
 		(dnp no)
 		(property "Reference" "R95"
-			(at 57.15 88.138 0)
+			(at 55.88 89.916 0)
 			(effects
 				(font
@@
 		)
 		(property "Value" "10K"
-			(at 62.738 92.202 0)
+			(at 55.88 91.948 0)
 			(effects
 				(font
@@
 		(dnp no)
 		(property "Reference" "R100"
-			(at 135.128 55.626 90)
+			(at 144.018 57.912 0)
 			(effects
 				(font
@@
 		)
 		(property "Value" "10K"
-			(at 142.24 57.404 0)
+			(at 143.002 59.944 0)
 			(effects
 				(font
@@
 		(dnp no)
 		(property "Reference" "R84"
-			(at 210.312 84.074 90)
+			(at 202.438 82.55 0)
 			(effects
 				(font
@@
 		)
 		(property "Value" "10K"
-			(at 203.2 82.296 0)
+			(at 202.438 84.582 0)
 			(effects
 				(font
@@
 		(dnp no)
 		(property "Reference" "R83"
-			(at 197.866 99.822 90)
+			(at 195.58 95.25 90)
 			(effects
 				(font
@@
 		)
 		(property "Value" "10K"
-			(at 192.786 99.568 90)
+			(at 196.088 100.584 90)
 			(effects
 				(font
@@
 		)
 		(property "Value" "10K"
-			(at 141.986 105.41 0)
+			(at 135.382 106.426 0)
 			(effects
 				(font
@@
 		(dnp yes)
 		(property "Reference" "R98"
-			(at 110.998 61.722 90)
+			(at 103.886 61.214 90)
 			(effects
 				(font
@@
 		)
 		(property "Value" "10K"
-			(at 105.918 61.722 90)
+			(at 110.998 61.214 90)
 			(effects
 				(font
@@
 		)
 		(property "Value" "10K"
-			(at 62.484 99.314 0)
-			(effects
-				(font
+			(at 55.88 98.044 0)
+			(effects
+				(font

Commit message: new
Parts:
- added U11: TPS22918DBVR, Package_TO_SOT_SMD:SOT-23-6, symbol TPS22918DBVR:TPS22918DBVR
- D11: footprint PESD0402-140:DIO_PESD0402-140 -> Diode_SMD:D_0402_1005Metric
- L2: footprint LQG15HS47NJ02D:INDC1005X55N -> Inductor_SMD:L_0402_1005Metric
- Q1: footprint MMBT3904LT1G:SOT95P240X111-3N -> Package_TO_SOT_SMD:SOT-23
- U15: footprint TPS22946YZPR:BGA6C50P2X3_140X90X50 -> Package_BGA:Texas_DSBGA-6_0.704x1.054mm_Layout2x3_P0.35mm
- U6: footprint SOT-363_DIO -> Package_TO_SOT_SMD:SOT-323_SC-70
Changed lines of the file:
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@@
 			)
 		)
-		(property "Footprint" "TPS22946YZPR:BGA6C50P2X3_140X90X50"
+		(property "Footprint" "Package_BGA:Texas_DSBGA-6_0.704x1.054mm_Layout2x3_P0.35mm"
 			(at 123.19 54.61 0)
 			(effects
@@
 			)
 		)
-		(property "Footprint" "LQG15HS47NJ02D:INDC1005X55N"
+		(property "Footprint" "Inductor_SMD:L_0402_1005Metric"
 			(at 95.25 69.85 0)
 			(effects
@@
 			)
 		)
-		(property "Footprint" "MMBT3904LT1G:SOT95P240X111-3N"
+		(property "Footprint" "Package_TO_SOT_SMD:SOT-23"
 			(at 205.74 97.79 0)
 			(effects
@@
 	)
 	(symbol
+		(lib_id "TPS22918DBVR:TPS22918DBVR")
+		(at 119.38 17.78 0)
+		(unit 1)
+		(exclude_from_sim no)
+		(in_bom yes)
+		(on_board yes)
+		(dnp no)
+		(fields_autoplaced yes)
+		(property "Reference" "U11"
+			(at 119.38 2.54 0)
+			(effects
+				(font
+					(size 1.27 1.27)
+				)
+			)
+		)
+		(property "Value" "TPS22918DBVR"
+			(at 119.38 5.08 0)
+			(effects
+				(font
+					(size 1.27 1.27)
+				)
+			)
+		)
+		(property "Footprint" "Package_TO_SOT_SMD:SOT-23-6"
+			(at 119.38 17.78 0)
+			(effects
+				(font
+					(size 1.27 1.27)
+				)
+				(justify bottom)
+				(hide yes)
+			)
+		)
+		(property "Datasheet" ""
+			(at 119.38 17.78 0)
+			(effects
+				(font
+					(size 1.27 1.27)
+				)
+				(hide yes)
+			)
+		)
+		(property "Description" ""
+			(at 119.38 17.78 0)
+			(effects
+				(font
+					(size 1.27 1.27)
+				)
+				(hide yes)
+			)
+		)
+		(pin "4"
+		)
+		(pin "2"
+		)
+		(pin "6"
+		)
+		(pin "1"
+		)
+		(pin "3"
+		)
+		(pin "5"
+		)
+		(instances
+			(project "GNSS"
+				(path "/a70dad34-b24c-4b58-b91c-f14576b5da7d/b1f00880-f738-473f-92f4-04222a609f67"
+					(reference "U11")
+					(unit 1)
+				)
+			)
+		)
+	)
+	(symbol
 		(lib_id "Device:R_Small_US")
 		(at 137.16 104.14 180)
@@
 			)
 		)
-		(property "Footprint" "SOT-363_DIO"
+		(property "Footprint" "Package_TO_SOT_SMD:SOT-323_SC-70"
 			(at 71.12 102.87 0)
 			(effects
@@
 		(dnp no)
 		(property "Reference" "D11"
-			(at 82.55 70.104 90)
+			(at 81.534 68.834 90)
 			(effects
 				(font
@@
 			)
 		)
-		(property "Footprint" "PESD0402-140:DIO_PESD0402-140"
+		(property "Footprint" "Diode_SMD:D_0402_1005Metric"
 			(at 86.36 68.58 0)
 			(effects

Commit message: new
Parts:
- removed U11: TPS22918DBVR, Package_TO_SOT_SMD:SOT-23-6, symbol TPS22918DBVR:TPS22918DBVR
Changed lines of the file:
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@@
-	)
-	(symbol
-		(lib_id "TPS22918DBVR:TPS22918DBVR")
-		(at 119.38 17.78 0)
-		(unit 1)
-		(exclude_from_sim no)
-		(in_bom yes)
-		(on_board yes)
-		(dnp no)
-		(fields_autoplaced yes)
-		(property "Reference" "U11"
-			(at 119.38 2.54 0)
-			(effects
-				(font
-					(size 1.27 1.27)
-				)
-			)
-		)
-		(property "Value" "TPS22918DBVR"
-			(at 119.38 5.08 0)
-			(effects
-				(font
-					(size 1.27 1.27)
-				)
-			)
-		)
-		(property "Footprint" "Package_TO_SOT_SMD:SOT-23-6"
-			(at 119.38 17.78 0)
-			(effects
-				(font
-					(size 1.27 1.27)
-				)
-				(justify bottom)
-				(hide yes)
-			)
-		)
-		(property "Datasheet" ""
-			(at 119.38 17.78 0)
-			(effects
-				(font
-					(size 1.27 1.27)
-				)
-				(hide yes)
-			)
-		)
-		(property "Description" ""
-			(at 119.38 17.78 0)
-			(effects
-				(font
-					(size 1.27 1.27)
-				)
-				(hide yes)
-			)
-		)
-		(pin "4"
-		)
-		(pin "2"
-		)
-		(pin "6"
-		)
-		(pin "1"
-		)
-		(pin "3"
-		)
-		(pin "5"
-		)
-		(instances
-			(project "GNSS"
-				(path "/a70dad34-b24c-4b58-b91c-f14576b5da7d/b1f00880-f738-473f-92f4-04222a609f67"
-					(reference "U11")
-					(unit 1)
-				)
-			)
-		)
 	)
 	(symbol

Commit message: new
Changed lines of the file:
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@@
 		)
 		(property "Footprint" "Package_TO_SOT_SMD:SOT-323_SC-70"
-			(at 71.12 102.87 0)
+			(at 72.898 104.648 0)
 			(effects
 				(font
