File: CAN.kicad_sch (KiCad schematic)
At the start: 13 parts, among them J2 Conn, U5 TCAN1042VDRBRQ1

Commit message: 123
Connections:
- net +3V3: now also FB6.1; no longer FB6.2
- net +3V3_CAN: now also FB6.2; no longer FB6.1
- net VIN: now also FB5.1; no longer FB5.2
- net VIN_CAN: now also FB5.2; no longer FB5.1

Commit message: new
Parts:
- D10, D12: footprint PESD0402-140:DIO_PESD0402-140 -> Diode_SMD:D_0402_1005Metric
Changed lines of the file:
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@@
 			)
 		)
-		(property "Footprint" "PESD0402-140:DIO_PESD0402-140"
+		(property "Footprint" "Diode_SMD:D_0402_1005Metric"
 			(at 198.12 104.14 0)
 			(effects
@@
 			)
 		)
-		(property "Footprint" "PESD0402-140:DIO_PESD0402-140"
+		(property "Footprint" "Diode_SMD:D_0402_1005Metric"
 			(at 198.12 114.3 0)
 			(effects
