File: content.kicad_sch (KiCad schematic)
At the start: 0 parts

Commit message: new
Other:
- note added: "15"
- note added: "BLOCK DIAGRAM"
- note added: "CAN"
- note added: "ESP"
- note added: "IMU"
- note added: "POWER 1"
- note added: "POWER 2"
- note added: "POWER ARCH"
- note added: "SDCARD"
- note added: "USB HUB"
- note added: "ZED F9P"
- note removed: "ESP & CAN"
- note removed: "IMU & SDCARD"
- note removed: "POWER"
- note removed: "POWER_ARCHITECTURE"
- note removed: "USB_HUB"
- note removed: "ZED_ZF9P"

Commit message: new
Other:
- note added: "16"
- note added: "17"
- note added: "18"
Changed lines of the file:
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@@
+		)
+	)
+	(text "15"
+		(exclude_from_sim no)
+		(at 193.294 130.048 0)
+		(effects
+			(font
+				(size 3.81 3.81)
+				(bold yes)
+			)
+		)
+	)
+	(text "17"
+		(exclude_from_sim no)
+		(at 193.548 144.78 0)
+		(effects
+			(font
+				(size 3.81 3.81)
+				(bold yes)
+			)
 		)
 	)
@@
 	(text "8"
 		(exclude_from_sim no)
-		(at 194.31 79.756 0)
+		(at 193.548 79.756 0)
 		(effects
 			(font
@@
 		)
 	)
+	(text "16"
+		(exclude_from_sim no)
+		(at 193.294 137.414 0)
+		(effects
+			(font
+				(size 3.81 3.81)
+				(bold yes)
+			)
+		)
+	)
 	(text "5"
 		(exclude_from_sim no)
@@
 	(text "ANTENNA"
 		(exclude_from_sim no)
-		(at 138.938 78.74 0)
+		(at 138.938 86.36 0)
 		(effects
 			(font
@@
 	(text "ARDUINO"
 		(exclude_from_sim no)
-		(at 139.446 108.712 0)
+		(at 139.446 129.794 0)
 		(effects
 			(font
@@
 	(text "CAN"
 		(exclude_from_sim no)
-		(at 138.43 101.346 0)
+		(at 138.43 122.936 0)
 		(effects
 			(font
@@
 	(text "7"
 		(exclude_from_sim no)
-		(at 194.056 72.39 0)
+		(at 194.056 72.136 0)
 		(effects
 			(font
@@
 	(text "ETHERNET"
 		(exclude_from_sim no)
-		(at 139.7 116.078 0)
+		(at 139.7 101.092 0)
 		(effects
 			(font
@@
 	(text "SDCARD"
 		(exclude_from_sim no)
-		(at 139.954 130.048 0)
+		(at 139.7 115.824 0)
+		(effects
+			(font
+				(size 3.81 3.81)
+				(bold yes)
+			)
+		)
+	)
+	(text "18"
+		(exclude_from_sim no)
+		(at 193.802 152.908 0)
 		(effects
 			(font
@@
 	(text "CONTROLLER"
 		(exclude_from_sim no)
-		(at 139.446 86.106 0)
+		(at 139.192 71.882 0)
 		(effects
 			(font
@@
 	(text "IMU"
 		(exclude_from_sim no)
-		(at 139.446 123.19 0)
+		(at 139.192 108.966 0)
 		(effects
 			(font
@@
 	(text "ZED F9P"
 		(exclude_from_sim no)
-		(at 139.446 71.628 0)
-		(effects
-			(font
+		(at 138.938 79.248 0)
+		(effects
+			(font
